File: hardware/bat_rf/bat_rf.kicad_sch (KiCad schematic)
At the start: 1 part

Commit message: hardware edit
Parts:
- added R1: R, symbol Device:R
Changed lines of the file:
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@@
+    )
+  )
+  (symbol (lib_id "Device:R") (at 124.46 68.58 0) (unit 1)
+    (in_bom yes) (on_board yes) (dnp no) (fields_autoplaced)
+    (property "Reference" "R1" (at 127 67.945 0)
+      (effects (font (size 1.27 1.27)) (justify left))
+    )
+    (property "Value" "R" (at 127 70.485 0)
+      (effects (font (size 1.27 1.27)) (justify left))
+    )
+    (property "Footprint" "" (at 122.682 68.58 90)
+      (effects (font (size 1.27 1.27)) hide)
+    )
+    (property "Datasheet" "~" (at 124.46 68.58 0)
+      (effects (font (size 1.27 1.27)) hide)
+    )
+    (pin "1")
+    (pin "2")
+    (instances
+      (project "bat_rf"
+        (path "/4b9911c3-08ff-4557-9b31-2480476fb503"
+          (reference "R1") (unit 1)
+        )
+      )
     )
   )
