File: hardware/bat_rf/bat_rf.kicad_sch (KiCad schematic)
At the start: 91 parts, among them J1 USB_C_Receptacle_PowerOnly_6P, J4 Conn_01x02, J5 Conn_01x04, Q1 NMOS, SW2 RESET, U1 TPS54331, U3 ESP8684-WROOM-02UC, U4 CS5090E

Commit message: espBat update
Parts:
- FB1: footprint Capacitor_SMD:C_0603_1608Metric_Pad1.08x0.95mm_HandSolder -> Capacitor_SMD:C_0805_2012Metric_Pad1.18x1.45mm_HandSolder
Changed lines of the file:
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@@
       (effects (font (size 1.27 1.27)))
     )
-    (property "Footprint" "Capacitor_SMD:C_0603_1608Metric_Pad1.08x0.95mm_HandSolder" (at 268.732 46.99 90)
+    (property "Footprint" "Capacitor_SMD:C_0805_2012Metric_Pad1.18x1.45mm_HandSolder" (at 268.732 46.99 90)
       (effects (font (size 1.27 1.27)) hide)
     )
