File: hardware/bat_rf/bat_rf.kicad_sch (KiCad schematic)
At the start: 54 parts, among them J1 USB_C_Receptacle_PowerOnly_6P, J2 Conn_01x02, J3 burningPort, Q1 NMOS, SW1 SW_DPDT_x2, SW2 RESET, U1 TPS5430DDA, U2 AMS1117, U3 ESP8684-WROOM-02UC, U4 CS5090E

Commit message: hardware update
Parts:
- removed C14, C5, C6: 47u/25V, symbol Device:C_Small
- removed C15: 100n, symbol Device:C_Small
- removed C16, C18: 10u, symbol Device:C
- removed C17, C19: 100n, symbol Device:C
- removed D1: 1N5819WS, Diode_SMD:D_SOD-323, symbol Diode:1N5819WS
- removed D2: LED, LED_SMD:LED_0603_1608Metric_Pad1.05x0.95mm_HandSolder, symbol Device:LED
- removed J2: Conn_01x02, symbol Connector_Generic:Conn_01x02
- removed L2: L, symbol Device:L
- removed R1: 10k, Resistor_SMD:R_0603_1608Metric_Pad0.98x0.95mm_HandSolder, symbol Device:R
- removed R2: 3.3k, Resistor_SMD:R_0603_1608Metric_Pad0.98x0.95mm_HandSolder, symbol Device:R
- removed R3: 4.7k, Resistor_SMD:R_0603_1608Metric_Pad0.98x0.95mm_HandSolder, symbol Device:R
- removed SW1: SW_DPDT_x2, symbol Switch:SW_DPDT_x2
- removed U1: TPS5430DDA, Package_SO:TI_SO-PowerPAD-8_ThermalVias, symbol Regulator_Switching:TPS5430DDA
- removed U2: AMS1117, Package_TO_SOT_SMD:SOT-223-3_TabPin2, symbol Regulator_Linear:AMS1117
- added C16, C39: 22u, Capacitor_SMD:C_0805_2012Metric_Pad1.18x1.45mm_HandSolder, symbol Device:C_Small
- added C17, C23, C24, C25, C26, C27, C28, C29, C30, C31, C32, C33, C34, C35, C36: 100n, Capacitor_SMD:C_0603_1608Metric_Pad1.08x0.95mm_HandSolder, symbol Device:C_Small
- added C18: 8.2n, Capacitor_SMD:C_0603_1608Metric_Pad1.08x0.95mm_HandSolder, symbol Device:C_Small
- added C19: 1n, Capacitor_SMD:C_0603_1608Metric_Pad1.08x0.95mm_HandSolder, symbol Device:C_Small
- added C37: 2.2u, Capacitor_SMD:C_0603_1608Metric_Pad1.08x0.95mm_HandSolder, symbol Device:C
- added C38: 10p, Capacitor_SMD:C_0603_1608Metric_Pad1.08x0.95mm_HandSolder, symbol Device:C_Small
- added D10, D11, D3, D7, D8, D9: WS2812B, LED_SMD:LED_WS2812B_PLCC4_5.0x5.0mm_P3.2mm, symbol LED:WS2812B
- added D12: 3A, Diode_SMD:D_MELF, symbol Diode:1N5711UR
- added D13, D14: LED, LED_SMD:LED_0603_1608Metric_Pad1.05x0.95mm_HandSolder, symbol Device:LED
- added J4: Conn_01x02, bat_rf:CONN-TH_XT30U-M, symbol Connector_Generic:Conn_01x02
- added J5: Conn_01x04, Connector_PinHeader_2.54mm:PinHeader_1x04_P2.54mm_Vertical_SMD_Pin1Left, symbol Connector_Generic:Conn_01x04
- added L3: 4.5u, bat_rf:IND-SMD_L7.0-W6.6_0630CDMCCDS, symbol Device:L
- added LED2, LED3, LED4, LED5, LED6, LED7: XL-4020RGBC-WS2812B, bat_rf:LED-SMD_4P-L4.0-W1.7_M4020-03003-RGB-862-001, symbol bat_rf:XL-4020RGBC-WS2812B
- added R13, R14, R17: 1k, Resistor_SMD:R_0603_1608Metric_Pad0.98x0.95mm_HandSolder, symbol Device:R
- added R15, R16: 10.2k, Resistor_SMD:R_0603_1608Metric_Pad0.98x0.95mm_HandSolder, symbol Device:R
- added R8: 29.4k, Resistor_SMD:R_0603_1608Metric_Pad0.98x0.95mm_HandSolder, symbol Device:R
- added SW3: SW_DPDT_x2, bat_rf:SW-TH_3P-SS12D06-1, symbol Switch:SW_DPDT_x2
- added U1: TPS54331, bat_rf:SOP8-PAD, symbol bat_rf:TPS54331
- BT3: footprint (none) -> bat_rf:BAT-SMD_BH-18650-B1BA007
- BZ1: footprint (none) -> Buzzer_Beeper:Buzzer_12x9.5RM7.6
- C1: value 10n -> 22u; footprint (none) -> Capacitor_SMD:C_0805_2012Metric_Pad1.18x1.45mm_HandSolder
- C10, C11, C13, C20, C8: footprint (none) -> Capacitor_SMD:C_0805_2012Metric_Pad1.18x1.45mm_HandSolder
- C12, C21, C22, C7, C9, FB1: footprint (none) -> Capacitor_SMD:C_0603_1608Metric_Pad1.08x0.95mm_HandSolder
- C2: value 100n -> 22u; footprint (none) -> Capacitor_SMD:C_0805_2012Metric_Pad1.18x1.45mm_HandSolder
- C3, C4: value 22u/25V -> 22u; footprint (none) -> Capacitor_SMD:C_0805_2012Metric_Pad1.18x1.45mm_HandSolder
- J3: footprint (none) -> Connector_PinHeader_2.54mm:PinHeader_1x06_P2.54mm_Vertical
- L1: footprint (none) -> bat_rf:IND-SMD_L7.0-W6.6_0630CDMCCDS
- LED1: footprint kicad_lceda:LED-SMD_4P-L4.0-W1.7_M4020-03003-RGB-862-001 -> bat_rf:LED-SMD_4P-L4.0-W1.7_M4020-03003-RGB-862-001
- Q1: footprint (none) -> Package_TO_SOT_SMD:SOT-23
- R10: value 10k -> 3m
- R6, R7: footprint (none) -> Resistor_SMD:R_0603_1608Metric_Pad0.98x0.95mm_HandSolder
- R9: value 5.1k -> 7m
- SW2: footprint (none) -> Button_Switch_SMD:SW_SPST_B3U-1000P
Connections:
- net +5V is gone; now on net +3V3: BZ1.1 (-), D5.1 (K)
- net +3V3: now also C1.2, C2.2, C3.2, C4.2, D4.1 (VDD), LED1.3 (VDD), C23.2, C24.2, C25.2, C26.2, C27.2, C28.2, C29.2, C30.2, C31.2, C32.2, C33.2, C34.2, C35.2, C39.2, D10.1 (VDD), D11.1 (VDD), D3.1 (VDD), D7.1 (VDD), D8.1 (VDD), D9.1 (VDD), J5.1 (Pin_1), L3.2, LED2.3 (VDD), LED3.3 (VDD), LED4.3 (VDD), LED5.3 (VDD), LED6.3 (VDD), R13.1, R15.2, R17.1
- net +BATT: now also R9.2, C16.1, SW3.2 (B), U1.2 (VIN); no longer C2.2, C3.2, C4.2
- net GNDD: now also R10.1, C37.2, J5.4 (Pin_4); no longer Q1.3 (S), R7.1
- net GNDPWR: now also C1.1, D4.3 (VSS), LED1.1 (VSS), Q1.3 (S), R7.1, U3.4 (IO5), C16.2, C18.1, C19.2, C23.1, C24.1, C25.1, C26.1, C27.1, C28.1, C29.1, C30.1, C31.1, C32.1, C33.1, C34.1, C35.1, C36.1, C38.2, C39.1, D10.3 (VSS), D11.3 (VSS), D12.2 (A), D13.1 (K), D14.1 (K), D3.3 (VSS), D7.3 (VSS), D8.3 (VSS), D9.3 (VSS), J4.2 (Pin_2), LED2.1 (VSS), LED3.1 (VSS), LED4.1 (VSS), LED5.1 (VSS), LED6.1 (VSS), LED7.1 (VSS), R16.1, U1.7 (GND)
- net at R9.1: now also R10.2, C37.1, R14.2
- net at LED1.2 (DO): now also D10.4 (DIN)
- net at LED1.4 (DI): now also LED2.2 (DO)
- net beep: now reaches R6.1
- net beep: now also U3.16 (IO2)
- net at D4.4 (DIN): now also D3.2 (DOUT)
- net RGB: now reaches U3.15 (IO3)
- net RGB: now also LED7.4 (DI)
- net ESP_RX: now reaches U3.17 (IO1)
- net ESP_RX: now also J5.3 (Pin_3)
- net ESP_TX: now reaches U3.18 (IO0)
- net ESP_TX: now also J5.2 (Pin_2)
- net BAT_FB: now reaches U3.5 (IO6)
- net BAT_FB: now also R14.1
- new net: C17.2, D12.1 (K), L3.1, U1.8 (PH)
- new net: C19.1, R8.2
- new net: D13.2 (A), R13.2
- new net: C38.1, R8.1, U1.6 (COMP)
- new net: D14.2 (A), R17.2
- new net: C36.2, LED7.3 (VDD)
- new net: R15.1, R16.2, U1.5 (VSNS)
- new net: J4.1 (Pin_1), SW3.1 (A)
- new net: LED5.4 (DI), LED6.2 (DO)
- new net: LED6.4 (DI), LED7.2 (DO)
- new net: C17.1, U1.1 (BOOT)
- new net: C18.2, U1.4 (SS)
- new net: D3.4 (DIN), D7.2 (DOUT)
- new net: D10.2 (DOUT), D11.4 (DIN)
- new net: D8.4 (DIN), D9.2 (DOUT)
- new net: D11.2 (DOUT), D9.4 (DIN)
- new net: LED4.4 (DI), LED5.2 (DO)
- new net: LED2.4 (DI), LED3.2 (DO)
- new net: LED3.4 (DI), LED4.2 (DO)
- new net: D7.4 (DIN), D8.2 (DOUT)
- no-connect marks 5 -> 11
Other:
- note added: "MCU"
- moved on the sheet: BZ1, C20, C21, C22, D4, D5, FB1, J3, LED1, Q1, R10, R4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

Commit message: esp32 sch update
Parts:
- removed BT3: Battery, bat_rf:BAT-SMD_BH-18650-B1BA007, symbol Device:Battery
- removed C26, C27, C28, C29: 100n, Capacitor_SMD:C_0603_1608Metric_Pad1.08x0.95mm_HandSolder, symbol Device:C_Small
- removed D10, D11, D3, D4, D7, D8, D9: WS2812B, LED_SMD:LED_WS2812B_PLCC4_5.0x5.0mm_P3.2mm, symbol LED:WS2812B
- removed J3: burningPort, Connector_PinHeader_2.54mm:PinHeader_1x06_P2.54mm_Vertical, symbol Connector_Generic:Conn_01x06
- removed SW3: SW_DPDT_x2, bat_rf:SW-TH_3P-SS12D06-1, symbol Switch:SW_DPDT_x2
- added BT1: doubleBatCell, bat_rf:BAT-SMD_BH-18650-B1BA007, symbol bat_rf:doubleBatCell
- added C14, C15, C5, C6: 100n, Capacitor_SMD:C_0603_1608Metric_Pad1.08x0.95mm_HandSolder, symbol Device:C_Small
- added H1, H2, H3, H4: MountingHole, MountingHole:MountingHole_2.2mm_M2_Pad, symbol Mechanical:MountingHole
- added LED10, LED11, LED12, LED13, LED14, LED8, LED9: XL-4020RGBC-WS2812B, bat_rf:LED-SMD_4P-L4.0-W1.7_M4020-03003-RGB-862-001, symbol bat_rf:XL-4020RGBC-WS2812B
- added TP1, TP2, TP3, TP4, TP5, TP6: TestPoint, TestPoint:TestPoint_Pad_D1.0mm, symbol Connector:TestPoint
- BZ1: footprint Buzzer_Beeper:Buzzer_12x9.5RM7.6 -> Buzzer_Beeper:MagneticBuzzer_Kobitone_254-EMB84Q-RO
- J1: footprint bat_rf:GCT_USB4515-GF-A_REVA -> bat_rf:USB-C-SMD_HX-TYPE-C-6PIN
Connections:
- net +3V3: now also C36.2, LED7.3 (VDD), C14.2, C15.2, C5.2, C6.2, LED10.3 (VDD), LED11.3 (VDD), LED12.3 (VDD), LED13.3 (VDD), LED14.3 (VDD), LED8.3 (VDD), LED9.3 (VDD), TP1.1
- net +BATT: now also J4.1 (Pin_1), BT1.1 (+)
- net BAT_FB: now also U3.18 (IO0); no longer U3.5 (IO6)
- net EN: now also TP4.1
- net ESP_RX: now also U3.6 (IO7); no longer U3.17 (IO1)
- net ESP_TX: now also U3.5 (IO6); no longer U3.18 (IO0)
- net GNDD: now also TP6.1
- net GNDPWR: now also BT1.4 (-), C14.1, C15.1, C5.1, C6.1, LED10.1 (VSS), LED11.1 (VSS), LED12.1 (VSS), LED13.1 (VSS), LED14.1 (VSS), LED8.1 (VSS), LED9.1 (VSS); no longer D13.1 (K), U3.4 (IO5)
- net IO9: now also TP5.1
- net RGB: now also U3.10 (IO10); no longer U3.15 (IO3)
- net RXD: now also TP3.1
- net TXD: now also TP2.1
- net beep: now also U3.14 (IO18); no longer U3.16 (IO2)
- net at LED1.2 (DO): now also LED10.4 (DI)
- new net: LED8.4 (DI), LED9.2 (DO)
- new net: LED11.4 (DI), LED12.2 (DO)
- new net: LED12.4 (DI), LED13.2 (DO)
- new net: LED13.4 (DI), LED14.2 (DO)
- new net: LED10.2 (DO), LED9.4 (DI)
- new net: BT1.2 (-), BT1.3 (+)
- new net LED: D13.1 (K), U3.17 (IO1)
- no-connect marks 11 -> 12
Other:
- moved on the sheet: C10, C11, C12, C13, C30, C31, C32, C33, C34, C35, C36, C37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

Commit message: rfBat PCB sent to manufacturing
Parts:
- removed J5: Conn_01x04, Connector_PinHeader_2.54mm:PinHeader_1x04_P2.54mm_Vertical_SMD_Pin1Left, symbol Connector_Generic:Conn_01x04
- added J2: Conn_01x04, bat_rf:CONN-SMD_4P-P2.54_XH2.54-4AB_vertical, symbol Connector_Generic:Conn_01x04
- D12: footprint Diode_SMD:D_MELF -> Diode_SMD:D_SMA
- FB1: footprint Capacitor_SMD:C_0603_1608Metric_Pad1.08x0.95mm_HandSolder -> Inductor_SMD:L_1206_3216Metric_Pad1.22x1.90mm_HandSolder
- renumbered LED14 to LED11, LED13 to LED12, LED12 to LED13, LED11 to LED14
Connections:
- net +3V3: now also J2.4 (Pin_4)
- net ESP_RX: now also J2.2 (Pin_2)
- net ESP_TX: now also J2.3 (Pin_3)
- net GNDD: now also J2.1 (Pin_1)
- net at LED8.2 (DO): now also LED11.4 (DI)
- no-connect marks 12 -> 10
Changed lines of the file:
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@@
   )
   (no_connect (at 90.17 39.37))
-  (no_connect (at 100.33 138.43))
   (no_connect (at 40.64 39.37))
-  (no_connect (at 29.21 107.95))
   (no_connect (at 113.03 167.64))
   (no_connect (at 113.03 165.1))
@@
     (stroke (width 0) (type default))
   )
+  (wire (pts (xy 29.21 107.95) (xy 29.21 116.84))
+    (stroke (width 0) (type default))
+  )
   (wire (pts (xy 143.51 31.75) (xy 143.51 34.29))
     (stroke (width 0) (type default))
@@
     (stroke (width 0) (type default))
   )
+  (wire (pts (xy 102.87 116.84) (xy 102.87 138.43))
+    (stroke (width 0) (type default))
+  )
   (wire (pts (xy 250.19 139.7) (xy 252.73 139.7))
     (stroke (width 0) (type default))
@@
     (stroke (width 0) (type default))
   )
-  (wire (pts (xy 100.33 138.43) (xy 99.06 138.43))
-    (stroke (width 0) (type default))
-  )
   (polyline (pts (xy 175.26 76.2) (xy 281.94 76.2))
     (stroke (width 0) (type default))
@@
     (stroke (width 0) (type default))
   )
+  (wire (pts (xy 99.06 138.43) (xy 102.87 138.43))
+    (stroke (width 0) (type default))
+  )
   (wire (pts (xy 262.89 85.09) (xy 262.89 87.63))
     (stroke (width 0) (type default))
@@
     (stroke (width 0) (type default))
   )
+  (wire (pts (xy 29.21 116.84) (xy 102.87 116.84))
+    (stroke (width 0) (type default))
+  )
   (wire (pts (xy 200.66 97.79) (xy 205.74 97.79))
     (stroke (width 0) (type default))
@@
     (effects (font (size 1.27 1.27)) (justify left bottom))
   )
+  (label "ESP_TX" (at 260.35 90.17 0) (fields_autoplaced)
+    (effects (font (size 1.27 1.27)) (justify left bottom))
+  )
   (label "beep" (at 238.76 139.7 180) (fields_autoplaced)
     (effects (font (size 1.27 1.27)) (justify right bottom))
@@
     (effects (font (size 1.27 1.27)) (justify left bottom))
   )
-  (label "ESP_TX" (at 260.35 90.17 0) (fields_autoplaced)
+  (label "ESP_RX" (at 260.35 92.71 0) (fields_autoplaced)
     (effects (font (size 1.27 1.27)) (justify left bottom))
   )
@@
     (effects (font (size 1.27 1.27)) (justify left bottom))
   )
-  (label "ESP_RX" (at 260.35 92.71 0) (fields_autoplaced)
-    (effects (font (size 1.27 1.27)) (justify left bottom))
-  )
   (label "TXD" (at 43.18 170.18 0) (fields_autoplaced)
     (effects (font (size 1.27 1.27)) (justify left bottom))
@@
       (effects (font (size 1.27 1.27)))
     )
-    (property "Footprint" "Diode_SMD:D_MELF" (at 186.69 33.655 0)
+    (property "Footprint" "Diode_SMD:D_SMA" (at 186.69 33.655 0)
       (effects (font (size 1.27 1.27)) hide)
     )
@@
     )
   )
+  (symbol (lib_id "Connector_Generic:Conn_01x04") (at 255.27 92.71 180) (unit 1)
+    (in_bom yes) (on_board yes) (dnp no)
+    (property "Reference" "J2" (at 255.27 100.33 0)
+      (effects (font (size 1.27 1.27)))
+    )
+    (property "Value" "Conn_01x04" (at 255.27 97.79 0)
+      (effects (font (size 1.27 1.27)))
+    )
+    (property "Footprint" "bat_rf:CONN-SMD_4P-P2.54_XH2.54-4AB_vertical" (at 255.27 92.71 0)
+      (effects (font (size 1.27 1.27)) hide)
+    )
+    (property "Datasheet" "~" (at 255.27 92.71 0)
+      (effects (font (size 1.27 1.27)) hide)
+    )
+    (pin "1")
+    (pin "2")
+    (pin "3")
+    (pin "4")
+    (instances
+      (project "bat_rf"
+        (path "/4b9911c3-08ff-4557-9b31-2480476fb503"
+          (reference "J2") (unit 1)
+        )
+      )
+    )
+  )
   (symbol (lib_id "Device:R") (at 237.49 96.52 0) (mirror y) (unit 1)
     (in_bom yes) (on_board yes) (dnp no)
@@
       (effects (font (size 1.27 1.27)))
     )
-    (property "Footprint" "Capacitor_SMD:C_0603_1608Metric_Pad1.08x0.95mm_HandSolder" (at 268.732 46.99 90)
+    (property "Footprint" "Inductor_SMD:L_1206_3216Metric_Pad1.22x1.90mm_HandSolder" (at 268.732 46.99 90)
       (effects (font (size 1.27 1.27)) hide)
     )
@@
   (symbol (lib_id "bat_rf:XL-4020RGBC-WS2812B") (at 54.61 134.62 0) (mirror y) (unit 1)
     (in_bom yes) (on_board yes) (dnp no)
-    (property "Reference" "LED12" (at 53.34 142.24 0)
+    (property "Reference" "LED13" (at 53.34 142.24 0)
       (effects (font (size 1.27 1.27)))
     )
@@
       (project "bat_rf"
         (path "/4b9911c3-08ff-4557-9b31-2480476fb503"
-          (reference "LED12") (unit 1)
+          (reference "LED13") (unit 1)
         )
       )
@@
   (symbol (lib_id "bat_rf:XL-4020RGBC-WS2812B") (at 73.66 134.62 0) (mirror y) (unit 1)
     (in_bom yes) (on_board yes) (dnp no)
-    (property "Reference" "LED13" (at 72.39 142.24 0)
+    (property "Reference" "LED12" (at 72.39 142.24 0)
       (effects (font (size 1.27 1.27)))
     )
@@
       (project "bat_rf"
         (path "/4b9911c3-08ff-4557-9b31-2480476fb503"
-          (reference "LED13") (unit 1)
+          (reference "LED12") (unit 1)
         )
       )
@@
   (symbol (lib_id "bat_rf:XL-4020RGBC-WS2812B") (at 92.71 134.62 0) (mirror y) (unit 1)
     (in_bom yes) (on_board yes) (dnp no)
-    (property "Reference" "LED14" (at 91.44 142.24 0)
+    (property "Reference" "LED11" (at 91.44 142.24 0)
       (effects (font (size 1.27 1.27)))
     )
@@
       (project "bat_rf"
         (path "/4b9911c3-08ff-4557-9b31-2480476fb503"
-          (reference "LED14") (unit 1)
+          (reference "LED11") (unit 1)
         )
       )
@@
   (symbol (lib_id "bat_rf:XL-4020RGBC-WS2812B") (at 35.56 134.62 0) (mirror y) (unit 1)
     (in_bom yes) (on_board yes) (dnp no)
-    (property "Reference" "LED11" (at 34.29 142.24 0)
+    (property "Reference" "LED14" (at 34.29 142.24 0)
       (effects (font (size 1.27 1.27)))
     )
@@
       (project "bat_rf"
         (path "/4b9911c3-08ff-4557-9b31-2480476fb503"
-          (reference "LED11") (unit 1)
+          (reference "LED14") (unit 1)
         )
       )
@@
         )
       )
-    )
-  )
-  (symbol (lib_id "Connector_Generic:Conn_01x04") (at 255.27 90.17 0) (mirror y) (unit 1)
-    (in_bom yes) (on_board yes) (dnp no) (fields_autoplaced)
-    (property "Reference" "J5" (at 255.27 82.55 0)
-      (effects (font (size 1.27 1.27)))
-    )
-    (property "Value" "Conn_01x04" (at 255.27 85.09 0)
-      (effects (font (size 1.27 1.27)))
-    )
-    (property "Footprint" "Connector_PinHeader_2.54mm:PinHeader_1x04_P2.54mm_Vertical_SMD_Pin1Left" (at 255.27 90.17 0)
-      (effects (font (size 1.27 1.27)) hide)
-    )
-    (property "Datasheet" "~" (at 255.27 90.17 0)
-      (effects (font (size 1.27 1.27)) hide)
-    )
-    (pin "1")
-    (pin "2")
-    (pin "3")
-    (pin "4")
-    (instances
-      (project "bat_rf"
-        (path "/4b9911c3-08ff-4557-9b31-2480476fb503"
-          (reference "J5") (unit 1)
-        )
-      )

Commit message: batRf to v1.1
Parts:
- added D1: 3A, Diode_SMD:D_SMA, symbol Diode:1N5711UR
- added TP7, TP8, TP9: TestPoint, TestPoint:TestPoint_Pad_D1.0mm, symbol Connector:TestPoint
- R16: value 10.2k -> 3.24k
Connections:
- net BAT_FB: now also TP8.1
- net RGB: now also TP9.1
- net beep: now also TP7.1
- net at C10.1, C11.1, C9.1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: now also D1.1 (K)
- net at L1.2, U4.3 (LX): now also D1.2 (A)
Other:
- moved on the sheet: C10, C11, C7, C8, C9, L1

Commit message: 更新rfBat PCB
Parts:
- removed BT1: doubleBatCell, bat_rf:BAT-SMD_BH-18650-B1BA007, symbol bat_rf:doubleBatCell
- removed C11: 22u, Capacitor_SMD:C_0805_2012Metric_Pad1.18x1.45mm_HandSolder, symbol Device:C_Small
- removed C12, C7, C9: 1u, Capacitor_SMD:C_0603_1608Metric_Pad1.08x0.95mm_HandSolder, symbol Device:C_Small
- removed C13, C8: 10u, Capacitor_SMD:C_0805_2012Metric_Pad1.18x1.45mm_HandSolder, symbol Device:C_Small
- removed D1: 3A, Diode_SMD:D_SMA, symbol Diode:1N5711UR
- removed D6: RED, LED_SMD:LED_0603_1608Metric_Pad1.05x0.95mm_HandSolder, symbol Device:LED
- removed L1: 2.2u, bat_rf:IND-SMD_L7.0-W6.6_0630CDMCCDS, symbol Device:L
- removed R11, R12: 1k, Resistor_SMD:R_0603_1608Metric_Pad0.98x0.95mm_HandSolder, symbol Device:R
- removed U4: CS5090E, bat_rf:ESOP-8_L4.9-W3.9-P1.27-LS6.0-BL-EP, symbol bat_rf:CS5090E
- added BT2: doubleBatCell, bat_rf:BAT-SMD_BH-18650-B1BA007, symbol bat_rf:doubleBatCell
- added C26: 22u, Capacitor_SMD:C_0805_2012Metric_Pad1.18x1.45mm_HandSolder, symbol Device:C_Small
- added C27: 100n, Capacitor_SMD:C_0603_1608Metric_Pad1.08x0.95mm_HandSolder, symbol Device:C_Small
- added C28, C29, C40: 10u, Capacitor_SMD:C_0805_2012Metric_Pad1.18x1.45mm_HandSolder, symbol Device:C_Small
- added D2: RED, Capacitor_SMD:C_0805_2012Metric_Pad1.18x1.45mm_HandSolder, symbol Device:LED
- added L2: 2.2uH, Inductor_SMD_Wurth:L_Wurth_WE-LQSH-4020, symbol Device:L
- added R1: 0.5R, Resistor_SMD:R_0603_1608Metric_Pad0.98x0.95mm_HandSolder, symbol Device:R
- added R18: 51k, Resistor_SMD:R_0603_1608Metric_Pad0.98x0.95mm_HandSolder, symbol Device:R
- added R2: 5k1, Resistor_SMD:R_0603_1608Metric_Pad0.98x0.95mm_HandSolder, symbol Device:R
- added R3: 100R, Resistor_SMD:R_0603_1608Metric_Pad0.98x0.95mm_HandSolder, symbol Device:R
- added U2: IP2325_5M_WHJC, bat_rf:ESOP-8_L4.9-W3.9-P1.27-LS6.0-BL-EP3.1, symbol bat_rf:IP2325_5M_WHJC
Connections:
- net +BATT: now also BT2.1 (+), C40.1, U2.2 (VOUT)
- net GNDPWR: now also BT2.4 (-), C26.2, C28.2, C29.2, C40.2, D2.1 (K), R18.1, R2.1, U2.9 (GND)
- net at C10.1: now also C26.1, U2.1 (VSYS)
- net at J1.A9 (VBUS), J1.B9 (VBUS): now also C28.1, L2.1, R1.1, R2.2
- new net: D2.2 (A), R3.1
- new net: R3.2, U2.5 (LED)
- new net: R18.2, U2.4 (NTC)
- new net: BT2.2 (-), BT2.3 (+)
- new net: C27.1, U2.7 (BST)
- new net: C27.2, L2.2, U2.8 (LX)
- new net: C29.1, R1.2, U2.6 (VIN)

Commit message: update espBat
Parts:
- removed C1, C16, C2, C3, C39, C4: 22u, Capacitor_SMD:C_0805_2012Metric_Pad1.18x1.45mm_HandSolder, symbol Device:C_Small
- removed C17, C24, C25: 100n, Capacitor_SMD:C_0603_1608Metric_Pad1.08x0.95mm_HandSolder, symbol Device:C_Small
- removed C18: 8.2n, Capacitor_SMD:C_0603_1608Metric_Pad1.08x0.95mm_HandSolder, symbol Device:C_Small
- removed C19: 1n, Capacitor_SMD:C_0603_1608Metric_Pad1.08x0.95mm_HandSolder, symbol Device:C_Small
- removed C38: 10p, Capacitor_SMD:C_0603_1608Metric_Pad1.08x0.95mm_HandSolder, symbol Device:C_Small
- removed D12: 3A, Diode_SMD:D_SMA, symbol Diode:1N5711UR
- removed D14: LED, LED_SMD:LED_0603_1608Metric_Pad1.05x0.95mm_HandSolder, symbol Device:LED
- removed FB1: FerriteBead, Inductor_SMD:L_1206_3216Metric_Pad1.22x1.90mm_HandSolder, symbol Device:FerriteBead
- removed J4: Conn_01x02, bat_rf:CONN-TH_XT30U-M, symbol Connector_Generic:Conn_01x02
- removed L3: 4.5u, bat_rf:IND-SMD_L7.0-W6.6_0630CDMCCDS, symbol Device:L
- removed LED11, LED12: XL-4020RGBC-WS2812B, bat_rf:LED-SMD_4P-L4.0-W1.7_M4020-03003-RGB-862-001, symbol bat_rf:XL-4020RGBC-WS2812B
- removed R15: 10.2k, Resistor_SMD:R_0603_1608Metric_Pad0.98x0.95mm_HandSolder, symbol Device:R
- removed R16: 3.24k, Resistor_SMD:R_0603_1608Metric_Pad0.98x0.95mm_HandSolder, symbol Device:R
- removed R17: 1k, Resistor_SMD:R_0603_1608Metric_Pad0.98x0.95mm_HandSolder, symbol Device:R
- removed U1: TPS54331, bat_rf:SOP8-PAD, symbol bat_rf:TPS54331
- added C1, C3, C8, C9: 100n, symbol Device:C
- added C11, C2, C4, C7: 10u, symbol Device:C
- added D1: BAT54C, Package_TO_SOT_SMD:SOT-23, symbol Diode:BAT54C
- added Q2: PMOS, symbol Simulation_SPICE:PMOS
- added Q3: NMOS, symbol Simulation_SPICE:NMOS
- added R11: 33k, symbol Device:R
- added SW3: SW_MEC_5E, symbol Switch:SW_MEC_5E
- added U4, U5: AMS1117, Package_TO_SOT_SMD:SOT-223-3_TabPin2, symbol Regulator_Linear:AMS1117
- R8: value 29.4k -> 33k; footprint Resistor_SMD:R_0603_1608Metric_Pad0.98x0.95mm_HandSolder -> (none)
Connections:
- net +3V3: now also R8.1, Q2.3 (S); no longer BZ1.1 (-), C14.2, C15.2, C20.1, C21.1, C23.2, C30.2, C31.2, C32.2, C33.2, C34.2, C35.2, C36.2, C5.2, C6.2, D5.1 (K), J2.4 (Pin_4), LED1.3 (VDD), LED10.3 (VDD), LED13.3 (VDD), LED14.3 (VDD), LED2.3 (VDD), LED3.3 (VDD), LED4.3 (VDD), LED5.3 (VDD), LED6.3 (VDD), LED7.3 (VDD), LED8.3 (VDD), LED9.3 (VDD), R4.2, R5.2, TP1.1, U3.1 (3V3)
- net at R8.2: now also D1.2, Q2.2 (G), Q3.1 (D)
- net at LED8.2 (DO): now also LED13.4 (DI)
- new net: C3.1, C4.1, U4.2 (VO)
- new net: C1.1, C2.1, U4.3 (VI)
- new net: C11.1, C9.1, U5.3 (VI)
- new net: D1.3, SW3.3 (K), SW3.4 (A)
- new net: C7.1, C8.1, U5.2 (VO)
- new net: C14.2, LED10.3 (VDD)
- new net +5V: BZ1.1 (-), C15.2, C23.2, C30.2, C31.2, C32.2, C33.2, C34.2, C35.2, C36.2, C5.2, C6.2, D5.1 (K), LED1.3 (VDD), LED13.3 (VDD), LED14.3 (VDD), LED2.3 (VDD), LED3.3 (VDD), LED4.3 (VDD), LED5.3 (VDD), LED6.3 (VDD), LED7.3 (VDD), LED8.3 (VDD), LED9.3 (VDD)
- new net GND: C1.2, C11.2, C2.2, C3.2, C4.2, C7.2, C8.2, C9.2, Q3.3 (S), R11.1, SW3.1, SW3.2, U4.1 (ADJ), U5.1 (ADJ)
- new net KEY: D1.1, J2.4 (Pin_4)
- new net POWER_EN: Q3.2 (G), R11.2
- new net VCC: C20.1, C21.1, Q2.1 (D), R4.2, R5.2, TP1.1, U3.1 (3V3)
- no-connect marks 10 -> 9
Other:
- note removed: "电源"
