File: hardware/bat_rf/_autosave-bat_rf.kicad_pcb (KiCad board)
At the start: 2 copper layers, 13.2 x 6 mm, 83 parts, among them J1 USB_C_Receptacle_PowerOnly_6P, J3 burningPort, J4 Conn_01x02, J5 Conn_01x04, Q1 NMOS, SW2 RESET, SW3 SW_DPDT_x2, U1 TPS54331, U3 ESP8684-WROOM-02UC, U4 CS5090E

Commit message: hardware update
Parts:
- moved U3 102.1 mm to (57.0, 95.7)
- moved C1 16.3 mm to (90.0, 60.8)
- moved C10 16.3 mm to (90.0, 75.9)
- moved C12 16.3 mm to (46.5, 65.6)
- moved C17 16.3 mm to (46.5, 68.1)
- moved C18 16.3 mm to (46.5, 70.6)
- moved C19 16.3 mm to (46.5, 73.1)
- moved C22 16.3 mm to (46.5, 78.2)
- moved C23 16.3 mm to (46.5, 80.7)
- moved C25 16.3 mm to (50.8, 60.6)
- moved C27 16.3 mm to (50.8, 65.6)
- moved C28 16.3 mm to (50.8, 68.1)
- moved C29 16.3 mm to (50.8, 70.6)
- moved C3 16.3 mm to (90.0, 66.9)
- moved C30 16.3 mm to (50.8, 73.1)
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Other:
- outline, holes or cut-outs redrawn
