File: hardware/bldcDriver/bldcDriver.kicad_pcb (KiCad board)
At the start: 4 copper layers, 89.8 x 41.5 mm, 187 parts, among them CN1 MR30PW-F, CN2 MR30PW-F, J1 Conn_01x02, J2 Conn_01x06, J3 Conn_01x06, J4 Conn_01x03, J5 Conn_01x06, Q1 KNY3406C, Q10 KNY3406C, Q11 KNY3406C, Q12 KNY3406C, Q13 PMOS, Q14 S8050, Q2 KNY3406C, Q3 KNY3406C, Q4 KNY3406C, Q5 KNY3406C, Q6 KNY3406C, Q7 KNY3406C, Q8 KNY3406C, Q9 KNY3406C, U1 FD6288T, U10 AMS1117, U11 FD6288T, U2 STM32G431RBTx, U3 TPS5430DDA, U4 MPU-6050, U6 TLV9062xD, U7 MT3608, U8 TLV9062xD, U9 TLV9062xD, Y1 25MHz

Commit message: update driver pcb
Parts:
- J2: moved to B.Cu
- moved C39 3.76 mm to (41.4, 64.2)
- moved Q5 3.76 mm to (48.0, 64.0)
- moved R25 3.76 mm to (63.9, 63.2)
- moved Q6 3.76 mm to (55.8, 64.0)
- moved R18 3.76 mm to (65.3, 55.2)
- moved C29 3.76 mm to (41.5, 53.4)
- moved C33 3.76 mm to (41.5, 55.5)
- moved C35 3.76 mm to (41.4, 62.0)
- moved C41 3.76 mm to (41.4, 57.7)
- moved C45 3.76 mm to (41.4, 60.0)
- moved Q9 3.76 mm to (47.9, 58.4)
- moved R21 3.76 mm to (61.9, 60.3)
- moved R45 3.76 mm to (62.6, 57.6)
- moved R7 3.76 mm to (61.9, 49.0)
- moved C36 3.76 mm to (65.4, 58.6)
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Routing:
- net GNDPWR: track 208.5 -> 148.5 mm, vias 88 -> 67
- net /inverter/1SH_W: track 51.9 -> 6.40 mm, vias 11 -> 0
- net /VREF_OP1: track 52.5 -> 20.0 mm, vias 2 -> 0
- net /inverter/1GH_B: track 30.7 -> 0.22 mm, vias 2 -> 0
- net /inverter/1SH_U: track 38.3 -> 8.87 mm, vias 11 -> 1
- net /OP_VCC: track 95.7 -> 67.1 mm, vias 6 -> 5
- net /M1_ADC2_IN7: track 39.5 -> 11.4 mm
- net /inverter/1SH_V: track 26.1 -> 0.00 mm, vias 9 -> 0
- net /1B_ISENSOR-: track 25.8 -> 0.00 mm, vias 1 -> 0
- net Net-(Q9-G): track 24.0 -> 0.00 mm
- net /inverter/1GL_B: track 23.3 -> 0.00 mm
- net /M1_ADC1_IN4: track 32.8 -> 9.69 mm
- net /inverter/1GL_C: track 23.0 -> 0.00 mm
- net /1A_ISENSOR-: track 21.6 -> 0.00 mm, vias 1 -> 0
- net /1B_ISENSOR+: track 19.6 -> 0.00 mm, vias 1 -> 0
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- removed copper zone on B.Cu, net /inverter/1SH_U
- removed copper zone on B.Cu, net /inverter/1SH_V
- removed copper zone on B.Cu, net /inverter/1SH_W
- removed copper zone on B.Cu, net Net-(Q2-S-Pad1)
- removed copper zone on B.Cu, net Net-(Q6-S-Pad1)
