File: hardware/main/bldcDriver.kicad_sch (KiCad schematic)
At the start: 101 parts, among them J1 Conn_01x02, J2 Conn_01x06, J3 Conn_01x06, J4 Conn_01x03, J5 Conn_01x06, Q13 PMOS, Q14 S8050, U10 AMS1117, U3 TPS5430DDA, U4 MPU-6050, U5 STM32G431CBUx, U6 TLV9062xD, U7 MT3608, U8 TLV9062xD, U9 TLV9062xD, Y1 25MHz

Commit message: update driver pcb
Parts:
- removed C42: 10u, Capacitor_SMD:C_0805_2012Metric_Pad1.18x1.45mm_HandSolder, symbol Device:C_Small
- removed C44, C51, C53, C55, C57, C58, C60, C61, C66: 100n, Capacitor_SMD:C_0603_1608Metric_Pad1.08x0.95mm_HandSolder, symbol Device:C_Small
- removed C52, C54, C56, C59: 4.7u, Capacitor_SMD:C_0603_1608Metric_Pad1.08x0.95mm_HandSolder, symbol Device:C_Small
- removed C62, C63, C64, C65: 2.2n, Capacitor_SMD:C_0603_1608Metric_Pad1.08x0.95mm_HandSolder, symbol Device:C_Small
- removed D9: 1N5712UR, Diode_SMD:D_MELF, symbol Diode:1N5712UR
- removed L2: 10u, Inductor_SMD:L_Taiyo-Yuden_MD-4040, symbol Device:L
- removed Q13: PMOS, Package_TO_SOT_SMD:SOT-23, symbol Simulation_SPICE:PMOS
- removed Q14: S8050, Package_TO_SOT_SMD:SOT-23, symbol Transistor_BJT:BC107
- removed R35, R36, R50, R51, R53, R56, R57, R59, R6, R62, R63, R67, R68: 1k, Resistor_SMD:R_0603_1608Metric_Pad0.98x0.95mm_HandSolder, symbol Device:R_Small
- removed R37, R38, R4, R52, R54, R58, R60, R64, R65, R69, R70: 10k, Resistor_SMD:R_0603_1608Metric_Pad0.98x0.95mm_HandSolder, symbol Device:R_Small
- removed R39: 63.4k, Resistor_SMD:R_0603_1608Metric_Pad0.98x0.95mm_HandSolder, symbol Device:R_Small
- removed R40: 3.3k, Resistor_SMD:R_0603_1608Metric_Pad0.98x0.95mm_HandSolder, symbol Device:R_Small
- removed R5, R55, R61, R66, R71: 100R, Resistor_SMD:R_0603_1608Metric_Pad0.98x0.95mm_HandSolder, symbol Device:R_Small
- removed U10: AMS1117, Package_TO_SOT_SMD:SOT-223-3_TabPin2, symbol Regulator_Linear:AMS1117
- removed U6, U8, U9: TLV9062xD, Package_SO:SOIC-8_3.9x4.9mm_P1.27mm, symbol Amplifier_Operational:TLV9062xD
- removed U7: MT3608, Package_TO_SOT_SMD:SOT-23-6, symbol Regulator_Switching:MT3608
- added C27: 100n, Capacitor_SMD:C_0603_1608Metric_Pad1.08x0.95mm_HandSolder, symbol Device:C_Small
- added R20, R21: 10k, Resistor_SMD:R_0603_1608Metric_Pad0.98x0.95mm_HandSolder, symbol Device:R_Small
- added U6, U7, U8, U9: TP181A1-CR, balancerDriver:SC70-6_L2.1-W1.3-P0.65-LS2.3-BL, symbol bldcDriver:TP181A1-CR
- C10, C9: value 47u -> 100n; footprint Capacitor_SMD:C_1206_3216Metric_Pad1.33x1.80mm_HandSolder -> Capacitor_SMD:C_0603_1608Metric_Pad1.08x0.95mm_HandSolder
- C11: value 10u -> 100n; footprint Capacitor_SMD:C_0805_2012Metric_Pad1.18x1.45mm_HandSolder -> Capacitor_SMD:C_0603_1608Metric_Pad1.08x0.95mm_HandSolder
- D8: footprint Diode_SMD:D_MELF -> balancerDriver:SMA_L4.3-W2.6-LS5.0-RD
- FB3: footprint Capacitor_SMD:C_0603_1608Metric_Pad1.08x0.95mm_HandSolder -> Capacitor_SMD:C_1206_3216Metric_Pad1.33x1.80mm_HandSolder
- R2: value 3.3k -> 5.9k
Connections:
- net +5V is gone; now on net +3V3: C2.2, C3.2, C4.2, C8.2, L1.2, R1.1, R3.1
- net USART1_RX is gone; now on net USART2_RX: J4.2 (Pin_2)
- net USART1_TX is gone; now on net USART2_TX: J4.3 (Pin_3)
- net +3V3: now also R20.1; no longer C11.2, FB3.2
- net GNDD: now also FB3.2; no longer C11.1
- net GNDPWR: no longer C10.1, C9.1
- net I2C2_SCL: no longer U5.4 (PC15)
- net NSS2: now also U5.12 (PA4)
- net SPI1_MISO: now also U5.14 (PA6)
- net SPI1_MOSI: now also U5.15 (PA7)
- net SPI1_SCK: now also U5.13 (PA5)
- net SWCLK: now also U5.37 (PA14)
- net SWDIO: now also U5.36 (PA13)
- net TIM1_CH1: now also U5.30 (PA8); no longer U5.39 (PC10)
- net TIM1_CH2: now also U5.31 (PA9); no longer U5.40 (PC11)
- net TIM1_CH3: now also U5.32 (PA10); no longer U5.2 (PC13)
- net TIM8_CH1: now also U5.44 (PB6); no longer U5.17 (PB0)
- net TIM8_CH2: now also U5.46 (PB8); no longer U5.18 (PB1)
- net TIM8_CH3: now also U5.47 (PB9); no longer U5.19 (PB2)
- net USART3_RX: now also U5.24 (PB11)
- net USART3_TX: now also U5.22 (PB10)
- net at C9.2: now also U6.3 (V+)
- net USART2_TX: now reaches U5.10 (PA2)
- net USART2_RX: now reaches U5.11 (PA3)
- net I2C1_SCL: now reaches U5.38 (PA15)
- net +12V: no longer names the net of C10.2
- net +12V: now also U7.3 (V+)
- net OP_VCC renamed GNDA
- net GNDA: now also C10.1, C11.1, C9.1, C27.1, R21.2, U6.2 (GND), U6.5 (IN-), U7.2 (GND), U7.5 (IN-), U8.2 (GND), U8.5 (IN-), U9.2 (GND), U9.5 (IN-)
- new net: C11.2, U8.3 (V+)
- new net: C27.2, U9.3 (V+)
- new net 1CS1: U6.4 (IN+)
- new net 1CS2: U7.4 (IN+)
- new net 2CS1: U8.4 (IN+)
- new net 2CS2: U9.4 (IN+)
- new net VREF: R20.2, R21.1, U6.1 (REF), U7.1 (REF), U8.1 (REF), U9.1 (REF)
Other:
- sheet inverter ports: added 1CS1, 1CS2, 2CS1, 2CS2; removed 1A_ISENSOR+, 1A_ISENSOR-, 1B_ISENSOR+, 1B_ISENSOR-, 2A_ISENSOR+, 2A_ISENSOR-, 2B_ISENSOR+, 2B_ISENSOR-, TIM1_CH1N, TIM1_CH2N, TIM1_CH3N, TIM8_CH1N, TIM8_CH2N, TIM8_CH3N
- moved on the sheet: C1, C13, C17, C18, C19, C2, C22, C23, C24, C3, C4, C5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

Commit message: update driver pcb
Parts:
- FB3: footprint Capacitor_SMD:C_1206_3216Metric_Pad1.33x1.80mm_HandSolder -> Capacitor_SMD:C_0603_1608Metric_Pad1.08x0.95mm_HandSolder
- L1: footprint Inductor_SMD:L_Sumida_CDMC6D28_7.25x6.5mm -> Inductor_SMD:L_Taiyo-Yuden_NR-40xx_HandSoldering
- Y1: footprint Crystal:Crystal_SMD_SeikoEpson_FA238-4Pin_3.2x2.5mm_HandSoldering -> Crystal:Crystal_SMD_SeikoEpson_FA238-4Pin_3.2x2.5mm
Connections:
- net GNDA: no longer U6.5 (IN-), U7.5 (IN-), U8.5 (IN-), U9.5 (IN-)
- net GNDD: now also J4.3 (Pin_3); no longer J4.1 (Pin_1)
- net I2C1_SDA: now also U5.45 (PB7)
- net NSS1: now also U5.12 (PA4); no longer U5.16 (PC4)
- net NSS2: now also U5.43 (PB5); no longer U5.12 (PA4)
- net USART2_TX: now also J4.1 (Pin_1); no longer J4.3 (Pin_3)
- net 1CS1 renamed 1CS1+
- net 1CS2 renamed 1CS2+
- net 2CS1 renamed 2CS1+
- net 2CS2 renamed 2CS2+
- new net 1CS1-: U6.5 (IN-)
- new net 1CS2-: U7.5 (IN-)
- new net 2CS1-: U8.5 (IN-)
- new net 2CS2-: U9.5 (IN-)
Other:
- sheet inverter ports: added 1CS1+, 1CS1-, 1CS2+, 1CS2-, 2CS1+, 2CS1-, 2CS2+, 2CS2-; removed 1CS1, 1CS2, 2CS1, 2CS2
- moved on the sheet: J4

Commit message: update driver pcb
Connections:
- net I2C2_SCL is gone; now on net I2C1_SCL: R73.2, U4.23 (SCL)
- net I2C2_SDA is gone; now on net I2C1_SDA: R72.2, U4.24 (SDA)
- net ADC2_IN5: now reaches U7.6 (OUT)
- net ADC2_IN5: now also U5.16 (PC4)
- net ADC2_IN15: now reaches U9.6 (OUT)
- net ADC2_IN15: now also U5.28 (PB15)
- net ADC1_IN15: now reaches U5.17 (PB0)
- net ADC1_IN15: now also U6.6 (OUT)
- net ADC1_IN11: now reaches U5.25 (PB12)
- net ADC1_IN5: now reaches U5.27 (PB14)
Other:
- moved on the sheet: C10, C11, C13, C22, C23, C24, C27, C9, FB1, FB3, J4, J5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

Commit message: update driver pcb
Connections:
- net NSS1: now also U5.43 (PB5); no longer U5.12 (PA4)
- net NSS2: now also U5.12 (PA4); no longer U5.43 (PB5)
Other:
- moved on the sheet: C10, C11, C27, C9, FB3, R20, R21, U6, U7, U8, U9

Commit message: update driver pcb
Connections:
- net ADC1_IN11: now also U8.6 (OUT)
- net ADC1_IN15: no longer U6.6 (OUT)
- net ADC1_IN5: now also U6.6 (OUT)
- net ADC2_IN15: now also U7.6 (OUT); no longer U9.6 (OUT)
- net NSS1: now also J5.6 (Pin_6), U5.41 (PB3); no longer J5.3 (Pin_3), U5.43 (PB5)
- net NSS2: now also J3.6 (Pin_6), U5.2 (PC13); no longer J3.3 (Pin_3), U5.12 (PA4)
- net SPI1_MISO: now also J3.4 (Pin_4); no longer J3.5 (Pin_5), J5.5 (Pin_5)
- net SPI1_MOSI: now also J3.5 (Pin_5); no longer J3.6 (Pin_6), J5.6 (Pin_6)
- net SPI1_SCK: now also J3.3 (Pin_3); no longer J3.4 (Pin_4), J5.4 (Pin_4)
- net ADC2_IN12: now reaches U5.19 (PB2)
- net ADC2_IN12: now also U9.6 (OUT)
- net SPI3_SCK: now reaches U5.39 (PC10)
- net SPI3_SCK: now also J5.3 (Pin_3)
- net SPI3_MISO: now reaches U5.40 (PC11)
- net SPI3_MISO: now also J5.4 (Pin_4)
- net ADC2_IN5: no longer names the net of U5.16 (PC4)
- net ADC2_IN5: no longer U7.6 (OUT)
- new net SPI3_MOSI: J5.5 (Pin_5), U5.43 (PB5)
Changed lines of the file:
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@@
-		)
-	)
-	(label "SPI1_SCK"
-		(at 325.12 186.69 180)
-		(fields_autoplaced yes)
-		(effects
-			(font
-				(size 1.27 1.27)
-			)
-			(justify right bottom)
 		)
 	)
@@
 		)
 	)
-	(label "NSS2"
-		(at 377.19 187.96 180)
-		(fields_autoplaced yes)
-		(effects
-			(font
-				(size 1.27 1.27)
-			)
-			(justify right bottom)
-		)
-	)
 	(label "2CS1+"
 		(at 138.43 165.1 0)
@@
 		)
 	)
-	(label "ADC1_IN11"
-		(at 99.06 157.48 0)
-		(fields_autoplaced yes)
-		(effects
-			(font
-				(size 1.27 1.27)
-			)
-			(justify left bottom)
-		)
-	)
 	(label "2CS1-"
 		(at 138.43 162.56 0)
@@
 		)
 	)
+	(label "SPI3_SCK"
+		(at 341.63 69.85 180)
+		(fields_autoplaced yes)
+		(effects
+			(font
+				(size 1.27 1.27)
+			)
+			(justify right bottom)
+		)
+	)
 	(label "1CS2-"
 		(at 215.9 194.31 180)
@@
 		)
 	)
-	(label "ADC2_IN5"
-		(at 341.63 64.77 180)
-		(fields_autoplaced yes)
-		(effects
-			(font
-				(size 1.27 1.27)
-			)
-			(justify right bottom)
-		)
-	)
-	(label "SPI1_MISO"
-		(at 377.19 182.88 180)
+	(label "SPI1_SCK"
+		(at 377.19 187.96 180)
+		(fields_autoplaced yes)
+		(effects
+			(font
+				(size 1.27 1.27)
+			)
+			(justify right bottom)
+		)
+	)
+	(label "NSS2"
+		(at 377.19 180.34 180)
 		(fields_autoplaced yes)
 		(effects
@@
 		)
 	)
-	(label "SPI1_MOSI"
-		(at 325.12 181.61 180)
-		(fields_autoplaced yes)
-		(effects
-			(font
-				(size 1.27 1.27)
-			)
-			(justify right bottom)
-		)
-	)
-	(label "NSS2"
-		(at 374.65 57.15 0)
-		(fields_autoplaced yes)
-		(effects
-			(font
-				(size 1.27 1.27)
-			)
-			(justify left bottom)
+	(label "SPI3_MISO"
+		(at 341.63 72.39 180)
+		(fields_autoplaced yes)
+		(effects
+			(font
+				(size 1.27 1.27)
+			)
+			(justify right bottom)
 		)
 	)
@@
 		)
 	)
-	(label "SPI1_MISO"
-		(at 325.12 184.15 180)
+	(label "SPI1_MOSI"
+		(at 377.19 182.88 180)
 		(fields_autoplaced yes)
 		(effects
@@
 		)
 	)
+	(label "ADC2_IN12"
+		(at 341.63 90.17 180)
+		(fields_autoplaced yes)
+		(effects
+			(font
+				(size 1.27 1.27)
+			)
+			(justify right bottom)
+		)
+	)
 	(label "TIM1_CH1"
 		(at 374.65 67.31 0)
@@
 		)
 	)
-	(label "SPI1_MOSI"
-		(at 377.19 180.34 180)
-		(fields_autoplaced yes)
-		(effects
-			(font
-				(size 1.27 1.27)
-			)
-			(justify right bottom)
-		)
-	)
 	(label "2CS1+"
 		(at 251.46 185.42 0)
@@
 		)
 	)
+	(label "SPI3_MOSI"
+		(at 325.12 184.15 180)
+		(fields_autoplaced yes)
+		(effects
+			(font
+				(size 1.27 1.27)
+			)
+			(justify right bottom)
+		)
+	)
+	(label "ADC2_IN15"
+		(at 90.17 187.96 0)
+		(fields_autoplaced yes)
+		(effects
+			(font
+				(size 1.27 1.27)
+			)
+			(justify left bottom)
+		)
+	)
+	(label "NSS1"
+		(at 325.12 181.61 180)
+		(fields_autoplaced yes)
+		(effects
+			(font
+				(size 1.27 1.27)
+			)
+			(justify right bottom)
+		)
+	)
 	(label "SWCLK"
 		(at 374.65 82.55 0)
@@
 		)
 	)
-	(label "NSS1"
-		(at 341.63 97.79 180)
-		(fields_autoplaced yes)
-		(effects
-			(font
-				(size 1.27 1.27)
-			)
-			(justify right bottom)
-		)
-	)
 	(label "TIM1_CH1"
 		(at 251.46 162.56 0)
@@
 		)
 	)
+	(label "NSS2"
+		(at 341.63 74.93 180)
+		(fields_autoplaced yes)
+		(effects
+			(font
+				(size 1.27 1.27)
+			)
+			(justify right bottom)
+		)
+	)
 	(label "VREF"
 		(at 121.92 187.96 180)
@@
 		)
 	)
+	(label "SPI1_MISO"
+		(at 377.19 185.42 180)
+		(fields_autoplaced yes)
+		(effects
+			(font
+				(size 1.27 1.27)
+			)
+			(justify right bottom)
+		)
+	)
 	(label "TIM1_CH2"
 		(at 374.65 69.85 0)
@@
 		)
 	)
-	(label "SPI1_SCK"
-		(at 377.19 185.42 180)
-		(fields_autoplaced yes)
-		(effects
-			(font
-				(size 1.27 1.27)
-			)
-			(justify right bottom)
-		)
-	)
 	(label "USART2_TX"
 		(at 328.93 223.52 0)
@@
 		)
 	)
+	(label "SPI3_MISO"
+		(at 325.12 186.69 180)
+		(fields_autoplaced yes)
+		(effects
+			(font
+				(size 1.27 1.27)
+			)
+			(justify right bottom)
+		)
+	)
 	(label "2CS1-"
 		(at 251.46 193.04 0)
@@
 		)
 	)
-	(label "ADC1_IN15"
-		(at 90.17 160.02 0)
-		(fields_autoplaced yes)
-		(effects
-			(font
-				(size 1.27 1.27)
-			)
-			(justify left bottom)
+	(label "NSS1"
+		(at 341.63 92.71 180)
+		(fields_autoplaced yes)
+		(effects
+			(font
+				(size 1.27 1.27)
+			)
+			(justify right bottom)
 		)
 	)
@@
 		)
 	)
+	(label "ADC1_IN5"
+		(at 90.17 160.02 0)
+		(fields_autoplaced yes)
+		(effects
+			(font
+				(size 1.27 1.27)
+			)
+			(justify left bottom)
+		)
+	)
 	(label "SPI1_MOSI"
 		(at 374.65 64.77 0)
@@
 		)
 	)
+	(label "SPI3_MOSI"
+		(at 341.63 97.79 180)
+		(fields_autoplaced yes)
+		(effects
+			(font
+				(size 1.27 1.27)
+			)
+			(justify right bottom)
+		)
+	)
 	(label "USART2_TX"
 		(at 374.65 52.07 0)
@@
 		)
 	)
-	(label "ADC2_IN5"
-		(at 90.17 187.96 0)
-		(fields_autoplaced yes)
-		(effects
-			(font
-				(size 1.27 1.27)
-			)
-			(justify left bottom)
-		)
-	)
-	(label "NSS1"
-		(at 325.12 189.23 180)
-		(fields_autoplaced yes)
-		(effects
-			(font
-				(size 1.27 1.27)
-			)
-			(justify right bottom)
-		)
-	)
 	(label "TIM8_CH3"
 		(at 341.63 107.95 180)
@@
 		)
 	)
+	(label "SPI3_SCK"
+		(at 325.12 189.23 180)
+		(fields_autoplaced yes)
+		(effects
+			(font
+				(size 1.27 1.27)
+			)
+			(justify right bottom)
+		)
+	)
 	(label "TIM8_CH1"
 		(at 215.9 162.56 180)
@@
 		)
 	)
-	(label "ADC2_IN15"
-		(at 139.7 187.96 0)
+	(label "ADC1_IN11"
+		(at 138.43 160.02 0)
 		(fields_autoplaced yes)
 		(effects
@@
 		(fields_autoplaced yes)
 		(effects
+			(font
+				(size 1.27 1.27)
+			)
+			(justify left bottom)
+		)
+	)
+	(label "ADC2_IN12"
+		(at 139.7 187.96 0)
+		(fields_autoplaced yes)
+		(effects
