File: hardware/main/bldcDriver.kicad_sch (KiCad schematic)
At the start: 50 parts, among them J1 Conn_01x02, J2 Conn_01x06, J3 Conn_01x06, J4 Conn_01x03, J5 Conn_01x06, U3 TPS5430DDA, U4 MPU-6050, U5 STM32G431CBUx, U6 TP181A1-CR, U7 TP181A1-CR, U8 TP181A1-CR, U9 TP181A1-CR, Y1 25MHz

Commit message: update motor pcb
Parts:
- removed U6, U7, U8, U9: TP181A1-CR, balancerDriver:SC70-6_L2.1-W1.3-P0.65-LS2.3-BL, symbol bldcDriver:TP181A1-CR
- added C38, C43, C44: 4.7u, Capacitor_SMD:C_0603_1608Metric_Pad1.08x0.95mm_HandSolder, symbol Device:C_Small
- added C39, C40, C45, C46, C47, C48: 100n, Capacitor_SMD:C_0603_1608Metric_Pad1.08x0.95mm_HandSolder, symbol Device:C_Small
- added C41, C42: 2.2n, Capacitor_SMD:C_0603_1608Metric_Pad1.08x0.95mm_HandSolder, symbol Device:C_Small
- added R30, R32, R38, R39, R40, R41, R42, R43, R44, R46: 1k, Resistor_SMD:R_0603_1608Metric_Pad0.98x0.95mm_HandSolder, symbol Device:R_Small
- added R31, R33, R34, R36, R45, R47, R48, R51: 10k, Resistor_SMD:R_0603_1608Metric_Pad0.98x0.95mm_HandSolder, symbol Device:R_Small
- added R35, R37, R50, R52: 100R, Resistor_SMD:R_0603_1608Metric_Pad0.98x0.95mm_HandSolder, symbol Device:R_Small
- added U6, U7, U8: TLV9062xD, Package_SO:SOIC-8_3.9x4.9mm_P1.27mm, symbol Amplifier_Operational:TLV9062xD
- C11, C27: value 100n -> 2.2n
- C9: value 100n -> 4.7u
- R20, R21: value 10k -> 1k
Connections:
- net +3V3: now also FB3.2, J2.1 (Pin_1), J5.5 (Pin_5); no longer J2.3 (Pin_3), J5.2 (Pin_2), R20.1
- net 1CS1+: now also R21.2
- net 1CS1-: now also R32.2
- net 1CS2+: now also R43.2
- net 1CS2-: now also R46.2
- net 2CS1+: now also R20.2
- net 2CS1-: now also R30.2
- net 2CS2+: now also R42.2
- net 2CS2-: now also R44.2
- net ADC1_IN11: now also C41.2, R50.2
- net ADC1_IN5: now also C27.2, R37.2
- net ADC2_IN12: now also C11.2, R35.2
- net ADC2_IN15: now also C42.2, R52.2
- net GNDD: now also C10.1, C11.1, C27.1, C9.1, J2.2 (Pin_2), J4.1 (Pin_1), J5.6 (Pin_6), C38.1, C39.1, C40.1, C41.1, C42.1, C43.1, C44.1, C45.1, C46.1, C47.1, C48.1, R39.1, R41.1, U6.4 (V-), U7.4 (V-), U8.4 (V-); no longer FB3.2, J2.4 (Pin_4), J4.3 (Pin_3), J5.1 (Pin_1)
- net MPU_INT: now also U5.12 (PA4)
- net NSS1: now also J5.1 (Pin_1), U5.41 (PB3); no longer J5.6 (Pin_6), U5.2 (PC13)
- net SPI3_MISO: now also J5.3 (Pin_3); no longer J5.4 (Pin_4)
- net SPI3_MOSI: now also J5.2 (Pin_2); no longer J5.5 (Pin_5)
- net SPI3_SCK: now also J5.4 (Pin_4); no longer J5.3 (Pin_3)
- net USART2_TX: now also J4.3 (Pin_3); no longer J4.1 (Pin_1)
- net USART3_RX: now also J2.4 (Pin_4); no longer J2.2 (Pin_2)
- net USART3_TX: now also J2.3 (Pin_3); no longer J2.1 (Pin_1)
- net OP_VCC: now reaches C10.2
- net OP_VCC: now also C9.2, FB3.1, C40.2, C45.2, C46.2, R38.2, U6.8 (V+), U7.8 (V+), U8.8 (V+)
- removed net GNDA: C10.1, C11.1, C27.1, C9.1, FB3.1, R21.2
- net VREF: no longer names the net of R21.1
- net VREF: now also R36.1, U7.2 (-); no longer R20.2
- new net: R44.1, R45.1, U6.5 (+)
- new net: R46.1, R47.1, U7.5 (+)
- new net: R43.1, R51.1, U7.6 (-)
- new net: R51.2, R52.1, U7.7
- new net: R34.2, R35.1, U6.1
- new net: R32.1, R33.1, U7.3 (+)
- new net: R42.1, R48.1, U6.6 (-)
- new net: R48.2, R50.1, U6.7
- new net: R20.1, R34.1, U6.2 (-)
- new net: R30.1, R31.1, U6.3 (+)
- new net: R36.2, R37.1, U7.1
- new net INA1+: C38.2, C39.2, R38.1, R39.2, R40.2, U8.3 (+)
- new net INA2+: R40.1, R41.2, U8.5 (+)
- new net VREF_OP1: C44.2, C48.2, R33.2, R47.2, U8.1, U8.2 (-)
- new net VREF_OP2: C43.2, C47.2, R31.2, R45.2, U8.6 (-), U8.7
- no-connect marks 3 -> 4
Other:
- moved on the sheet: J4
