File: hardware/main/_autosave-bldcDriver.kicad_sch (KiCad schematic)
At the start: 50 parts, among them J1 Conn_01x02, J2 Conn_01x06, J3 Conn_01x06, J4 Conn_01x03, J5 Conn_01x06, U3 TPS5430DDA, U4 MPU-6050, U5 STM32G431CBUx, U6 TP181A1-CR, U7 TP181A1-CR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

Commit message: update driver pcb
Connections:
- net USART3_RX: now also J2.2 (Pin_2); no longer J2.1 (Pin_1)
- net USART3_TX: now also J2.1 (Pin_1); no longer J2.2 (Pin_2)
Changed lines of the file:
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@@
+		)
+	)
+	(label "USART3_TX"
+		(at 375.92 219.71 180)
+		(fields_autoplaced yes)
+		(effects
+			(font
+				(size 1.27 1.27)
+			)
+			(justify right bottom)
 		)
 	)
@@
 		)
 	)
-	(label "USART3_TX"
-		(at 375.92 222.25 180)
-		(fields_autoplaced yes)
-		(effects
-			(font
-				(size 1.27 1.27)
-			)
-			(justify right bottom)
-		)
-	)
 	(label "VREF"
 		(at 40.64 172.72 0)
@@
 		)
 	)
+	(label "USART3_RX"
+		(at 375.92 222.25 180)
+		(fields_autoplaced yes)
+		(effects
+			(font
+				(size 1.27 1.27)
+			)
+			(justify right bottom)
+		)
+	)
 	(label "TIM8_CH1"
 		(at 215.9 162.56 180)
@@
 		)
 	)
-	(label "USART3_RX"
-		(at 375.92 219.71 180)
-		(fields_autoplaced yes)
-		(effects
-			(font
-				(size 1.27 1.27)
-			)
-			(justify right bottom)
-		)
-	)
