File: hardware/main/bldcDriver.kicad_pcb (KiCad board)
At the start: 2 copper layers, 89.8 x 41.5 mm, 135 parts, among them CN1 MR30PW-F, CN2 MR30PW-F, J1 Conn_01x02, J2 Conn_01x06, J3 Conn_01x06, J4 Conn_01x03, J5 Conn_01x06, Q1 EMB09N03V, Q10 EMB09N03V, Q11 EMB09N03V, Q12 EMB09N03V, Q13 EMB09N03V, Q13 PMOS, Q14 EMB09N03V, Q14 S8050, Q15 EMB09N03V, Q16 EMB09N03V, Q2 EMB09N03V, Q7 EMB09N03V, Q8 EMB09N03V, Q9 EMB09N03V, U1 EG2133, U10 AMS1117, U2 EG2133, U3 TPS5430DDA, U4 MPU-6050, U5 STM32G431CBUx, U6 TP181A1-CR, U7 MT3608, U7 TP181A1-CR, U8 TP181A1-CR, U9 TP181A1-CR, Y1 25MHz

Commit message: update driver pcb
Parts:
- removed the C10 at (73.6, 150.9)
- removed the C10 at (51.9, 142.4)
- removed the C11 at (51.9, 144.9)
- removed the C11 at (168.7, 123.2)
- removed C42: 10u, Capacitor_SMD:C_0805_2012Metric_Pad1.18x1.45mm_HandSolder
- removed C44, C51: 100n, Capacitor_SMD:C_0603_1608Metric_Pad1.08x0.95mm_HandSolder
- removed the C9 at (51.9, 139.8)
- removed the C9 at (73.6, 147.6)
- removed the D9 at (39.2, 90.4)
- removed the D9 at (85.2, 162.4)
- removed L2: 10u, Inductor_SMD:L_Taiyo-Yuden_MD-4040
- removed the Q13 at (141.7, 178.7)
- removed the Q14 at (92.1, 170.9)
- removed R37, R38: 10k, Resistor_SMD:R_0603_1608Metric_Pad0.98x0.95mm_HandSolder
- removed R39: 63.4k, Resistor_SMD:R_0603_1608Metric_Pad0.98x0.95mm_HandSolder
- removed the R4 at (83.1, 149.6)
- removed the R4 at (44.3, 90.0)
- removed R40: 3.3k, Resistor_SMD:R_0603_1608Metric_Pad0.98x0.95mm_HandSolder
- removed the R5 at (44.3, 92.5)
- removed the R5 at (83.1, 152.2)
- removed the R6 at (83.1, 154.7)
- removed the R6 at (44.3, 95.0)
- removed U10: AMS1117, Package_TO_SOT_SMD:SOT-223-3_TabPin2
- removed the U7 at (73.1, 163.9)
- added C10: 100n, Capacitor_SMD:C_0603_1608Metric_Pad1.08x0.95mm_HandSolder, F.Cu at (60.7, 57.8)
- added C11: 100n, Capacitor_SMD:C_0603_1608Metric_Pad1.08x0.95mm_HandSolder, F.Cu at (92.1, 63.7)
- added C28: 1n, Capacitor_SMD:C_0603_1608Metric_Pad1.08x0.95mm_HandSolder, B.Cu at (51.0, 69.7)
- added C35: 1n, Capacitor_SMD:C_0603_1608Metric_Pad1.08x0.95mm_HandSolder, B.Cu at (51.0, 54.5)
- added C36: 1n, Capacitor_SMD:C_0603_1608Metric_Pad1.08x0.95mm_HandSolder, B.Cu at (102.4, 66.9)
- added C37: 1n, Capacitor_SMD:C_0603_1608Metric_Pad1.08x0.95mm_HandSolder, B.Cu at (102.5, 52.1)
- added C9: 100n, Capacitor_SMD:C_0603_1608Metric_Pad1.08x0.95mm_HandSolder, F.Cu at (60.7, 61.2)
- added D9: 1N4148W, Diode_SMD:D_SOD-123, B.Cu at (41.1, 63.3)
- added R22: 100R, Resistor_SMD:R_0603_1608Metric_Pad0.98x0.95mm_HandSolder, B.Cu at (49.3, 68.2)
- added R23: 100R, Resistor_SMD:R_0603_1608Metric_Pad0.98x0.95mm_HandSolder, B.Cu at (52.7, 68.2)
- added R24: 100R, Resistor_SMD:R_0603_1608Metric_Pad0.98x0.95mm_HandSolder, B.Cu at (49.4, 53.0)
- added R25: 100R, Resistor_SMD:R_0603_1608Metric_Pad0.98x0.95mm_HandSolder, B.Cu at (52.7, 53.0)
- added R26: 100R, Resistor_SMD:R_0603_1608Metric_Pad0.98x0.95mm_HandSolder, B.Cu at (104.1, 68.4)
- added R27: 100R, Resistor_SMD:R_0603_1608Metric_Pad0.98x0.95mm_HandSolder, B.Cu at (100.7, 68.4)
- added R28: 100R, Resistor_SMD:R_0603_1608Metric_Pad0.98x0.95mm_HandSolder, B.Cu at (104.2, 53.6)
- added R29: 100R, Resistor_SMD:R_0603_1608Metric_Pad0.98x0.95mm_HandSolder, B.Cu at (100.8, 53.6)
- added R4: 10R, Resistor_SMD:R_0603_1608Metric_Pad0.98x0.95mm_HandSolder, B.Cu at (41.7, 61.3)
- added R5: 10R, Resistor_SMD:R_0603_1608Metric_Pad0.98x0.95mm_HandSolder, B.Cu at (45.7, 61.3)
- added R6: 10R, Resistor_SMD:R_0603_1608Metric_Pad0.98x0.95mm_HandSolder, B.Cu at (41.8, 53.9)
- added TP1: TestPoint, TestPoint:TestPoint_Pad_1.0x1.0mm, F.Cu at (37.3, 60.6)
- added TP2: TestPoint, TestPoint:TestPoint_Pad_1.0x1.0mm, F.Cu at (35.9, 58.9)
- added TP3: TestPoint, TestPoint:TestPoint_Pad_1.0x1.0mm, F.Cu at (37.3, 57.1)
- added TP4: TestPoint, TestPoint:TestPoint_Pad_1.0x1.0mm, F.Cu at (117.0, 59.0)
- added TP5: TestPoint, TestPoint:TestPoint_Pad_1.0x1.0mm, F.Cu at (118.5, 60.7)
- added TP6: TestPoint, TestPoint:TestPoint_Pad_1.0x1.0mm, F.Cu at (117.0, 62.5)
- C1, C2, C3, C4, C5, C6, C7, C8, D1, D16, D17, D18, D19, D20, D21, D22, D23, D24, D5, D6, D8, J1, Q1, Q10, Q11, Q12, Q13, Q14, Q15, Q16, Q2, Q7, Q8, Q9, R1, R13, R14, R15, R16, R17, R18, R19, R2, R3, R7, R8, U3: moved to B.Cu
- FB3: footprint Capacitor_SMD:C_1206_3216Metric_Pad1.33x1.80mm_HandSolder -> Capacitor_SMD:C_0603_1608Metric_Pad1.08x0.95mm_HandSolder
- L1: footprint Inductor_SMD:L_Sumida_CDMC6D28_7.25x6.5mm -> Inductor_SMD:L_Taiyo-Yuden_NR-40xx_HandSoldering; moved to B.Cu
- R10, R11, R12, R9: footprint Resistor_SMD:R_2512_6332Metric_Pad1.40x3.35mm_HandSolder -> Resistor_SMD:R_1206_3216Metric_Pad1.30x1.75mm_HandSolder; moved to B.Cu
- Y1: footprint Crystal:Crystal_SMD_SeikoEpson_FA238-4Pin_3.2x2.5mm_HandSoldering -> Crystal:Crystal_SMD_SeikoEpson_FA238-4Pin_3.2x2.5mm
- moved FB2 139.6 mm to (64.5, 38.6)
- moved L1 133.5 mm to (56.6, 41.3), turned to 90 degrees
- moved D1 130.3 mm to (43.6, 40.4), turned to 180 degrees
- moved R12 116.7 mm to (103.2, 55.5)
- moved R3 115.3 mm to (43.5, 38.8), turned to 180 degrees
- moved C8 107.4 mm to (46.1, 39.8), turned to 90 degrees
- moved C4 106.6 mm to (48.1, 40.7), turned to 90 degrees
- moved U8 105.8 mm to (94.8, 63.6), turned to -90 degrees
- moved U9 105.4 mm to (94.8, 60.5), turned to -90 degrees
- moved C3 102.8 mm to (50.5, 40.7), turned to 90 degrees
- moved R11 100.3 mm to (103.1, 70.4)
- moved C2 99.0 mm to (53.0, 40.7), turned to 90 degrees
- moved R2 97.7 mm to (63.8, 48.9)
- moved R1 96.8 mm to (63.8, 47.3), turned to 180 degrees
- moved R9 96.7 mm to (50.1, 66.2), turned to 180 degrees
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Connections:
- CN2 pad 1: /inverter/2VS3 -> /inverter/2VS1
- CN2 pad 3: /inverter/2VS1 -> /inverter/2VS3
- D16 pad 1: /inverter/2HO1 -> /inverter/2HO3
- D17 pad 1: /inverter/2LO1 -> /inverter/2LO3
- D20 pad 1: /inverter/2HO3 -> /inverter/2HO1
- D21 pad 1: /inverter/2LO3 -> /inverter/2LO1
- D23 pad 1: /inverter/1HO3 -> /inverter/1HO1
- D24 pad 1: /inverter/1LO3 -> /inverter/1LO1
- D5 pad 1: /inverter/1HO1 -> /inverter/1HO3
- D6 pad 1: /inverter/1LO1 -> /inverter/1LO3
- J4 pad 1: GNDD -> /USART2_TX
- J4 pad 3: /USART2_TX -> GNDD
- Q1 pad 1: /1CS1 -> Net-(Q1-S-Pad1)
- Q1 pad 2: /1CS1 -> Net-(Q1-S-Pad1)
- Q1 pad 3: /1CS1 -> Net-(Q1-S-Pad1)
- Q1 pad 5: /inverter/1VS1 -> /inverter/1VS3
- Q1 pad 6: /inverter/1VS1 -> /inverter/1VS3
- Q1 pad 7: /inverter/1VS1 -> /inverter/1VS3
- Q1 pad 8: /inverter/1VS1 -> /inverter/1VS3
- Q11 pad 1: /inverter/2VS3 -> /inverter/2VS1
- Q11 pad 2: /inverter/2VS3 -> /inverter/2VS1
- Q11 pad 3: /inverter/2VS3 -> /inverter/2VS1
- Q12 pad 1: /2CS2 -> Net-(Q12-S-Pad1)
- Q12 pad 2: /2CS2 -> Net-(Q12-S-Pad1)
- Q12 pad 3: /2CS2 -> Net-(Q12-S-Pad1)
- Q12 pad 5: /inverter/2VS3 -> /inverter/2VS1
- Q12 pad 6: /inverter/2VS3 -> /inverter/2VS1
- Q12 pad 7: /inverter/2VS3 -> /inverter/2VS1
- Q12 pad 8: /inverter/2VS3 -> /inverter/2VS1
- Q13 pad 1: /inverter/1VS1 -> /inverter/1VS3
- Q13 pad 2: /inverter/1VS1 -> /inverter/1VS3
- Q13 pad 3: /inverter/1VS1 -> /inverter/1VS3
- Q15 pad 1: /inverter/1VS3 -> /inverter/1VS1
- Q15 pad 2: /inverter/1VS3 -> /inverter/1VS1
- Q15 pad 3: /inverter/1VS3 -> /inverter/1VS1
- Q16 pad 1: /1CS2 -> Net-(Q16-S-Pad1)
- Q16 pad 2: /1CS2 -> Net-(Q16-S-Pad1)
- Q16 pad 3: /1CS2 -> Net-(Q16-S-Pad1)
- Q16 pad 5: /inverter/1VS3 -> /inverter/1VS1
- Q16 pad 6: /inverter/1VS3 -> /inverter/1VS1
- Q16 pad 7: /inverter/1VS3 -> /inverter/1VS1
- Q16 pad 8: /inverter/1VS3 -> /inverter/1VS1
- Q7 pad 1: /inverter/2VS1 -> /inverter/2VS3
- Q7 pad 2: /inverter/2VS1 -> /inverter/2VS3
- Q7 pad 3: /inverter/2VS1 -> /inverter/2VS3
- Q8 pad 1: /2CS1 -> Net-(Q8-S-Pad1)
- Q8 pad 2: /2CS1 -> Net-(Q8-S-Pad1)
- Q8 pad 3: /2CS1 -> Net-(Q8-S-Pad1)
- Q8 pad 5: /inverter/2VS1 -> /inverter/2VS3
- Q8 pad 6: /inverter/2VS1 -> /inverter/2VS3
- Q8 pad 7: /inverter/2VS1 -> /inverter/2VS3
- Q8 pad 8: /inverter/2VS1 -> /inverter/2VS3
- R10 pad 2: /1CS2 -> Net-(Q16-S-Pad1)
- R11 pad 2: /2CS1 -> Net-(Q8-S-Pad1)
- R12 pad 2: /2CS2 -> Net-(Q12-S-Pad1)
- R13 pad 1: /inverter/2HO1 -> /inverter/2HO3
- R14 pad 1: /inverter/2LO1 -> /inverter/2LO3
- R17 pad 1: /inverter/2HO3 -> /inverter/2HO1
- R18 pad 1: /inverter/2LO3 -> /inverter/2LO1
- R19 pad 1: /inverter/1LO3 -> /inverter/1LO1
- R7 pad 1: /inverter/1LO1 -> /inverter/1LO3
- R8 pad 1: /inverter/1HO1 -> /inverter/1HO3
- R9 pad 2: /1CS1 -> Net-(Q1-S-Pad1)
- U5 pad 12: /NSS2 -> /NSS1
- U5 pad 16: /NSS1 -> unconnected-(U5-PC4-Pad16)
- U5 pad 43: unconnected-(U5-PB5-Pad43) -> /NSS2
- U5 pad 45: unconnected-(U5-PB7-Pad45) -> /I2C1_SDA
- U6 pad 4: /1CS1 -> /1CS1+
- U6 pad 5: GNDA -> /1CS1-
- U7 pad 4: /1CS2 -> /1CS2+
- U7 pad 5: GNDA -> /1CS2-
- U8 pad 4: /2CS1 -> /2CS1+
- U8 pad 5: GNDA -> /2CS1-
- U9 pad 4: /2CS2 -> /2CS2+
- U9 pad 5: GNDA -> /2CS2-
Routing:
- net /SPI1_MOSI: track 0.00 -> 90.5 mm, vias 0 -> 2
- net /SPI1_MISO: track 0.00 -> 89.9 mm, vias 0 -> 2
- net /SPI1_SCK: track 0.00 -> 86.6 mm, vias 0 -> 2
- net /VREF: track 0.00 -> 68.9 mm
- net /NSS1: track 0.00 -> 41.5 mm
- net /NSS2: track 0.00 -> 39.1 mm, vias 0 -> 2
- net /inverter/1VS3: track 0.00 -> 39.1 mm, vias 0 -> 9
- net +3V3: track 0.00 -> 37.0 mm, vias 0 -> 4
- net /inverter/1VS2: track 0.00 -> 28.7 mm, vias 0 -> 9
- net /inverter/1VS1: track 0.00 -> 27.5 mm, vias 0 -> 8
- net /inverter/2HO1: track 0.00 -> 27.1 mm, vias 0 -> 2
- net /inverter/1LO3: track 0.00 -> 26.9 mm
- net /USART2_RX: track 0.00 -> 26.2 mm, vias 0 -> 2
- net /inverter/2LO3: track 0.00 -> 24.8 mm, vias 0 -> 2
- net /inverter/1HO3: track 0.00 -> 22.9 mm, vias 0 -> 2
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- added copper zone on B.Cu, net +3V3
- added copper zone on B.Cu, net /2CS1+
- added copper zone on B.Cu, net /2CS2+
- added copper zone on B.Cu, net /inverter/1VS1
- added copper zone on B.Cu, net /inverter/1VS2
- added copper zone on B.Cu, net /inverter/1VS3
- added copper zone on B.Cu, net /inverter/2VS1
- added copper zone on B.Cu, net /inverter/2VS2
- added copper zone on B.Cu, net /inverter/2VS3
- added copper zone on F.Cu, net GNDPWR
- added copper zone on B.Cu, net Net-(D8-K)
- added copper zone on B.Cu, net Net-(Q1-S-Pad1)
- added copper zone on B.Cu, net Net-(Q16-S-Pad1)
- added copper zone on B.Cu, net Net-(Q8-S-Pad1)
- removed copper zone on F.Cu, net +3V3

Commit message: update driver pcb
Parts:
- C10, C11, C13, C17, C18, C19, C20, C21, C22, C23, C24, C27, C67, C68, C9, FB1, FB2, FB3, J3, J5, R20, R21, R49, R72, R73, U4, U5, U6, U7, U8, U9, Y1: moved to B.Cu
- moved J2 42.4 mm to (71.7, 70.3)
- moved U7 15.9 mm to (73.2, 61.7), turned to -90 degrees
- moved C10 15.8 mm to (76.1, 61.5), turned to -90 degrees
- moved C9 15.8 mm to (76.1, 65.0), turned to -90 degrees
- moved U6 15.7 mm to (73.2, 64.8), turned to -90 degrees
- moved D10 13.2 mm to (60.9, 65.8), turned to -90 degrees
- moved U8 12.7 mm to (82.2, 65.2), turned to 90 degrees
- moved C11 12.7 mm to (79.5, 65.1), turned to 90 degrees
- moved U9 12.7 mm to (82.3, 62.5), turned to 90 degrees
- moved C27 12.7 mm to (79.5, 61.7), turned to 90 degrees
- moved C18 12.5 mm to (84.6, 54.0), turned to 0 degrees
- moved C20 12.5 mm to (84.6, 52.4), turned to 0 degrees
- moved D3 12.2 mm to (94.6, 54.0), turned to 90 degrees
- moved C17 12.1 mm to (72.4, 48.1), turned to 180 degrees
- moved C19 11.9 mm to (72.4, 46.6), turned to 180 degrees
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Connections:
- CN2 pad 1: /inverter/2VS1 -> /inverter/2VS3
- CN2 pad 3: /inverter/2VS3 -> /inverter/2VS1
- D16 pad 1: /inverter/2HO3 -> /inverter/2HO1
- D17 pad 1: /inverter/2LO3 -> /inverter/2LO1
- D20 pad 1: /inverter/2HO1 -> /inverter/2HO3
- D21 pad 1: /inverter/2LO1 -> /inverter/2LO3
- Q11 pad 1: /inverter/2VS1 -> /inverter/2VS3
- Q11 pad 2: /inverter/2VS1 -> /inverter/2VS3
- Q11 pad 3: /inverter/2VS1 -> /inverter/2VS3
- Q12 pad 5: /inverter/2VS1 -> /inverter/2VS3
- Q12 pad 6: /inverter/2VS1 -> /inverter/2VS3
- Q12 pad 7: /inverter/2VS1 -> /inverter/2VS3
- Q12 pad 8: /inverter/2VS1 -> /inverter/2VS3
- Q7 pad 1: /inverter/2VS3 -> /inverter/2VS1
- Q7 pad 2: /inverter/2VS3 -> /inverter/2VS1
- Q7 pad 3: /inverter/2VS3 -> /inverter/2VS1
- Q8 pad 5: /inverter/2VS3 -> /inverter/2VS1
- Q8 pad 6: /inverter/2VS3 -> /inverter/2VS1
- Q8 pad 7: /inverter/2VS3 -> /inverter/2VS1
- Q8 pad 8: /inverter/2VS3 -> /inverter/2VS1
- R13 pad 1: /inverter/2HO3 -> /inverter/2HO1
- R14 pad 1: /inverter/2LO3 -> /inverter/2LO1
- R17 pad 1: /inverter/2HO1 -> /inverter/2HO3
- R18 pad 1: /inverter/2LO1 -> /inverter/2LO3
- R72 pad 2: /I2C2_SDA -> /I2C1_SDA
- R73 pad 2: /I2C2_SCL -> /I2C1_SCL
- TP4 pad 1: /inverter/2VS1 -> /inverter/2VS3
- TP6 pad 1: /inverter/2VS3 -> /inverter/2VS1
- U1 pad 1: /TIM8_CH1 -> /TIM1_CH3
- U1 pad 2: /TIM8_CH2 -> /TIM1_CH2
- U1 pad 3: /TIM8_CH3 -> /TIM1_CH1
- U1 pad 4: /TIM8_CH1 -> /TIM1_CH3
- U1 pad 5: /TIM8_CH2 -> /TIM1_CH2
- U1 pad 6: /TIM8_CH3 -> /TIM1_CH1
- U2 pad 1: /TIM1_CH1 -> /TIM8_CH3
- U2 pad 2: /TIM1_CH2 -> /TIM8_CH2
- U2 pad 3: /TIM1_CH3 -> /TIM8_CH1
- U2 pad 4: /TIM1_CH1 -> /TIM8_CH3
- U2 pad 5: /TIM1_CH2 -> /TIM8_CH2
- U2 pad 6: /TIM1_CH3 -> /TIM8_CH1
- U4 pad 23: /I2C2_SCL -> /I2C1_SCL
- U4 pad 24: /I2C2_SDA -> /I2C1_SDA
- U5 pad 16: unconnected-(U5-PC4-Pad16) -> /ADC2_IN5
- U5 pad 17: unconnected-(U5-PB0-Pad17) -> /ADC1_IN15
- U5 pad 25: unconnected-(U5-PB12-Pad25) -> /ADC1_IN11
- U5 pad 27: unconnected-(U5-PB14-Pad27) -> /ADC1_IN5
- U5 pad 28: unconnected-(U5-PB15-Pad28) -> /ADC2_IN15
- U6 pad 6: unconnected-(U6-OUT-Pad6) -> /ADC1_IN15
- U7 pad 6: unconnected-(U7-OUT-Pad6) -> /ADC2_IN5
- U9 pad 6: unconnected-(U9-OUT-Pad6) -> /ADC2_IN15
Routing:
- net GNDPWR: track 7.97 -> 113.2 mm, vias 0 -> 31
- net /SPI1_MOSI: track 90.5 -> 0.00 mm, vias 2 -> 0
- net /SPI1_MISO: track 89.9 -> 0.00 mm, vias 2 -> 0
- net /SPI1_SCK: track 86.6 -> 0.00 mm, vias 2 -> 0
- net /VREF: track 68.9 -> 19.5 mm
- net /NSS1: track 41.5 -> 0.00 mm
- net /NSS2: track 39.1 -> 0.00 mm, vias 2 -> 0
- net /USART2_RX: track 26.2 -> 1.62 mm, vias 2 -> 1
- net /1CS2+: track 9.23 -> 33.3 mm, vias 1 -> 2
- net /inverter/2VS3: track 19.0 -> 39.5 mm, vias 8 -> 9
- net /USART2_TX: track 21.6 -> 1.52 mm, vias 2 -> 1
- net /inverter/1LO2: track 21.5 -> 3.53 mm
- net +3V3: track 37.0 -> 53.0 mm, vias 4 -> 6
- net /1CS2-: track 10.2 -> 24.8 mm, vias 1 -> 2
- net /2CS1-: track 8.46 -> 22.6 mm, vias 1 -> 0
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
Commit message: update driver pcb
Parts:
- moved FB1 8.37 mm to (75.4, 32.5)
- moved J4 4.53 mm to (98.3, 38.4)
- moved J5 0.20 mm to (35.4, 42.3)
- moved C68 0.13 mm to (80.6, 45.6)
- moved Y1 0.10 mm to (77.8, 45.6)
- turned FB2 to 0 degrees
Connections:
- U5 pad 12: /NSS1 -> /NSS2
- U5 pad 43: /NSS2 -> /NSS1
Routing:
- net +3V3: track 53.0 -> 121.9 mm, vias 6 -> 0
- net /NSS2: track 0.00 -> 38.6 mm
- net /SPI1_SCK: track 0.00 -> 37.7 mm
- net /SPI1_MISO: track 0.00 -> 37.5 mm
- net /SPI1_MOSI: track 0.00 -> 37.3 mm
- net /I2C1_SCL: track 0.00 -> 17.5 mm, vias 0 -> 2
- net /I2C1_SDA: track 0.00 -> 13.5 mm, vias 0 -> 2
- net /inverter/2VS2: track 25.8 -> 31.9 mm, vias 8 -> 9
- net /YI: track 0.00 -> 5.98 mm
- net GNDD: track 5.98 -> 1.66 mm, vias 3 -> 1
- net Net-(U4-VDD): track 6.52 -> 10.5 mm
- net /YO: track 0.00 -> 3.90 mm
- net GNDPWR: track 113.2 -> 110.6 mm, vias 31 -> 27
- net /VREF: track 19.5 -> 21.7 mm, vias 0 -> 2
- net Net-(U4-REGOUT): track 0.00 -> 1.83 mm
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
Commit message: update driver pcb
Connections:
- J3 pad 3: /NSS2 -> /SPI1_SCK
- J3 pad 4: /SPI1_SCK -> /SPI1_MISO
- J3 pad 5: /SPI1_MISO -> /SPI1_MOSI
- J3 pad 6: /SPI1_MOSI -> /NSS2
- J5 pad 3: /NSS1 -> /SPI3_SCK
- J5 pad 4: /SPI1_SCK -> /SPI3_MISO
- J5 pad 5: /SPI1_MISO -> /SPI3_MOSI
- J5 pad 6: /SPI1_MOSI -> /NSS1
- U5 pad 12: /NSS2 -> unconnected-(U5-PA4-Pad12)
- U5 pad 16: /ADC2_IN5 -> unconnected-(U5-PC4-Pad16)
- U5 pad 19: unconnected-(U5-PB2-Pad19) -> /ADC2_IN12
- U5 pad 2: unconnected-(U5-PC13-Pad2) -> /NSS2
- U5 pad 39: unconnected-(U5-PC10-Pad39) -> /SPI3_SCK
- U5 pad 40: unconnected-(U5-PC11-Pad40) -> /SPI3_MISO
- U5 pad 41: unconnected-(U5-PB3-Pad41) -> /NSS1
- U5 pad 43: /NSS1 -> /SPI3_MOSI
- U6 pad 6: /ADC1_IN15 -> /ADC1_IN5
- U7 pad 6: /ADC2_IN5 -> /ADC2_IN15
- U8 pad 6: unconnected-(U8-OUT-Pad6) -> /ADC1_IN11
- U9 pad 6: /ADC2_IN15 -> /ADC2_IN12
Routing:
- net /NSS2: track 38.6 -> 0.72 mm, vias 0 -> 1
- net /SPI1_SCK: track 37.7 -> 7.58 mm
- net /SPI3_SCK: track 0.00 -> 21.5 mm, vias 0 -> 1
- net /SPI3_MISO: track 0.00 -> 20.3 mm, vias 0 -> 1
- net /SPI3_MOSI: track 0.00 -> 19.8 mm, vias 0 -> 1
- net /SPI1_MISO: track 37.5 -> 19.4 mm
- net /ADC2_IN12: track 0.00 -> 12.7 mm, vias 0 -> 2
- net /ADC1_IN5: track 0.00 -> 12.6 mm, vias 0 -> 2
- net /ADC1_IN11: track 0.00 -> 11.8 mm, vias 0 -> 2
- net /ADC2_IN15: track 0.00 -> 10.4 mm, vias 0 -> 2
- net +3V3: track 121.9 -> 112.6 mm
- net GNDA: track 3.73 -> 12.9 mm
- net /I2C1_SCL: track 17.5 -> 19.8 mm
- net GNDPWR: track 110.6 -> 109.5 mm
- net /NSS1: track 0.00 -> 1.07 mm
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
Commit message: update driver pcb
Parts:
- FB2: footprint Capacitor_SMD:C_1206_3216Metric_Pad1.33x1.80mm_HandSolder -> Capacitor_SMD:C_0603_1608Metric_Pad1.08x0.95mm_HandSolder
- J1: moved to F.Cu
- moved J2 12.2 mm to (83.9, 70.3), turned to -90 degrees
- moved J4 3.40 mm to (94.9, 38.3), turned to -90 degrees
- moved J1 0.51 mm to (35.3, 50.7)
- moved C68 0.23 mm to (80.6, 45.4)
Connections:
- J2 pad 1: /USART3_RX -> /USART3_TX
- J2 pad 2: /USART3_TX -> /USART3_RX
- J2 pad 3: /SWDIO -> +3V3
- J2 pad 4: /SWCLK -> GNDD
- J2 pad 5: +3V3 -> /SWDIO
- J2 pad 6: GNDD -> /SWCLK
- U5 pad 16: unconnected-(U5-PC4-Pad16) -> /NSS2
- U5 pad 2: /NSS2 -> /NSS1
- U5 pad 41: /NSS1 -> unconnected-(U5-PB3-Pad41)
Routing:
- net GNDD: track 1.66 -> 167.3 mm, vias 1 -> 17
- net +3V3: track 112.6 -> 170.2 mm, vias 0 -> 5
- net /NSS1: track 1.07 -> 46.3 mm, vias 0 -> 2
- net /NSS2: track 0.72 -> 37.5 mm, vias 1 -> 0
- net /SPI1_SCK: track 7.58 -> 38.2 mm
- net /SPI3_MOSI: track 19.8 -> 42.5 mm, vias 1 -> 2
- net +BATT: track 0.00 -> 22.6 mm, vias 0 -> 45
- net /SPI3_MISO: track 20.3 -> 42.6 mm, vias 1 -> 2
- net /USART2_TX: track 0.00 -> 21.6 mm, vias 0 -> 1
- net /SPI3_SCK: track 21.5 -> 42.3 mm, vias 1 -> 2
- net /USART2_RX: track 0.00 -> 20.3 mm, vias 0 -> 1
- net /USART3_TX: track 0.00 -> 19.6 mm, vias 0 -> 1
- net /SPI1_MISO: track 19.4 -> 37.9 mm
- net /inverter/1LO2: track 3.53 -> 21.9 mm, vias 0 -> 2
- net /SWCLK: track 0.00 -> 17.5 mm, vias 0 -> 1
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- added copper zone on In2.Cu, net +BATT
- added copper zone on F.Cu, net GNDD
- added copper zone on In1.Cu, net GNDPWR
- added copper zone on B.Cu, net Net-(Q12-S-Pad1)
- removed copper zone on B.Cu, net +BATT
- removed copper zone on B.Cu, net /2CS2+
- removed copper zone on F.Cu, net GNDPWR
Other:
- copper layers 2 -> 4
