File: hardware/main/bldcDriver.kicad_pcb (KiCad board)
At the start: 4 copper layers, 89.8 x 41.5 mm, 134 parts, among them CN1 MR30PW-F, CN2 MR30PW-F, J1 Conn_01x02, J2 Conn_01x06, J3 Conn_01x06, J4 Conn_01x03, J5 Conn_01x06, Q1 EMB09N03V, Q10 EMB09N03V, Q11 EMB09N03V, Q12 EMB09N03V, Q13 EMB09N03V, Q14 EMB09N03V, Q15 EMB09N03V, Q16 EMB09N03V, Q2 EMB09N03V, Q7 EMB09N03V, Q8 EMB09N03V, Q9 EMB09N03V, U1 EG2133, U2 EG2133, U3 TPS5430DDA, U4 MPU-6050, U5 STM32G431CBUx, U6 TP181A1-CR, U7 TP181A1-CR, U8 TP181A1-CR, U9 TP181A1-CR, Y1 25MHz

Commit message: update body
Parts:
- moved J1 1.07 mm to (35.6, 51.7)
Changed lines of the file:
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@@
 	(footprint "balancerDriver:CONN-TH_XT30UPB-M"
 		(layer "F.Cu")
-		(at 35.3 50.7 -90)
+		(at 35.62 51.72 -90)
 		(property "Reference" "J1"
 			(at 0 -3.207 90)
@@
 			)
 		)
-		(property ki_fp_filters "Connector*:*_1x??_*")
-		(sheetname "根目录")
-		(sheetfile "bldcDriver.kicad_sch")
 		(attr through_hole)
-		(fp_line
-			(start 5.1 2.6)
-			(end -2.506 2.6)
-			(stroke
-				(width 0.254)
-				(type solid)
-			)
-			(layer "F.SilkS")
-		)
-		(fp_line
-			(start -3.429 1.905)
-			(end -4.445 0.889)
-			(stroke
-				(width 0.254)
-				(type solid)
-			)
-			(layer "F.SilkS")
-		)
-		(fp_line
-			(start 4.445 1.905)
-			(end -3.429 1.905)
-			(stroke
-				(width 0.254)
-				(type solid)
-			)
-			(layer "F.SilkS")
-		)
-		(fp_line
-			(start -4.445 0.889)
-			(end -4.445 -1.016)
-			(stroke
-				(width 0.254)
-				(type solid)
-			)
-			(layer "F.SilkS")
-		)
-		(fp_line
-			(start -4.445 -1.016)
-			(end -3.429 -2.032)
-			(stroke
-				(width 0.254)
-				(type solid)
-			)
-			(layer "F.SilkS")
-		)
-		(fp_line
-			(start -3.429 -2.032)
-			(end 4.445 -2.032)
-			(stroke
-				(width 0.254)
-				(type solid)
-			)
-			(layer "F.SilkS")
-		)
-		(fp_line
-			(start 4.445 -2.032)
-			(end 4.445 1.905)
-			(stroke
-				(width 0.254)
-				(type solid)
-			)
-			(layer "F.SilkS")
-		)
-		(fp_line
-			(start -2.597 -2.6)
-			(end 5.1 -2.6)
-			(stroke
-				(width 0.254)
-				(type solid)
-			)
-			(layer "F.SilkS")
-		)
-		(fp_line
-			(start 5.1 -2.6)
-			(end 5.1 2.6)
-			(stroke
-				(width 0.254)
-				(type solid)
-			)
-			(layer "F.SilkS")
-		)
-		(fp_arc
-			(start -2.506 2.6)
-			(mid -5.14388 0.04546)
-			(end -2.596919 -2.599739)
-			(stroke
-				(width 0.254)
-				(type solid)
-			)
-			(layer "F.SilkS")
-		)
-		(fp_poly
-			(pts
-				(xy -2.667 -2.413) (xy -3.138 -2.367) (xy -3.59 -2.229) (xy -4.008 -2.006) (xy -4.373 -1.706) (xy -4.673 -1.341)
-				(xy -4.896 -0.923) (xy -5.034 -0.471) (xy -5.08 0) (xy -5.034 0.471) (xy -4.896 0.923) (xy -4.673 1.341)
-				(xy -4.373 1.706) (xy -4.008 2.006) (xy -3.59 2.229) (xy -3.138 2.367) (xy -2.667 2.413) (xy -2.642 2.415)
-				(xy -2.618 2.423) (xy -2.596 2.434) (xy -2.577 2.45) (xy -2.561 2.469) (xy -2.55 2.491) (xy -2.542 2.515)
-				(xy -2.54 2.54) (xy -2.542 2.565) (xy -2.55 2.589) (xy -2.561 2.611) (xy -2.577 2.63) (xy -2.596 2.646)
-				(xy -2.618 2.657) (xy -2.642 2.665) (xy -2.667 2.667) (xy -3.187 2.616) (xy -3.688 2.464) (xy -4.149 2.218)
-				(xy -4.553 1.886) (xy -4.885 1.482) (xy -5.131 1.021) (xy -5.283 0.52) (xy -5.334 0) (xy -5.283 -0.52)
-				(xy -5.131 -1.021) (xy -4.885 -1.482) (xy -4.553 -1.886) (xy -4.149 -2.218) (xy -3.688 -2.464) (xy -3.187 -2.616)
-				(xy -2.667 -2.667) (xy -2.642 -2.665) (xy -2.618 -2.657) (xy -2.596 -2.646) (xy -2.577 -2.63) (xy -2.561 -2.611)
-				(xy -2.55 -2.589) (xy -2.542 -2.565) (xy -2.54 -2.54) (xy -2.542 -2.515) (xy -2.55 -2.491) (xy -2.561 -2.469)
-				(xy -2.577 -2.45) (xy -2.596 -2.434) (xy -2.618 -2.423) (xy -2.642 -2.415) (xy -2.667 -2.413)
-			)
-			(stroke
-				(width 0.12)
-				(type solid)
-			)
-			(fill solid)
-			(layer "Dwgs.User")
-		)
-		(fp_circle
-			(center -5.1 2.8)
-			(end -5.07 2.8)
-			(stroke
-				(width 0.06)
-				(type solid)
-			)
-			(fill none)
-			(layer "Eco2.User")
-		)
 		(fp_circle
 			(center -2.5 0)
@@
 			(layer "Eco2.User")
 		)
-		(fp_circle
-			(center 2.5 0)
-			(end 2.9 0)
-			(stroke
-				(width 0.8)
-				(type solid)
-			)
-			(fill none)
-			(layer "Eco2.User")
-		)
-		(fp_line
-			(start -5.1 2.8)
-			(end -5.1 -2.8)
-			(stroke
-				(width 0.12)
-				(type solid)
-			)
-			(layer "F.CrtYd")
-		)
-		(fp_line
-			(start 5.1 2.8)
-			(end -5.1 2.8)
-			(stroke
-				(width 0.12)
-				(type solid)
-			)
-			(layer "F.CrtYd")
-		)
-		(fp_line
-			(start -5.1 -2.8)
-			(end 5.1 -2.8)
-			(stroke
-				(width 0.12)
-				(type solid)
-			)
-			(layer "F.CrtYd")
-		)
-		(fp_line
-			(start 5.1 -2.8)
-			(end 5.1 2.8)
-			(stroke
-				(width 0.12)
-				(type solid)
-			)
-			(layer "F.CrtYd")
-		)
 		(fp_text user "+"
-			(at 5.334 0.008 90)
+			(at 3.21 -0.02 90)
 			(layer "F.SilkS")
 			(effects
@@
 		)
 		(fp_text user "-"
-			(at -6.223 -0.119 90)
+			(at -5.02 0.07 90)
 			(layer "F.SilkS")
 			(effects
@@
 		)
 		(pad "2" thru_hole circle
-			(at 2.5 0 270)
+			(at 1.5 0 270)
 			(size 2.5 2.5)
 			(drill 1.8)

Commit message: update motor pcb
Parts:
- removed C12, C14, C33, C34: 22u, Capacitor_SMD:C_0805_2012Metric_Pad1.18x1.45mm_HandSolder
- removed U9: TP181A1-CR, balancerDriver:SC70-6_L2.1-W1.3-P0.65-LS2.3-BL
- added C38: 4.7u, Capacitor_SMD:C_0603_1608Metric_Pad1.08x0.95mm_HandSolder, B.Cu at (74.3, 56.5)
- added C39: 100n, Capacitor_SMD:C_0603_1608Metric_Pad1.08x0.95mm_HandSolder, B.Cu at (71.8, 57.4)
- added C40: 100n, Capacitor_SMD:C_0603_1608Metric_Pad1.08x0.95mm_HandSolder, B.Cu at (68.7, 50.6)
- added C41: 2.2n, Capacitor_SMD:C_0603_1608Metric_Pad1.08x0.95mm_HandSolder, B.Cu at (79.0, 60.2)
- added C42: 2.2n, Capacitor_SMD:C_0603_1608Metric_Pad1.08x0.95mm_HandSolder, B.Cu at (65.0, 59.6)
- added C43: 4.7u, Capacitor_SMD:C_0603_1608Metric_Pad1.08x0.95mm_HandSolder, B.Cu at (67.2, 53.9)
- added C44: 4.7u, Capacitor_SMD:C_0603_1608Metric_Pad1.08x0.95mm_HandSolder, B.Cu at (79.2, 51.4)
- added C45: 100n, Capacitor_SMD:C_0603_1608Metric_Pad1.08x0.95mm_HandSolder, B.Cu at (82.4, 60.2)
- added C46: 100n, Capacitor_SMD:C_0603_1608Metric_Pad1.08x0.95mm_HandSolder, B.Cu at (68.3, 60.2)
- added C47: 100n, Capacitor_SMD:C_0603_1608Metric_Pad1.08x0.95mm_HandSolder, B.Cu at (68.7, 54.0)
- added C48: 100n, Capacitor_SMD:C_0603_1608Metric_Pad1.08x0.95mm_HandSolder, B.Cu at (77.7, 51.4)
- added R30: 1k, Resistor_SMD:R_0603_1608Metric_Pad0.98x0.95mm_HandSolder, B.Cu at (89.0, 66.0)
- added R31: 10k, Resistor_SMD:R_0603_1608Metric_Pad0.98x0.95mm_HandSolder, B.Cu at (90.5, 66.0)
- added R32: 1k, Resistor_SMD:R_0603_1608Metric_Pad0.98x0.95mm_HandSolder, B.Cu at (75.8, 66.7)
- added R33: 10k, Resistor_SMD:R_0603_1608Metric_Pad0.98x0.95mm_HandSolder, B.Cu at (75.8, 65.2)
- added R34: 10k, Resistor_SMD:R_0603_1608Metric_Pad0.98x0.95mm_HandSolder, B.Cu at (89.0, 62.6)
- added R35: 100R, Resistor_SMD:R_0603_1608Metric_Pad0.98x0.95mm_HandSolder, B.Cu at (89.1, 60.2)
- added R36: 10k, Resistor_SMD:R_0603_1608Metric_Pad0.98x0.95mm_HandSolder, B.Cu at (74.9, 62.7)
- added R37: 100R, Resistor_SMD:R_0603_1608Metric_Pad0.98x0.95mm_HandSolder, B.Cu at (75.1, 60.2)
- added R38: 1k, Resistor_SMD:R_0603_1608Metric_Pad0.98x0.95mm_HandSolder, B.Cu at (79.2, 54.8)
- added R39: 1k, Resistor_SMD:R_0603_1608Metric_Pad0.98x0.95mm_HandSolder, B.Cu at (77.7, 54.8)
- added R40: 1k, Resistor_SMD:R_0603_1608Metric_Pad0.98x0.95mm_HandSolder, B.Cu at (70.2, 57.4)
- added R41: 1k, Resistor_SMD:R_0603_1608Metric_Pad0.98x0.95mm_HandSolder, B.Cu at (68.7, 57.4)
- added R42: 1k, Resistor_SMD:R_0603_1608Metric_Pad0.98x0.95mm_HandSolder, B.Cu at (78.5, 64.1)
- added R43: 1k, Resistor_SMD:R_0603_1608Metric_Pad0.98x0.95mm_HandSolder, B.Cu at (64.3, 63.5)
- added R44: 1k, Resistor_SMD:R_0603_1608Metric_Pad0.98x0.95mm_HandSolder, B.Cu at (82.5, 67.2)
- added R45: 10k, Resistor_SMD:R_0603_1608Metric_Pad0.98x0.95mm_HandSolder, B.Cu at (80.0, 67.4)
- added R46: 1k, Resistor_SMD:R_0603_1608Metric_Pad0.98x0.95mm_HandSolder, B.Cu at (65.9, 66.8)
- added R47: 10k, Resistor_SMD:R_0603_1608Metric_Pad0.98x0.95mm_HandSolder, B.Cu at (68.4, 67.2)
- added R48: 10k, Resistor_SMD:R_0603_1608Metric_Pad0.98x0.95mm_HandSolder, B.Cu at (80.0, 64.1)
- added R50: 100R, Resistor_SMD:R_0603_1608Metric_Pad0.98x0.95mm_HandSolder, B.Cu at (79.1, 61.7)
- added R51: 10k, Resistor_SMD:R_0603_1608Metric_Pad0.98x0.95mm_HandSolder, B.Cu at (65.9, 63.5)
- added R52: 100R, Resistor_SMD:R_0603_1608Metric_Pad0.98x0.95mm_HandSolder, B.Cu at (65.0, 61.0)
- C11, C27: value 100n -> 2.2n
- C15, C32: value 100n -> 1u
- C9: value 100n -> 4.7u
- R20, R21: value 10k -> 1k
- U6, U7, U8: value TP181A1-CR -> TLV9062xD; footprint balancerDriver:SC70-6_L2.1-W1.3-P0.65-LS2.3-BL -> Package_SO:SOIC-8_3.9x4.9mm_P1.27mm
- moved U8 15.1 mm to (73.2, 53.0), turned to 180 degrees
- moved FB1 14.8 mm to (90.1, 34.5)
- moved C22 14.7 mm to (91.6, 34.5)
- moved C23 14.6 mm to (93.1, 34.5)
- moved R72 14.6 mm to (90.9, 43.6)
- moved R73 14.6 mm to (92.4, 43.6)
- moved C24 14.5 mm to (93.9, 43.6)
- moved U4 14.5 mm to (92.8, 39.2)
- moved R49 14.5 mm to (94.6, 34.5)
- moved C13 14.4 mm to (96.2, 37.1)
- moved FB3 13.2 mm to (83.7, 54.7), turned to 90 degrees
- moved R20 13.0 mm to (90.5, 62.6), turned to 90 degrees
- moved C9 11.9 mm to (82.2, 54.7)
- moved J4 11.8 mm to (106.5, 40.7), turned to 90 degrees
- moved U6 11.4 mm to (84.5, 63.7), turned to 180 degrees
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Connections:
- C10 pad 1: GNDA -> GNDD
- C10 pad 2: Net-(U7-V+) -> /OP_VCC
- C11 pad 1: GNDA -> GNDD
- C11 pad 2: Net-(U8-V+) -> /ADC2_IN12
- C27 pad 1: GNDA -> GNDD
- C27 pad 2: Net-(U9-V+) -> /ADC1_IN5
- C9 pad 1: GNDA -> GNDD
- C9 pad 2: Net-(U6-V+) -> /OP_VCC
- FB3 pad 1: GNDA -> /OP_VCC
- FB3 pad 2: GNDD -> +3V3
- J2 pad 1: /USART3_TX -> +3V3
- J2 pad 2: /USART3_RX -> GNDD
- J2 pad 3: +3V3 -> /USART3_TX
- J2 pad 4: GNDD -> /USART3_RX
- J4 pad 1: /USART2_TX -> GNDD
- J4 pad 3: GNDD -> /USART2_TX
- J5 pad 1: GNDD -> /NSS1
- J5 pad 2: +3V3 -> /SPI3_MOSI
- J5 pad 3: /SPI3_SCK -> /SPI3_MISO
- J5 pad 4: /SPI3_MISO -> /SPI3_SCK
- J5 pad 5: /SPI3_MOSI -> +3V3
- J5 pad 6: /NSS1 -> GNDD
- R20 pad 1: +3V3 -> Net-(U6A--)
- R20 pad 2: /VREF -> /2CS1+
- R21 pad 1: /VREF -> Net-(U7A--)
- R21 pad 2: GNDA -> /1CS1+
- U5 pad 12: unconnected-(U5-PA4-Pad12) -> /MPU_INT
- U5 pad 2: /NSS1 -> unconnected-(U5-PC13-Pad2)
- U5 pad 41: unconnected-(U5-PB3-Pad41) -> /NSS1
- U6 pad 1: /VREF -> Net-(R34-Pad2)
- U6 pad 2: GNDA -> Net-(U6A--)
- U6 pad 3: Net-(U6-V+) -> Net-(U6A-+)
- U6 pad 4: /1CS1+ -> GNDD
- U6 pad 5: /1CS1- -> Net-(U6B-+)
- U6 pad 6: /ADC1_IN5 -> Net-(U6B--)
- U7 pad 1: /VREF -> Net-(R36-Pad2)
- U7 pad 2: GNDA -> Net-(U7A--)
- U7 pad 3: Net-(U7-V+) -> Net-(U7A-+)
- U7 pad 4: /1CS2+ -> GNDD
- U7 pad 5: /1CS2- -> Net-(U7B-+)
- U7 pad 6: /ADC2_IN15 -> Net-(U7B--)
- U8 pad 1: /VREF -> /VREF_OP1
- U8 pad 2: GNDA -> /VREF_OP1
- U8 pad 3: Net-(U8-V+) -> /INA1+
- U8 pad 4: /2CS1+ -> GNDD
- U8 pad 5: /2CS1- -> /INA2+
- U8 pad 6: /ADC1_IN11 -> /VREF_OP2
Routing:
- net GNDD: track 167.3 -> 13.7 mm, vias 17 -> 46
- net GNDPWR: track 111.9 -> 36.4 mm, vias 31 -> 46
- net /OP_VCC: track 0.00 -> 39.7 mm, vias 0 -> 2
- net /VREF_OP2: track 0.00 -> 35.7 mm, vias 0 -> 2
- net /VREF_OP1: track 0.00 -> 28.9 mm, vias 0 -> 2
- net GNDA: track 28.5 -> 0.00 mm, vias 3 -> 0
- net /1CS1+: track 26.1 -> 49.0 mm
- net /VREF: track 21.7 -> 0.00 mm, vias 2 -> 0
- net /MPU_INT: track 4.66 -> 24.2 mm
- net /inverter/2VS3: track 39.5 -> 22.9 mm, vias 9 -> 13
- net +BATT: track 22.6 -> 7.09 mm, vias 45 -> 81
- net /inverter/1VS3: track 39.1 -> 24.5 mm, vias 9 -> 14
- net /1CS1-: track 23.9 -> 37.5 mm
- net /ADC2_IN15: track 10.4 -> 23.4 mm
- net /inverter/2VS2: track 31.9 -> 19.6 mm, vias 9 -> 14
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