File: hardware/main/untitled.kicad_sch (KiCad schematic)
At the start: 58 parts, among them CN1 MR30PW-F, CN2 MR30PW-F, Q1 NMOS, Q10 NMOS, Q11 NMOS, Q12 NMOS, Q2 NMOS, Q3 NMOS, Q4 NMOS, Q5 NMOS, Q6 NMOS, Q7 NMOS, Q8 NMOS, Q9 NMOS, U1 EG2133, U2 EG2133

Commit message: update driver pcb
Parts:
- removed D12, D13, D14, D15: 1N4148W, Diode_SMD:D_SOD-123, symbol Diode:1N4148W
- removed Q1, Q10, Q11, Q12, Q2, Q3, Q4, Q5, Q6, Q7, Q8, Q9: NMOS, symbol Simulation_SPICE:NMOS
- removed R10, R11, R12, R9: 10R, symbol Device:R_Small
- added D22, D23, D24, D9: 1N4148W, Diode_SMD:D_SOD-123, symbol Diode:1N4148W
- added Q1, Q10, Q11, Q12, Q13, Q14, Q15, Q16, Q2, Q7, Q8, Q9: EMB09N03V, balancerDriver:POWERTDFN-8_L3.1-W3.1-P0.65-LS3.3-BL, symbol bldcDriver:EMB09N03V
- added R10, R11, R12, R9: 10mR, Resistor_SMD:R_2512_6332Metric_Pad1.40x3.35mm_HandSolder, symbol Device:R
- added R19, R4, R5, R6: 10R, Resistor_SMD:R_0603_1608Metric_Pad0.98x0.95mm_HandSolder, symbol Device:R_Small
- C12, C14, C33, C34: value 100n -> 22u; footprint Capacitor_SMD:C_0603_1608Metric_Pad1.08x0.95mm_HandSolder -> Capacitor_SMD:C_0805_2012Metric_Pad1.18x1.45mm_HandSolder
- CN1, CN2: footprint balancerDriver:CONN-TH_MR30PW-F -> balancerDriver:CONN-SMD_3P-P1.00_BX-SH1.0-3PWT
- D10, D11, D2, D3, D4, D7: footprint (none) -> balancerDriver:SOD-123FL_L2.7-W1.8-LS3.8-RD
- R13, R14, R15, R16, R17, R18, R7, R8: footprint (none) -> Resistor_SMD:R_0603_1608Metric_Pad0.98x0.95mm_HandSolder
Connections:
- net +12V is gone; now on net +BATT: D10.2 (A), D11.2 (A), D2.2 (A), D3.2 (A), D4.2 (A), D7.2 (A)
- net 1SH_U is gone; now on net 1VS3: CN1.1
- net 1SH_V is gone; now on net 1VS2: CN1.2
- net 1SH_W is gone; now on net 1VS1: CN1.3
- net 2SH_U is gone; now on net 2VS1: CN2.3
- net 2SH_V is gone; now on net 2VS2: CN2.2
- net 2SH_W is gone; now on net 2VS3: CN2.1
- net +BATT: now also Q11.5 (D), Q11.6 (D), Q11.7 (D), Q11.8 (D), Q13.5 (D), Q13.6 (D), Q13.7 (D), Q13.8 (D), Q15.5 (D), Q15.6 (D), Q15.7 (D), Q15.8 (D), Q2.5 (D), Q2.6 (D), Q2.7 (D), Q2.8 (D), Q7.5 (D), Q7.6 (D), Q7.7 (D), Q7.8 (D), Q9.5 (D), Q9.6 (D), Q9.7 (D), Q9.8 (D)
- net 1HO2: now also D9.1 (K), R4.1
- net 1HO3: now also D23.1 (K), R6.1
- net 1LO2: now also D22.1 (K), R5.1; no longer D19.1 (K), R16.1
- net 1LO3: now also D24.1 (K), R19.1
- net 1VS1: now also Q1.5 (D), Q1.6 (D), Q1.7 (D), Q1.8 (D), Q13.1 (S), Q13.2 (S), Q13.3 (S)
- net 1VS2: now also Q14.5 (D), Q14.6 (D), Q14.7 (D), Q14.8 (D), Q2.1 (S), Q2.2 (S), Q2.3 (S)
- net 1VS3: now also Q15.1 (S), Q15.2 (S), Q15.3 (S), Q16.5 (D), Q16.6 (D), Q16.7 (D), Q16.8 (D)
- net 2LO1: now also D17.1 (K), R14.1
- net 2LO2: now also D19.1 (K), R16.1
- net 2VS1: now also Q7.1 (S), Q7.2 (S), Q7.3 (S), Q8.5 (D), Q8.6 (D), Q8.7 (D), Q8.8 (D); no longer D17.1 (K), R14.1
- net 2VS2: now also Q10.5 (D), Q10.6 (D), Q10.7 (D), Q10.8 (D), Q9.1 (S), Q9.2 (S), Q9.3 (S)
- net 2VS3: now also Q11.1 (S), Q11.2 (S), Q11.3 (S), Q12.5 (D), Q12.6 (D), Q12.7 (D), Q12.8 (D)
- net GNDPWR: now also Q10.1 (S), Q10.2 (S), Q10.3 (S), Q14.1 (S), Q14.2 (S), Q14.3 (S), R10.1, R11.1, R12.1, R9.1
- net at D17.2 (A), R14.2: now also Q8.4 (G)
- net at D16.2 (A), R13.2: now also Q7.4 (G)
- net at D18.2 (A), R15.2: now also Q9.4 (G)
- net at D20.2 (A), R17.2: now also Q11.4 (G)
- net at D6.2 (A), R7.2: now also Q1.4 (G)
- net at D5.2 (A), R8.2: now also Q13.4 (G)
- net at D21.2 (A), R18.2: now also Q12.4 (G)
- net at D19.2 (A), R16.2: now also Q10.4 (G)
- new net: D22.2 (A), Q14.4 (G), R5.2
- new net: D24.2 (A), Q16.4 (G), R19.2
- new net: D9.2 (A), Q2.4 (G), R4.2
- new net: D23.2 (A), Q15.4 (G), R6.2
- new net 1CS1: Q1.1 (S), Q1.2 (S), Q1.3 (S), R9.2
- new net 1CS2: Q16.1 (S), Q16.2 (S), Q16.3 (S), R10.2
- new net 2CS1: Q8.1 (S), Q8.2 (S), Q8.3 (S), R11.2
- new net 2CS2: Q12.1 (S), Q12.2 (S), Q12.3 (S), R12.2
Other:
- moved on the sheet: CN1, D5, D6, R7, R8

Commit message: update driver pcb
Parts:
- added C28, C35, C36, C37: 1n, Capacitor_SMD:C_0603_1608Metric_Pad1.08x0.95mm_HandSolder, symbol Device:C_Small
- added R22, R23, R24, R25, R26, R27, R28, R29: 100R, Resistor_SMD:R_0603_1608Metric_Pad0.98x0.95mm_HandSolder, symbol Device:R
- added TP1, TP2, TP3, TP4, TP5, TP6: TestPoint, TestPoint:TestPoint_Pad_1.0x1.0mm, symbol Connector:TestPoint
- R10, R11, R12, R9: footprint Resistor_SMD:R_2512_6332Metric_Pad1.40x3.35mm_HandSolder -> Resistor_SMD:R_1206_3216Metric_Pad1.30x1.75mm_HandSolder
Connections:
- net 1HO1: now also D23.1 (K), R6.1; no longer D5.1 (K), R8.1
- net 1HO3: now also D5.1 (K), R8.1; no longer D23.1 (K), R6.1
- net 1LO1: now also D24.1 (K), R19.1; no longer D6.1 (K), R7.1
- net 1LO3: now also D6.1 (K), R7.1; no longer D24.1 (K), R19.1
- net 1VS1: now also Q15.1 (S), Q15.2 (S), Q15.3 (S), Q16.5 (D), Q16.6 (D), Q16.7 (D), Q16.8 (D), TP3.1; no longer Q1.5 (D), Q1.6 (D), Q1.7 (D), Q1.8 (D), Q13.1 (S), Q13.2 (S), Q13.3 (S)
- net 1VS2: now also TP2.1
- net 1VS3: now also Q1.5 (D), Q1.6 (D), Q1.7 (D), Q1.8 (D), Q13.1 (S), Q13.2 (S), Q13.3 (S), TP1.1; no longer Q15.1 (S), Q15.2 (S), Q15.3 (S), Q16.5 (D), Q16.6 (D), Q16.7 (D), Q16.8 (D)
- net 2HO1: now also D20.1 (K), R17.1; no longer D16.1 (K), R13.1
- net 2HO3: now also D16.1 (K), R13.1; no longer D20.1 (K), R17.1
- net 2LO1: now also D21.1 (K), R18.1; no longer D17.1 (K), R14.1
- net 2LO3: now also D17.1 (K), R14.1; no longer D21.1 (K), R18.1
- net 2VS1: now also CN2.1, Q11.1 (S), Q11.2 (S), Q11.3 (S), Q12.5 (D), Q12.6 (D), Q12.7 (D), Q12.8 (D), TP4.1; no longer CN2.3, Q7.1 (S), Q7.2 (S), Q7.3 (S), Q8.5 (D), Q8.6 (D), Q8.7 (D), Q8.8 (D)
- net 2VS2: now also TP5.1
- net 2VS3: now also CN2.3, Q7.1 (S), Q7.2 (S), Q7.3 (S), Q8.5 (D), Q8.6 (D), Q8.7 (D), Q8.8 (D), TP6.1; no longer CN2.1, Q11.1 (S), Q11.2 (S), Q11.3 (S), Q12.5 (D), Q12.6 (D), Q12.7 (D), Q12.8 (D)
- net GNDPWR: now also R23.1, R25.1, R27.1, R29.1
- net 1CS1: no longer names the net of Q1.1 (S), Q1.2 (S), Q1.3 (S), R9.2
- net 1CS1: now also R22.1
- net 1CS2: no longer names the net of Q16.1 (S), Q16.2 (S), Q16.3 (S), R10.2
- net 1CS2: now also R24.1
- net 2CS1: no longer names the net of Q8.1 (S), Q8.2 (S), Q8.3 (S), R11.2
- net 2CS1: now also R26.1
- net 2CS2: no longer names the net of Q12.1 (S), Q12.2 (S), Q12.3 (S), R12.2
- net 2CS2: now also R28.1
- new net 1CS1+: C28.2, R22.2
- new net 1CS1-: C28.1, R23.2
- new net 1CS2+: C35.2, R24.2
- new net 1CS2-: C35.1, R25.2
- new net 2CS1+: C36.2, R26.2
- new net 2CS1-: C36.1, R27.2
- new net 2CS2+: C37.2, R28.2
- new net 2CS2-: C37.1, R29.2
Other:
- moved on the sheet: R10, R11, R12, R9

Commit message: update driver pcb
Connections:
- net 2HO1: now also D16.1 (K), R13.1; no longer D20.1 (K), R17.1
- net 2HO3: now also D20.1 (K), R17.1; no longer D16.1 (K), R13.1
- net 2LO1: now also D17.1 (K), R14.1; no longer D21.1 (K), R18.1
- net 2LO3: now also D21.1 (K), R18.1; no longer D17.1 (K), R14.1
- net 2VS1: now also CN2.3, Q7.1 (S), Q7.2 (S), Q7.3 (S), Q8.5 (D), Q8.6 (D), Q8.7 (D), Q8.8 (D), TP6.1; no longer CN2.1, Q11.1 (S), Q11.2 (S), Q11.3 (S), Q12.5 (D), Q12.6 (D), Q12.7 (D), Q12.8 (D), TP4.1
- net 2VS3: now also CN2.1, Q11.1 (S), Q11.2 (S), Q11.3 (S), Q12.5 (D), Q12.6 (D), Q12.7 (D), Q12.8 (D), TP4.1; no longer CN2.3, Q7.1 (S), Q7.2 (S), Q7.3 (S), Q8.5 (D), Q8.6 (D), Q8.7 (D), Q8.8 (D), TP6.1
- net TIM1_CH1: now also U1.3 (HIN3), U1.6 (LIN3#); no longer U2.1 (HIN1), U2.4 (LIN1#)
- net TIM1_CH2: now also U1.2 (HIN2), U1.5 (LIN2#); no longer U2.2 (HIN2), U2.5 (LIN2#)
- net TIM1_CH3: now also U1.1 (HIN1), U1.4 (LIN1#); no longer U2.3 (HIN3), U2.6 (LIN3#)
- net TIM8_CH1: now also U2.3 (HIN3), U2.6 (LIN3#); no longer U1.1 (HIN1), U1.4 (LIN1#)
- net TIM8_CH2: now also U2.2 (HIN2), U2.5 (LIN2#); no longer U1.2 (HIN2), U1.5 (LIN2#)
- net TIM8_CH3: now also U2.1 (HIN1), U2.4 (LIN1#); no longer U1.3 (HIN3), U1.6 (LIN3#)
Other:
- moved on the sheet: C28, C35, CN1, D22, D23, D24, D5, D6, D9, Q1, Q13, Q14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

Commit message: update motor pcb
Parts:
- removed C12, C14, C33, C34: 22u, Capacitor_SMD:C_0805_2012Metric_Pad1.18x1.45mm_HandSolder, symbol Device:C_Small
- C15, C32: value 100n -> 1u
