File: hardware/rfBat/bat_rf.kicad_sch (KiCad schematic)
At the start: 83 parts, among them J1 USB_C_Receptacle_PowerOnly_6P, J2 Conn_01x04, Q1 NMOS, Q2 PMOS, Q3 NMOS, SW2 RESET, SW3 SW_MEC_5E, U1 ESP8684-WROOM-01C, U2 IP2325_5M_WHJC, U4 AMS1117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

Commit message: update rfBat pcb
Parts:
- removed C11, C7: 10u, Capacitor_SMD:C_0805_2012Metric_Pad1.18x1.45mm_HandSolder, symbol Device:C
- removed C8, C9: 100n, Capacitor_SMD:C_0603_1608Metric_Pad1.08x0.95mm_HandSolder, symbol Device:C
- removed TP7, TP8, TP9: TestPoint, TestPoint:TestPoint_Pad_D1.0mm, symbol Connector:TestPoint
- removed U5: AMS1117, Package_TO_SOT_SMD:SOT-223-3_TabPin2, symbol Regulator_Linear:AMS1117
- added C11, C17, C9: 100n, Capacitor_SMD:C_0603_1608Metric_Pad1.08x0.95mm_HandSolder, symbol Device:C_Small
- added C15, C8: 10u, Capacitor_SMD:C_0805_2012Metric_Pad1.18x1.45mm_HandSolder, symbol Device:C_Small
- added C7: 10n, Capacitor_SMD:C_0603_1608Metric_Pad1.08x0.95mm_HandSolder, symbol Device:C_Small
- added FB1: FerriteBead_Small, Capacitor_SMD:C_0805_2012Metric_Pad1.18x1.45mm_HandSolder, symbol Device:FerriteBead_Small
- added J3: Conn_01x02_Socket, bat_rf:CONN-TH_XT30UPB-F, symbol Connector:Conn_01x02_Socket
- added LED11, LED12: XL-4020RGBC-WS2812B, bat_rf:LED-SMD_4P-L4.0-W1.7_M4020-03003-RGB-862-001, symbol bat_rf:XL-4020RGBC-WS2812B
- added U3: SPX3819M5-L-3-3, Package_TO_SOT_SMD:SOT-23-5, symbol Regulator_Linear:SPX3819M5-L-3-3
- J2: footprint bat_rf:CONN-SMD_4P-P2.54_XH2.54-4AB_vertical -> Connector_Samtec_MicroMate:Samtec_T1M-04-X-S-V_1x04-1MP_P1.0mm_Terminal_Vertical
- L2: footprint Inductor_SMD_Wurth:L_Wurth_WE-LQSH-4020 -> Inductor_SMD:L_Vishay_IHLP-4040
- R11: footprint Button_Switch_SMD:SW_SPST_B3S-1000 -> Resistor_SMD:R_0603_1608Metric_Pad0.98x0.95mm_HandSolder
- SW3: footprint Button_Switch_SMD:SW_Push_1P1T_NO_6x6mm_H9.5mm -> bat_rf:SW-SMD_EVQPUD02K
- U4: footprint Package_TO_SOT_SMD:SOT-223-3_TabPin2 -> Package_TO_SOT_SMD:SOT-89-3_Handsoldering
Connections:
- net +3V3: now also C8.1, C9.1, U3.5 (OUT)
- net +5V: now also C1.1, C2.1, U4.3 (VI), C11.2, C15.1, C17.2, LED11.3 (VDD), LED12.3 (VDD), U3.1 (IN), U3.3 (EN)
- net +BATT: now also C3.1, C4.1, U4.2 (VO), J3.2 (Pin_2)
- net GNDD: now also Q3.3 (S), R11.1, SW3.1, SW3.2, C15.2, C7.2, C8.2, C9.2, FB1.2, U3.2 (GND)
- net GNDPWR: now also C1.2, C2.2, C3.2, C4.2, U4.1 (ADJ), C11.1, C17.1, FB1.1, J3.1 (Pin_1), LED11.1 (VSS), LED12.1 (VSS)
- net at LED8.2 (DO): now also LED12.4 (DI)
- removed net GND: C1.2, C2.2, C3.2, C4.2, Q3.3 (S), R11.1, SW3.1, SW3.2, U4.1 (ADJ)
- new net: C7.1, U3.4 (BP)
- new net: LED11.4 (DI), LED12.2 (DO)
Other:
- moved on the sheet: C14, C30, C31, C32, C33, C34, C35, C36, C5, C6, D13, J2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

Commit message: update rfBat pcb
Parts:
- added D3, D4: LED, LED_SMD:LED_0603_1608Metric_Pad1.05x0.95mm_HandSolder, symbol Device:LED
- added R15, R5: 1k, Resistor_SMD:R_0603_1608Metric_Pad0.98x0.95mm_HandSolder, symbol Device:R
Connections:
- net +3V3: no longer R13.1
- net BAT_FB: now also U1.5 (GPIO4/ADC1_CH4/FSPIHD/MTMS/LEDPWM); no longer U1.20 (GPIO3/ADC1_CH3/LEDPWM)
- net EN: now also C16.1, R12.1, U1.3 (EN)
- net ESP_RX: now also U1.17 (GPIO8); no longer U1.7 (GPIO6/FSPICLK/MTCK/LEDPWM)
- net ESP_TX: now also U1.16 (GPIO7/FSPID/MTDO/LEDPWM); no longer U1.6 (GPIO5/FSPIWP/MTDI/LEDPWM)
- net IO9: now also R4.1, U1.18 (GPIO9)
- net KEY: now also U1.12 (GPIO18); no longer U1.5 (GPIO4/ADC1_CH4/FSPIHD/MTMS/LEDPWM)
- net POWER_EN: now also U1.7 (GPIO6/FSPICLK/MTCK/LEDPWM); no longer U1.2 (GPIO1/ADC1_CH1)
- net VCC: now also R13.1, R15.1, R5.1
- net beep: now also U1.2 (GPIO1/ADC1_CH1); no longer U1.19 (GPIO10/FSPICS0/LEDPWM)
- net LED renamed BLUE
- net BLUE: now also U1.6 (GPIO5/FSPIWP/MTDI/LEDPWM); no longer U1.4 (GPIO2/ADC1_CH2/FSPIQ)
- new net: D4.2 (A), R15.2
- new net: D3.2 (A), R5.2
- new net GREEN: D3.1 (K), U1.4 (GPIO2/ADC1_CH2/FSPIQ)
- new net YELLOW: D4.1 (K), U1.20 (GPIO3/ADC1_CH3/LEDPWM)
Other:
- moved on the sheet: BZ1, C37, D13, D5, Q1, R10, R13, R14, R6, R7, R9

Commit message: rfBat ready to manufacture
Parts:
- added D6: LED, LED_SMD:LED_0603_1608Metric_Pad1.05x0.95mm_HandSolder, symbol Device:LED
- added R16: 1k, Resistor_SMD:R_0603_1608Metric_Pad0.98x0.95mm_HandSolder, symbol Device:R
- added TP10, TP12, TP7, TP8, TP9: TestPoint, TestPoint:TestPoint_Pad_D1.0mm, symbol Connector:TestPoint
- L2: footprint Inductor_SMD:L_Vishay_IHLP-4040 -> Inductor_SMD:L_Taiyo-Yuden_NR-40xx_HandSoldering
Connections:
- net +3V3: now also R16.1, TP8.1
- net +5V: now also TP7.1
- net BAT_FB: now also U1.2 (GPIO1/ADC1_CH1); no longer U1.5 (GPIO4/ADC1_CH4/FSPIHD/MTMS/LEDPWM)
- net GNDD: now also D6.1 (K), TP10.1
- net GNDPWR: now also TP9.1
- net GREEN: now also U1.5 (GPIO4/ADC1_CH4/FSPIHD/MTMS/LEDPWM); no longer U1.4 (GPIO2/ADC1_CH2/FSPIQ)
- net at C28.1, J1.A9 (VBUS), J1.B9 (VBUS)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: now also TP12.1
- net beep renamed BEEP
- net BEEP: now also U1.4 (GPIO2/ADC1_CH2/FSPIQ); no longer U1.2 (GPIO1/ADC1_CH1)
- new net: D6.2 (A), R16.2
- no-connect marks 9 -> 10
Other:
- moved on the sheet: D1, J3, Q2, Q3, R11, R8, SW3

Commit message: update rfBat
Parts:
- removed BT2: doubleBatCell, bat_rf:BAT-SMD_BH-18650-B1BA007, symbol bat_rf:doubleBatCell
- removed J2: Conn_01x04, Connector_Samtec_MicroMate:Samtec_T1M-04-X-S-V_1x04-1MP_P1.0mm_Terminal_Vertical, symbol Connector_Generic:Conn_01x04
- removed J3: Conn_01x02_Socket, bat_rf:CONN-TH_XT30UPB-F, symbol Connector:Conn_01x02_Socket
- added BT1: doubleBatCell, bat_rf:batCase_18650x2, symbol bat_rf:doubleBatCell
- added J2: Conn_01x02_Socket, bat_rf:CONN-TH_XT30UPB-F, symbol Connector:Conn_01x02_Socket
- added J4: Conn_01x03, bat_rf:CONN-SMD_3P-P1.00_WAFER-SH1.0-3PWB, symbol Connector_Generic:Conn_01x03
- added Q4: KNY3406C, bat_rf:PDFN-8_L4.9-W5.8-P1.27-LS6.1-BL, symbol bat_rf:KNY3406C
- added TP11: TestPoint, TestPoint:TestPoint_Pad_D1.0mm, symbol Connector:TestPoint
Connections:
- net +BATT: now also BT1.1 (+), J2.2 (Pin_2), TP11.1
- net BAT_FB: now also U1.20 (GPIO3/ADC1_CH3/LEDPWM); no longer U1.2 (GPIO1/ADC1_CH1)
- net BEEP: now also U1.2 (GPIO1/ADC1_CH1); no longer U1.4 (GPIO2/ADC1_CH2/FSPIQ)
- net BLUE: now also R13.1; no longer D13.1 (K)
- net ESP_RX: now also J4.3 (Pin_3)
- net ESP_TX: now also J4.2 (Pin_2)
- net GNDD: now also J4.1 (Pin_1); no longer Q3.3 (S), R11.1, SW3.1, SW3.2
- net GNDPWR: now also D13.1 (K), D3.1 (K), D4.1 (K), Q3.3 (S), R11.1, SW3.1, SW3.2, BT1.4 (-), Q4.1 (S), Q4.2 (S), Q4.3 (S)
- net GREEN: now also R5.1, U1.4 (GPIO2/ADC1_CH2/FSPIQ); no longer D3.1 (K), U1.5 (GPIO4/ADC1_CH4/FSPIHD/MTMS/LEDPWM)
- net VCC: no longer R13.1, R15.1, R5.1
- net YELLOW: now also R15.1, U1.19 (GPIO10/FSPICS0/LEDPWM); no longer D4.1 (K), U1.20 (GPIO3/ADC1_CH3/LEDPWM)
- new net: J2.1 (Pin_1), Q4.5 (D), Q4.6 (D), Q4.7 (D), Q4.8 (D), Q4.9 (D)
- new net: BT1.2 (-), BT1.3 (+)
- new net BAT_EN: Q4.4 (G), U1.5 (GPIO4/ADC1_CH4/FSPIHD/MTMS/LEDPWM)
- no-connect marks 10 -> 9
Other:
- moved on the sheet: C10, C12, C13, C16, C26, C27, C28, C29, C37, C40, D13, D2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

Commit message: motor sch update
Parts:
- BT1: footprint bat_rf:batCase_18650x2 -> bat_rf:BAT-SMD_BH-18650-B1BA007
Changed lines of the file:
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@@
 			)
 		)
-		(property "Footprint" "bat_rf:batCase_18650x2"
+		(property "Footprint" "bat_rf:BAT-SMD_BH-18650-B1BA007"
 			(at 125.73 46.99 0)
 			(effects

Commit message: update pcbs
Parts:
- removed TP10: TestPoint, TestPoint:TestPoint_Pad_D1.0mm, symbol Connector:TestPoint
- removed U1: ESP8684-WROOM-01C, bat_rf:WIRELM-SMD_ESP8684-WROOM0-1C, symbol bat_rf:ESP8684-WROOM-01C
- added U1: ESP32-C3-WROOM-02-N4, bat_rf:BULETM-SMD_18P-L20.0-W18.0-P1.50_ESP32-C3-WROOM, symbol bat_rf:ESP32-C3-WROOM-02-N4
- D13, D3, D4, D6: footprint LED_SMD:LED_0603_1608Metric_Pad1.05x0.95mm_HandSolder -> LED_SMD:LED_0402_1005Metric_Pad0.77x0.64mm_HandSolder
- D2: footprint Capacitor_SMD:C_0805_2012Metric_Pad1.18x1.45mm_HandSolder -> LED_SMD:LED_0402_1005Metric_Pad0.77x0.64mm_HandSolder
- SW2: footprint Button_Switch_SMD:SW_SPST_B3U-1000P -> Button_Switch_SMD:SW_Push_1P1T_NO_CK_KMR2
Connections:
- net +5V: now also C14.2, LED10.3 (VDD), U4.2 (VO); no longer U4.3 (VI)
- net +BATT: now also U4.3 (VI); no longer U4.2 (VO)
- net BAT_EN: now also U1.4 (IO5)
- net BAT_FB: now also U1.15 (IO3)
- net BEEP: now also U1.17 (IO1)
- net BLUE: now also U1.7 (IO8)
- net EN: now also U1.2 (EN)
- net ESP_RX: now also U1.10 (IO10)
- net ESP_TX: now also U1.13 (IO18)
- net GNDD: now also U1.19 (EP), U1.9 (GND)
- net GREEN: now also U1.3 (IO4)
- net IO9: now also U1.8 (IO9)
- net KEY: now also U1.6 (IO7)
- net POWER_EN: now also U1.5 (IO6)
- net RGB: now also U1.18 (IO0)
- net RXD: now also U1.11 (RXD)
- net TXD: now also U1.12 (TXD)
- net VCC: now also U1.1 (3V3)
- net YELLOW: now also U1.16 (IO2)
- no-connect marks 9 -> 4
Other:
- moved on the sheet: C12, C13, C16, R12, R4

Commit message: f
Parts:
- removed SW2: RESET, Button_Switch_SMD:SW_Push_1P1T_NO_CK_KMR2, symbol Switch:SW_Push
- added SW1: 3*4*2.5MM_贴片4脚, bat_rf:SW-SMD_4P-L4.2-W3.3-P2.15-LS5.1, symbol bat_rf:3*4*2.5MM_贴片4脚
Connections:
- net BLUE: now also U1.10 (IO10); no longer U1.7 (IO8)
- net EN: now also SW1.1
- net ESP_RX: now also U1.13 (IO18); no longer U1.10 (IO10)
- net ESP_TX: now also U1.14 (IO19); no longer U1.13 (IO18)
- net GNDD: now also SW1.3
- net IO9: no longer R4.1
- new net: R4.1, U1.7 (IO8)
- no-connect marks 4 -> 5

Commit message: update controller pcb
Parts:
- BZ1: footprint Buzzer_Beeper:MagneticBuzzer_Kobitone_254-EMB84Q-RO -> bat_rf:BUZ-SMD_FUET-9045
- J2: footprint bat_rf:CONN-TH_XT30UPB-F -> bat_rf:CONN-TH_XT30U-F
Changed lines of the file:
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@@
 			)
 		)
-		(property "Footprint" "Buzzer_Beeper:MagneticBuzzer_Kobitone_254-EMB84Q-RO"
+		(property "Footprint" "bat_rf:BUZ-SMD_FUET-9045"
 			(at 276.225 121.92 90)
 			(effects
@@
 			)
 		)
-		(property "Footprint" "bat_rf:CONN-TH_XT30UPB-F"
+		(property "Footprint" "bat_rf:CONN-TH_XT30U-F"
 			(at 97.79 54.61 0)
 			(effects
