File: hardware/rfBat/bat_rf.kicad_sch (KiCad schematic)
At the start: 89 parts, among them J1 USB_C_Receptacle_PowerOnly_6P, J2 Conn_01x01_Pin, J3 Conn_01x06, J4 Conn_01x03, J5 Conn_01x01_Pin, Q1 NPN, Q3 AO4407, Q5 AllPower__AP2300, SW1 3*4*2.5MM_贴片4脚, SW3 TS-1199A-B-B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

Commit message: update pcb
Parts:
- added C1, C4: 22u, Capacitor_SMD:C_0603_1608Metric_Pad1.08x0.95mm_HandSolder, symbol Device:C
- added C18, C2, C7: 100n, Capacitor_SMD:C_0603_1608Metric_Pad1.08x0.95mm_HandSolder, symbol Device:C
- added C3, C8: 47u, Capacitor_SMD:C_0603_1608Metric_Pad1.08x0.95mm_HandSolder, symbol Device:C
- added L1: 10uH, symbol Device:L
- added R22: 160k, Resistor_SMD:R_0603_1608Metric_Pad0.98x0.95mm_HandSolder, symbol Device:R
- added R23: 100k, Resistor_SMD:R_0603_1608Metric_Pad0.98x0.95mm_HandSolder, symbol Device:R
- R11: value 1k -> 22k
Connections:
- net +5V: now also C4.1, C7.1, C8.1, L1.2, R22.2
- net GNDD: now also R11.2, U3.2 (GND), C1.2, C2.2, C3.2, C4.2, C7.2, C8.2
- net VCC: now also U3.5 (IN), C1.1, C2.1, C3.1, R23.2
- net at R11.1: now also U3.3 (FB), R22.1
- net at U3.1 (BS): now also C18.1
- net at U3.4 (EN): now also R23.1
- net at U3.6 (SW): now also C18.2, L1.1
Other:
- moved on the sheet: C15, C9, D6, FB1, R11, R16, TP1, U3, U7

Commit message: update motor pcb
Parts:
- removed J4: Conn_01x03, bat_rf:CONN-SMD_3P-P1.00_WAFER-SH1.0-3PWB, symbol Connector_Generic:Conn_01x03
- removed Q3: AO4407, bat_rf:SOP-8_L5.0-W4.0-P1.27-LS6.0-BL, symbol bat_rf:AO4407
- added FPC1: 1.0K-N-3PB, bat_rf:FPC-SMD_3P-P1.00_HDGC_1.0K-N-3PB, symbol bat_rf:1.0K-N-3PB
- added Q2: AON7403, bat_rf:PQFN-8_L3.1-W3.1-P0.65-LS3.3-BL, symbol bat_rf:AON7403
- added TP2: TestPoint, TestPoint:TestPoint_Pad_D1.0mm, symbol Connector:TestPoint
- L1: footprint (none) -> Inductor_SMD:L_Chilisin_BMRA00040420
- Q1: footprint (none) -> Package_TO_SOT_SMD:SOT-23
- SW3: footprint Button_Switch_SMD:SW_SPST_B3U-1000P -> bat_rf:SW-SMD_L4.0-W2.9-LS5.0
Connections:
- net +3V3: now also J3.1 (Pin_1), TP2.1; no longer J3.3 (Pin_3)
- net +BATT: now also Q2.1 (S), Q2.2 (S), Q2.3 (S)
- net EN: now also J3.3 (Pin_3); no longer J3.2 (Pin_2)
- net ESP_RX: now also FPC1.3
- net ESP_TX: now also FPC1.1
- net GNDD: now also FPC1.2
- net IO9: now also J3.2 (Pin_2); no longer J3.1 (Pin_1)
- net VCC: now also Q2.5 (D), Q2.6 (D), Q2.7 (D), Q2.8 (D)
- net at R19.2, R8.1: now also Q2.4 (G)
- no-connect marks 7 -> 9
Other:
- moved on the sheet: D6, R16

Commit message: update rfBat pcb
Parts:
- removed FPC1: 1.0K-N-3PB, bat_rf:FPC-SMD_3P-P1.00_HDGC_1.0K-N-3PB, symbol bat_rf:1.0K-N-3PB
- removed Q1: NPN, Package_TO_SOT_SMD:SOT-23, symbol Simulation_SPICE:NPN
- added J4: Conn_01x04, symbol Connector_Generic:Conn_01x04
- added P1: FPC_0.5MM_4P_Vertical_mounting_type_H2.0mm, bat_rf:FPC-SMD_4P-L7.5-W2.0-P0.50, symbol bat_rf:FPC_0.5MM_4P_Vertical_mounting_type_H2.0mm
- added U4: SS8050_C7420370, bat_rf:SOT-23-3_L2.9-W1.3-P1.90-LS2.4-BR, symbol bat_rf:SS8050_C7420370
- C1, C4: value 22u -> 2.2u
- C3, C8: value 47u -> 10u
Connections:
- net +3V3: now also P1.4
- net ESP_RX: now also P1.3
- net ESP_TX: now also P1.1
- net GNDD: now also P1.2
- net GNDPWR: now also U4.2 (E)
- net K1: now also U4.3 (C)
- net at R20.2, R21.1: now also U4.1 (B)

Commit message: update firmware
Parts:
- removed Q2: AON7403, bat_rf:PQFN-8_L3.1-W3.1-P0.65-LS3.3-BL, symbol bat_rf:AON7403
- added Q1: IRFH7440TRPBF, bat_rf:DFN-8_L5.8-W4.9-P1.27-LS6.0-BL-1, symbol bat_rf:IRFH7440TRPBF
- added TP3, TP4: TestPoint, TestPoint:TestPoint_Pad_D1.0mm, symbol Connector:TestPoint
Connections:
- net +BATT: now also Q1.1 (S), Q1.2 (S), Q1.3 (S)
- net ESP_RX: now also TP3.1
- net ESP_TX: now also TP4.1
- net VCC: now also Q1.5 (D), Q1.6 (D), Q1.7 (D), Q1.8 (D), Q1.9 (D)
- net at R19.2, R8.1: now also Q1.4 (G)

Commit message: update motor pcb
Parts:
- added TP5: TestPoint, TestPoint:TestPoint_Pad_D1.0mm, symbol Connector:TestPoint
Connections:
- net BAT_FB: now also TP5.1
Changed lines of the file:
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@@
 		)
 	)
+	(wire
+		(pts
+			(xy 130.81 144.78) (xy 139.7 144.78)
+		)
+		(stroke
+			(width 0)
+			(type default)
+		)
+	)
 	(polyline
 		(pts
@@
 					(unit 1)
 				)
+			)
+		)
+	)
+	(symbol
+		(lib_id "Connector:TestPoint")
+		(at 139.7 144.78 270)
+		(unit 1)
+		(exclude_from_sim no)
+		(in_bom yes)
+		(on_board yes)
+		(dnp no)
+		(property "Reference" "TP5"
+			(at 144.78 144.78 90)
+			(effects
+				(font
+					(size 1.27 1.27)
+				)
+				(justify left)
+			)
+		)
+		(property "Value" "TestPoint"
+			(at 144.78 146.0499 90)
+			(effects
+				(font
+					(size 1.27 1.27)
+				)
+				(justify left)
+				(hide yes)
+			)
+		)
+		(property "Footprint" "TestPoint:TestPoint_Pad_D1.0mm"
+			(at 139.7 149.86 0)
+			(effects
+				(font
+					(size 1.27 1.27)
+				)
+				(hide yes)
+			)
+		)
+		(property "Datasheet" "~"
+			(at 139.7 149.86 0)
+			(effects
+				(font
+					(size 1.27 1.27)
+				)
+				(hide yes)
+			)
+		)
+		(property "Description" "test point"
+			(at 139.7 144.78 0)
+			(effects
+				(font
+					(size 1.27 1.27)
+				)
+				(hide yes)
+			)
+		)
+		(pin "1"
+		)
+		(instances
+			(project "bat_rf"
+				(path "/4b9911c3-08ff-4557-9b31-2480476fb503"
+					(reference "TP5")
+					(unit 1)
+				)
