File: hardware/rfBat/bat_rf.kicad_pcb (KiCad board)
At the start: 2 copper layers, 89.8 x 41.5 mm, 98 parts, among them J1 USB_C_Receptacle_PowerOnly_6P, J2 Conn_01x02_Socket, J4 Conn_01x03, Q1 NMOS, Q2 PMOS, Q3 NMOS, Q4 KNY3406C, SW1 3*4*2.5MM_贴片4脚, SW3 SW_MEC_5E, U1 ESP32-C3-WROOM-02-N4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

Commit message: update body
Parts:
- J2: footprint bat_rf:CONN-TH_XT30UPB-F -> bat_rf:CONN-TH_XT30U-F
- moved J2 0.06 mm to (68.0, 89.4)

Commit message: update controller pcb
Parts:
- BZ1: footprint Buzzer_Beeper:MagneticBuzzer_Kobitone_254-EMB84Q-RO -> bat_rf:BUZ-SMD_FUET-9045
- moved BZ1 2.37 mm to (88.4, 94.0), turned to -90 degrees

Commit message: update rfBat pcb
Parts:
- removed D1: BAT54C, Package_TO_SOT_SMD:SOT-23
- removed Q1: NMOS, Package_TO_SOT_SMD:SOT-23
- removed SW3: SW_MEC_5E, bat_rf:SW-SMD_EVQPUD02K
- removed TP12: TestPoint, TestPoint:TestPoint_Pad_D1.0mm
- added D7: BAT54C, bat_rf:BAT54C, B.Cu at (93.5, 81.0)
- added Q5: AllPower__AP2300, bat_rf:SOT-23, B.Cu at (87.5, 103.0)
- added SW2: 3*4*2.5MM_贴片4脚, bat_rf:SW-SMD_4P-L4.2-W3.3-P2.15-LS5.1, F.Cu at (152.5, 89.5)
- J1: moved to B.Cu
- Q2: value PMOS -> AllPower__AP2300; footprint Package_TO_SOT_SMD:SOT-23 -> bat_rf:SOT-23
- Q3: value NMOS -> AO3401; footprint Package_TO_SOT_SMD:SOT-23 -> bat_rf:AO3401
- moved D6 13.0 mm to (82.8, 87.8), turned to -90 degrees
- moved R16 8.42 mm to (85.5, 87.9), turned to 180 degrees
- moved TP8 5.70 mm to (90.8, 77.5)
- moved R11 5.40 mm to (93.6, 87.9), turned to 0 degrees
- moved Q2 4.78 mm to (93.6, 85.1), turned to -90 degrees
- moved L2 4.59 mm to (141.5, 87.2)
- moved Q3 4.29 mm to (90.4, 87.0), turned to 180 degrees
- moved R8 3.34 mm to (89.8, 84.4), turned to 0 degrees
- moved TP11 2.65 mm to (132.3, 87.0)
- moved BZ1 1.84 mm to (89.4, 95.6)
- moved D5 0.84 mm to (92.0, 102.9)
- moved R6 0.69 mm to (92.1, 105.6)
- moved J2 0.26 mm to (67.8, 89.4), turned to -90 degrees
- moved BT1 0.25 mm to (109.4, 89.5)
- turned J1 to -90 degrees
Connections:
- Q2 pad 1: VCC -> /POWER_EN
- Q2 pad 2: Net-(Q2-G) -> GNDD
- Q2 pad 3: +3V3 -> Net-(Q2-D)
- Q3 pad 1: Net-(Q2-G) -> Net-(Q2-D)
- Q3 pad 2: /POWER_EN -> +3V3
- Q3 pad 3: GNDPWR -> VCC
- R11 pad 1: GNDPWR -> GNDD
- R16 pad 1: +3V3 -> VCC
- R8 pad 2: Net-(Q2-G) -> Net-(Q2-D)
Routing:
- net Net-(C28-Pad1): track 49.9 -> 0.55 mm, vias 8 -> 0
- net Net-(U2-LX): track 40.7 -> 2.65 mm, vias 4 -> 0
- net Net-(SW3-A): track 26.6 -> 0.00 mm, vias 4 -> 0
- net Net-(D7-C): track 0.00 -> 24.2 mm, vias 0 -> 4
- net +5V: track 239.2 -> 256.8 mm, vias 3 -> 0
- net VCC: track 57.3 -> 73.1 mm
- net /KEY: track 19.1 -> 31.5 mm
- net Net-(Q2-G): track 11.1 -> 0.00 mm, vias 2 -> 0
- net Net-(U2-LED): track 13.8 -> 2.84 mm
- net Net-(Q2-D): track 0.00 -> 10.1 mm
- net +3V3: track 0.00 -> 6.62 mm
- net GNDD: track 67.4 -> 73.1 mm, vias 18 -> 19
- net /BAT_EN: track 28.5 -> 23.6 mm
- net Net-(BZ1-+): track 6.40 -> 10.2 mm
- net GNDPWR: track 116.9 -> 113.4 mm, vias 53 -> 46
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- removed copper zone on B.Cu, net Net-(C28-Pad1)
Other:
- board text added: "ON"
- board text removed: "USB_P"

Commit message: update rfBat pcb
Parts:
- moved C6 2.63 mm to (151.8, 82.6), turned to 180 degrees
- moved SW1 0.45 mm to (112.5, 78.2)
- moved BT1 0.13 mm to (109.6, 89.5)
- moved J2 0.06 mm to (67.8, 89.5)
Routing:
- net GNDD: track 73.1 -> 205.7 mm, vias 19 -> 18
- net Net-(D7-C): track 24.2 -> 66.1 mm, vias 4 -> 1
- net +BATT: track 124.1 -> 140.8 mm
- net Net-(J2-Pin_1): track 11.7 -> 27.4 mm
- net +5V: track 256.8 -> 269.0 mm
- net Net-(U2-LED): track 2.84 -> 13.9 mm, vias 0 -> 2
- net /KEY: track 31.5 -> 21.7 mm
- net Net-(U2-LX): track 2.65 -> 11.6 mm, vias 0 -> 2
- net GNDPWR: track 113.4 -> 116.8 mm, vias 46 -> 47
- net Net-(LED8-DI): track 20.7 -> 22.9 mm
- net Net-(LED4-DI): track 20.7 -> 22.8 mm
- net /IO9: track 10.2 -> 9.61 mm
- added copper zone on B.Cu, net Net-(C28-Pad1)
- removed copper zone on B.Cu, net +5V
- removed copper zone on B.Cu, net GNDD
Other:
- board text added: "V2.3"
- board text removed: "V2.2"

Commit message: update rfBat firmware
Parts:
- removed BZ1: Buzzer, bat_rf:BUZ-SMD_FUET-9045
- removed C15: 10u, Capacitor_SMD:C_0805_2012Metric_Pad1.18x1.45mm_HandSolder
- removed C9: 100n, Capacitor_SMD:C_0603_1608Metric_Pad1.08x0.95mm_HandSolder
- removed Q3: AO3401, bat_rf:AO3401
- removed SW1: 3*4*2.5MM_贴片4脚, bat_rf:SW-SMD_4P-L4.2-W3.3-P2.15-LS5.1
- removed TP8: TestPoint, TestPoint:TestPoint_Pad_D1.0mm
- removed U3: SPX3819M5-L-3-3, Package_TO_SOT_SMD:SOT-23-5
- added Q1: AON7403, bat_rf:PQFN-8_L3.1-W3.1-P0.65-LS3.3-BL, B.Cu at (84.8, 81.7)
- added SW3: TS-1199A-B-B, Button_Switch_SMD:SW_SPST_B3U-1000P, B.Cu at (118.9, 84.3)
- added U5: MLT-8530-5V, bat_rf:BUZ-SMD_4P-L8.5-W8.5-TL, B.Cu at (89.8, 96.3)
- added U6: TPLP2992IM5X-3.3, bat_rf:SOT-23-5_L2.9-W1.6-P0.95-LS2.8-BL, B.Cu at (89.5, 78.0)
- C37: value 2.2u -> 100n
- C7: value 10n -> 1u
- C8: value 10u -> 1u; footprint Capacitor_SMD:C_0805_2012Metric_Pad1.18x1.45mm_HandSolder -> Capacitor_SMD:C_0603_1608Metric_Pad1.08x0.95mm_HandSolder
- D13: value LED -> B_LED; footprint LED_SMD:LED_0402_1005Metric_Pad0.77x0.64mm_HandSolder -> LED_SMD:LED_0603_1608Metric_Pad1.05x0.95mm_HandSolder
- D2, D6: footprint LED_SMD:LED_0402_1005Metric_Pad0.77x0.64mm_HandSolder -> LED_SMD:LED_0603_1608Metric_Pad1.05x0.95mm_HandSolder
- D3: value LED -> G_LED; footprint LED_SMD:LED_0402_1005Metric_Pad0.77x0.64mm_HandSolder -> LED_SMD:LED_0603_1608Metric_Pad1.05x0.95mm_HandSolder
- D4: value LED -> Y_LED; footprint LED_SMD:LED_0402_1005Metric_Pad0.77x0.64mm_HandSolder -> LED_SMD:LED_0603_1608Metric_Pad1.05x0.95mm_HandSolder
- R13, R15, R5: value 1k -> 3k
- R3: value 100R -> 3k
- R9: value 7m -> 7.5m
- moved TP7 20.3 mm to (78.8, 90.6)
- moved D6 16.3 mm to (94.4, 76.4)
- moved R16 11.9 mm to (94.4, 80.1), turned to 90 degrees
- moved R11 11.0 mm to (82.7, 88.2)
- moved Q2 10.9 mm to (82.7, 85.4)
- moved D7 8.66 mm to (86.6, 86.3)
- moved R8 8.48 mm to (81.8, 81.6), turned to 90 degrees
- moved C8 6.74 mm to (89.7, 80.9)
- moved TP9 5.80 mm to (112.5, 74.7)
- moved C7 4.86 mm to (89.2, 75.6), turned to 0 degrees
- moved D2 1.08 mm to (151.2, 75.0)
- moved D13 0.90 mm to (67.6, 75.0)
- turned TP1 to 180 degrees
Connections:
- C11 pad 2: +5V -> VCC
- C12 pad 1: VCC -> +3V3
- C13 pad 1: VCC -> +3V3
- C14 pad 2: +5V -> VCC
- C17 pad 2: +5V -> VCC
- C30 pad 2: +5V -> VCC
- C31 pad 2: +5V -> VCC
- C32 pad 2: +5V -> VCC
- C33 pad 2: +5V -> VCC
- C34 pad 2: +5V -> VCC
- C35 pad 2: +5V -> VCC
- C36 pad 2: +5V -> VCC
- C5 pad 2: +5V -> VCC
- C6 pad 2: +5V -> VCC
- C7 pad 1: Net-(U3-BP) -> VCC
- D5 pad 1: +5V -> VCC
- LED1 pad 3: +5V -> VCC
- LED10 pad 3: +5V -> VCC
- LED11 pad 3: +5V -> VCC
- LED12 pad 3: +5V -> VCC
- LED2 pad 3: +5V -> VCC
- LED3 pad 3: +5V -> VCC
- LED4 pad 3: +5V -> VCC
- LED5 pad 3: +5V -> VCC
- LED6 pad 3: +5V -> VCC
- LED7 pad 3: +5V -> VCC
- LED8 pad 3: +5V -> VCC
- LED9 pad 3: +5V -> VCC
- R12 pad 2: VCC -> +3V3
- R16 pad 1: VCC -> +3V3
- R4 pad 2: VCC -> +3V3
- R8 pad 1: +3V3 -> +5V
- TP1 pad 1: VCC -> +3V3
- U1 pad 1: VCC -> +3V3
Routing:
- net +5V: track 269.0 -> 20.7 mm
- net VCC: track 73.1 -> 264.6 mm, vias 2 -> 0
- net +3V3: track 6.62 -> 75.2 mm, vias 0 -> 4
- net GNDD: track 205.7 -> 216.5 mm, vias 18 -> 16
- net /POWER_EN: track 15.3 -> 24.7 mm
- net Net-(D7-C): track 66.1 -> 75.1 mm, vias 1 -> 3
- net /BLUE: track 65.0 -> 56.0 mm, vias 4 -> 2
- net Net-(D2-A): track 8.13 -> 15.7 mm
- net /KEY: track 21.7 -> 28.1 mm, vias 0 -> 2
- net Net-(D5-A): track 10.2 -> 5.72 mm
- net /EN: track 32.3 -> 35.7 mm
- net Net-(U3-BP): track 2.02 -> 0.00 mm
- net +BATT: track 140.8 -> 142.3 mm
- net Net-(D13-A): track 3.33 -> 4.66 mm
- net Net-(Q1-G): track 10.1 -> 10.9 mm, vias 0 -> 2
- removed copper zone on B.Cu, net +3V3
Other:
- outline, holes or cut-outs redrawn
- board text added: "ON/OFF"
- board text added: "V2.4"
- board text removed: "ON"
- board text removed: "V2.3"
- board text removed: "VCC"

Commit message: update controller pcb
Routing:
- net GNDPWR: track 116.8 -> 116.0 mm
Changed lines of the file:
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@@
 	)
 	(via blind
-		(at 149.2565 92.225)
+		(at 148.2565 92.600388)
 		(size 1.2)
 		(drill 0.6)
@@
 	)
 	(segment
-		(start 149.2565 92.225)
-		(end 148.5625 92.225)
-		(width 0.6)
-		(layer "B.Cu")
-		(net 2)
-	)
-	(segment
 		(start 84.925 71.925)
 		(end 85 72)
@@
 	)
 	(segment
+		(start 148.187112 92.600388)
+		(end 146.2625 94.525)
+		(width 0.6)
+		(layer "B.Cu")
+		(net 2)
+	)
+	(segment
 		(start 129.125 92.625)
 		(end 129 92.5)
@@
 	)
 	(segment
+		(start 148.631888 92.225)
+		(end 149.472135 92.225)
+		(width 0.6)
+		(layer "B.Cu")
+		(net 2)
+	)
+	(segment
 		(start 133.7 98.4375)
 		(end 131.7625 98.4375)
@@
 	)
 	(segment
+		(start 148.2565 92.600388)
+		(end 148.631888 92.225)
+		(width 0.6)
+		(layer "B.Cu")
+		(net 2)
+	)
+	(segment
 		(start 124.475 70.025)
 		(end 124.5 70)
@@
 	)
 	(segment
-		(start 149.2565 92.225)
-		(end 146.2375 92.225)
-		(width 0.6)
-		(layer "B.Cu")
-		(net 2)
-	)
-	(segment
 		(start 138.5 91.665)
 		(end 137.8325 92.3325)
@@
 	)
 	(segment
-		(start 148.5625 92.225)
-		(end 146.2625 94.525)
-		(width 0.6)
-		(layer "B.Cu")
-		(net 2)
-	)
-	(segment
 		(start 84.375 70.125)
 		(end 84.5 70)
@@
 		(end 77.075 77)
 		(width 0.5)
-		(layer "B.Cu")
-		(net 2)
-	)
-	(segment
-		(start 149.2565 92.225)
-		(end 149.472135 92.225)
-		(width 0.6)
 		(layer "B.Cu")
 		(net 2)
@@
 	)
 	(segment
+		(start 148.2565 92.600388)
+		(end 147.881112 92.225)
+		(width 0.6)
+		(layer "B.Cu")
+		(net 2)
+	)
+	(segment
 		(start 79.575 106.425)
 		(end 79.5 106.5)
@@
 	)
 	(segment
+		(start 146.2375 92.225)
+		(end 146.125 92.3375)
+		(width 0.6)
+		(layer "B.Cu")
+		(net 2)
+	)
+	(segment
 		(start 102.375 72.125)
 		(end 102.5 72)
@@
 		(end 85.5 106)
 		(width 0.5)
+		(layer "B.Cu")
+		(net 2)
+	)
+	(segment
+		(start 148.2565 92.600388)
+		(end 148.187112 92.600388)
+		(width 0.6)
 		(layer "B.Cu")
 		(net 2)
@@
 	)
 	(segment
+		(start 147.881112 92.225)
+		(end 146.2375 92.225)
+		(width 0.6)
+		(layer "B.Cu")
+		(net 2)
+	)
+	(segment
 		(start 98.35 108.8)
 		(end 97.6 108.8)
@@
 		(layer "B.Cu")
 		(net 2)
-	)
-	(segment
-		(start 146.2375 92.225)
-		(end 146.125 92.3375)
-		(width 0.6)
-		(layer "B.Cu")
-		(net 2)

Commit message: update rfBat pcb
Parts:
- removed Q4: KNY3406C, bat_rf:PDFN-8_L4.9-W5.8-P1.27-LS6.1-BL
- removed TP1, TP2, TP3, TP4, TP5, TP6: TestPoint, TestPoint:TestPoint_Pad_D1.0mm
- removed U6: TPLP2992IM5X-3.3, bat_rf:SOT-23-5_L2.9-W1.6-P0.95-LS2.8-BL
- added C15: 1u, Capacitor_SMD:C_0603_1608Metric_Pad1.08x0.95mm_HandSolder, B.Cu at (81.3, 80.5)
- added C9: 1u, Capacitor_SMD:C_0603_1608Metric_Pad1.08x0.95mm_HandSolder, B.Cu at (81.3, 78.0)
- added J3: Conn_01x06, kicadLib:CONN-SMD_6P-P1.00_XYECONN_XY-SH1.0-6A61, B.Cu at (107.2, 81.5)
- added R17: 500R, Resistor_SMD:R_0603_1608Metric_Pad0.98x0.95mm_HandSolder, B.Cu at (84.1, 101.8)
- added U7: XC6220B331MR, Package_TO_SOT_SMD:SOT-23-5, B.Cu at (93.7, 73.1)
- Q1: value AON7403 -> Q_PMOS_GDS; footprint bat_rf:PQFN-8_L3.1-W3.1-P0.65-LS3.3-BL -> Package_TO_SOT_SMD:TO-252-2
- moved Q1 9.81 mm to (75.0, 82.2)
- moved C1 6.17 mm to (82.5, 85.8)
- moved C4 6.17 mm to (82.2, 76.8)
- moved D7 6.17 mm to (92.8, 86.1)
- moved R8 6.17 mm to (88.0, 81.4)
- moved C2 6.17 mm to (82.7, 87.8)
- moved C3 6.17 mm to (82.0, 78.9)
- moved FB1 6.17 mm to (87.3, 78.3)
- moved Q2 6.17 mm to (88.9, 85.2)
- moved R11 6.17 mm to (88.8, 88.0)
- moved U4 6.17 mm to (83.7, 82.3)
- moved C7 1.60 mm to (90.8, 75.7)
- moved C8 1.60 mm to (91.3, 81.0)
Connections:
- C11 pad 2: VCC -> +5V
- C14 pad 2: VCC -> +5V
- C17 pad 2: VCC -> +5V
- C3 pad 1: +BATT -> VCC
- C30 pad 2: VCC -> +5V
- C31 pad 2: VCC -> +5V
- C32 pad 2: VCC -> +5V
- C33 pad 2: VCC -> +5V
- C34 pad 2: VCC -> +5V
- C35 pad 2: VCC -> +5V
- C36 pad 2: VCC -> +5V
- C4 pad 1: +BATT -> VCC
- C5 pad 2: VCC -> +5V
- C6 pad 2: VCC -> +5V
- D5 pad 1: VCC -> +5V
- J2 pad 1: Net-(J2-Pin_1) -> GNDPWR
- J2 pad 2: +BATT -> VCC
- LED1 pad 3: VCC -> +5V
- LED10 pad 3: VCC -> +5V
- LED11 pad 3: VCC -> +5V
- LED12 pad 3: VCC -> +5V
- LED2 pad 3: VCC -> +5V
- LED3 pad 3: VCC -> +5V
- LED4 pad 3: VCC -> +5V
- LED5 pad 3: VCC -> +5V
- LED6 pad 3: VCC -> +5V
- LED7 pad 3: VCC -> +5V
- LED8 pad 3: VCC -> +5V
- LED9 pad 3: VCC -> +5V
- Q1 pad 1: +5V -> Net-(Q1-G)
- Q1 pad 2: +5V -> +BATT
- Q1 pad 3: +5V -> VCC
- Q5 pad 2: GNDPWR -> Net-(Q5-S)
- R8 pad 1: +5V -> +BATT
- U1 pad 4: /BAT_EN -> unconnected-(U1-IO5-Pad4)
- U4 pad 3: +BATT -> VCC
- U5 pad 1: VCC -> +5V
Routing:
- net VCC: track 264.6 -> 170.5 mm
- net +5V: track 20.7 -> 92.2 mm
- net +BATT: track 142.3 -> 83.5 mm, vias 9 -> 3
- net /BLUE: track 56.0 -> 24.8 mm
- net Net-(J2-Pin_1): track 27.4 -> 0.00 mm
- net unconnected-(U1-IO5-Pad4): track 0.00 -> 23.6 mm, vias 0 -> 2
- net /BAT_EN: track 23.6 -> 0.00 mm, vias 2 -> 0
- net /EN: track 35.7 -> 21.9 mm
- net Net-(D7-C): track 75.1 -> 61.8 mm, vias 3 -> 2
- net /TXD: track 16.1 -> 3.20 mm
- net Net-(Q1-G): track 10.9 -> 0.00 mm
- net Net-(Q2-D): track 0.00 -> 10.9 mm
- net GNDPWR: track 116.0 -> 111.8 mm, vias 47 -> 44
- net +3V3: track 75.2 -> 71.1 mm
- net /IO9: track 9.61 -> 5.71 mm
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- removed copper zone on B.Cu, net +BATT
Other:
- board text removed: "3V3"
- board text removed: "BOOT"
- board text removed: "EN"
- board text removed: "GNDD"
- board text removed: "RXD"
- board text removed: "TXD"
