File: hardware/rfBat/bat_rf.kicad_pcb (KiCad board)
At the start: 2 copper layers, 89.8 x 41.5 mm, 91 parts, among them J1 USB_C_Receptacle_PowerOnly_6P, J2 Conn_01x02_Socket, J3 Conn_01x06, J4 Conn_01x03, Q1 Q_PMOS_GDS, Q2 AllPower__AP2300, Q5 AllPower__AP2300, SW2 3*4*2.5MM_贴片4脚, SW3 TS-1199A-B-B, U1 ESP32-C3-WROOM-02-N4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

Commit message: update rfbat pcb
Parts:
- removed C7, C8: 1u, Capacitor_SMD:C_0603_1608Metric_Pad1.08x0.95mm_HandSolder
- added J5: Conn_01x01_Pin, TestPoint:TestPoint_Pad_D4.0mm, B.Cu at (76.0, 97.8)
- added TP1: TestPoint, TestPoint:TestPoint_Pad_D1.0mm, B.Cu at (113.4, 77.9)
- J2: value Conn_01x02_Socket -> Conn_01x01_Pin; footprint bat_rf:CONN-TH_XT30U-F -> TestPoint:TestPoint_Pad_D4.0mm; moved to B.Cu
- moved SW2 86.1 mm to (66.4, 89.1)
- moved TP7 16.4 mm to (84.4, 75.2)
- moved C15 13.8 mm to (94.3, 85.0), turned to 0 degrees
- moved C9 13.1 mm to (94.3, 78.9), turned to 0 degrees
- moved C2 12.1 mm to (88.2, 77.0), turned to 90 degrees
- moved C1 11.4 mm to (90.1, 77.3), turned to 90 degrees
- moved D7 11.1 mm to (82.0, 83.2)
- moved D6 11.1 mm to (89.7, 86.5)
- moved R8 10.0 mm to (79.6, 86.9), turned to -90 degrees
- moved U7 8.92 mm to (94.3, 82.0), turned to -90 degrees
- moved J2 8.81 mm to (76.2, 92.0), turned to 180 degrees
- moved FB1 7.08 mm to (94.2, 76.7)
- moved R16 7.08 mm to (91.4, 86.5), turned to -90 degrees
- moved Q2 6.51 mm to (82.6, 86.8), turned to 0 degrees
- moved U4 4.37 mm to (88.0, 81.5)
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Connections:
- C15 pad 2: GND -> GNDPWR
- C9 pad 2: GND -> GNDPWR
- J2 pad 1: GNDPWR -> VCC
- J3 pad 1: GNDD -> /IO9
- J3 pad 2: /IO9 -> /EN
- J3 pad 3: /EN -> +3V3
- J3 pad 4: /RXD -> /TXD
- J3 pad 5: /TXD -> /RXD
- J3 pad 6: +3V3 -> GNDD
- U7 pad 2: GND -> GNDPWR
Routing:
- net +5V: track 92.2 -> 268.6 mm, vias 0 -> 2
- net VCC: track 170.5 -> 23.3 mm
- net Net-(D7-C): track 61.8 -> 21.3 mm, vias 2 -> 1
- net /BLUE: track 24.8 -> 57.4 mm
- net GNDPWR: track 111.8 -> 142.5 mm, vias 44 -> 56
- net +BATT: track 83.5 -> 111.9 mm, vias 3 -> 41
- net GNDD: track 218.0 -> 193.7 mm, vias 16 -> 10
- net unconnected-(U1-IO5-Pad4): track 23.6 -> 0.00 mm, vias 2 -> 0
- net Net-(BT1-+-Pad3): track 22.2 -> 45.5 mm
- net +3V3: track 71.1 -> 55.1 mm, vias 4 -> 0
- net /EN: track 21.9 -> 36.3 mm, vias 0 -> 2
- net /TXD: track 3.20 -> 17.6 mm
- net Net-(Q2-D): track 10.9 -> 0.00 mm
- net Net-(D2-A): track 15.7 -> 7.47 mm
- net Net-(Q1-G): track 0.00 -> 7.47 mm, vias 2 -> 0
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Other:
- board text added: "+"
- board text added: "B"
- board text added: "CHARGE"
- board text added: "DGND"
- board text added: "DOWNlOAD"
- board text added: "E"
- board text added: "G"
- board text added: "M2"
- board text added: "R"
- board text added: "RX"
- board text added: "T"
- board text added: "TX"
- board text added: "V"
- board text added: "V2.5"
- board text removed: "ESP_RX"
- board text removed: "ESP_TX"
- board text removed: "V2.4"

Commit message: update pcb
Parts:
- added C1: 22u, Capacitor_SMD:C_0603_1608Metric_Pad1.08x0.95mm_HandSolder, F.Cu at (95.0, 37.7)
- added C18: 100n, Capacitor_SMD:C_0603_1608Metric_Pad1.08x0.95mm_HandSolder, F.Cu at (99.4, 40.2)
- added C2: 100n, Capacitor_SMD:C_0603_1608Metric_Pad1.08x0.95mm_HandSolder, F.Cu at (95.0, 40.2)
- added C3: 47u, Capacitor_SMD:C_0603_1608Metric_Pad1.08x0.95mm_HandSolder, F.Cu at (95.0, 42.7)
- added C4: 22u, Capacitor_SMD:C_0603_1608Metric_Pad1.08x0.95mm_HandSolder, F.Cu at (95.0, 45.2)
- added C7: 100n, Capacitor_SMD:C_0603_1608Metric_Pad1.08x0.95mm_HandSolder, F.Cu at (95.0, 47.7)
- added C8: 47u, Capacitor_SMD:C_0603_1608Metric_Pad1.08x0.95mm_HandSolder, F.Cu at (99.4, 37.7)
- added D1: 1N4148W, Diode_SMD:D_SOD-123, F.Cu at (102.3, 50.6)
- added D7: 1N4148W, Diode_SMD:D_SOD-123, F.Cu at (102.3, 54.0)
- added L1: 10uH, Inductor_SMD:L_Chilisin_BMRA00040420, F.Cu at (109.3, 43.9)
- added Q1: NPN, Package_TO_SOT_SMD:SOT-23, F.Cu at (107.6, 51.3)
- added Q3: AO4407, bat_rf:SOP-8_L5.0-W4.0-P1.27-LS6.0-BL, F.Cu at (96.3, 53.2)
- added R11: 22k, Resistor_SMD:R_0603_1608Metric_Pad0.98x0.95mm_HandSolder, F.Cu at (99.4, 45.2)
- added R19: 100R, Resistor_SMD:R_0603_1608Metric_Pad0.98x0.95mm_HandSolder, F.Cu at (99.4, 47.7)
- added R20: 1k, Resistor_SMD:R_0603_1608Metric_Pad0.98x0.95mm_HandSolder, F.Cu at (103.7, 37.7)
- added R21: 10k, Resistor_SMD:R_0603_1608Metric_Pad0.98x0.95mm_HandSolder, F.Cu at (103.7, 40.2)
- added R22: 160k, Resistor_SMD:R_0603_1608Metric_Pad0.98x0.95mm_HandSolder, F.Cu at (103.7, 42.7)
- added R23: 100k, Resistor_SMD:R_0603_1608Metric_Pad0.98x0.95mm_HandSolder, F.Cu at (103.7, 45.2)
- added R8: 10k, Resistor_SMD:R_0603_1608Metric_Pad0.98x0.95mm_HandSolder, F.Cu at (99.4, 42.7)
- added SW1: 3*4*2.5MM_贴片4脚, bat_rf:SW-SMD_4P-L4.2-W3.3-P2.15-LS5.1, F.Cu at (109.3, 38.7)
- added U3: MT2492, bat_rf:SOT-23-6_L2.9-W1.6-P0.95-LS2.8-BL, F.Cu at (107.7, 55.8)
Connections:
- C15 pad 2: GNDPWR -> GNDD
- C9 pad 2: GNDPWR -> GNDD
- U7 pad 2: GNDPWR -> GNDD
Routing:
- net GNDD: track 193.7 -> 198.0 mm, vias 10 -> 12
- net GNDPWR: track 142.5 -> 138.2 mm, vias 56 -> 54

Commit message: update motor pcb
Parts:
- removed the C1 at (90.1, 77.3)
- removed the C2 at (88.2, 77.0)
- removed the C3 at (83.1, 79.1)
- removed the C4 at (81.2, 78.8)
- removed the D7 at (82.0, 83.2)
- removed J4: Conn_01x03, bat_rf:CONN-SMD_3P-P1.00_WAFER-SH1.0-3PWB
- removed the Q1 at (75.0, 82.2)
- removed Q3: AO4407, bat_rf:SOP-8_L5.0-W4.0-P1.27-LS6.0-BL
- removed the R11 at (85.5, 86.8)
- removed the R8 at (79.6, 86.9)
- removed SW2: 3*4*2.5MM_贴片4脚, bat_rf:SW-SMD_4P-L4.2-W3.3-P2.15-LS5.1
- removed U4: AMS1117, Package_TO_SOT_SMD:SOT-89-3_Handsoldering
- added FPC1: 1.0K-N-3PB, bat_rf:FPC-SMD_3P-P1.00_HDGC_1.0K-N-3PB, B.Cu at (127.1, 78.6)
- added TP2: TestPoint, TestPoint:TestPoint_Pad_D1.0mm, B.Cu at (100.0, 75.9)
- C1, C18, C2, C3, C4, C7, C8, D1, D7, L1, Q1, R11, R19, R20, R21, R22, R23, R8, U3: moved to B.Cu
- Q2: value AllPower__AP2300 -> AON7403; footprint bat_rf:SOT-23 -> bat_rf:PQFN-8_L3.1-W3.1-P0.65-LS3.3-BL
- SW3: footprint Button_Switch_SMD:SW_SPST_B3U-1000P -> bat_rf:SW-SMD_L4.0-W2.9-LS5.0
- moved SW1 66.2 mm to (66.4, 89.2), turned to -90 degrees
- moved C8 51.3 mm to (85.9, 87.1), turned to -90 degrees
- moved R22 47.5 mm to (83.5, 85.6)
- moved R20 46.4 mm to (80.4, 77.8), turned to 90 degrees
- moved R8 46.3 mm to (73.0, 80.7), turned to -90 degrees
- moved L1 43.7 mm to (88.8, 82.5), turned to -90 degrees
- moved R21 43.6 mm to (77.8, 75.2)
- moved C18 43.5 mm to (85.6, 81.4), turned to 90 degrees
- moved D1 43.2 mm to (79.1, 87.0), turned to -90 degrees
- moved C4 42.6 mm to (87.4, 87.1), turned to -90 degrees
- moved C1 42.3 mm to (84.5, 78.6)
- moved R11 42.0 mm to (83.5, 84.1)
- moved Q1 40.0 mm to (77.6, 77.8)
- moved C7 39.9 mm to (88.9, 87.1), turned to -90 degrees
- moved R19 39.8 mm to (73.9, 78.3), turned to 180 degrees
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Connections:
- J3 pad 1: /IO9 -> +3V3
- J3 pad 2: /EN -> /IO9
- J3 pad 3: +3V3 -> /EN
- Q2 pad 1: /POWER_EN -> +BATT
- Q2 pad 2: GNDD -> +BATT
- Q2 pad 3: Net-(Q1-G) -> +BATT
- R19 pad 2: Net-(Q3-G) -> Net-(Q2-G)
- R8 pad 1: Net-(Q3-G) -> Net-(Q2-G)
Routing:
- net GNDPWR: track 138.2 -> 100.4 mm, vias 54 -> 45
- net Net-(D7-C): track 21.3 -> 0.00 mm, vias 1 -> 0
- net Net-(D1-K): track 0.00 -> 14.4 mm, vias 0 -> 1
- net /IO9: track 9.61 -> 23.3 mm
- net GNDD: track 198.0 -> 210.6 mm, vias 12 -> 10
- net +BATT: track 111.9 -> 103.4 mm, vias 41 -> 23
- net /POWER_EN: track 25.0 -> 32.7 mm
- net Net-(Q1-G): track 7.47 -> 0.00 mm
- net /TXD: track 17.6 -> 24.6 mm
- net /RXD: track 16.8 -> 22.8 mm
- net Net-(Q1-B): track 0.00 -> 5.41 mm, vias 0 -> 2
- net /EN: track 36.3 -> 41.6 mm, vias 2 -> 0
- net /K1: track 0.00 -> 5.04 mm
- net +5V: track 268.6 -> 263.6 mm
- net Net-(U3-SW): track 0.00 -> 4.74 mm
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- added copper zone on B.Cu, net +BATT
- added copper zone on F.Cu, net +BATT
Other:
- board text added: "3V3"
- board text added: "V2.6"
- board text removed: "V2.5"

Commit message: update rfBat pcb
Parts:
- removed FPC1: 1.0K-N-3PB, bat_rf:FPC-SMD_3P-P1.00_HDGC_1.0K-N-3PB
- removed Q1: NPN, Package_TO_SOT_SMD:SOT-23
- added P1: FPC_0.5MM_4P_Vertical_mounting_type_H2.0mm, bat_rf:FPC-SMD_4P-L7.5-W2.0-P0.50, B.Cu at (124.8, 79.0)
- added U4: SS8050_C7420370, bat_rf:SOT-23-3_L2.9-W1.3-P1.90-LS2.4-BR, B.Cu at (77.5, 77.7)
- C1, C4: value 22u -> 2.2u
- C3, C8: value 47u -> 10u
- moved C8 3.00 mm to (88.9, 87.1)
- moved C7 1.51 mm to (87.4, 87.1)
- moved C4 1.50 mm to (85.9, 87.1)
Routing:
- net +3V3: track 54.7 -> 69.3 mm
- net GNDD: track 210.6 -> 197.1 mm, vias 10 -> 12
- net /ESP_TX: track 26.1 -> 19.6 mm
- net /EN: track 41.6 -> 36.8 mm
- net GNDPWR: track 100.4 -> 98.8 mm, vias 45 -> 46
- net Net-(U4-B): track 5.41 -> 4.21 mm, vias 2 -> 0
- net /IO9: track 23.3 -> 22.1 mm
- net /K1: track 5.04 -> 5.89 mm
- net /ESP_RX: track 19.1 -> 18.4 mm

Commit message: update firmware
Parts:
- removed Q2: AON7403, bat_rf:PQFN-8_L3.1-W3.1-P0.65-LS3.3-BL
- added Q1: IRFH7440TRPBF, bat_rf:DFN-8_L5.8-W4.9-P1.27-LS6.0-BL-1, B.Cu at (75.5, 81.0)
- added TP3: TestPoint, TestPoint:TestPoint_Pad_D1.0mm, B.Cu at (124.0, 82.6)
- added TP4: TestPoint, TestPoint:TestPoint_Pad_D1.0mm, B.Cu at (126.0, 83.0)
- added TP5: TestPoint, TestPoint:TestPoint_Pad_D1.0mm, B.Cu at (126.0, 94.8)
- moved R8 3.51 mm to (73.0, 77.2), turned to 180 degrees
- moved R19 2.92 mm to (76.6, 77.2)
- moved C18 2.53 mm to (88.1, 81.4)
- moved D1 2.53 mm to (81.6, 87.0)
- moved R23 2.53 mm to (84.6, 77.7)
- moved U7 2.53 mm to (97.4, 83.4)
- moved C1 2.53 mm to (87.0, 78.6)
- moved C15 2.53 mm to (97.5, 80.4)
- moved C2 2.53 mm to (87.0, 77.1)
- moved C3 2.53 mm to (87.0, 75.6)
- moved C4 2.53 mm to (88.4, 87.1)
- moved C7 2.53 mm to (89.9, 87.1)
- moved C8 2.53 mm to (91.4, 87.1)
- moved C9 2.53 mm to (94.7, 83.7)
- moved D6 2.53 mm to (96.8, 77.8)
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Routing:
- net Net-(LED3-DI): track 18.5 -> 35.8 mm, vias 0 -> 1
- net +BATT: track 103.4 -> 114.2 mm, vias 23 -> 15
- net +3V3: track 69.3 -> 65.8 mm
- net GNDD: track 197.1 -> 193.5 mm
- net Net-(D1-K): track 14.4 -> 17.9 mm
- net /K1: track 5.89 -> 8.91 mm
- net +5V: track 263.6 -> 266.2 mm
- net /KEY: track 26.3 -> 23.7 mm
- net /POWER_EN: track 32.7 -> 30.4 mm
- net GNDPWR: track 98.8 -> 100.9 mm
- net Net-(U4-B): track 4.21 -> 5.13 mm, vias 0 -> 1
- net Net-(Q1-G): track 3.11 -> 4.01 mm
- removed copper zone on F.Cu, net +BATT
Other:
- board text removed: "MCU"

Commit message: update bat PCB
Other:
- board text added: "V2.7"
- board text removed: "V2.6"
Changed lines of the file:
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@@
 		)
 	)
-	(gr_text "V2.6"
+	(gr_text "V2.7"
 		(at 140 77.3 0)
 		(layer "B.SilkS" knockout)
