File: hardware/controller/_autosave-controller.kicad_sch (KiCad schematic)
At the start: 48 parts, among them J1 USB_C_Receptacle_PowerOnly_6P, J2 Bat, Q1 AO3401, Q2 AllPower__AP2300, SW2 RKJXV1224005, SW3 RKJXV1224005, SW4 TC-1102N-C-AS-B, SW5 TS-1199A-B-B, SW6 TC-1102N-C-AS-B, SW8 TS-1199A-B-B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

Commit message: update controller pcb
Connections:
- net EN: now also SW8.2; no longer SW8.1
- net GND: now also SW8.1; no longer SW8.2
Changed lines of the file:
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@@
 		(lib_id "espController:TS-1199A-B-B")
 		(at 63.5 173.99 0)
+		(mirror x)
 		(unit 1)
 		(exclude_from_sim no)
@@
 		(on_board yes)
 		(dnp no)
-		(fields_autoplaced yes)
 		(property "Reference" "SW8"
-			(at 66.04 172.7199 0)
+			(at 66.04 175.2601 0)
 			(effects
 				(font
@@
 		)
 		(property "Value" "TS-1199A-B-B"
-			(at 66.04 175.2599 0)
+			(at 66.04 172.7201 0)
 			(effects
 				(font
@@
 		)
 		(property "Footprint" "espController:SW-SMD_L6.0-W6.0-P6.00-LS6.6"
-			(at 63.5 171.323 0)
+			(at 63.5 176.657 0)
 			(effects
 				(font
@@
 		)
 		(property "Datasheet" "http://www.szlcsc.com/product/details_724359.html"
-			(at 63.5 176.403 0)
+			(at 63.5 171.577 0)
 			(effects
 				(font
@@
 		)
 		(property "Description" "C692476"
-			(at 63.5 181.483 0)
+			(at 63.5 166.497 0)
 			(effects
 				(font
@@
 		)
 		(property "uuid" "std:a8f90e8ccef74c11ad070f97756e49fb"
-			(at 63.5 181.483 0)
+			(at 63.5 166.497 0)
 			(effects
 				(font
