File: hardware/controller/controller.kicad_pcb (KiCad board)
At the start: 2 copper layers, 0 parts

Commit message: update controller pcb
Other:
- board outline added: 100 x 53.9 mm

Commit message: update controller pcb
Parts:
- added C1: 100n, Capacitor_SMD:C_0603_1608Metric_Pad1.08x0.95mm_HandSolder, B.Cu at (133.5, 83.7)
- added C10: 10u, Capacitor_SMD:C_0805_2012Metric_Pad1.18x1.45mm_HandSolder, B.Cu at (122.9, 75.4)
- added C11: 100n, Capacitor_SMD:C_0603_1608Metric_Pad1.08x0.95mm_HandSolder, B.Cu at (116.8, 101.4)
- added C2: 10u, Capacitor_SMD:C_0805_2012Metric_Pad1.18x1.45mm_HandSolder, F.Cu at (131.1, 58.0)
- added C3: 100n, Capacitor_SMD:C_0603_1608Metric_Pad1.08x0.95mm_HandSolder, F.Cu at (129.2, 58.2)
- added C4: 1u, Capacitor_SMD:C_0603_1608Metric_Pad1.08x0.95mm_HandSolder, B.Cu at (122.2, 97.0)
- added C5: 10u, Capacitor_SMD:C_0805_2012Metric_Pad1.18x1.45mm_HandSolder, B.Cu at (128.9, 96.8)
- added C6: 2.2u, Capacitor_SMD:C_0603_1608Metric_Pad1.08x0.95mm_HandSolder, B.Cu at (113.8, 81.0)
- added C7: 10u, Capacitor_SMD:C_0805_2012Metric_Pad1.18x1.45mm_HandSolder, B.Cu at (127.5, 71.3)
- added C8: 100n, Capacitor_SMD:C_0603_1608Metric_Pad1.08x0.95mm_HandSolder, B.Cu at (127.4, 73.1)
- added C9: 100n, Capacitor_SMD:C_0603_1608Metric_Pad1.08x0.95mm_HandSolder, B.Cu at (124.8, 75.6)
- added D1: RED, LED_SMD:LED_0603_1608Metric_Pad1.05x0.95mm_HandSolder, B.Cu at (125.1, 94.2)
- added D2: GREEN, LED_SMD:LED_0603_1608Metric_Pad1.05x0.95mm_HandSolder, B.Cu at (121.2, 94.3)
- added D3: WS2812B, LED_SMD:LED_WS2812B_PLCC4_5.0x5.0mm_P3.2mm, F.Cu at (122.8, 102.3)
- added H1: MountingHole, MountingHole:MountingHole_2.2mm_M2_Pad, F.Cu at (103.3, 95.0)
- added H2: MountingHole, MountingHole:MountingHole_2.2mm_M2_Pad, F.Cu at (143.3, 66.9)
- added H3: MountingHole, MountingHole:MountingHole_2.2mm_M2_Pad, F.Cu at (143.3, 95.0)
- added H4: MountingHole, MountingHole:MountingHole_2.2mm_M2_Pad, F.Cu at (103.3, 66.9)
- added J1: USB_C_Receptacle_PowerOnly_6P, bat_rf:USB-C-SMD_HX-TYPE-C-6PIN, B.Cu at (122.8, 102.4)
- added J2: Bat, Connector_PinSocket_2.54mm:PinSocket_1x02_P2.54mm_Vertical, F.Cu at (137.7, 66.5)
- added R1: 10k, Resistor_SMD:R_0603_1608Metric_Pad0.98x0.95mm_HandSolder, B.Cu at (131.9, 83.7)
- added R2: 10k, Resistor_SMD:R_0603_1608Metric_Pad0.98x0.95mm_HandSolder, B.Cu at (134.4, 67.0)
- added R3: 1k, Resistor_SMD:R_0603_1608Metric_Pad0.98x0.95mm_HandSolder, B.Cu at (120.6, 97.0)
- added R4: 1.5k, Resistor_SMD:R_0603_1608Metric_Pad0.98x0.95mm_HandSolder, B.Cu at (119.0, 97.0)
- added R5: 7m, Resistor_SMD:R_0603_1608Metric_Pad0.98x0.95mm_HandSolder, B.Cu at (113.8, 84.4)
- added R6: 3m, Resistor_SMD:R_0603_1608Metric_Pad0.98x0.95mm_HandSolder, B.Cu at (113.8, 82.9)
- added R7: 1k, Resistor_SMD:R_0603_1608Metric_Pad0.98x0.95mm_HandSolder, B.Cu at (113.8, 79.2)
- added SW1: 3*4*2.5MM_贴片4脚, bat_rf:SW-SMD_4P-L4.2-W3.3-P2.15-LS5.1, F.Cu at (138.0, 76.3)
- added SW2: RKJXV1224005, espController:SW-TH_RKJXV1224005, F.Cu at (89.0, 80.1)
- added SW3: RKJXV1224005, espController:SW-TH_RKJXV1224005, F.Cu at (154.9, 80.0)
- added SW4: TC-1102N-C-AS-B, espController:SW-TH_TC-1102N-C-AS-B, F.Cu at (108.4, 59.1)
- added SW5: TS-1199A-B-B, espController:SW-SMD_L6.0-W6.0-P6.00-LS6.6, F.Cu at (134.5, 103.1)
- added SW6: TC-1102N-C-AS-B, espController:SW-TH_TC-1102N-C-AS-B, F.Cu at (138.3, 59.1)
- added SW7: SK-12D07-L3-B, Button_Switch_SMD:SW_SPDT_CK_JS102011SAQN, F.Cu at (123.0, 58.1)
- added SW8: TS-1199A-B-B, espController:SW-SMD_L6.0-W6.0-P6.00-LS6.6, F.Cu at (112.3, 103.0)
- added TP1: TestPoint, TestPoint:TestPoint_Pad_D1.0mm, F.Cu at (108.7, 85.3)
- added TP2: TestPoint, TestPoint:TestPoint_Pad_D1.0mm, F.Cu at (108.7, 76.3)
- added TP3: TestPoint, TestPoint:TestPoint_Pad_D1.0mm, F.Cu at (108.7, 78.6)
- added TP4: TestPoint, TestPoint:TestPoint_Pad_D1.0mm, F.Cu at (108.7, 83.1)
- added TP5: TestPoint, TestPoint:TestPoint_Pad_D1.0mm, F.Cu at (108.7, 80.9)
- added TP6: TestPoint, TestPoint:TestPoint_Pad_D1.0mm, F.Cu at (108.7, 74.1)
- added TP7: TestPoint, TestPoint:TestPoint_Pad_D1.0mm, F.Cu at (137.9, 86.1)
- added U1: TP4059, espController:SOT-23-6_L2.9-W1.6-P0.95-LS2.8-BR, B.Cu at (125.3, 97.1)
- added U2: ESP32-C3-WROOM-02-N4, bat_rf:BULETM-SMD_18P-L20.0-W18.0-P1.50_ESP32-C3-WROOM, B.Cu at (123.3, 63.0)
- added U3: AMS1117, Package_TO_SOT_SMD:SOT-89-3_Handsoldering, B.Cu at (129.6, 76.4)
Routing:
- net +3V3: track 0.00 -> 149.3 mm, vias 0 -> 2
- net +BATT: track 0.00 -> 72.5 mm
- net /IO9: track 0.00 -> 63.3 mm, vias 0 -> 2
- net /EN: track 0.00 -> 56.1 mm, vias 0 -> 5
- net GND: track 0.00 -> 49.7 mm, vias 0 -> 16
- net /ADC1_CH1: track 0.00 -> 46.4 mm
- net /R_D_SW: track 0.00 -> 45.0 mm, vias 0 -> 1
- net /ADC2_CH0: track 0.00 -> 43.5 mm
- net /RGB: track 0.00 -> 43.5 mm, vias 0 -> 1
- net /L_D_SW: track 0.00 -> 42.9 mm, vias 0 -> 1
- net /ADC1_CH2: track 0.00 -> 40.0 mm
- net /L_BUTTON: track 0.00 -> 32.9 mm, vias 0 -> 1
- net /ADC1_CH4: track 0.00 -> 29.1 mm
- net /ADC1_CH3: track 0.00 -> 19.0 mm
- net VCC: track 0.00 -> 16.8 mm, vias 0 -> 1
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- added copper zone on F.Cu, net GND
- added copper zone on B.Cu, net Net-(U1-VCC)
Other:
- board text added: "+"
- board text added: "3V3"
- board text added: "B"
- board text added: "E"
- board text added: "G"
- board text added: "R"
- board text added: "RESET"
- board text added: "T"
- board text added: "V"

Commit message: update controller pcb
Parts:
- removed U2: ESP32-C3-WROOM-02-N4, bat_rf:BULETM-SMD_18P-L20.0-W18.0-P1.50_ESP32-C3-WROOM
- added U4: ESP32-C3-WROOM-02-N4, espController:ESP32-C3-WROOM-02, B.Cu at (123.4, 62.9)
- J2: footprint Connector_PinSocket_2.54mm:PinSocket_1x02_P2.54mm_Vertical -> espController:CN-XH2P
- SW1: value 3*4*2.5MM_贴片4脚 -> SW_SPST; footprint bat_rf:SW-SMD_4P-L4.2-W3.3-P2.15-LS5.1 -> Button_Switch_SMD:SW_SPST_B3U-1000P
- moved SW1 0.50 mm to (138.0, 76.8)
- moved J2 0.24 mm to (137.5, 66.4), turned to 90 degrees
Connections:
- SW1 pad 2: unconnected-(SW1-Pad2) -> GND

Commit message: update rfBat pcb
Parts:
- SW4, SW6: moved to B.Cu
- U4: moved to F.Cu
- turned SW4 to 45 degrees
- turned SW6 to -45 degrees
- turned U4 to 0 degrees
Routing:
- net /L_U_SW: track 6.10 -> 0.00 mm
- net GND: track 49.7 -> 55.8 mm

Commit message: update rfBat pcb
Parts:
- removed SW1: SW_SPST, Button_Switch_SMD:SW_SPST_B3U-1000P
- removed SW7: SK-12D07-L3-B, Button_Switch_SMD:SW_SPDT_CK_JS102011SAQN
- added D4: BAT54C, Package_TO_SOT_SMD:SOT-23, B.Cu at (164.8, 48.9)
- added Q1: AO3401, Package_TO_SOT_SMD:SOT-23, B.Cu at (170.4, 46.1)
- added Q2: AllPower__AP2300, Package_TO_SOT_SMD:SOT-23, B.Cu at (171.9, 52.6)
- added R8: 33k, Resistor_SMD:R_0603_1608Metric_Pad0.98x0.95mm_HandSolder, B.Cu at (170.4, 49.1)
- added R9: 33k, Resistor_SMD:R_0603_1608Metric_Pad0.98x0.95mm_HandSolder, B.Cu at (171.8, 55.5)
- C1, C10, C4, C5, C6, C7, C8, C9, D1, D2, R1, R3, R4, R5, R6, R7, U1, U3: moved to F.Cu
- C2, C3: moved to B.Cu
- J2: footprint espController:CN-XH2P -> espController:CONN-SMD_2P-P2.54-XH2.54-WT
- moved C10 78.1 mm to (182.0, 126.4)
- moved C9 75.2 mm to (180.1, 126.6)
- moved C8 71.5 mm to (177.5, 124.1), turned to 180 degrees
- moved C7 71.3 mm to (177.4, 122.3), turned to 180 degrees
- moved U3 68.5 mm to (175.3, 127.4), turned to 180 degrees
- moved R4 54.6 mm to (163.6, 128.5)
- moved R3 52.0 mm to (162.0, 128.5)
- moved R5 51.7 mm to (116.2, 136.0), turned to 180 degrees
- moved R6 51.7 mm to (116.1, 134.5), turned to 0 degrees
- moved R7 51.7 mm to (116.1, 130.8), turned to 0 degrees
- moved C6 51.7 mm to (116.1, 132.6), turned to 180 degrees
- moved D2 51.1 mm to (161.4, 125.8), turned to 0 degrees
- moved C4 49.5 mm to (160.4, 128.5)
- moved D1 45.2 mm to (157.5, 125.7), turned to 0 degrees
- moved U1 44.9 mm to (157.3, 128.6), turned to 180 degrees
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Connections:
- C11 pad 2: Net-(D3-VDD) -> VCC
- C2 pad 1: +3V3 -> VCC
- C3 pad 1: +3V3 -> VCC
- C7 pad 1: VCC -> +BATT
- C8 pad 1: VCC -> +BATT
- D3 pad 1: Net-(D3-VDD) -> VCC
- R1 pad 2: +3V3 -> VCC
- R2 pad 2: +3V3 -> VCC
- SW2 pad 1: +3V3 -> VCC
- SW2 pad 4: +3V3 -> VCC
- SW3 pad 1: +3V3 -> VCC
- SW3 pad 4: +3V3 -> VCC
- SW5 pad 1: /R_D_SW -> Net-(D4-C)
- SW8 pad 1: /L_D_SW -> /EN
- TP1 pad 1: +3V3 -> VCC
- U3 pad 3: VCC -> +BATT
- U4 pad 1: +3V3 -> VCC
Routing:
- net +3V3: track 149.3 -> 0.00 mm, vias 2 -> 0
- net +BATT: track 72.5 -> 0.00 mm
- net /IO9: track 63.3 -> 0.00 mm, vias 2 -> 0
- net /EN: track 56.1 -> 0.00 mm, vias 5 -> 0
- net GND: track 55.8 -> 0.00 mm, vias 16 -> 0
- net /ADC1_CH1: track 46.4 -> 0.00 mm
- net /R_D_SW: track 45.0 -> 0.00 mm, vias 1 -> 0
- net /ADC2_CH0: track 43.5 -> 0.00 mm
- net /RGB: track 43.5 -> 0.00 mm, vias 1 -> 0
- net /L_D_SW: track 42.9 -> 0.00 mm, vias 1 -> 0
- net /ADC1_CH2: track 40.0 -> 0.00 mm
- net /L_BUTTON: track 32.9 -> 0.00 mm, vias 1 -> 0
- net /ADC1_CH4: track 29.1 -> 0.00 mm
- net /ADC1_CH3: track 19.0 -> 0.00 mm
- net VCC: track 16.8 -> 0.00 mm, vias 1 -> 0
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- removed copper zone on F.Cu, net GND
- removed copper zone on B.Cu, net Net-(U1-VCC)

Commit message: update controller pcb
Parts:
- removed TP7: TestPoint, TestPoint:TestPoint_Pad_D1.0mm
- C11, C2, C3, D4, Q1, Q2, R2, R8, R9: moved to F.Cu
- J2: moved to B.Cu
- moved J2 79.7 mm to (104.5, 84.5)
- moved C10 76.6 mm to (113.4, 92.2), turned to -90 degrees
- moved C9 73.4 mm to (115.3, 92.0), turned to -90 degrees
- moved C8 66.5 mm to (117.9, 94.5), turned to 0 degrees
- moved U3 66.1 mm to (120.0, 91.2), turned to 0 degrees
- moved C7 64.8 mm to (118.0, 96.3), turned to 0 degrees
- moved R8 61.2 mm to (125.0, 90.2), turned to 90 degrees
- moved Q1 61.2 mm to (128.0, 90.2), turned to 0 degrees
- moved Q2 55.8 mm to (127.6, 86.4), turned to -90 degrees
- moved D4 52.7 mm to (132.1, 90.1), turned to -90 degrees
- moved R9 52.3 mm to (127.6, 83.5)
- moved C6 48.1 mm to (113.4, 84.6), turned to 90 degrees
- moved R5 48.0 mm to (114.9, 88.0), turned to -90 degrees
- moved R6 46.5 mm to (113.4, 88.0), turned to 90 degrees
- moved R7 46.2 mm to (115.0, 84.6), turned to -90 degrees
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Connections:
- SW8 pad 1: /EN -> GND
- SW8 pad 2: GND -> /EN
Routing:
- added copper zone on B.Cu, net GND
Other:
- board text added: "ON"
- board text removed: "3V3"

Commit message: update motor pcb
Parts:
- moved C6 16.5 mm to (129.9, 84.0)
- moved R5 16.5 mm to (131.4, 87.4)
- moved R6 16.5 mm to (129.9, 87.4)
- moved R7 16.5 mm to (131.5, 84.0)
- moved Q2 7.57 mm to (120.9, 82.8)
- moved Q1 7.26 mm to (121.6, 86.7), turned to 90 degrees
- moved R8 7.18 mm to (118.8, 86.6)
- moved D4 6.31 mm to (125.8, 90.4)
- moved R1 5.55 mm to (111.4, 86.8)
- moved C1 5.55 mm to (113.0, 86.8)
- moved R9 3.88 mm to (123.8, 82.7), turned to 90 degrees
- moved R4 3.35 mm to (129.9, 93.6), turned to 180 degrees
- moved D2 3.32 mm to (132.7, 95.2), turned to 90 degrees
- moved TP4 3.30 mm to (123.2, 78.5)
- moved SW5 2.40 mm to (134.4, 103.1)
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Connections:
- J2 pad 1: GND -> +BATT
- J2 pad 2: +BATT -> GND
- SW2 pad 2: /ADC1_CH1 -> /ADC1_CH4
- SW2 pad 5: /ADC1_CH2 -> /ADC2_CH0
- SW3 pad 2: /ADC1_CH4 -> /ADC1_CH1
- SW3 pad 5: /ADC2_CH0 -> /ADC1_CH2
- SW3 pad a: /IO9 -> /R_BUTTON
- SW3 pad c: /IO9 -> /R_BUTTON
- SW5 pad 1: Net-(D4-C) -> GND
- SW5 pad 2: GND -> Net-(D4-C)
- U4 pad 10: /R_D_SW -> /KEY
- U4 pad 13: /L_D_SW -> /POWER_EN
- U4 pad 14: /L_BUTTON -> /R_BUTTON
- U4 pad 18: /L_U_SW -> /R_U_SW
- U4 pad 5: /R_U_SW -> /L_BUTTON
Routing:
- net VCC: track 0.00 -> 177.3 mm, vias 0 -> 2
- net +BATT: track 0.00 -> 48.4 mm, vias 0 -> 3
- net /EN: track 0.00 -> 47.9 mm, vias 0 -> 3
- net GND: track 0.00 -> 47.1 mm, vias 0 -> 23
- net /ADC1_CH4: track 0.00 -> 39.3 mm, vias 0 -> 1
- net /L_BUTTON: track 0.00 -> 37.9 mm, vias 0 -> 1
- net /ADC1_CH2: track 0.00 -> 36.5 mm
- net /RGB: track 0.00 -> 35.4 mm, vias 0 -> 2
- net /ADC2_CH0: track 0.00 -> 34.6 mm, vias 0 -> 1
- net /R_BUTTON: track 0.00 -> 30.0 mm, vias 0 -> 1
- net Net-(U1-VCC): track 0.00 -> 24.9 mm, vias 0 -> 2
- net /ADC1_CH1: track 0.00 -> 23.5 mm
- net Net-(D4-C): track 0.00 -> 17.2 mm, vias 0 -> 2
- net /KEY: track 0.00 -> 17.1 mm
- net /ADC1_CH3: track 0.00 -> 16.9 mm
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Other:
- board text added: "ON/OFF"
- board text added: "V1.0"
- board text removed: "ON"

Commit message: update rfBat firmware
Parts:
- C6: value 2.2u -> 100n
- R5: value 7m -> 7.5m
Connections:
- C11 pad 2: VCC -> +BATT
- D3 pad 1: VCC -> +BATT
- SW2 pad a: /L_BUTTON -> /IO9
- SW2 pad c: /L_BUTTON -> /IO9
- U4 pad 5: /L_BUTTON -> /L_U_SW
Routing:
- net /L_BUTTON: track 37.9 -> 0.00 mm, vias 1 -> 0
- net /IO9: track 8.48 -> 37.2 mm, vias 0 -> 2
- net VCC: track 177.3 -> 150.9 mm, vias 2 -> 1
- net /L_U_SW: track 0.00 -> 14.6 mm, vias 0 -> 1
- net +BATT: track 48.4 -> 52.8 mm
- net /RGB: track 35.4 -> 36.0 mm, vias 2 -> 4
Other:
- outline, holes or cut-outs redrawn
- board text added: "V1.1"
- board text removed: "V1.0"
