File: hardware/controller/controller.kicad_pcb (KiCad board)
At the start: 2 copper layers, 100 x 53.9 mm, 47 parts, among them J1 USB_C_Receptacle_PowerOnly_6P, J2 Bat, Q1 AO3401, Q2 AllPower__AP2300, SW2 RKJXV1224005, SW3 RKJXV1224005, SW4 TC-1102N-C-AS-B, SW5 TS-1199A-B-B, SW6 TC-1102N-C-AS-B, SW8 TS-1199A-B-B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

Commit message: update controller pcb
Parts:
- removed C10: 10u, Capacitor_SMD:C_0805_2012Metric_Pad1.18x1.45mm_HandSolder
- removed C8: 100n, Capacitor_SMD:C_0603_1608Metric_Pad1.08x0.95mm_HandSolder
- added D5: GREEN, LED_SMD:LED_0603_1608Metric_Pad1.05x0.95mm_HandSolder, F.Cu at (116.8, 87.0)
- added R10: 5k, Resistor_SMD:R_0603_1608Metric_Pad0.98x0.95mm_HandSolder, F.Cu at (115.2, 87.0)
- C7: value 10u -> 1u; footprint Capacitor_SMD:C_0805_2012Metric_Pad1.18x1.45mm_HandSolder -> Capacitor_SMD:C_0603_1608Metric_Pad1.08x0.95mm_HandSolder
- C9: value 100n -> 1u
- D2: value GREEN -> BLUE
- U3: value AMS1117 -> XC6220B331MR; footprint Package_TO_SOT_SMD:SOT-89-3_Handsoldering -> Package_TO_SOT_SMD:SOT-23-5
- moved U3 6.14 mm to (115.5, 95.3), turned to 90 degrees
- moved C7 5.33 mm to (112.8, 95.4), turned to 90 degrees
- moved C9 0.22 mm to (115.5, 92.2), turned to 0 degrees
Connections:
- U3 pad 1: GND -> +BATT
- U3 pad 2: +3V3 -> GND
Routing:
- net Net-(D2-K): track 10.5 -> 5.67 mm
- net Net-(U1-VCC): track 24.9 -> 29.3 mm
- net VCC: track 150.9 -> 154.2 mm
- net GND: track 47.1 -> 44.9 mm, vias 23 -> 20
- net Net-(D5-K): track 0.00 -> 1.67 mm
- net +BATT: track 52.8 -> 53.5 mm
Other:
- outline, holes or cut-outs redrawn
- board text added: "V1.2"
- board text removed: "V1.1"
