File: hardware/controller/controller.kicad_pcb (KiCad board)
At the start: 2 copper layers, 100 x 53.9 mm, 43 parts, among them J1 USB_C_Receptacle_PowerOnly_6P, J2 Bat, J3 Conn_01x06, Q1 AO3401, Q2 AllPower__AP2300, Q3 AllPower__AP2300, SW1 TS-1199A-B-B, SW2 RKJXV1224005, SW3 RKJXV1224005, SW5 TS-1199A-B-B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

Commit message: update controller
Parts:
- removed C6: 100n, Capacitor_SMD:C_0603_1608Metric_Pad1.08x0.95mm_HandSolder
- removed R5: 2m, Resistor_SMD:R_0603_1608Metric_Pad0.98x0.95mm_HandSolder
- removed R6: 3m, Resistor_SMD:R_0603_1608Metric_Pad0.98x0.95mm_HandSolder
- removed R7: 1k, Resistor_SMD:R_0603_1608Metric_Pad0.98x0.95mm_HandSolder
- added SW4: SW_Push, espController:SW-TH_TC-1102N-C-AS-B, B.Cu at (108.6, 59.2)
- added SW6: SW_Push, espController:SW-TH_TC-1102N-C-AS-B, B.Cu at (138.0, 59.0)
- R10: value 5k -> 3k6
Routing:
- net /ADC1_CH3: track 34.3 -> 0.16 mm, vias 2 -> 1
- net Net-(C6-Pad1): track 6.45 -> 0.00 mm
- net GND: track 48.0 -> 45.7 mm, vias 20 -> 18
Other:
- board text added: "V1.4"
- board text removed: "V1.3"
