File: hardware/controller/controller.kicad_sch (KiCad schematic)
At the start: 45 parts, among them J1 USB_C_Receptacle_PowerOnly_6P, J2 Bat, SW1 3*4*2.5MM_贴片4脚, SW2 RKJXV1224005, SW3 RKJXV1224005, SW4 TC-1102N-C-AS-B, SW5 TS-1199A-B-B, SW6 TS-1199A-B-B, SW7 TC-1102N-C-AS-B, SW9 SK-12D07-L3-B, U1 TP4059, U2 ESP32-C3-WROOM-02-N4, U3 AMS1117

Commit message: update controller pcb
Parts:
- C11, C4: footprint (none) -> Capacitor_SMD:C_0603_1608Metric_Pad1.08x0.95mm_HandSolder
- R3, R4: footprint (none) -> Resistor_SMD:R_0603_1608Metric_Pad0.98x0.95mm_HandSolder
Changed lines of the file:
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@@
 			)
 		)
-		(property "Footprint" ""
+		(property "Footprint" "Resistor_SMD:R_0603_1608Metric_Pad0.98x0.95mm_HandSolder"
 			(at 69.85 36.83 0)
 			(effects
@@
 			)
 		)
-		(property "Footprint" ""
+		(property "Footprint" "Capacitor_SMD:C_0603_1608Metric_Pad1.08x0.95mm_HandSolder"
 			(at 60.96 38.1 0)
 			(effects
@@
 			)
 		)
-		(property "Footprint" ""
+		(property "Footprint" "Capacitor_SMD:C_0603_1608Metric_Pad1.08x0.95mm_HandSolder"
 			(at 210.82 34.29 0)
 			(effects
@@
 			)
 		)
-		(property "Footprint" ""
+		(property "Footprint" "Resistor_SMD:R_0603_1608Metric_Pad0.98x0.95mm_HandSolder"
 			(at 83.82 44.45 0)
 			(effects

Commit message: update controller pcb
Parts:
- removed SW2, SW3: RKJXV1224005, bat_rf:SW-TH_RKJXV1224005, symbol bat_rf:RKJXV1224005
- removed SW4, SW7: TC-1102N-C-AS-B, bat_rf:SW-TH_TC-1102N-C-AS-B, symbol bat_rf:TC-1102N-C-AS-B
- removed SW5, SW6: TS-1199A-B-B, bat_rf:SW-SMD_L6.0-W6.0-P6.00-LS6.6, symbol bat_rf:TS-1199A-B-B
- removed SW9: SK-12D07-L3-B, bat_rf:SW-TH_SK-12D07-X-X, symbol bat_rf:SK-12D07-L3-B
- added SW2, SW3: RKJXV1224005, espController:SW-TH_RKJXV1224005, symbol espController:RKJXV1224005
- added SW4, SW6: TC-1102N-C-AS-B, espController:SW-TH_TC-1102N-C-AS-B, symbol espController:TC-1102N-C-AS-B
- added SW5, SW8: TS-1199A-B-B, espController:SW-SMD_L6.0-W6.0-P6.00-LS6.6, symbol espController:TS-1199A-B-B
- added SW7: SK-12D07-L3-B, Button_Switch_SMD:SW_SPDT_CK_JS102011SAQN, symbol espController:SK-12D07-L3-B
- C5: footprint (none) -> Capacitor_SMD:C_0805_2012Metric_Pad1.18x1.45mm_HandSolder
- D1, D2: footprint (none) -> LED_SMD:LED_0603_1608Metric_Pad1.05x0.95mm_HandSolder
- J2: footprint (none) -> Connector_PinSocket_2.54mm:PinSocket_1x02_P2.54mm_Vertical
- U1: footprint kicad_lceda:SOT-23-6_L2.9-W1.6-P0.95-LS2.8-BR -> espController:SOT-23-6_L2.9-W1.6-P0.95-LS2.8-BR
Connections:
- net +3V3: now also R2.2, SW2.1 (B), SW2.4 (A), SW3.1 (B), SW3.4 (A)
- net +BATT: now also J2.2 (Pin_2), SW7.2; no longer J2.1 (Pin_1)
- net GND: now also J2.1 (Pin_1), SW2.10 (GND), SW2.3 (A), SW2.6 (B), SW2.7 (GND), SW2.8 (GND), SW2.9 (GND), SW2.b, SW2.d, SW3.10 (GND), SW3.3 (A), SW3.6 (B), SW3.7 (GND), SW3.8 (GND), SW3.9 (GND), SW3.b, SW3.d, SW4.2, SW4.3, SW4.4, SW5.2, SW6.1, SW6.3, SW6.4, SW8.2; no longer J2.2 (Pin_2)
- net IO9: now also SW3.a, SW3.c
- net RGB: now also D3.4 (DIN), U2.6 (IO7); no longer U2.18 (IO0)
- net VCC: now also SW7.3
- net L_D_SW: now reaches U2.13 (IO18)
- net L_D_SW: now also SW8.1
- net L_BUTTON: now reaches U2.14 (IO19)
- net L_BUTTON: now also SW2.a, SW2.c
- net ADC1_CH4: now reaches U2.3 (IO4)
- net ADC1_CH4: now also SW3.2 (DTA)
- net ADC2_CH0: now reaches U2.4 (IO5)
- net ADC2_CH0: now also SW3.5 (DTA)
- net R_U_SW: now reaches U2.5 (IO6)
- net R_U_SW: now also SW6.2
- net BAT_FB renamed ADC1_CH3
- net BEEP renamed ADC1_CH1
- net ADC1_CH1: now also SW2.2 (DTA)
- net BLUE renamed R_D_SW
- net R_D_SW: now also SW5.1
- net YELLOW renamed ADC1_CH2
- net ADC1_CH2: now also SW2.5 (DTA)
- new net L_U_SW: SW4.1, U2.18 (IO0)

Commit message: update controller pcb
Parts:
- removed U2: ESP32-C3-WROOM-02-N4, bat_rf:BULETM-SMD_18P-L20.0-W18.0-P1.50_ESP32-C3-WROOM, symbol bat_rf:ESP32-C3-WROOM-02-N4
- added U4: ESP32-C3-WROOM-02-N4, espController:ESP32-C3-WROOM-02, symbol espController:ESP32-C3-WROOM-02-N4
Connections:
- net +3V3: now also U4.1 (3V3)
- net ADC1_CH1: now also U4.17 (IO1)
- net ADC1_CH2: now also U4.16 (IO2)
- net ADC1_CH3: now also U4.15 (IO3)
- net ADC1_CH4: now also U4.3 (IO4)
- net ADC2_CH0: now also U4.4 (IO5)
- net EN: now also U4.2 (EN)
- net GND: now also U4.19 (EP), U4.9 (GND)
- net IO9: now also U4.8 (IO9)
- net L_BUTTON: now also U4.14 (IO19)
- net L_D_SW: now also U4.13 (IO18)
- net L_U_SW: now also U4.18 (IO0)
- net RGB: now also U4.6 (IO7)
- net RXD: now also U4.11 (RXD)
- net R_D_SW: now also U4.10 (IO10)
- net R_U_SW: now also U4.5 (IO6)
- net TXD: now also U4.12 (TXD)
- net at R2.1: now also U4.7 (IO8)
Changed lines of the file:
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@@
 	)
 	(symbol
+		(lib_id "espController:ESP32-C3-WROOM-02-N4")
+		(at 135.89 158.75 0)
+		(unit 1)
+		(exclude_from_sim no)
+		(in_bom yes)
+		(on_board yes)
+		(dnp no)
+		(fields_autoplaced yes)
+		(property "Reference" "U4"
+			(at 135.89 139.7 0)
+			(effects
+				(font
+					(size 1.27 1.27)
+				)
+			)
+		)
+		(property "Value" "ESP32-C3-WROOM-02-N4"
+			(at 135.89 142.24 0)
+			(effects
+				(font
+					(size 1.27 1.27)
+				)
+			)
+		)
+		(property "Footprint" "espController:ESP32-C3-WROOM-02"
+			(at 135.89 147.2438 0)
+			(effects
+				(font
+					(size 1.27 1.27)
+				)
+				(hide yes)
+			)
+		)
+		(property "Datasheet" ""
+			(at 135.89 152.3238 0)
+			(effects
+				(font
+					(size 1.27 1.27)
+				)
+				(hide yes)
+			)
+		)
+		(property "Description" "C9900000362"
+			(at 135.89 157.4038 0)
+			(effects
+				(font
+					(size 1.27 1.27)
+				)
+				(hide yes)
+			)
+		)
+		(property "uuid" "std:80e57613425b46c2881201d76cb7a63c"
+			(at 135.89 157.4038 0)
+			(effects
+				(font
+					(size 1.27 1.27)
+				)
+				(hide yes)
+			)
+		)
+		(pin "3"
+		)
+		(pin "8"
+		)
+		(pin "4"
+		)
+		(pin "5"
+		)
+		(pin "7"
+		)
+		(pin "9"
+		)
+		(pin "6"
+		)
+		(pin "2"
+		)
+		(pin "11"
+		)
+		(pin "10"
+		)
+		(pin "1"
+		)
+		(pin "12"
+		)
+		(pin "16"
+		)
+		(pin "17"
+		)
+		(pin "14"
+		)
+		(pin "13"
+		)
+		(pin "15"
+		)
+		(pin "18"
+		)
+		(pin "19"
+		)
+		(instances
+			(project "controller"
+				(path "/ac6122ee-da02-46ca-bfd7-d634b1b1f53e"
+					(reference "U4")
+					(unit 1)
+				)
+			)
+		)
+	)
+	(symbol
 		(lib_id "power:GND")
 		(at 196.85 148.59 0)
@@
 					(unit 1)
 				)
-			)
-		)
-	)
-	(symbol
-		(lib_id "bat_rf:ESP32-C3-WROOM-02-N4")
-		(at 135.89 158.75 0)
-		(unit 1)
-		(exclude_from_sim no)
-		(in_bom yes)
-		(on_board yes)
-		(dnp no)
-		(fields_autoplaced yes)
-		(property "Reference" "U2"
-			(at 135.89 139.7 0)
-			(effects
-				(font
-					(size 1.27 1.27)
-				)
-			)
-		)
-		(property "Value" "ESP32-C3-WROOM-02-N4"
-			(at 135.89 142.24 0)
-			(effects
-				(font
-					(size 1.27 1.27)
-				)
-			)
-		)
-		(property "Footprint" "bat_rf:BULETM-SMD_18P-L20.0-W18.0-P1.50_ESP32-C3-WROOM"
-			(at 135.89 147.2438 0)
-			(effects
-				(font
-					(size 1.27 1.27)
-				)
-				(hide yes)
-			)
-		)
-		(property "Datasheet" ""
-			(at 135.89 152.3238 0)
-			(effects
-				(font
-					(size 1.27 1.27)
-				)
-				(hide yes)
-			)
-		)
-		(property "Description" "C9900000362"
-			(at 135.89 157.4038 0)
-			(effects
-				(font
-					(size 1.27 1.27)
-				)
-				(hide yes)
-			)
-		)
-		(property "uuid" "std:80e57613425b46c2881201d76cb7a63c"
-			(at 135.89 157.4038 0)
-			(effects
-				(font
-					(size 1.27 1.27)
-				)
-				(hide yes)
-			)
-		)
-		(pin "11"
-		)
-		(pin "15"
-		)
-		(pin "3"
-		)
-		(pin "16"
-		)
-		(pin "18"
-		)
-		(pin "19"
-		)
-		(pin "5"
-		)
-		(pin "6"
-		)
-		(pin "10"
-		)
-		(pin "7"
-		)
-		(pin "1"
-		)
-		(pin "14"
-		)
-		(pin "4"
-		)
-		(pin "13"
-		)
-		(pin "17"
-		)
-		(pin "8"
-		)
-		(pin "12"
-		)
-		(pin "9"
-		)
-		(pin "2"
-		)
-		(instances
-			(project "controller"
-				(path "/ac6122ee-da02-46ca-bfd7-d634b1b1f53e"
-					(reference "U2")
-					(unit 1)
-				)

Commit message: update rfBat pcb
Parts:
- removed SW1: 3*4*2.5MM_贴片4脚, bat_rf:SW-SMD_4P-L4.2-W3.3-P2.15-LS5.1, symbol bat_rf:3*4*2.5MM_贴片4脚
- added SW1: SW_SPST, Button_Switch_SMD:SW_SPST_B3U-1000P, symbol Switch:SW_SPST
- J2: footprint Connector_PinSocket_2.54mm:PinSocket_1x02_P2.54mm_Vertical -> espController:CN-XH2P
Connections:
- net EN: now also SW1.1 (A)
- net GND: now also SW1.2 (B)
- no-connect marks 6 -> 5
Changed lines of the file:
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@@
 	)
 	(junction
+		(at 52.07 181.61)
+		(diameter 0)
+		(color 0 0 0 0)
+	)
+	(junction
 		(at 139.7 91.44)
 		(diameter 0)
@@
 	)
 	(junction
-		(at 52.07 179.07)
-		(diameter 0)
-		(color 0 0 0 0)
-	)
-	(junction
 		(at 128.27 36.83)
 		(diameter 0)
@@
 	)
 	(no_connect
-		(at 64.77 171.45)
-	)
-	(no_connect
 		(at 228.6 43.18)
 	)
@@
 	(wire
 		(pts
+			(xy 52.07 181.61) (xy 52.07 182.88)
+		)
+		(stroke
+			(width 0)
+			(type default)
+		)
+	)
+	(wire
+		(pts
 			(xy 186.69 82.55) (xy 187.96 82.55)
 		)
@@
 	(wire
 		(pts
-			(xy 52.07 176.53) (xy 52.07 179.07)
+			(xy 52.07 176.53) (xy 52.07 181.61)
 		)
 		(stroke
@@
 	(wire
 		(pts
-			(xy 49.53 171.45) (xy 54.61 171.45)
+			(xy 49.53 171.45) (xy 58.42 171.45)
 		)
 		(stroke
@@
 	(wire
 		(pts
+			(xy 52.07 181.61) (xy 58.42 181.61)
+		)
+		(stroke
+			(width 0)
+			(type default)
+		)
+	)
+	(wire
+		(pts
 			(xy 200.66 80.01) (xy 201.93 80.01)
 		)
@@
 	(wire
 		(pts
-			(xy 52.07 179.07) (xy 52.07 182.88)
-		)
-		(stroke
-			(width 0)
-			(type default)
-		)
-	)
-	(wire
-		(pts
 			(xy 102.87 147.32) (xy 102.87 148.59)
 		)
@@
 	(wire
 		(pts
-			(xy 52.07 179.07) (xy 54.61 179.07)
-		)
-		(stroke
-			(width 0)
-			(type default)
-		)
-	)
-	(wire
-		(pts
 			(xy 252.73 113.03) (xy 252.73 110.49)
 		)
@@
 	)
 	(symbol
+		(lib_id "Switch:SW_SPST")
+		(at 58.42 176.53 270)
+		(unit 1)
+		(exclude_from_sim no)
+		(in_bom yes)
+		(on_board yes)
+		(dnp no)
+		(fields_autoplaced yes)
+		(property "Reference" "SW1"
+			(at 60.96 175.2599 90)
+			(effects
+				(font
+					(size 1.27 1.27)
+				)
+				(justify left)
+			)
+		)
+		(property "Value" "SW_SPST"
+			(at 60.96 177.7999 90)
+			(effects
+				(font
+					(size 1.27 1.27)
+				)
+				(justify left)
+			)
+		)
+		(property "Footprint" "Button_Switch_SMD:SW_SPST_B3U-1000P"
+			(at 58.42 176.53 0)
+			(effects
+				(font
+					(size 1.27 1.27)
+				)
+				(hide yes)
+			)
+		)
+		(property "Datasheet" "~"
+			(at 58.42 176.53 0)
+			(effects
+				(font
+					(size 1.27 1.27)
+				)
+				(hide yes)
+			)
+		)
+		(property "Description" "Single Pole Single Throw (SPST) switch"
+			(at 58.42 176.53 0)
+			(effects
+				(font
+					(size 1.27 1.27)
+				)
+				(hide yes)
+			)
+		)
+		(pin "1"
+		)
+		(pin "2"
+		)
+		(instances
+			(project "controller"
+				(path "/ac6122ee-da02-46ca-bfd7-d634b1b1f53e"
+					(reference "SW1")
+					(unit 1)
+				)
+			)
+		)
+	)
+	(symbol
 		(lib_id "espController:SK-12D07-L3-B")
 		(at 166.37 36.83 270)
@@
 	)
 	(symbol
-		(lib_id "bat_rf:3*4*2.5MM_贴片4脚")
-		(at 59.69 176.53 0)
-		(unit 1)
-		(exclude_from_sim no)
-		(in_bom yes)
-		(on_board yes)
-		(dnp no)
-		(fields_autoplaced yes)
-		(property "Reference" "SW1"
-			(at 59.69 166.37 0)
-			(effects
-				(font
-					(size 1.27 1.27)
-				)
-			)
-		)
-		(property "Value" "3*4*2.5MM_贴片4脚"
-			(at 59.69 168.91 0)
-			(effects
-				(font
-					(size 1.27 1.27)
-				)
-				(hide yes)
-			)
-		)
-		(property "Footprint" "bat_rf:SW-SMD_4P-L4.2-W3.3-P2.15-LS5.1"
-			(at 59.69 171.45 0)
-			(effects
-				(font
-					(size 1.27 1.27)
-				)
-				(hide yes)
-			)
-		)
-		(property "Datasheet" ""
-			(at 59.69 176.53 0)
-			(effects
-				(font
-					(size 1.27 1.27)
-				)
-				(hide yes)
-			)
-		)
-		(property "Description" "C9900020788"
-			(at 59.69 181.61 0)
-			(effects
-				(font
-					(size 1.27 1.27)
-				)
-				(hide yes)
-			)
-		)
-		(property "uuid" "std:cca39041c27d4052af9d3c1225cc14e7"
-			(at 59.69 181.61 0)
-			(effects
-				(font
-					(size 1.27 1.27)
-				)
-				(hide yes)
-			)
-		)
-		(pin "1"
-		)
-		(pin "4"
-		)
-		(pin "3"
-		)
-		(pin "2"
-		)
-		(instances
-			(project "controller"
-				(path "/ac6122ee-da02-46ca-bfd7-d634b1b1f53e"
-					(reference "SW1")
-					(unit 1)
-				)
-			)
-		)
-	)
-	(symbol
 		(lib_id "power:GND")
 		(at 128.27 38.1 0)
@@
 			)
 		)
-		(property "Footprint" "Connector_PinSocket_2.54mm:PinSocket_1x02_P2.54mm_Vertical"
+		(property "Footprint" "espController:CN-XH2P"
 			(at 135.89 34.29 0)
 			(effects

Commit message: update rfBat pcb
Parts:
- removed SW1: SW_SPST, Button_Switch_SMD:SW_SPST_B3U-1000P, symbol Switch:SW_SPST
- removed SW7: SK-12D07-L3-B, Button_Switch_SMD:SW_SPDT_CK_JS102011SAQN, symbol espController:SK-12D07-L3-B
- added D4: BAT54C, bat_rf:BAT54C, symbol bat_rf:BAT54C
- added Q1: AO3401, bat_rf:AO3401, symbol bat_rf:AO3401
- added Q2: AllPower__AP2300, bat_rf:SOT-23, symbol bat_rf:AllPower__AP2300
- added R8, R9: 33k, Resistor_SMD:R_0603_1608Metric_Pad0.98x0.95mm_HandSolder, symbol Device:R
Connections:
- net +3V3: now also Q1.2 (S), R8.1
- net EN: now also SW8.1
- net GND: now also Q2.2 (S), R9.1
- net L_D_SW: no longer SW8.1
- net R_D_SW: no longer SW5.1
- net VCC: now also Q1.3 (D)
- new net: D4.3 (C), SW5.1
- new net: D4.2 (A), Q1.1 (G), Q2.3 (D), R8.2
- new net KEY: D4.1 (A)
- new net POWER_EN: Q2.1 (G), R9.2
- no-connect marks 5 -> 3
Other:
- moved on the sheet: C11, D3, SW5, SW6, SW8

Commit message: update motor pcb
Parts:
- removed TP7: TestPoint, TestPoint:TestPoint_Pad_D1.0mm, symbol Connector:TestPoint
- D4: footprint bat_rf:BAT54C -> Package_TO_SOT_SMD:SOT-23
- J2: footprint espController:CN-XH2P -> espController:CONN-SMD_2P-P2.54-XH2.54-WT
- Q1: footprint bat_rf:AO3401 -> Package_TO_SOT_SMD:SOT-23
- Q2: footprint bat_rf:SOT-23 -> Package_TO_SOT_SMD:SOT-23
Connections:
- net L_D_SW is gone; now on net POWER_EN: U4.13 (IO18)
- net R_D_SW is gone; now on net KEY: U4.10 (IO10)
- net +3V3: no longer C2.1, C3.1, R1.2, R2.2, SW2.1 (B), SW2.4 (A), SW3.1 (B), SW3.4 (A), TP1.1, U4.1 (3V3)
- net +BATT: now also C7.1, C8.1, J2.1 (Pin_1), U3.3 (VI); no longer J2.2 (Pin_2)
- net ADC1_CH1: now also SW3.2 (DTA); no longer SW2.2 (DTA)
- net ADC1_CH2: now also SW3.5 (DTA); no longer SW2.5 (DTA)
- net ADC1_CH4: now also SW2.2 (DTA); no longer SW3.2 (DTA)
- net ADC2_CH0: now also SW2.5 (DTA); no longer SW3.5 (DTA)
- net EN: now also SW8.2; no longer SW8.1
- net GND: now also J2.2 (Pin_2), SW5.1, SW8.1; no longer J2.1 (Pin_1), SW5.2, SW8.2
- net IO9: no longer SW3.a, SW3.c
- net L_BUTTON: now also U4.5 (IO6); no longer U4.14 (IO19)
- net L_U_SW: no longer U4.18 (IO0)
- net R_U_SW: now also U4.18 (IO0); no longer U4.5 (IO6)
- net VCC: now also C11.2, C2.1, C3.1, D3.1 (VDD), R1.2, R2.2, SW2.1 (B), SW2.4 (A), SW3.1 (B), SW3.4 (A), TP1.1, U4.1 (3V3); no longer C7.1, C8.1, U3.3 (VI)
- net at D4.3 (C): now also SW5.2; no longer SW5.1
- new net R_BUTTON: SW3.a, SW3.c, U4.14 (IO19)
Other:
- moved on the sheet: C6, R5, R6, R7, SW4, SW5, SW6

Commit message: update rfBat firmware
Parts:
- C6: value 2.2u -> 100n
- R5: value 7m -> 7.5m
Connections:
- net +BATT: now also C11.2, D3.1 (VDD)
- net IO9: now also SW2.a, SW2.c
- net L_U_SW: now also U4.5 (IO6)
- net VCC: no longer C11.2, D3.1 (VDD)
- removed net L_BUTTON: SW2.a, SW2.c, U4.5 (IO6)
Changed lines of the file:
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@@
 		)
 	)
-	(label "L_BUTTON"
-		(at 125.73 157.48 180)
+	(label "ADC2_CH0"
+		(at 207.01 113.03 90)
+		(fields_autoplaced yes)
+		(effects
+			(font
+				(size 1.27 1.27)
+			)
+			(justify left bottom)
+		)
+	)
+	(label "IO9"
+		(at 125.73 165.1 180)
 		(fields_autoplaced yes)
 		(effects
@@
 		)
 	)
-	(label "ADC2_CH0"
-		(at 207.01 113.03 90)
+	(label "IO9"
+		(at 199.39 135.89 180)
 		(fields_autoplaced yes)
 		(effects
@@
 				(size 1.27 1.27)
 			)
-			(justify left bottom)
+			(justify right bottom)
 		)
 	)
@@
 		)
 	)
+	(label "L_U_SW"
+		(at 165.1 77.47 0)
+		(fields_autoplaced yes)
+		(effects
+			(font
+				(size 1.27 1.27)
+			)
+			(justify left bottom)
+		)
+	)
 	(label "R_U_SW"
 		(at 146.05 147.32 0)
@@
 		)
 	)
+	(label "IO9"
+		(at 214.63 135.89 0)
+		(fields_autoplaced yes)
+		(effects
+			(font
+				(size 1.27 1.27)
+			)
+			(justify left bottom)
+		)
+	)
 	(label "ADC1_CH3"
 		(at 146.05 154.94 0)
@@
 		)
 	)
-	(label "L_BUTTON"
-		(at 214.63 135.89 0)
-		(fields_autoplaced yes)
-		(effects
-			(font
-				(size 1.27 1.27)
-			)
-			(justify left bottom)
-		)
-	)
-	(label "L_BUTTON"
-		(at 199.39 135.89 180)
-		(fields_autoplaced yes)
-		(effects
-			(font
-				(size 1.27 1.27)
-			)
-			(justify right bottom)
-		)
-	)
-	(label "L_U_SW"
-		(at 165.1 77.47 0)
-		(fields_autoplaced yes)
-		(effects
-			(font
-				(size 1.27 1.27)
-			)
-			(justify left bottom)
-		)
-	)
 	(label "L_U_SW"
-		(at 118.11 138.43 0)
+		(at 125.73 157.48 180)
 		(fields_autoplaced yes)
 		(effects
@@
 				(size 1.27 1.27)
 			)
-			(justify left bottom)
+			(justify right bottom)
 		)
 	)
@@
 		)
 	)
-	(label "IO9"
-		(at 125.73 165.1 180)
-		(fields_autoplaced yes)
-		(effects
-			(font
-				(size 1.27 1.27)
-			)
-			(justify right bottom)
-		)
-	)
 	(label "ADC1_CH3"
 		(at 129.54 107.95 0)
@@
 			)
 		)
-		(property "Value" "2.2u"
+		(property "Value" "100n"
 			(at 111.76 116.84 0)
 			(effects
@@
 			)
 		)
-		(property "Value" "7m"
+		(property "Value" "7.5m"
 			(at 123.19 101.6 0)
 			(effects
@@
 	)
 	(symbol
-		(lib_id "power:VCC")
-		(at 172.72 33.02 0)
+		(lib_id "Device:C")
+		(at 110.49 152.4 0)
 		(unit 1)
 		(exclude_from_sim no)
@@
 		(on_board yes)
 		(dnp no)
-		(property "Reference" "#PWR044"
-			(at 172.72 36.83 0)
+		(property "Reference" "C3"
+			(at 106.68 149.86 0)
 			(effects
 				(font
 					(size 1.27 1.27)
 				)
-				(hide yes)
+				(justify left)
 			)
 		)
-		(property "Value" "VCC"
-			(at 172.466 28.194 90)
+		(property "Value" "100n"
+			(at 105.41 154.94 0)
 			(effects
 				(font
 					(size 1.27 1.27)
 				)
+				(justify left)
 			)
 		)
-		(property "Footprint" ""
-			(at 172.72 33.02 0)
+		(property "Footprint" "Capacitor_SMD:C_0603_1608Metric_Pad1.08x0.95mm_HandSolder"
+			(at 111.4552 156.21 0)
 			(effects
 				(font
@@
 			)
 		)
-		(property "Datasheet" ""
-			(at 172.72 33.02 0)
+		(property "Datasheet" "~"
+			(at 110.49 152.4 0)
 			(effects
 				(font
@@
 			)
 		)
-		(property "Description" "Power symbol creates a global label with name \"VCC\""
-			(at 172.72 33.02 0)
+		(property "Description" ""
+			(at 110.49 152.4 0)
 			(effects
 				(font
@@
 		(pin "1"
 		)
+		(pin "2"
+		)
 		(instances
 			(project "controller"
 				(path "/ac6122ee-da02-46ca-bfd7-d634b1b1f53e"
-					(reference "#PWR044")
+					(reference "C3")
 					(unit 1)
 				)
@@
 	)
 	(symbol
-		(lib_id "Device:C")
-		(at 110.49 152.4 0)
+		(lib_id "power:GND")
+		(at 194.31 118.11 180)
 		(unit 1)
 		(exclude_from_sim no)
@@
 		(on_board yes)
 		(dnp no)
-		(property "Reference" "C3"
-			(at 106.68 149.86 0)
+		(fields_autoplaced yes)
+		(property "Reference" "#PWR029"
+			(at 194.31 111.76 0)
 			(effects
 				(font
 					(size 1.27 1.27)
 				)
-				(justify left)
+				(hide yes)
 			)
 		)
-		(property "Value" "100n"
-			(at 105.41 154.94 0)
+		(property "Value" "GND"
+			(at 194.31 113.03 0)
 			(effects
 				(font
 					(size 1.27 1.27)
 				)
-				(justify left)
+				(hide yes)
 			)
 		)
-		(property "Footprint" "Capacitor_SMD:C_0603_1608Metric_Pad1.08x0.95mm_HandSolder"
-			(at 111.4552 156.21 0)
+		(property "Footprint" ""
+			(at 194.31 118.11 0)
 			(effects
 				(font
@@
 			)
 		)
-		(property "Datasheet" "~"
-			(at 110.49 152.4 0)
+		(property "Datasheet" ""
+			(at 194.31 118.11 0)
 			(effects
 				(font
@@
 			)
 		)
-		(property "Description" ""
-			(at 110.49 152.4 0)
+		(property "Description" "Power symbol creates a global label with name \"GND\" , ground"
+			(at 194.31 118.11 0)
 			(effects
 				(font
@@
 		(pin "1"
 		)
-		(pin "2"
-		)
 		(instances
 			(project "controller"
 				(path "/ac6122ee-da02-46ca-bfd7-d634b1b1f53e"
-					(reference "C3")
+					(reference "#PWR029")
 					(unit 1)
 				)
@@
 	)
 	(symbol
-		(lib_id "power:GND")
-		(at 194.31 118.11 180)
+		(lib_id "power:+BATT")
+		(at 172.72 33.02 0)
 		(unit 1)
 		(exclude_from_sim no)
@@
 		(on_board yes)
 		(dnp no)
-		(fields_autoplaced yes)
-		(property "Reference" "#PWR029"
-			(at 194.31 111.76 0)
+		(property "Reference" "#PWR044"
+			(at 172.72 36.83 0)
 			(effects
 				(font
@@
 			)
 		)
-		(property "Value" "GND"
-			(at 194.31 113.03 0)
+		(property "Value" "+BATT"
+			(at 175.26 29.21 0)
 			(effects
 				(font
 					(size 1.27 1.27)
 				)
-				(hide yes)
 			)
 		)
 		(property "Footprint" ""
-			(at 194.31 118.11 0)
+			(at 172.72 33.02 0)
 			(effects
 				(font
@@
 		)
 		(property "Datasheet" ""
-			(at 194.31 118.11 0)
+			(at 172.72 33.02 0)
 			(effects
 				(font
@@
 			)
 		)
-		(property "Description" "Power symbol creates a global label with name \"GND\" , ground"
-			(at 194.31 118.11 0)
+		(property "Description" ""
+			(at 172.72 33.02 0)
 			(effects
 				(font
@@
 			(project "controller"
 				(path "/ac6122ee-da02-46ca-bfd7-d634b1b1f53e"
-					(reference "#PWR029")
+					(reference "#PWR044")
 					(unit 1)
 				)

Commit message: update controller pcb
Parts:
- removed C10: 10u, Capacitor_SMD:C_0805_2012Metric_Pad1.18x1.45mm_HandSolder, symbol Device:C
- removed C8: 100n, Capacitor_SMD:C_0603_1608Metric_Pad1.08x0.95mm_HandSolder, symbol Device:C
- removed U3: AMS1117, Package_TO_SOT_SMD:SOT-89-3_Handsoldering, symbol Regulator_Linear:AMS1117
- added D5: GREEN, LED_SMD:LED_0603_1608Metric_Pad1.05x0.95mm_HandSolder, symbol Device:LED
- added R10: 5k, Resistor_SMD:R_0603_1608Metric_Pad0.98x0.95mm_HandSolder, symbol Device:R
- added U3: XC6220B331MR, Package_TO_SOT_SMD:SOT-23-5, symbol Regulator_Linear:XC6220B331MR
- C7: value 10u -> 1u; footprint Capacitor_SMD:C_0805_2012Metric_Pad1.18x1.45mm_HandSolder -> Capacitor_SMD:C_0603_1608Metric_Pad1.08x0.95mm_HandSolder
- C9: value 100n -> 1u
- D2: value GREEN -> BLUE
Connections:
- net +3V3: now also U3.5 (VOUT)
- net +BATT: now also U3.1 (VIN), U3.3 (CE)
- net GND: now also R10.2, U3.2 (GND)
- net VCC: now also D5.2 (A)
- new net: D5.1 (K), R10.1
Other:
- moved on the sheet: C6, C7, C9, R5, R6, R7
