File: hardware/controller/controller.kicad_sch (KiCad schematic)
At the start: 42 parts, among them J1 USB_C_Receptacle_PowerOnly_6P, J2 Bat, J3 Conn_01x06, Q1 AO3401, Q2 AllPower__AP2300, SW2 RKJXV1224005, SW3 RKJXV1224005, SW4 TC-1102N-C-AS-B, SW5 TS-1199A-B-B, SW6 TC-1102N-C-AS-B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

Commit message: update controller pcb
Parts:
- removed SW4, SW6: TC-1102N-C-AS-B, espController:SW-TH_TC-1102N-C-AS-B, symbol espController:TC-1102N-C-AS-B
- removed SW8: TS-1199A-B-B, espController:SW-SMD_L6.0-W6.0-P6.00-LS6.6, symbol espController:TS-1199A-B-B
- added BUZZER2: MLT-5020_COPY, espController:BUZ-SMD_L5.0-W5.5-P4.60, symbol espController:MLT-5020_COPY
- added Q3: AllPower__AP2300, Package_TO_SOT_SMD:SOT-23, symbol bat_rf:AllPower__AP2300
- added R11: 33k, Resistor_SMD:R_0603_1608Metric_Pad0.98x0.95mm_HandSolder, symbol Device:R
- added SW1: TS-1199A-B-B, espController:SW-SMD_L6.0-W6.0-P6.00-LS6.6, symbol espController:TS-1199A-B-B
Connections:
- net +3V3: now also J3.2 (Pin_2), BUZZER2.1 (+); no longer J3.1 (Pin_1)
- net ADC1_CH0: now also SW2.2 (DTA); no longer SW2.5 (DTA)
- net ADC1_CH4: now also SW2.5 (DTA); no longer SW2.2 (DTA)
- net EN: now also J3.3 (Pin_3), SW1.2; no longer J3.4 (Pin_4)
- net GND: now also J3.1 (Pin_1), Q3.2 (S), R11.1, SW1.1; no longer J3.6 (Pin_6)
- net IO9: now also J3.6 (Pin_6); no longer J3.5 (Pin_5), SW2.a, SW2.c
- net RXD: now also J3.5 (Pin_5); no longer J3.3 (Pin_3)
- net TXD: now also J3.4 (Pin_4); no longer J3.2 (Pin_2)
- net L_U_SW renamed L_BUTTON
- net L_BUTTON: now also SW2.a, SW2.c
- net R_U_SW renamed BEEPER
- net BEEPER: now also Q3.1 (G), R11.2
- new net: BUZZER2.2 (-), Q3.3 (D)
Other:
- moved on the sheet: C11, C6, C7, C9, D3, J3, R5, R6, R7, U3

Commit message: update motor
Parts:
- R10: value 5k -> 3k6
Changed lines of the file:
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@@
 			)
 		)
-		(property "Value" "5k"
-			(at 210.82 49.276 0)
+		(property "Value" "3k6"
+			(at 217.17 49.53 0)
 			(effects
 				(font

Commit message: update controller
Parts:
- removed C6: 100n, Capacitor_SMD:C_0603_1608Metric_Pad1.08x0.95mm_HandSolder, symbol Device:C
- removed R5: 2m, Resistor_SMD:R_0603_1608Metric_Pad0.98x0.95mm_HandSolder, symbol Device:R
- removed R6: 3m, Resistor_SMD:R_0603_1608Metric_Pad0.98x0.95mm_HandSolder, symbol Device:R
- removed R7: 1k, Resistor_SMD:R_0603_1608Metric_Pad0.98x0.95mm_HandSolder, symbol Device:R
- added SW4, SW6: SW_Push, symbol Switch:SW_Push
Connections:
- net +3V3: now also SW4.2, SW6.2
- net ADC1_CH3: now also SW6.1
- net IO9: now also SW4.1
Other:
- moved on the sheet: BUZZER2, C7, C9, Q3, R11, U3
