File: hardware/motor/_autosave-bldcDriver.kicad_sch (KiCad schematic)
At the start: 81 parts, among them J1 Conn_01x02, J2 Conn_01x06, J3 Conn_01x06, J4 Conn_01x03, J5 Conn_01x06, U3 MT2492, U4 MPU-6050, U5 STM32G431CBUx, U6 TLV9062xD, U7 TLV9062xD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

Commit message: update pcb
Parts:
- FB2: footprint Capacitor_SMD:C_0603_1608Metric_Pad1.08x0.95mm_HandSolder -> Capacitor_SMD:C_1206_3216Metric_Pad1.33x1.80mm_HandSolder
Changed lines of the file:
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@@
 			)
 		)
-		(property "Footprint" "Capacitor_SMD:C_0603_1608Metric_Pad1.08x0.95mm_HandSolder"
+		(property "Footprint" "Capacitor_SMD:C_1206_3216Metric_Pad1.33x1.80mm_HandSolder"
 			(at 109.22 81.788 90)
 			(effects
