File: hardware/motor/_autosave-bldcDriver.kicad_sch (KiCad schematic)
At the start: 90 parts, among them J1 Conn_01x02, J2 Conn_01x06, P1 FPC_0.5MM_4P_Vertical_mountin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, SW1 SW_Push, SW2 SW_Push, U10 HC-FPC-0.5-6P-CSH20, U3 TPS5430DDA, U4 HC-FPC-0.5-6P-CSH20, U5 STM32G431CBUx, U6 TLV9062xD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

Commit message: update driver pcb
Connections:
- net +3V3: now also P1.3; no longer P1.4
- net GNDD: now also P1.1; no longer P1.2
- net USART2_RX: now also P1.2; no longer P1.1
- net USART2_TX: now also P1.4; no longer P1.3
Changed lines of the file:
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@@
 	(wire
 		(pts
+			(xy 341.63 228.6) (xy 341.63 229.87)
+		)
+		(stroke
+			(width 0)
+			(type default)
+		)
+	)
+	(wire
+		(pts
 			(xy 67.31 151.13) (xy 60.96 151.13)
 		)
@@
 	(wire
 		(pts
-			(xy 328.93 226.06) (xy 339.09 226.06)
-		)
-		(stroke
-			(width 0)
-			(type default)
-		)
-	)
-	(wire
-		(pts
 			(xy 146.05 33.02) (xy 140.97 33.02)
 		)
@@
 	(wire
 		(pts
+			(xy 328.93 223.52) (xy 339.09 223.52)
+		)
+		(stroke
+			(width 0)
+			(type default)
+		)
+	)
+	(wire
+		(pts
 			(xy 91.44 38.1) (xy 102.87 38.1)
 		)
@@
 	(wire
 		(pts
-			(xy 328.93 220.98) (xy 339.09 220.98)
-		)
-		(stroke
-			(width 0)
-			(type default)
-		)
-	)
-	(wire
-		(pts
 			(xy 95.25 43.18) (xy 91.44 43.18)
 		)
@@
 	(wire
 		(pts
+			(xy 328.93 228.6) (xy 341.63 228.6)
+		)
+		(stroke
+			(width 0)
+			(type default)
+		)
+	)
+	(wire
+		(pts
 			(xy 146.05 245.11) (xy 152.4 245.11)
 		)
@@
 		)
 	)
-	(label "USART2_RX"
-		(at 328.93 228.6 0)
-		(fields_autoplaced yes)
-		(effects
-			(font
-				(size 1.27 1.27)
-			)
-			(justify left bottom)
-		)
-	)
 	(label "KEY"
 		(at 237.49 167.64 0)
@@
 		)
 	)
+	(label "USART2_RX"
+		(at 328.93 226.06 0)
+		(fields_autoplaced yes)
+		(effects
+			(font
+				(size 1.27 1.27)
+			)
+			(justify left bottom)
+		)
+	)
 	(label "VREF_OP"
 		(at 45.72 175.26 180)
@@
 		)
 	)
-	(label "SPI3_SCK"
-		(at 325.12 189.23 180)
+	(label "USART2_TX"
+		(at 328.93 220.98 0)
 		(fields_autoplaced yes)
 		(effects
@@
 				(size 1.27 1.27)
 			)
-			(justify right bottom)
+			(justify left bottom)
 		)
 	)
-	(label "USART2_TX"
-		(at 328.93 223.52 0)
+	(label "SPI3_SCK"
+		(at 325.12 189.23 180)
 		(fields_autoplaced yes)
 		(effects
@@
 				(size 1.27 1.27)
 			)
-			(justify left bottom)
+			(justify right bottom)
 		)
 	)
@@
 	)
 	(symbol
-		(lib_id "power:GNDD")
-		(at 339.09 226.06 90)
+		(lib_id "Device:R_Small")
+		(at 48.26 175.26 270)
 		(unit 1)
 		(exclude_from_sim no)
@@
 		(on_board yes)
 		(dnp no)
-		(fields_autoplaced yes)
-		(property "Reference" "#PWR016"
-			(at 345.44 226.06 0)
+		(property "Reference" "R33"
+			(at 50.546 174.244 90)
 			(effects
 				(font
 					(size 1.27 1.27)
 				)
-				(hide yes)
+				(justify left)
 			)
 		)
-		(property "Value" "GNDD"
-			(at 342.9 226.06 0)
+		(property "Value" "10k"
+			(at 50.546 176.276 90)
 			(effects
 				(font
 					(size 1.27 1.27)
 				)
-				(hide yes)
+				(justify left)
 			)
 		)
-		(property "Footprint" ""
-			(at 339.09 226.06 0)
+		(property "Footprint" "Resistor_SMD:R_0603_1608Metric_Pad0.98x0.95mm_HandSolder"
+			(at 48.26 175.26 0)
 			(effects
 				(font
@@
 			)
 		)
-		(property "Datasheet" ""
-			(at 339.09 226.06 0)
+		(property "Datasheet" "~"
+			(at 48.26 175.26 0)
 			(effects
 				(font
@@
 			)
 		)
-		(property "Description" "Power symbol creates a global label with name \"GNDD\" , digital ground"
-			(at 339.09 226.06 0)
+		(property "Description" "Resistor, small symbol"
+			(at 48.26 175.26 0)
 			(effects
 				(font
@@
 		(pin "1"
 		)
+		(pin "2"
+		)
 		(instances
 			(project "bldcDriver"
 				(path "/024b6358-58d2-4f27-baff-bf9e44899c87"
-					(reference "#PWR016")
+					(reference "R33")
 					(unit 1)
 				)
@@
 	)
 	(symbol
-		(lib_id "Device:R_Small")
-		(at 48.26 175.26 270)
+		(lib_id "power:GNDD")
+		(at 388.62 114.3 0)
 		(unit 1)
 		(exclude_from_sim no)
@@
 		(on_board yes)
 		(dnp no)
-		(property "Reference" "R33"
-			(at 50.546 174.244 90)
+		(fields_autoplaced yes)
+		(property "Reference" "#PWR039"
+			(at 388.62 120.65 0)
 			(effects
 				(font
 					(size 1.27 1.27)
 				)
-				(justify left)
+				(hide yes)
 			)
 		)
-		(property "Value" "10k"
-			(at 50.546 176.276 90)
+		(property "Value" "GNDD"
+			(at 388.62 118.11 0)
 			(effects
 				(font
 					(size 1.27 1.27)
 				)
-				(justify left)
 			)
 		)
-		(property "Footprint" "Resistor_SMD:R_0603_1608Metric_Pad0.98x0.95mm_HandSolder"
-			(at 48.26 175.26 0)
+		(property "Footprint" ""
+			(at 388.62 114.3 0)
 			(effects
 				(font
@@
 			)
 		)
-		(property "Datasheet" "~"
-			(at 48.26 175.26 0)
+		(property "Datasheet" ""
+			(at 388.62 114.3 0)
 			(effects
 				(font
@@
 			)
 		)
-		(property "Description" "Resistor, small symbol"
-			(at 48.26 175.26 0)
+		(property "Description" "Power symbol creates a global label with name \"GNDD\" , digital ground"
+			(at 388.62 114.3 0)
 			(effects
 				(font
@@
 		(pin "1"
 		)
-		(pin "2"
-		)
 		(instances
 			(project "bldcDriver"
 				(path "/024b6358-58d2-4f27-baff-bf9e44899c87"
-					(reference "R33")
+					(reference "#PWR039")
 					(unit 1)
 				)
@@
 	)
 	(symbol
-		(lib_id "power:GNDD")
-		(at 388.62 114.3 0)
+		(lib_id "power:+3V3")
+		(at 339.09 223.52 270)
+		(mirror x)
 		(unit 1)
 		(exclude_from_sim no)
@@
 		(on_board yes)
 		(dnp no)
-		(fields_autoplaced yes)
-		(property "Reference" "#PWR039"
-			(at 388.62 120.65 0)
+		(property "Reference" "#PWR016"
+			(at 335.28 223.52 0)
 			(effects
 				(font
@@
 			)
 		)
-		(property "Value" "GNDD"
-			(at 388.62 118.11 0)
+		(property "Value" "+3V3"
+			(at 344.17 223.52 90)
 			(effects
 				(font
@@
 		)
 		(property "Footprint" ""
-			(at 388.62 114.3 0)
+			(at 339.09 223.52 0)
 			(effects
 				(font
@@
 		)
 		(property "Datasheet" ""
-			(at 388.62 114.3 0)
+			(at 339.09 223.52 0)
 			(effects
 				(font
@@
 			)
 		)
-		(property "Description" "Power symbol creates a global label with name \"GNDD\" , digital ground"
-			(at 388.62 114.3 0)
+		(property "Description" "Power symbol creates a global label with name \"+3V3\""
+			(at 339.09 223.52 0)
 			(effects
 				(font
@@
 			(project "bldcDriver"
 				(path "/024b6358-58d2-4f27-baff-bf9e44899c87"
-					(reference "#PWR039")
+					(reference "#PWR016")
 					(unit 1)
 				)
@@
 	)
 	(symbol
+		(lib_id "power:GNDD")
+		(at 341.63 229.87 0)
+		(unit 1)
+		(exclude_from_sim no)
+		(in_bom yes)
+		(on_board yes)
+		(dnp no)
+		(fields_autoplaced yes)
+		(property "Reference" "#PWR068"
+			(at 341.63 236.22 0)
+			(effects
+				(font
+					(size 1.27 1.27)
+				)
+				(hide yes)
+			)
+		)
+		(property "Value" "GNDD"
+			(at 341.63 233.68 0)
+			(effects
+				(font
+					(size 1.27 1.27)
+				)
+			)
+		)
+		(property "Footprint" ""
+			(at 341.63 229.87 0)
+			(effects
+				(font
+					(size 1.27 1.27)
+				)
+				(hide yes)
+			)
+		)
+		(property "Datasheet" ""
+			(at 341.63 229.87 0)
+			(effects
+				(font
+					(size 1.27 1.27)
+				)
+				(hide yes)
+			)
+		)
+		(property "Description" "Power symbol creates a global label with name \"GNDD\" , digital ground"
+			(at 341.63 229.87 0)
+			(effects
+				(font
+					(size 1.27 1.27)
+				)
+				(hide yes)
+			)
+		)
+		(pin "1"
+		)
+		(instances
+			(project "bldcDriver"
+				(path "/024b6358-58d2-4f27-baff-bf9e44899c87"
+					(reference "#PWR068")
+					(unit 1)
+				)
+			)
+		)
+	)
+	(symbol
 		(lib_id "power:VDDA")
 		(at 339.09 43.18 0)
@@
 		(on_board yes)
 		(dnp no)
-		(fields_autoplaced yes)
 		(property "Reference" "P1"
 			(at 318.77 222.2499 0)
@@
 					(unit 1)
 				)
-			)
-		)
-	)
-	(symbol
-		(lib_id "power:+3V3")
-		(at 339.09 220.98 270)
-		(unit 1)
-		(exclude_from_sim no)
-		(in_bom yes)
-		(on_board yes)
-		(dnp no)
-		(property "Reference" "#PWR068"
-			(at 335.28 220.98 0)
-			(effects
-				(font
-					(size 1.27 1.27)
-				)
-				(hide yes)
-			)
-		)
-		(property "Value" "+3V3"
-			(at 344.17 220.98 90)
-			(effects
-				(font
-					(size 1.27 1.27)
-				)
-			)
-		)
-		(property "Footprint" ""
-			(at 339.09 220.98 0)
-			(effects
-				(font
-					(size 1.27 1.27)
-				)
-				(hide yes)
-			)
-		)
-		(property "Datasheet" ""
-			(at 339.09 220.98 0)
-			(effects
-				(font
-					(size 1.27 1.27)
-				)
-				(hide yes)
-			)
-		)
-		(property "Description" "Power symbol creates a global label with name \"+3V3\""
-			(at 339.09 220.98 0)
-			(effects
-				(font
-					(size 1.27 1.27)
-				)
-				(hide yes)
-			)
-		)
-		(pin "1"
-		)
-		(instances
-			(project "bldcDriver"
-				(path "/024b6358-58d2-4f27-baff-bf9e44899c87"
-					(reference "#PWR068")
-					(unit 1)
-				)
