File: hardware/motor/untitled.kicad_sch (KiCad schematic)
At the start: 88 parts, among them CN1 MR30PW-F, CN2 MR30PW-F, Q1 EMB09N03V, Q10 EMB09N03V, Q11 EMB09N03V, Q12 EMB09N03V, Q13 EMB09N03V, Q14 EMB09N03V, Q15 EMB09N03V, Q16 EMB09N03V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

Commit message: update pcn
Connections:
- net +BATT: now also C15.1, C32.1, U1.7 (VCC), U2.7 (VCC)
Other:
- moved on the sheet: TP16
Changed lines of the file:
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@@
 	)
 	(junction
+		(at 60.96 97.79)
+		(diameter 0)
+		(color 0 0 0 0)
+	)
+	(junction
 		(at 251.46 167.64)
 		(diameter 0)
@@
 	)
 	(junction
+		(at 66.04 204.47)
+		(diameter 0)
+		(color 0 0 0 0)
+	)
+	(junction
 		(at 297.18 166.37)
 		(diameter 0)
@@
 	(wire
 		(pts
+			(xy 58.42 92.71) (xy 66.04 92.71)
+		)
+		(stroke
+			(width 0)
+			(type default)
+		)
+	)
+	(wire
+		(pts
 			(xy 114.3 180.34) (xy 114.3 196.85)
 		)
@@
 	(symbol
 		(lib_id "Connector:TestPoint")
-		(at 66.04 92.71 90)
+		(at 58.42 92.71 90)
 		(unit 1)
 		(exclude_from_sim no)
@@
 		(dnp no)
 		(property "Reference" "TP16"
-			(at 60.96 94.234 0)
+			(at 53.34 94.234 0)
 			(effects
 				(font
@@
 		)
 		(property "Value" "TestPoint"
-			(at 64.0079 90.17 0)
+			(at 56.3879 90.17 0)
 			(effects
 				(font
@@
 		)
 		(property "Footprint" "TestPoint:TestPoint_Pad_D1.0mm"
-			(at 66.04 87.63 0)
+			(at 58.42 87.63 0)
 			(effects
 				(font
@@
 		)
 		(property "Datasheet" "~"
-			(at 66.04 87.63 0)
+			(at 58.42 87.63 0)
 			(effects
 				(font
@@
 		)
 		(property "Description" "test point"
-			(at 66.04 92.71 0)
+			(at 58.42 92.71 0)
 			(effects
 				(font
@@
 	)
 	(symbol
+		(lib_id "power:+BATT")
+		(at 60.96 97.79 0)
+		(unit 1)
+		(exclude_from_sim no)
+		(in_bom yes)
+		(on_board yes)
+		(dnp no)
+		(fields_autoplaced yes)
+		(property "Reference" "#PWR066"
+			(at 60.96 101.6 0)
+			(effects
+				(font
+					(size 1.27 1.27)
+				)
+				(hide yes)
+			)
+		)
+		(property "Value" "+BATT"
+			(at 60.96 93.98 0)
+			(effects
+				(font
+					(size 1.27 1.27)
+				)
+			)
+		)
+		(property "Footprint" ""
+			(at 60.96 97.79 0)
+			(effects
+				(font
+					(size 1.27 1.27)
+				)
+				(hide yes)
+			)
+		)
+		(property "Datasheet" ""
+			(at 60.96 97.79 0)
+			(effects
+				(font
+					(size 1.27 1.27)
+				)
+				(hide yes)
+			)
+		)
+		(property "Description" "Power symbol creates a global label with name \"+BATT\""
+			(at 60.96 97.79 0)
+			(effects
+				(font
+					(size 1.27 1.27)
+				)
+				(hide yes)
+			)
+		)
+		(pin "1"
+		)
+		(instances
+			(project "bldcDriver"
+				(path "/024b6358-58d2-4f27-baff-bf9e44899c87/f49693e9-44aa-4011-a606-f09dffd6beb1"
+					(reference "#PWR066")
+					(unit 1)
+				)
+			)
+		)
+	)
+	(symbol
 		(lib_id "bldcDriver:EMB09N03V")
 		(at 250.19 203.2 270)
@@
 					(unit 1)
 				)
+			)
+		)
+	)
+	(symbol
+		(lib_id "power:+BATT")
+		(at 66.04 204.47 0)
+		(unit 1)
+		(exclude_from_sim no)
+		(in_bom yes)
+		(on_board yes)
+		(dnp no)
+		(fields_autoplaced yes)
+		(property "Reference" "#PWR067"
+			(at 66.04 208.28 0)
+			(effects
+				(font
+					(size 1.27 1.27)
+				)
+				(hide yes)
+			)
+		)
+		(property "Value" "+BATT"
+			(at 66.04 200.66 0)
+			(effects
+				(font
+					(size 1.27 1.27)
+				)
+			)
+		)
+		(property "Footprint" ""
+			(at 66.04 204.47 0)
+			(effects
+				(font
+					(size 1.27 1.27)
+				)
+				(hide yes)
+			)
+		)
+		(property "Datasheet" ""
+			(at 66.04 204.47 0)
+			(effects
+				(font
+					(size 1.27 1.27)
+				)
+				(hide yes)
+			)
+		)
+		(property "Description" "Power symbol creates a global label with name \"+BATT\""
+			(at 66.04 204.47 0)
+			(effects
+				(font
+					(size 1.27 1.27)
+				)
+				(hide yes)
+			)
+		)
+		(pin "1"
+		)
+		(instances
+			(project "bldcDriver"
+				(path "/024b6358-58d2-4f27-baff-bf9e44899c87/f49693e9-44aa-4011-a606-f09dffd6beb1"
+					(reference "#PWR067")
+					(unit 1)
+				)

Commit message: update motor pcb
Parts:
- added R49, R54, R55, R56, R57, R58: 3k, Resistor_SMD:R_0603_1608Metric_Pad0.98x0.95mm_HandSolder, symbol Device:R
Connections:
- net TIM1_CH1: now also R58.1
- net TIM1_CH2: now also R57.1
- net TIM1_CH3: now also R56.1
- net TIM8_CH1: now also R55.1
- net TIM8_CH2: now also R54.1
- net TIM8_CH3: now also R49.1
- new net GNDD: R49.2, R54.2, R55.2, R56.2, R57.2, R58.2

Commit message: update motor pcb
Parts:
- removed R49, R54, R55, R56, R57, R58: 3k, Resistor_SMD:R_0603_1608Metric_Pad0.98x0.95mm_HandSolder, symbol Device:R
- added TP26, TP27, TP28, TP9: TestPoint, TestPoint:TestPoint_Pad_D1.0mm, symbol Connector:TestPoint
Connections:
- net at Q16.1 (S), Q16.2 (S), Q16.3 (S)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: now also TP27.1
- net at Q1.1 (S), Q1.2 (S), Q1.3 (S)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: now also TP28.1
- net at Q8.1 (S), Q8.2 (S), Q8.3 (S)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: now also TP9.1
- net at Q12.1 (S), Q12.2 (S), Q12.3 (S)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: now also TP26.1
