File: hardware/motor/untitled.kicad_sch (KiCad schematic)
At the start: 92 parts, among them CN1 MR30PW-F, CN2 MR30PW-F, Q1 EMB09N03V, Q10 EMB09N03V, Q11 EMB09N03V, Q12 EMB09N03V, Q13 EMB09N03V, Q14 EMB09N03V, Q15 EMB09N03V, Q16 EMB09N03V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

Commit message: update motor
Parts:
- D10, D11, D2, D3, D4, D7: value D -> DSK34
Changed lines of the file:
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@@
 		(on_board yes)
 		(dnp no)
-		(fields_autoplaced yes)
 		(property "Reference" "D7"
-			(at 106.68 67.3099 90)
+			(at 104.14 66.04 90)
 			(effects
 				(font
@@
 			)
 		)
-		(property "Value" "D"
-			(at 106.68 69.8499 90)
+		(property "Value" "DSK34"
+			(at 101.6 66.04 0)
 			(effects
 				(font
@@
 			)
 		)
-		(property "Value" "D"
+		(property "Value" "DSK34"
 			(at 125.73 69.8499 90)
 			(effects
@@
 			)
 		)
-		(property "Value" "D"
+		(property "Value" "DSK34"
 			(at 120.65 176.5299 90)
 			(effects
@@
 		(on_board yes)
 		(dnp no)
-		(fields_autoplaced yes)
 		(property "Reference" "D2"
 			(at 111.76 173.9899 90)
@@
 			)
 		)
-		(property "Value" "D"
-			(at 111.76 176.5299 90)
+		(property "Value" "DSK34"
+			(at 106.68 170.18 0)
 			(effects
 				(font
@@
 			)
 		)
-		(property "Value" "D"
+		(property "Value" "DSK34"
 			(at 115.57 69.8499 90)
 			(effects
@@
 			)
 		)
-		(property "Value" "D"
+		(property "Value" "DSK34"
 			(at 130.81 176.5299 90)
 			(effects

Commit message: update motor pcb
Parts:
- added R40, R54, R55, R56, R57, R58: 3k, Resistor_SMD:R_0603_1608Metric_Pad0.98x0.95mm_HandSolder, symbol Device:R
- D10, D11, D2, D3, D4, D7: value DSK34 -> FR107
Connections:
- net TIM1_CH1: now also R58.1
- net TIM1_CH2: now also R57.1
- net TIM1_CH3: now also R56.1
- net TIM8_CH1: now also R55.1
- net TIM8_CH2: now also R54.1
- net TIM8_CH3: now also R40.1
- new net GNDD: R40.2, R54.2, R55.2, R56.2, R57.2, R58.2
Other:
- moved on the sheet: TP13, TP16
