File: hardware/motor/bldcDriver.kicad_sch (KiCad schematic)
At the start: 81 parts, among them J1 Conn_01x02, J2 Conn_01x06, J3 Conn_01x06, J4 Conn_01x03, J5 Conn_01x06, U3 MT2492, U4 MPU-6050, U5 STM32G431CBUx, U6 TLV9062xD, U7 TLV9062xD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

Commit message: update controller firmware
Parts:
- added TP10, TP11, TP12, TP18, TP7, TP9: TestPoint, TestPoint:TestPoint_Pad_D1.0mm, symbol Connector:TestPoint
- FB2: footprint Capacitor_SMD:C_0603_1608Metric_Pad1.08x0.95mm_HandSolder -> Capacitor_SMD:C_1206_3216Metric_Pad1.33x1.80mm_HandSolder
Connections:
- net +3V3: now also TP7.1
- net GNDD: now also TP18.1
- net at R51.2, R52.1, U7.7: now also TP10.1
- net at R34.2, R35.1, U6.1: now also TP12.1
- net at R48.2, R50.1, U6.7: now also TP11.1
- net at R36.2, R37.1, U7.1: now also TP9.1

Commit message: update motor firmware
Connections:
- net ADC1_IN11 renamed M2_CS_B
- net ADC1_IN5 renamed M1_CS_A
- net ADC2_IN12 renamed M2_CS_A
- net ADC2_IN15 renamed M1_CS_B
Changed lines of the file:
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@@
-		)
-	)
-	(label "ADC1_IN11"
-		(at 113.03 265.43 0)
-		(fields_autoplaced yes)
-		(effects
-			(font
-				(size 1.27 1.27)
-			)
-			(justify left bottom)
 		)
 	)
@@
 		)
 	)
-	(label "ADC1_IN5"
+	(label "M1_CS_A"
 		(at 341.63 120.65 180)
 		(fields_autoplaced yes)
@@
 		)
 	)
-	(label "ADC2_IN15"
-		(at 341.63 123.19 180)
-		(fields_autoplaced yes)
-		(effects
-			(font
-				(size 1.27 1.27)
-			)
-			(justify right bottom)
-		)
-	)
 	(label "USART3_TX"
 		(at 341.63 110.49 180)
@@
 		)
 	)
+	(label "M1_CS_B"
+		(at 341.63 123.19 180)
+		(fields_autoplaced yes)
+		(effects
+			(font
+				(size 1.27 1.27)
+			)
+			(justify right bottom)
+		)
+	)
 	(label "NSS2"
 		(at 377.19 180.34 180)
@@
 		)
 	)
-	(label "ADC2_IN12"
-		(at 57.15 264.16 0)
-		(fields_autoplaced yes)
-		(effects
-			(font
-				(size 1.27 1.27)
-			)
-			(justify left bottom)
-		)
-	)
 	(label "1CS1-"
 		(at 232.41 208.28 180)
@@
 		)
 	)
-	(label "ADC2_IN12"
+	(label "M2_CS_A"
 		(at 341.63 90.17 180)
 		(fields_autoplaced yes)
@@
 		)
 	)
-	(label "ADC2_IN15"
+	(label "M1_CS_B"
 		(at 114.3 210.82 0)
 		(fields_autoplaced yes)
@@
 		)
 	)
+	(label "M2_CS_B"
+		(at 113.03 265.43 0)
+		(fields_autoplaced yes)
+		(effects
+			(font
+				(size 1.27 1.27)
+			)
+			(justify left bottom)
+		)
+	)
 	(label "TIM1_CH2"
 		(at 374.65 69.85 0)
@@
 		)
 	)
-	(label "ADC1_IN5"
+	(label "M1_CS_A"
 		(at 58.42 209.55 0)
 		(fields_autoplaced yes)
@@
 		)
 	)
-	(label "ADC1_IN11"
+	(label "M2_CS_B"
 		(at 341.63 115.57 180)
 		(fields_autoplaced yes)
@@
 		)
 	)
+	(label "M2_CS_A"
+		(at 57.15 264.16 0)
+		(fields_autoplaced yes)
+		(effects
+			(font
+				(size 1.27 1.27)
+			)
+			(justify left bottom)
+		)
+	)

Commit message: update rfBat pcb
Parts:
- removed R53: 100k, Resistor_SMD:R_0603_1608Metric_Pad0.98x0.95mm_HandSolder, symbol Device:R_Small
- removed TP10, TP11, TP12, TP18, TP7, TP9: TestPoint, TestPoint:TestPoint_Pad_D1.0mm, symbol Connector:TestPoint
- removed U3: MT2492, balancerDriver:SOT-23-6_L2.9-W1.6-P0.95-LS2.8-BL, symbol bldcDriver:MT2492
- added C8: 100n, Capacitor_SMD:C_0603_1608Metric_Pad1.08x0.95mm_HandSolder, symbol Device:C_Small
- added D8: 1N5712UR, balancerDriver:SMA_L4.3-W2.6-LS5.0-RD, symbol Diode:1N5712UR
- added U3: TPS5430DDA, Package_SO:TI_SO-PowerPAD-8_ThermalVias, symbol Regulator_Switching:TPS5430DDA
- C1: value 100n -> 10n
- C3: value 100n -> 47u; footprint Capacitor_SMD:C_0603_1608Metric_Pad1.08x0.95mm_HandSolder -> Capacitor_SMD:C_1206_3216Metric_Pad1.33x1.80mm_HandSolder
- C4: value 22u -> 47u; footprint Capacitor_SMD:C_0805_2012Metric_Pad1.18x1.45mm_HandSolder -> Capacitor_SMD:C_1206_3216Metric_Pad1.33x1.80mm_HandSolder
- C5: value 47u -> 22u; footprint Capacitor_SMD:C_1206_3216Metric_Pad1.33x1.80mm_HandSolder -> Capacitor_SMD:C_0805_2012Metric_Pad1.18x1.45mm_HandSolder
- FB2: footprint Capacitor_SMD:C_1206_3216Metric_Pad1.33x1.80mm_HandSolder -> Capacitor_SMD:C_0603_1608Metric_Pad1.08x0.95mm_HandSolder
Connections:
- net +3V3: now also C2.2, C8.2; no longer C5.2
- net +BATT: now also C5.2, U3.7 (VIN); no longer C2.2
- net GNDPWR: now also C8.1, D8.2 (A), U3.6 (GND), U3.9 (GNDPAD)
- net at R1.2, R2.1: now also U3.4 (VSENSE)
- net at C1.1: now also U3.1 (BOOT)
- net at C1.2, L1.1: now also D8.1 (K), U3.8 (PH)
- net M1_CS_A renamed ADC1_IN5
- net M1_CS_B renamed ADC2_IN15
- net M2_CS_A renamed ADC2_IN12
- net M2_CS_B renamed ADC1_IN11
- no-connect marks 3 -> 4
Other:
- moved on the sheet: C6, C7, D1, J1, R3

Commit message: update rfbat pcb
Parts:
- removed D8: 1N5712UR, balancerDriver:SMA_L4.3-W2.6-LS5.0-RD, symbol Diode:1N5712UR
- removed U3: TPS5430DDA, Package_SO:TI_SO-PowerPAD-8_ThermalVias, symbol Regulator_Switching:TPS5430DDA
- added FB4: FerriteBead, Capacitor_SMD:C_0603_1608Metric_Pad1.08x0.95mm_HandSolder, symbol Device:FerriteBead
- added R53: 100k, Resistor_SMD:R_0603_1608Metric_Pad0.98x0.95mm_HandSolder, symbol Device:R_Small
- added SW1: SW_Push, symbol Switch:SW_Push
- added U3: MT2492, balancerDriver:SOT-23-6_L2.9-W1.6-P0.95-LS2.8-BL, symbol bldcDriver:MT2492
- C1: value 10n -> 100n
- C21: value 470n -> 100n
- C3: value 47u -> 100n; footprint Capacitor_SMD:C_1206_3216Metric_Pad1.33x1.80mm_HandSolder -> Capacitor_SMD:C_0603_1608Metric_Pad1.08x0.95mm_HandSolder
- C4: value 47u -> 22u; footprint Capacitor_SMD:C_1206_3216Metric_Pad1.33x1.80mm_HandSolder -> Capacitor_SMD:C_0805_2012Metric_Pad1.18x1.45mm_HandSolder
- C5: value 22u -> 47u; footprint Capacitor_SMD:C_0805_2012Metric_Pad1.18x1.45mm_HandSolder -> Capacitor_SMD:C_1206_3216Metric_Pad1.33x1.80mm_HandSolder
- C8: value 100n -> 470n
- FB2: footprint Capacitor_SMD:C_0603_1608Metric_Pad1.08x0.95mm_HandSolder -> Capacitor_SMD:C_1206_3216Metric_Pad1.33x1.80mm_HandSolder
Connections:
- net +3V3: now also C5.2, FB4.1; no longer C17.1, C2.2, C21.1, C8.2, U5.20 (VREF+), U5.21 (VDDA)
- net +BATT: now also C2.2, R53.2, U3.5 (IN); no longer C5.2
- net GNDD: now also C8.2, SW1.2
- net GNDPWR: now also U3.2 (GND); no longer C8.1
- net at C1.1: now also U3.1 (BS)
- net at C1.2, L1.1: now also U3.6 (SW)
- net at R1.2, R2.1: now also U3.3 (FB)
- net RESET: now reaches U5.7 (PG10)
- net RESET: now also C21.1, SW1.1
- net ADC1_IN15: no longer names the net of U5.17 (PB0)
- new net: R53.1, U3.4 (EN)
- new net VDDA: C17.1, C8.1, FB4.2, U5.20 (VREF+), U5.21 (VDDA)
- no-connect marks 4 -> 3
Other:
- moved on the sheet: C6, C7, D1, J1, R3
