File: hardware/motor/bldcDriver.kicad_sch (KiCad schematic)
At the start: 94 parts, among them J1 Conn_01x02, J2 Conn_01x06, J3 Conn_01x06, J4 Conn_01x03, J5 Conn_01x06, SW1 SW_Push, U3 TPS5430DDA, U4 MPU-6050, U5 STM32G431CBUx, U6 TLV9062xD, U7 TLV9062xD, U8 TLV9062xD, Y1 25MHz

Commit message: update pcn
Parts:
- removed J3, J5: Conn_01x06, balancerDriver:CONN-SMD_6P-P1.00_MEGASTAR_ZX-SH1.0-6PWT, symbol Connector_Generic:Conn_01x06
- removed R49: 10k, Resistor_SMD:R_0603_1608Metric_Pad0.98x0.95mm_HandSolder, symbol Device:R_Small
- removed R72, R73: 4.7k, Resistor_SMD:R_0603_1608Metric_Pad0.98x0.95mm_HandSolder, symbol Device:R_Small
- removed U4: MPU-6050, Sensor_Motion:InvenSense_QFN-24_4x4mm_P0.5mm, symbol Sensor_Motion:MPU-6050
- added C52: 100n, Capacitor_SMD:C_0603_1608Metric_Pad1.08x0.95mm_HandSolder, symbol Device:C_Small
- added SW2: SW_Push, balancerDriver:SW-SMD_L4.0-W2.9-LS5.0, symbol Switch:SW_Push
- added TP20, TP21, TP22, TP23, TP24, TP25: TestPoint, TestPoint:TestPoint_Pad_D1.0mm, symbol Connector:TestPoint
- added U10, U4: HC-FPC-0.5-6P-CSH20, balancerDriver:FPC-SMD_6P-P0.50_HC-FPC-0.5-6P-CSH20, symbol balancerDriver:HC-FPC-0.5-6P-CSH20
- added U9: MPU6500, balancerDriver:QFN-24_L3.0-W3.0-P0.40-BL-EP, symbol bldcDriver:MPU6500
- C23: value 100n -> 2.2u
- C24: value 2.2n -> 100n
- SW1: footprint Button_Switch_SMD:SW_SPST_B3U-1000P -> balancerDriver:SW-SMD_L4.0-W2.9-LS5.0
Connections:
- net +3V3: now also FB1.2, TP20.1, U10.5, U4.5; no longer FB1.1
- net GNDD: now also C5.1, C50.1, C6.1, C7.1, D1.2 (A), D8.1 (K), R2.2, U3.6 (GND), U3.9 (GNDPAD), C52.2, SW2.2, TP22.1, U10.6, U4.6, U9.11 (FSYNC), U9.18 (GND), U9.20 (RESV)
- net GNDPWR: now also TP21.1; no longer C5.1, C50.1, C6.1, C7.1, D1.2 (A), D8.1 (K), R2.2, U3.6 (GND), U3.9 (GNDPAD)
- net NSS1: now also U10.1
- net NSS2: now also U4.1
- net SPI1_MISO: now also TP24.1, U9.9 (SDO/AD0)
- net SPI1_MOSI: now also TP25.1, U9.24 (SDA/SDI)
- net SPI1_SCK: now also TP23.1, U9.23 (SCL/SCLK)
- net SPI3_MISO: now also U10.3, U4.3
- net SPI3_MOSI: now also U10.2, U4.2
- net SPI3_SCK: now also U10.4, U4.4
- net at C23.1: now also C13.1, C24.1, FB1.1, U9.13 (VDD), U9.8 (VDDIO)
- net MPU_INT: no longer names the net of U5.12 (PA4)
- new net: C22.1, U9.10 (REGOUT)
- new net KEY: C52.1, SW2.1
- new net SPI1_CS: U9.22 (nCS)
- no-connect marks 9 -> 27
Other:
- moved on the sheet: FB2

Commit message: update pcb
Connections:
- net SPI1_CS: now also U5.9 (PA1)
- net at U5.12 (PA4): now also TP10.1
- net I2C1_SDA: no longer names the net of U5.45 (PB7)
- no-connect marks 27 -> 28
Changed lines of the file:
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@@
 	)
 	(no_connect
+		(at 341.63 102.87)
+	)
+	(no_connect
 		(at 243.84 50.8)
 	)
@@
 		)
 	)
-	(label "I2C1_SDA"
-		(at 341.63 102.87 180)
-		(fields_autoplaced yes)
-		(effects
-			(font
-				(size 1.27 1.27)
-			)
-			(justify right bottom)
-		)
-	)
 	(label "VREF_OP1"
 		(at 149.86 116.84 0)
@@
 		)
 	)
+	(label "SPI1_CS"
+		(at 374.65 49.53 0)
+		(fields_autoplaced yes)
+		(effects
+			(font
+				(size 1.27 1.27)
+			)
+			(justify left bottom)
+		)
+	)
 	(label "VREF_OP1"
 		(at 52.07 184.15 180)
@@
 	)
 	(symbol
+		(lib_id "Connector:TestPoint")
+		(at 374.65 57.15 270)
+		(unit 1)
+		(exclude_from_sim no)
+		(in_bom yes)
+		(on_board yes)
+		(dnp no)
+		(property "Reference" "TP10"
+			(at 376.682 55.118 90)
+			(effects
+				(font
+					(size 1.27 1.27)
+				)
+				(justify left)
+			)
+		)
+		(property "Value" "TestPoint"
+			(at 376.6821 59.69 0)
+			(effects
+				(font
+					(size 1.27 1.27)
+				)
+				(justify left)
+				(hide yes)
+			)
+		)
+		(property "Footprint" "TestPoint:TestPoint_Pad_D1.0mm"
+			(at 374.65 62.23 0)
+			(effects
+				(font
+					(size 1.27 1.27)
+				)
+				(hide yes)
+			)
+		)
+		(property "Datasheet" "~"
+			(at 374.65 62.23 0)
+			(effects
+				(font
+					(size 1.27 1.27)
+				)
+				(hide yes)
+			)
+		)
+		(property "Description" "test point"
+			(at 374.65 57.15 0)
+			(effects
+				(font
+					(size 1.27 1.27)
+				)
+				(hide yes)
+			)
+		)
+		(pin "1"
+		)
+		(instances
+			(project "bldcDriver"
+				(path "/024b6358-58d2-4f27-baff-bf9e44899c87"
+					(reference "TP10")
+					(unit 1)
+				)
+			)
+		)
+	)
+	(symbol
 		(lib_id "power:+3V3")
 		(at 198.12 44.45 0)
@@
 					(unit 1)
 				)
-			)
-		)
-	)
-	(symbol
-		(lib_id "Connector:TestPoint")
-		(at 374.65 49.53 270)
-		(unit 1)
-		(exclude_from_sim no)
-		(in_bom yes)
-		(on_board yes)
-		(dnp no)
-		(property "Reference" "TP10"
-			(at 376.682 47.498 90)
-			(effects
-				(font
-					(size 1.27 1.27)
-				)
-				(justify left)
-			)
-		)
-		(property "Value" "TestPoint"
-			(at 376.6821 52.07 0)
-			(effects
-				(font
-					(size 1.27 1.27)
-				)
-				(justify left)
-				(hide yes)
-			)
-		)
-		(property "Footprint" "TestPoint:TestPoint_Pad_D1.0mm"
-			(at 374.65 54.61 0)
-			(effects
-				(font
-					(size 1.27 1.27)
-				)
-				(hide yes)
-			)
-		)
-		(property "Datasheet" "~"
-			(at 374.65 54.61 0)
-			(effects
-				(font
-					(size 1.27 1.27)
-				)
-				(hide yes)
-			)
-		)
-		(property "Description" "test point"
-			(at 374.65 49.53 0)
-			(effects
-				(font
-					(size 1.27 1.27)
-				)
-				(hide yes)
-			)
-		)
-		(pin "1"
-		)
-		(instances
-			(project "bldcDriver"
-				(path "/024b6358-58d2-4f27-baff-bf9e44899c87"
-					(reference "TP10")
-					(unit 1)
-				)

Commit message: update motor pcb
Parts:
- removed C38, C43, C44: 4.7u, Capacitor_SMD:C_0603_1608Metric_Pad1.08x0.95mm_HandSolder, symbol Device:C_Small
- removed C39, C40, C47, C48: 100n, Capacitor_SMD:C_0603_1608Metric_Pad1.08x0.95mm_HandSolder, symbol Device:C_Small
- removed R40, R41: 1k, Resistor_SMD:R_0603_1608Metric_Pad0.98x0.95mm_HandSolder, symbol Device:R_Small
- removed TP9: TestPoint, TestPoint:TestPoint_Pad_D1.0mm, symbol Connector:TestPoint
- removed U8: TLV9062xD, Package_SO:SOIC-8_3.9x4.9mm_P1.27mm, symbol Amplifier_Operational:TLV9062xD
- U9: footprint balancerDriver:QFN-24_L3.0-W3.0-P0.40-BL-EP -> balancerDriver:QFN24_3X3X0P9_IVS-L
Connections:
- net VREF_OP2 is gone; now on net VREF_OP: R31.2, R45.2
- net KEY: now also U5.3 (PC14)
- net SPI1_CS: now also U5.12 (PA4); no longer U5.9 (PA1)
- net VREF_OP1: no longer R33.2, R47.2
- net at TP10.1: now also U5.9 (PA1); no longer U5.12 (PA4)
- net INA1+ renamed VREF_OP
- net VREF_OP: now also R33.2, R47.2
Other:
- moved on the sheet: C10, C11, C27, C41, C42, C45, C46, C9, FB3, R20, R21, R30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

Commit message: update rfBat pcb
Connections:
- net +3V3: now also J2.6 (Pin_6); no longer J2.1 (Pin_1)
- net GNDD: now also J2.5 (Pin_5); no longer J2.2 (Pin_2)
- net SWCLK: now also J2.1 (Pin_1); no longer J2.6 (Pin_6)
- net SWDIO: now also J2.2 (Pin_2); no longer J2.5 (Pin_5)
- net USART3_RX: now also J2.3 (Pin_3); no longer J2.4 (Pin_4)
- net USART3_TX: now also J2.4 (Pin_4); no longer J2.3 (Pin_3)
Other:
- moved on the sheet: J2
Changed lines of the file:
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@@
 	(wire
 		(pts
-			(xy 372.11 219.71) (xy 375.92 219.71)
-		)
-		(stroke
-			(width 0)
-			(type default)
-		)
-	)
-	(wire
-		(pts
 			(xy 60.96 147.32) (xy 60.96 151.13)
 		)
@@
 	(wire
 		(pts
-			(xy 367.03 222.25) (xy 375.92 222.25)
-		)
-		(stroke
-			(width 0)
-			(type default)
-		)
-	)
-	(wire
-		(pts
 			(xy 102.87 33.02) (xy 107.95 33.02)
 		)
@@
 	(wire
 		(pts
+			(xy 367.03 219.71) (xy 375.92 219.71)
+		)
+		(stroke
+			(width 0)
+			(type default)
+		)
+	)
+	(wire
+		(pts
 			(xy 133.35 179.07) (xy 130.81 179.07)
 		)
@@
 	(wire
 		(pts
+			(xy 372.11 217.17) (xy 375.92 217.17)
+		)
+		(stroke
+			(width 0)
+			(type default)
+		)
+	)
+	(wire
+		(pts
 			(xy 300.99 83.82) (xy 308.61 83.82)
 		)
@@
 		)
 	)
-	(label "SWCLK"
-		(at 375.92 232.41 180)
-		(fields_autoplaced yes)
-		(effects
-			(font
-				(size 1.27 1.27)
-			)
-			(justify right bottom)
-		)
-	)
 	(label "TIM8_CH2"
 		(at 232.41 186.69 180)
@@
 		)
 	)
-	(label "USART3_TX"
-		(at 375.92 224.79 180)
-		(fields_autoplaced yes)
-		(effects
-			(font
-				(size 1.27 1.27)
-			)
-			(justify right bottom)
-		)
-	)
 	(label "NSS1"
 		(at 341.63 92.71 180)
@@
 		)
 	)
-	(label "SWDIO"
-		(at 375.92 229.87 180)
-		(fields_autoplaced yes)
-		(effects
-			(font
-				(size 1.27 1.27)
-			)
-			(justify right bottom)
-		)
-	)
 	(label "TIM1_CH2"
 		(at 267.97 185.42 0)
@@
 		)
 	)
+	(label "SWCLK"
+		(at 375.92 229.87 180)
+		(fields_autoplaced yes)
+		(effects
+			(font
+				(size 1.27 1.27)
+			)
+			(justify right bottom)
+		)
+	)
 	(label "YI"
 		(at 293.37 74.93 0)
@@
 		)
 	)
+	(label "USART3_RX"
+		(at 375.92 224.79 180)
+		(fields_autoplaced yes)
+		(effects
+			(font
+				(size 1.27 1.27)
+			)
+			(justify right bottom)
+		)
+	)
 	(label "TIM1_CH3"
 		(at 267.97 190.5 0)
@@
 		)
 	)
+	(label "SWDIO"
+		(at 375.92 227.33 180)
+		(fields_autoplaced yes)
+		(effects
+			(font
+				(size 1.27 1.27)
+			)
+			(justify right bottom)
+		)
+	)
 	(label "SPI3_SCK"
 		(at 377.19 187.96 180)
@@
 		)
 	)
-	(label "1CS2+"
-		(at 99.06 181.61 180)
+	(label "USART3_TX"
+		(at 375.92 222.25 180)
 		(fields_autoplaced yes)
 		(effects
@@
 		)
 	)
-	(label "1CS1+"
-		(at 43.18 180.34 180)
+	(label "1CS2+"
+		(at 99.06 181.61 180)
 		(fields_autoplaced yes)
 		(effects
@@
 		)
 	)
-	(label "USART3_RX"
-		(at 375.92 227.33 180)
+	(label "1CS1+"
+		(at 43.18 180.34 180)
 		(fields_autoplaced yes)
 		(effects
@@
 	)
 	(symbol
+		(lib_id "power:GNDD")
+		(at 367.03 219.71 270)
+		(unit 1)
+		(exclude_from_sim no)
+		(in_bom yes)
+		(on_board yes)
+		(dnp no)
+		(fields_autoplaced yes)
+		(property "Reference" "#PWR012"
+			(at 360.68 219.71 0)
+			(effects
+				(font
+					(size 1.27 1.27)
+				)
+				(hide yes)
+			)
+		)
+		(property "Value" "GNDD"
+			(at 363.22 219.7099 90)
+			(effects
+				(font
+					(size 1.27 1.27)
+				)
+				(justify right)
+				(hide yes)
+			)
+		)
+		(property "Footprint" ""
+			(at 367.03 219.71 0)
+			(effects
+				(font
+					(size 1.27 1.27)
+				)
+				(hide yes)
+			)
+		)
+		(property "Datasheet" ""
+			(at 367.03 219.71 0)
+			(effects
+				(font
+					(size 1.27 1.27)
+				)
+				(hide yes)
+			)
+		)
+		(property "Description" "Power symbol creates a global label with name \"GNDD\" , digital ground"
+			(at 367.03 219.71 0)
+			(effects
+				(font
+					(size 1.27 1.27)
+				)
+				(hide yes)
+			)
+		)
+		(pin "1"
+		)
+		(instances
+			(project "bldcDriver"
+				(path "/024b6358-58d2-4f27-baff-bf9e44899c87"
+					(reference "#PWR012")
+					(unit 1)
+				)
+			)
+		)
+	)
+	(symbol
 		(lib_id "Device:R_Small")
 		(at 50.8 250.19 0)
@@
 	)
 	(symbol
-		(lib_id "power:GNDD")
-		(at 367.03 222.25 270)
-		(unit 1)
-		(exclude_from_sim no)
-		(in_bom yes)
-		(on_board yes)
-		(dnp no)
-		(fields_autoplaced yes)
-		(property "Reference" "#PWR012"
-			(at 360.68 222.25 0)
-			(effects
-				(font
-					(size 1.27 1.27)
-				)
-				(hide yes)
-			)
-		)
-		(property "Value" "GNDD"
-			(at 363.22 222.2499 90)
-			(effects
-				(font
-					(size 1.27 1.27)
-				)
-				(justify right)
-				(hide yes)
-			)
-		)
-		(property "Footprint" ""
-			(at 367.03 222.25 0)
-			(effects
-				(font
-					(size 1.27 1.27)
-				)
-				(hide yes)
-			)
-		)
-		(property "Datasheet" ""
-			(at 367.03 222.25 0)
-			(effects
-				(font
-					(size 1.27 1.27)
-				)
-				(hide yes)
-			)
-		)
-		(property "Description" "Power symbol creates a global label with name \"GNDD\" , digital ground"
-			(at 367.03 222.25 0)
-			(effects
-				(font
-					(size 1.27 1.27)
-				)
-				(hide yes)
-			)
-		)
-		(pin "1"
-		)
-		(instances
-			(project "bldcDriver"
-				(path "/024b6358-58d2-4f27-baff-bf9e44899c87"
-					(reference "#PWR012")
-					(unit 1)
-				)
-			)
-		)
-	)
-	(symbol
 		(lib_id "Device:Crystal_GND24")
 		(at 300.99 74.93 0)
@@
 	(symbol
 		(lib_id "power:+3V3")
+		(at 372.11 217.17 90)
+		(unit 1)
+		(exclude_from_sim no)
+		(in_bom yes)
+		(on_board yes)
+		(dnp no)
+		(property "Reference" "#PWR034"
+			(at 375.92 217.17 0)
+			(effects
+				(font
+					(size 1.27 1.27)
+				)
+				(hide yes)
+			)
+		)
+		(property "Value" "+3V3"
+			(at 367.03 217.17 90)
+			(effects
+				(font
+					(size 1.27 1.27)
+				)
+			)
+		)
+		(property "Footprint" ""
+			(at 372.11 217.17 0)
+			(effects
+				(font
+					(size 1.27 1.27)
+				)
+				(hide yes)
+			)
+		)
+		(property "Datasheet" ""
+			(at 372.11 217.17 0)
+			(effects
+				(font
+					(size 1.27 1.27)
+				)
+				(hide yes)
+			)
+		)
+		(property "Description" "Power symbol creates a global label with name \"+3V3\""
+			(at 372.11 217.17 0)
+			(effects
+				(font
+					(size 1.27 1.27)
+				)
+				(hide yes)
+			)
+		)
+		(pin "1"
+		)
+		(instances
+			(project "bldcDriver"
+				(path "/024b6358-58d2-4f27-baff-bf9e44899c87"
+					(reference "#PWR034")
+					(unit 1)
+				)
+			)
+		)
+	)
+	(symbol
+		(lib_id "power:+3V3")
 		(at 374.65 190.5 90)
 		(unit 1)
@@
 		(lib_id "Connector_Generic:Conn_01x06")
 		(at 381 224.79 0)
+		(mirror x)
 		(unit 1)
 		(exclude_from_sim no)
@@
 		(on_board yes)
 		(dnp no)
-		(fields_autoplaced yes)
 		(property "Reference" "J2"
-			(at 383.54 225.425 0)
+			(at 383.54 224.155 0)
 			(effects
 				(font
@@
 		)
 		(property "Value" "Conn_01x06"
-			(at 383.54 227.965 0)
+			(at 383.54 221.615 0)
 			(effects
 				(font
@@
 					(unit 1)
 				)
-			)
-		)
-	)
-	(symbol
-		(lib_id "power:+3V3")
-		(at 372.11 219.71 90)
-		(unit 1)
-		(exclude_from_sim no)
-		(in_bom yes)
-		(on_board yes)
-		(dnp no)
-		(property "Reference" "#PWR036"
-			(at 375.92 219.71 0)
-			(effects
-				(font
-					(size 1.27 1.27)
-				)
-				(hide yes)
-			)
-		)
-		(property "Value" "+3V3"
-			(at 367.03 219.71 90)
-			(effects
-				(font
-					(size 1.27 1.27)
-				)
-			)
-		)
-		(property "Footprint" ""
-			(at 372.11 219.71 0)
-			(effects
-				(font
-					(size 1.27 1.27)
-				)
-				(hide yes)
-			)
-		)
-		(property "Datasheet" ""
-			(at 372.11 219.71 0)
-			(effects
-				(font
-					(size 1.27 1.27)
-				)
-				(hide yes)
-			)
-		)
-		(property "Description" "Power symbol creates a global label with name \"+3V3\""
-			(at 372.11 219.71 0)
-			(effects
-				(font
-					(size 1.27 1.27)
-				)
-				(hide yes)
-			)
-		)
-		(pin "1"
-		)
-		(instances
-			(project "bldcDriver"
-				(path "/024b6358-58d2-4f27-baff-bf9e44899c87"
-					(reference "#PWR036")
-					(unit 1)
-				)

Commit message: update motor pcb
Parts:
- removed J4: Conn_01x03, balancerDriver:CONN-SMD_3P-P1.00_WAFER-SH1.0-3PWB, symbol Connector_Generic:Conn_01x03
- added C38: 100n, Capacitor_SMD:C_0603_1608Metric_Pad1.08x0.95mm_HandSolder, symbol Device:C_Small
- added P1: FPC_0.5MM_4P_Vertical_mounting_type_H2.0mm, balancerDriver:FPC-SMD_4P-L7.5-W2.0-P0.50, symbol balancerDriver:FPC_0.5MM_4P_Vertical_mounting_type_H2.0mm
- added R40: 3k, Resistor_SMD:R_0603_1608Metric_Pad0.98x0.95mm_HandSolder, symbol Device:R
- added RV1: R_Potentiometer, balancerDriver:RES-ADJ-TH_3362P, symbol Device:R_Potentiometer
Connections:
- net +3V3: now also P1.4, RV1.1
- net GNDD: now also C38.2, P1.1, R40.2, RV1.3
- net TIM8_CH2: now also R40.1
- net USART2_RX: now also P1.2
- net USART2_TX: now also P1.3
- net I2C1_SCL: no longer names the net of U5.38 (PA15)
- new net: C38.1, RV1.2
- no-connect marks 28 -> 30

Commit message: update motor pcb
Parts:
- removed TP10: TestPoint, TestPoint:TestPoint_Pad_D1.0mm, symbol Connector:TestPoint
Connections:
- net ADC1_IN2: now reaches C38.1, RV1.2
- net ADC1_IN2: now also U5.9 (PA1)
Changed lines of the file:
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@@
 		)
 	)
+	(label "ADC1_IN2"
+		(at 218.44 134.62 180)
+		(fields_autoplaced yes)
+		(effects
+			(font
+				(size 1.27 1.27)
+			)
+			(justify right bottom)
+		)
+	)
 	(label "SPI1_SCK"
 		(at 243.84 45.72 0)
@@
 		)
 	)
+	(label "ADC1_IN2"
+		(at 374.65 49.53 0)
+		(fields_autoplaced yes)
+		(effects
+			(font
+				(size 1.27 1.27)
+			)
+			(justify left bottom)
+		)
+	)
 	(label "TIM1_CH2"
 		(at 374.65 69.85 0)
@@
 					(unit 1)
 				)
-			)
-		)
-	)
-	(symbol
-		(lib_id "Connector:TestPoint")
-		(at 374.65 49.53 270)
-		(unit 1)
-		(exclude_from_sim no)
-		(in_bom yes)
-		(on_board yes)
-		(dnp no)
-		(property "Reference" "TP10"
-			(at 376.682 47.498 90)
-			(effects
-				(font
-					(size 1.27 1.27)
-				)
-				(justify left)
-			)
-		)
-		(property "Value" "TestPoint"
-			(at 376.6821 52.07 0)
-			(effects
-				(font
-					(size 1.27 1.27)
-				)
-				(justify left)
-				(hide yes)
-			)
-		)
-		(property "Footprint" "TestPoint:TestPoint_Pad_D1.0mm"
-			(at 374.65 54.61 0)
-			(effects
-				(font
-					(size 1.27 1.27)
-				)
-				(hide yes)
-			)
-		)
-		(property "Datasheet" "~"
-			(at 374.65 54.61 0)
-			(effects
-				(font
-					(size 1.27 1.27)
-				)
-				(hide yes)
-			)
-		)
-		(property "Description" "test point"
-			(at 374.65 49.53 0)
-			(effects
-				(font
-					(size 1.27 1.27)
-				)
-				(hide yes)
-			)
-		)
-		(pin "1"
-		)
-		(instances
-			(project "bldcDriver"
-				(path "/024b6358-58d2-4f27-baff-bf9e44899c87"
-					(reference "TP10")
-					(unit 1)
-				)
