File: hardware/motor/bldcDriver.kicad_sch (KiCad schematic)
At the start: 90 parts, among them J1 Conn_01x02, J2 Conn_01x06, P1 FPC_0.5MM_4P_Vertical_mountin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, SW1 SW_Push, SW2 SW_Push, U10 HC-FPC-0.5-6P-CSH20, U3 TPS5430DDA, U4 HC-FPC-0.5-6P-CSH20, U5 STM32G431CBUx, U6 TLV9062xD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

Commit message: update ibom
Parts:
- added TP10: TestPoint, TestPoint:TestPoint_Pad_D1.0mm, symbol Connector:TestPoint
Connections:
- net +3V3: now also P1.1; no longer P1.4
- net GNDD: now also P1.3; no longer P1.2
- net USART2_RX: now also P1.4; no longer P1.1
- net USART2_TX: now also P1.2; no longer P1.3
- net at U5.38 (PA15): now also TP10.1
Changed lines of the file:
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@@
 	(wire
 		(pts
-			(xy 328.93 226.06) (xy 339.09 226.06)
-		)
-		(stroke
-			(width 0)
-			(type default)
-		)
-	)
-	(wire
-		(pts
 			(xy 146.05 33.02) (xy 140.97 33.02)
 		)
@@
 	(wire
 		(pts
+			(xy 328.93 223.52) (xy 341.63 223.52)
+		)
+		(stroke
+			(width 0)
+			(type default)
+		)
+	)
+	(wire
+		(pts
 			(xy 304.8 80.01) (xy 304.8 82.55)
 		)
@@
 	(wire
 		(pts
+			(xy 340.36 228.6) (xy 328.93 228.6)
+		)
+		(stroke
+			(width 0)
+			(type default)
+		)
+	)
+	(wire
+		(pts
 			(xy 195.58 62.23) (xy 208.28 62.23)
 		)
@@
 	(wire
 		(pts
-			(xy 328.93 220.98) (xy 339.09 220.98)
-		)
-		(stroke
-			(width 0)
-			(type default)
-		)
-	)
-	(wire
-		(pts
 			(xy 95.25 43.18) (xy 91.44 43.18)
 		)
@@
 		)
 	)
-	(label "USART2_RX"
-		(at 328.93 228.6 0)
-		(fields_autoplaced yes)
-		(effects
-			(font
-				(size 1.27 1.27)
-			)
-			(justify left bottom)
-		)
-	)
 	(label "KEY"
 		(at 237.49 167.64 0)
@@
 		)
 	)
+	(label "USART2_RX"
+		(at 328.93 220.98 0)
+		(fields_autoplaced yes)
+		(effects
+			(font
+				(size 1.27 1.27)
+			)
+			(justify left bottom)
+		)
+	)
 	(label "ADC2_IN12"
 		(at 50.8 255.27 0)
@@
 		)
 	)
+	(label "USART2_TX"
+		(at 328.93 226.06 0)
+		(fields_autoplaced yes)
+		(effects
+			(font
+				(size 1.27 1.27)
+			)
+			(justify left bottom)
+		)
+	)
 	(label "LED"
 		(at 257.81 152.4 0)
@@
 		)
 	)
-	(label "USART2_TX"
-		(at 328.93 223.52 0)
-		(fields_autoplaced yes)
-		(effects
-			(font
-				(size 1.27 1.27)
-			)
-			(justify left bottom)
-		)
-	)
 	(label "TIM8_CH1"
 		(at 207.01 219.71 180)
@@
 	)
 	(symbol
+		(lib_id "power:+3V3")
+		(at 340.36 228.6 270)
+		(mirror x)
+		(unit 1)
+		(exclude_from_sim no)
+		(in_bom yes)
+		(on_board yes)
+		(dnp no)
+		(property "Reference" "#PWR016"
+			(at 336.55 228.6 0)
+			(effects
+				(font
+					(size 1.27 1.27)
+				)
+				(hide yes)
+			)
+		)
+		(property "Value" "+3V3"
+			(at 345.44 228.6 90)
+			(effects
+				(font
+					(size 1.27 1.27)
+				)
+			)
+		)
+		(property "Footprint" ""
+			(at 340.36 228.6 0)
+			(effects
+				(font
+					(size 1.27 1.27)
+				)
+				(hide yes)
+			)
+		)
+		(property "Datasheet" ""
+			(at 340.36 228.6 0)
+			(effects
+				(font
+					(size 1.27 1.27)
+				)
+				(hide yes)
+			)
+		)
+		(property "Description" "Power symbol creates a global label with name \"+3V3\""
+			(at 340.36 228.6 0)
+			(effects
+				(font
+					(size 1.27 1.27)
+				)
+				(hide yes)
+			)
+		)
+		(pin "1"
+		)
+		(instances
+			(project "bldcDriver"
+				(path "/024b6358-58d2-4f27-baff-bf9e44899c87"
+					(reference "#PWR016")
+					(unit 1)
+				)
+			)
+		)
+	)
+	(symbol
 		(lib_id "power:VDDA")
 		(at 294.64 31.75 0)
@@
 	)
 	(symbol
-		(lib_id "power:GNDD")
-		(at 339.09 226.06 90)
-		(unit 1)
-		(exclude_from_sim no)
-		(in_bom yes)
-		(on_board yes)
-		(dnp no)
-		(fields_autoplaced yes)
-		(property "Reference" "#PWR016"
-			(at 345.44 226.06 0)
-			(effects
-				(font
-					(size 1.27 1.27)
-				)
-				(hide yes)
-			)
-		)
-		(property "Value" "GNDD"
-			(at 342.9 226.06 0)
-			(effects
-				(font
-					(size 1.27 1.27)
-				)
-				(hide yes)
-			)
-		)
-		(property "Footprint" ""
-			(at 339.09 226.06 0)
-			(effects
-				(font
-					(size 1.27 1.27)
-				)
-				(hide yes)
-			)
-		)
-		(property "Datasheet" ""
-			(at 339.09 226.06 0)
-			(effects
-				(font
-					(size 1.27 1.27)
-				)
-				(hide yes)
-			)
-		)
-		(property "Description" "Power symbol creates a global label with name \"GNDD\" , digital ground"
-			(at 339.09 226.06 0)
-			(effects
-				(font
-					(size 1.27 1.27)
-				)
-				(hide yes)
-			)
-		)
-		(pin "1"
-		)
-		(instances
-			(project "bldcDriver"
-				(path "/024b6358-58d2-4f27-baff-bf9e44899c87"
-					(reference "#PWR016")
-					(unit 1)
-				)
-			)
-		)
-	)
-	(symbol
 		(lib_id "Device:R_Small")
 		(at 48.26 175.26 270)
@@
 	(symbol
 		(lib_id "power:GNDD")
+		(at 341.63 223.52 90)
+		(unit 1)
+		(exclude_from_sim no)
+		(in_bom yes)
+		(on_board yes)
+		(dnp no)
+		(fields_autoplaced yes)
+		(property "Reference" "#PWR068"
+			(at 347.98 223.52 0)
+			(effects
+				(font
+					(size 1.27 1.27)
+				)
+				(hide yes)
+			)
+		)
+		(property "Value" "GNDD"
+			(at 345.44 223.5199 90)
+			(effects
+				(font
+					(size 1.27 1.27)
+				)
+				(justify right)
+			)
+		)
+		(property "Footprint" ""
+			(at 341.63 223.52 0)
+			(effects
+				(font
+					(size 1.27 1.27)
+				)
+				(hide yes)
+			)
+		)
+		(property "Datasheet" ""
+			(at 341.63 223.52 0)
+			(effects
+				(font
+					(size 1.27 1.27)
+				)
+				(hide yes)
+			)
+		)
+		(property "Description" "Power symbol creates a global label with name \"GNDD\" , digital ground"
+			(at 341.63 223.52 0)
+			(effects
+				(font
+					(size 1.27 1.27)
+				)
+				(hide yes)
+			)
+		)
+		(pin "1"
+		)
+		(instances
+			(project "bldcDriver"
+				(path "/024b6358-58d2-4f27-baff-bf9e44899c87"
+					(reference "#PWR068")
+					(unit 1)
+				)
+			)
+		)
+	)
+	(symbol
+		(lib_id "power:GNDD")
 		(at 107.95 208.28 0)
 		(unit 1)
@@
 	)
 	(symbol
+		(lib_id "Connector:TestPoint")
+		(at 374.65 85.09 270)
+		(unit 1)
+		(exclude_from_sim no)
+		(in_bom yes)
+		(on_board yes)
+		(dnp no)
+		(property "Reference" "TP10"
+			(at 379.476 85.344 90)
+			(effects
+				(font
+					(size 1.27 1.27)
+				)
+				(justify left)
+			)
+		)
+		(property "Value" "TestPoint"
+			(at 376.6821 87.63 0)
+			(effects
+				(font
+					(size 1.27 1.27)
+				)
+				(justify left)
+				(hide yes)
+			)
+		)
+		(property "Footprint" "TestPoint:TestPoint_Pad_D1.0mm"
+			(at 374.65 90.17 0)
+			(effects
+				(font
+					(size 1.27 1.27)
+				)
+				(hide yes)
+			)
+		)
+		(property "Datasheet" "~"
+			(at 374.65 90.17 0)
+			(effects
+				(font
+					(size 1.27 1.27)
+				)
+				(hide yes)
+			)
+		)
+		(property "Description" "test point"
+			(at 374.65 85.09 0)
+			(effects
+				(font
+					(size 1.27 1.27)
+				)
+				(hide yes)
+			)
+		)
+		(pin "1"
+		)
+		(instances
+			(project "bldcDriver"
+				(path "/024b6358-58d2-4f27-baff-bf9e44899c87"
+					(reference "TP10")
+					(unit 1)
+				)
+			)
+		)
+	)
+	(symbol
 		(lib_id "Device:R_Small")
 		(at 50.8 240.03 0)
@@
 		(on_board yes)
 		(dnp no)
-		(fields_autoplaced yes)
 		(property "Reference" "P1"
 			(at 318.77 222.2499 0)
@@
 					(unit 1)
 				)
-			)
-		)
-	)
-	(symbol
-		(lib_id "power:+3V3")
-		(at 339.09 220.98 270)
-		(unit 1)
-		(exclude_from_sim no)
-		(in_bom yes)
-		(on_board yes)
-		(dnp no)
-		(property "Reference" "#PWR068"
-			(at 335.28 220.98 0)
-			(effects
-				(font
-					(size 1.27 1.27)
-				)
-				(hide yes)
-			)
-		)
-		(property "Value" "+3V3"
-			(at 344.17 220.98 90)
-			(effects
-				(font
-					(size 1.27 1.27)
-				)
-			)
-		)
-		(property "Footprint" ""
-			(at 339.09 220.98 0)
-			(effects
-				(font
-					(size 1.27 1.27)
-				)
-				(hide yes)
-			)
-		)
-		(property "Datasheet" ""
-			(at 339.09 220.98 0)
-			(effects
-				(font
-					(size 1.27 1.27)
-				)
-				(hide yes)
-			)
-		)
-		(property "Description" "Power symbol creates a global label with name \"+3V3\""
-			(at 339.09 220.98 0)
-			(effects
-				(font
-					(size 1.27 1.27)
-				)
-				(hide yes)
-			)
-		)
-		(pin "1"
-		)
-		(instances
-			(project "bldcDriver"
-				(path "/024b6358-58d2-4f27-baff-bf9e44899c87"
-					(reference "#PWR068")
-					(unit 1)
-				)

Commit message: update motor
Parts:
- added TP29, TP30, TP31, TP32, TP33, TP34, TP35, TP36, TP37, TP38, TP39: TestPoint, TestPoint:TestPoint_Pad_D1.0mm, symbol Connector:TestPoint
Connections:
- net ADC1_IN2: now also TP37.1
- net GNDD: no longer C5.1, C50.1, C6.1, C7.1, D1.2 (A), D8.1 (K), R2.2, U3.6 (GND), U3.9 (GNDPAD)
- net GNDPWR: now also C5.1, C50.1, C6.1, C7.1, D1.2 (A), D8.1 (K), R2.2, U3.6 (GND), U3.9 (GNDPAD)
- net KEY: now also TP38.1
- net NSS1: now also TP32.1
- net NSS2: now also TP33.1
- net RESET: now also TP39.1
- net SPI3_MISO: now also TP30.1
- net SPI3_MOSI: now also TP29.1
- net SPI3_SCK: now also TP31.1
- net USART2_RX: now also TP34.1
- net USART2_TX: now also TP35.1
- net VREF_OP: now also TP36.1
Other:
- moved on the sheet: FB2, TP21, TP22

Commit message: update motor pcb
Parts:
- removed R40: 3k, Resistor_SMD:R_0603_1608Metric_Pad0.98x0.95mm_HandSolder, symbol Device:R
- removed TP36: TestPoint, TestPoint:TestPoint_Pad_D1.0mm, symbol Connector:TestPoint
- added C39, C43, C44: 4.7u, Capacitor_SMD:C_0603_1608Metric_Pad1.08x0.95mm_HandSolder, symbol Device:C_Small
- added C40, C47, C48, C53: 100n, Capacitor_SMD:C_0603_1608Metric_Pad1.08x0.95mm_HandSolder, symbol Device:C_Small
- added R41, R49: 1k, Resistor_SMD:R_0603_1608Metric_Pad0.98x0.95mm_HandSolder, symbol Device:R_Small
- added TP40: TestPoint, TestPoint:TestPoint_Pad_D1.0mm, symbol Connector:TestPoint
- added U8: TLV9062xD, Package_SO:SOIC-8_3.9x4.9mm_P1.27mm, symbol Amplifier_Operational:TLV9062xD
Connections:
- net ADC1_IN5: no longer C27.2, R37.2, TP17.1
- net GNDD: now also C39.1, C40.1, C43.1, C44.1, C47.1, C48.1, C53.1, R49.1, U8.4 (V-)
- net LED: no longer U5.17 (PB0)
- net OP_VCC: now also C39.2, C40.2, C47.2, R41.2, U8.8 (V+)
- net VREF_OP1: now also R33.2, R47.2, C43.2, C48.2, U8.1, U8.2 (-)
- net ADC1_IN12_COMP1_INP: now reaches U5.18 (PB1)
- net ADC1_IN12_COMP1_INP: now also C27.2, R37.2, TP17.1
- net ADC2_IN12 renamed ADC1_IN15_COMP4_INP
- net ADC1_IN15_COMP4_INP: now also U5.17 (PB0); no longer U5.19 (PB2)
- removed net VREF_OP: R31.2, R33.2, R38.1, R39.2, R45.2, R47.2
- new net INA1+: R38.1, R39.2, U8.3 (+)
- new net INA2+: R41.1, R49.2, TP40.1, U8.5 (+)
- new net VREF_OP2: C44.2, C53.2, R31.2, R45.2, U8.6 (-), U8.7
- no-connect marks 30 -> 29
Other:
- moved on the sheet: C10, C67, C68, C9, FB2, FB3, R38, R39, TP21, TP22, Y1

Commit message: update motor pcb
Parts:
- removed D12: LED, LED_SMD:LED_0805_2012Metric_Pad1.15x1.40mm_HandSolder, symbol Device:LED
- removed R53: 4.7k, Resistor_SMD:R_0603_1608Metric_Pad0.98x0.95mm_HandSolder, symbol Device:R_Small
- added C54: 100n, Capacitor_SMD:C_0603_1608Metric_Pad1.08x0.95mm_HandSolder, symbol Device:C_Small
- added D12: WS2812B, LED_SMD:LED_WS2812B_PLCC4_5.0x5.0mm_P3.2mm, symbol LED:WS2812B
Connections:
- new net GND: C54.1, D12.3 (VSS)
- new net RGB: D12.4 (DIN)
- new net VCC: C54.2, D12.1 (VDD)
- no-connect marks 29 -> 30
Other:
- moved on the sheet: C38, RV1, TP37

Commit message: update motor pcb
Parts:
- FB3: footprint Capacitor_SMD:C_0603_1608Metric_Pad1.08x0.95mm_HandSolder -> Capacitor_SMD:C_0805_2012Metric_Pad1.18x1.45mm_HandSolder
Connections:
- net ADC1_IN11: no longer U5.25 (PB12)
- net INA1+: now also U8.5 (+); no longer U8.3 (+)
- net INA2+: now also U8.3 (+); no longer U8.5 (+)
- net RGB: now also U5.8 (PA0)
- net VREF_OP1: now also U8.6 (-), U8.7; no longer U8.1, U8.2 (-)
- net VREF_OP2: now also U8.1, U8.2 (-); no longer U8.6 (-), U8.7
- net ADC1_IN5: no longer names the net of U5.27 (PB14)
- no-connect marks 30 -> 31
Changed lines of the file:
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@@
 	)
 	(no_connect
-		(at 374.65 46.99)
-	)
-	(no_connect
 		(at 332.74 176.53)
 	)
@@
 	)
 	(no_connect
+		(at 341.63 120.65)
+	)
+	(no_connect
 		(at 243.84 63.5)
 	)
@@
 	)
 	(no_connect
+		(at 341.63 115.57)
+	)
+	(no_connect
 		(at 208.28 44.45)
 	)
@@
 		)
 	)
-	(label "ADC1_IN5"
-		(at 341.63 120.65 180)
-		(fields_autoplaced yes)
-		(effects
-			(font
-				(size 1.27 1.27)
-			)
-			(justify right bottom)
-		)
-	)
 	(label "KEY"
 		(at 237.49 167.64 0)
@@
 	)
 	(label "RGB"
-		(at 325.12 76.2 180)
+		(at 374.65 46.99 0)
 		(fields_autoplaced yes)
 		(effects
@@
 				(size 1.27 1.27)
 			)
-			(justify right bottom)
+			(justify left bottom)
 		)
 	)
@@
 		)
 	)
-	(label "ADC1_IN11"
-		(at 341.63 115.57 180)
-		(fields_autoplaced yes)
-		(effects
-			(font
-				(size 1.27 1.27)
-			)
-			(justify right bottom)
-		)
-	)
 	(label "SPI3_SCK"
 		(at 325.12 189.23 180)
@@
 	)
 	(symbol
-		(lib_id "Amplifier_Operational:TLV9062xD")
-		(at 95.25 128.27 0)
-		(unit 2)
-		(exclude_from_sim no)
-		(in_bom yes)
-		(on_board yes)
-		(dnp no)
-		(fields_autoplaced yes)
-		(property "Reference" "U8"
-			(at 95.25 118.11 0)
-			(effects
-				(font
-					(size 1.27 1.27)
-				)
-			)
-		)
-		(property "Value" "TLV9062xD"
-			(at 95.25 120.65 0)
-			(effects
-				(font
-					(size 1.27 1.27)
-				)
-			)
-		)
-		(property "Footprint" "Package_SO:SOIC-8_3.9x4.9mm_P1.27mm"
-			(at 97.79 128.27 0)
-			(effects
-				(font
-					(size 1.27 1.27)
-				)
-				(hide yes)
-			)
-		)
-		(property "Datasheet" "https://www.ti.com/lit/ds/symlink/tlv9062.pdf"
-			(at 101.6 124.46 0)
-			(effects
-				(font
-					(size 1.27 1.27)
-				)
-				(hide yes)
-			)
-		)
-		(property "Description" "Dual operational amplifier, 300 uV Offset, SOIC-8"
-			(at 95.25 128.27 0)
-			(effects
-				(font
-					(size 1.27 1.27)
-				)
-				(hide yes)
-			)
-		)
-		(pin "1"
-		)
-		(pin "8"
-		)
-		(pin "2"
-		)
-		(pin "4"
-		)
-		(pin "3"
-		)
-		(pin "7"
-		)
-		(pin "6"
-		)
-		(pin "5"
-		)
-		(instances
-			(project "bldcDriver"
-				(path "/024b6358-58d2-4f27-baff-bf9e44899c87"
-					(reference "U8")
-					(unit 2)
-				)
-			)
-		)
-	)
-	(symbol
 		(lib_id "Connector:TestPoint")
 		(at 90.17 57.15 0)
@@
 	)
 	(symbol
-		(lib_id "Amplifier_Operational:TLV9062xD")
-		(at 50.8 127 0)
-		(unit 1)
-		(exclude_from_sim no)
-		(in_bom yes)
-		(on_board yes)
-		(dnp no)
-		(fields_autoplaced yes)
-		(property "Reference" "U8"
-			(at 50.8 116.84 0)
-			(effects
-				(font
-					(size 1.27 1.27)
-				)
-			)
-		)
-		(property "Value" "TLV9062xD"
-			(at 50.8 119.38 0)
-			(effects
-				(font
-					(size 1.27 1.27)
-				)
-			)
-		)
-		(property "Footprint" "Package_SO:SOIC-8_3.9x4.9mm_P1.27mm"
-			(at 53.34 127 0)
-			(effects
-				(font
-					(size 1.27 1.27)
-				)
-				(hide yes)
-			)
-		)
-		(property "Datasheet" "https://www.ti.com/lit/ds/symlink/tlv9062.pdf"
-			(at 57.15 123.19 0)
-			(effects
-				(font
-					(size 1.27 1.27)
-				)
-				(hide yes)
-			)
-		)
-		(property "Description" "Dual operational amplifier, 300 uV Offset, SOIC-8"
-			(at 50.8 127 0)
-			(effects
-				(font
-					(size 1.27 1.27)
-				)
-				(hide yes)
-			)
-		)
-		(pin "1"
-		)
-		(pin "8"
-		)
-		(pin "2"
-		)
-		(pin "4"
-		)
-		(pin "3"
-		)
-		(pin "7"
-		)
-		(pin "6"
-		)
-		(pin "5"
-		)
-		(instances
-			(project "bldcDriver"
-				(path "/024b6358-58d2-4f27-baff-bf9e44899c87"
-					(reference "U8")
-					(unit 1)
-				)
-			)
-		)
-	)
-	(symbol
 		(lib_id "Device:C_Small")
 		(at 323.85 36.83 0)
@@
 	)
 	(symbol
+		(lib_id "Amplifier_Operational:TLV9062xD")
+		(at 95.25 128.27 0)
+		(unit 1)
+		(exclude_from_sim no)
+		(in_bom yes)
+		(on_board yes)
+		(dnp no)
+		(fields_autoplaced yes)
+		(property "Reference" "U8"
+			(at 95.25 118.11 0)
+			(effects
+				(font
+					(size 1.27 1.27)
+				)
+			)
+		)
+		(property "Value" "TLV9062xD"
+			(at 95.25 120.65 0)
+			(effects
+				(font
+					(size 1.27 1.27)
+				)
+			)
+		)
+		(property "Footprint" "Package_SO:SOIC-8_3.9x4.9mm_P1.27mm"
+			(at 97.79 128.27 0)
+			(effects
+				(font
+					(size 1.27 1.27)
+				)
+				(hide yes)
+			)
+		)
+		(property "Datasheet" "https://www.ti.com/lit/ds/symlink/tlv9062.pdf"
+			(at 101.6 124.46 0)
+			(effects
+				(font
+					(size 1.27 1.27)
+				)
+				(hide yes)
+			)
+		)
+		(property "Description" "Dual operational amplifier, 300 uV Offset, SOIC-8"
+			(at 95.25 128.27 0)
+			(effects
+				(font
+					(size 1.27 1.27)
+				)
+				(hide yes)
+			)
+		)
+		(pin "1"
+		)
+		(pin "8"
+		)
+		(pin "2"
+		)
+		(pin "4"
+		)
+		(pin "3"
+		)
+		(pin "7"
+		)
+		(pin "6"
+		)
+		(pin "5"
+		)
+		(instances
+			(project "bldcDriver"
+				(path "/024b6358-58d2-4f27-baff-bf9e44899c87"
+					(reference "U8")
+					(unit 1)
+				)
+			)
+		)
+	)
+	(symbol
 		(lib_id "Device:R_Small")
 		(at 114.3 95.25 180)
@@
 			)
 		)
-		(property "Footprint" "Capacitor_SMD:C_0603_1608Metric_Pad1.08x0.95mm_HandSolder"
+		(property "Footprint" "Capacitor_SMD:C_0805_2012Metric_Pad1.18x1.45mm_HandSolder"
 			(at 44.45 85.852 90)
 			(effects
@@
 				)
 			)
+		)
+	)
+	(symbol
+		(lib_id "Amplifier_Operational:TLV9062xD")
+		(at 50.8 127 0)
+		(unit 2)
+		(exclude_from_sim no)
+		(in_bom yes)
+		(on_board yes)
+		(dnp no)
+		(fields_autoplaced yes)
+		(property "Reference" "U8"
+			(at 50.8 116.84 0)
+			(effects
+				(font
+					(size 1.27 1.27)
+				)
+			)
+		)
+		(property "Value" "TLV9062xD"
+			(at 50.8 119.38 0)
+			(effects
+				(font
+					(size 1.27 1.27)
+				)
+			)
+		)
+		(property "Footprint" "Package_SO:SOIC-8_3.9x4.9mm_P1.27mm"
+			(at 53.34 127 0)
+			(effects
+				(font
+					(size 1.27 1.27)
+				)
+				(hide yes)
+			)
+		)
+		(property "Datasheet" "https://www.ti.com/lit/ds/symlink/tlv9062.pdf"
+			(at 57.15 123.19 0)
+			(effects
+				(font
+					(size 1.27 1.27)
+				)
+				(hide yes)
+			)
+		)
+		(property "Description" "Dual operational amplifier, 300 uV Offset, SOIC-8"
+			(at 50.8 127 0)
+			(effects
+				(font
+					(size 1.27 1.27)
+				)
+				(hide yes)
+			)
+		)
+		(pin "1"
+		)
+		(pin "8"
+		)
+		(pin "2"
+		)
+		(pin "4"
+		)
+		(pin "3"
+		)
+		(pin "7"
+		)
+		(pin "6"
+		)
+		(pin "5"
+		)
+		(instances
+			(project "bldcDriver"
+				(path "/024b6358-58d2-4f27-baff-bf9e44899c87"
+					(reference "U8")
+					(unit 2)
+				)
+			)
