File: hardware/motor/bldcDriver.kicad_pcb (KiCad board)
At the start: 4 copper layers, 89.8 x 41.5 mm, 189 parts, among them CN1 MR30PW-F, CN2 MR30PW-F, J1 Conn_01x02, J2 Conn_01x06, J3 Conn_01x06, J4 Conn_01x03, J5 Conn_01x06, Q1 EMB09N03V, Q10 EMB09N03V, Q11 EMB09N03V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

Commit message: update pcn
Parts:
- removed J3, J5: Conn_01x06, balancerDriver:CONN-SMD_6P-P1.00_MEGASTAR_ZX-SH1.0-6PWT
- removed R49: 10k, Resistor_SMD:R_0603_1608Metric_Pad0.98x0.95mm_HandSolder
- removed R72, R73: 4.7k, Resistor_SMD:R_0603_1608Metric_Pad0.98x0.95mm_HandSolder
- added C52: 100n, Capacitor_SMD:C_0603_1608Metric_Pad1.08x0.95mm_HandSolder, B.Cu at (-13.1, 45.3)
- added SW2: SW_Push, balancerDriver:SW-SMD_L4.0-W2.9-LS5.0, F.Cu at (4.05, 51.2)
- added TP23: TestPoint, TestPoint:TestPoint_Pad_D1.0mm, F.Cu at (3.10, 35.6)
- added TP24: TestPoint, TestPoint:TestPoint_Pad_D1.0mm, F.Cu at (3.10, 38.6)
- added TP25: TestPoint, TestPoint:TestPoint_Pad_D1.0mm, F.Cu at (3.10, 41.7)
- added U10: HC-FPC-0.5-6P-CSH20, balancerDriver:FPC-SMD_6P-P0.50_HC-FPC-0.5-6P-CSH20, F.Cu at (36.5, 42.4)
- added U9: MPU6500, balancerDriver:QFN-24_L3.0-W3.0-P0.40-BL-EP, B.Cu at (-4.73, 51.1)
- C23: value 100n -> 2.2u
- C24: value 2.2n -> 100n
- D12, TP11, TP13, TP14, TP15, TP16, TP17, TP18, TP19, TP22, TP8: moved to F.Cu
- SW1: footprint Button_Switch_SMD:SW_SPST_B3U-1000P -> balancerDriver:SW-SMD_L4.0-W2.9-LS5.0; moved to F.Cu
- U4: value MPU-6050 -> HC-FPC-0.5-6P-CSH20; footprint Sensor_Motion:InvenSense_QFN-24_4x4mm_P0.5mm -> balancerDriver:FPC-SMD_6P-P0.50_HC-FPC-0.5-6P-CSH20; moved to F.Cu
- moved C13 109.4 mm to (-13.1, 35.3), turned to 180 degrees
- moved C24 107.0 mm to (-13.1, 42.8), turned to 180 degrees
- moved C23 106.4 mm to (-13.1, 40.3), turned to 180 degrees
- moved C22 104.8 mm to (-13.1, 37.8), turned to 180 degrees
- moved FB1 97.7 mm to (-6.60, 48.1), turned to 180 degrees
- moved U4 25.8 mm to (118.2, 43.4), turned to 90 degrees
- moved SW1 10.1 mm to (77.7, 32.4), turned to 0 degrees
- turned D12 to 0 degrees
- turned TP11 to 0 degrees
- turned TP13 to 0 degrees
- turned TP14 to 0 degrees
- turned TP15 to 0 degrees
- turned TP16 to 0 degrees
- turned TP17 to 0 degrees
- turned TP18 to 0 degrees
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Connections:
- C13 pad 1: Net-(U4-VDD) -> Net-(U9-VDD)
- C15 pad 1: Net-(U1-VCC) -> +BATT
- C22 pad 1: Net-(U4-VDD) -> Net-(U9-REGOUT)
- C23 pad 1: Net-(U4-REGOUT) -> Net-(U9-VDD)
- C24 pad 1: Net-(U4-CPOUT) -> Net-(U9-VDD)
- C32 pad 1: Net-(U2-VCC) -> +BATT
- C5 pad 1: GNDPWR -> GNDD
- C50 pad 1: GNDPWR -> GNDD
- C6 pad 1: GNDPWR -> GNDD
- C7 pad 1: GNDPWR -> GNDD
- D1 pad 2: GNDPWR -> GNDD
- D8 pad 1: GNDPWR -> GNDD
- FB1 pad 1: +3V3 -> Net-(U9-VDD)
- FB1 pad 2: Net-(U4-VDD) -> +3V3
- R2 pad 2: GNDPWR -> GNDD
- U1 pad 7: Net-(U1-VCC) -> +BATT
- U2 pad 7: Net-(U2-VCC) -> +BATT
- U3 pad 6: GNDPWR -> GNDD
- U3 pad 9: GNDPWR -> GNDD
- U4 pad 1: GNDD -> /NSS2
- U4 pad 2: unconnected-(U4-NC-Pad2) -> /SPI3_MOSI
- U4 pad 3: unconnected-(U4-NC-Pad3) -> /SPI3_MISO
- U4 pad 4: unconnected-(U4-NC-Pad4) -> /SPI3_SCK
- U4 pad 5: unconnected-(U4-NC-Pad5) -> +3V3
- U4 pad 6: unconnected-(U4-AUX_DA-Pad6) -> GNDD
- U4 pad 8: Net-(U4-VDD) -> unconnected-(U4-Pad8)
- U5 pad 12: /MPU_INT -> unconnected-(U5-PA4-Pad12)
Routing:
- net +3V3: track 194.2 -> 124.4 mm, vias 8 -> 7
- net /SPI3_SCK: track 39.2 -> 1.54 mm, vias 2 -> 1
- net /NSS1: track 37.5 -> 1.71 mm, vias 2 -> 1
- net /SPI3_MOSI: track 36.5 -> 0.93 mm, vias 2 -> 1
- net /SPI3_MISO: track 38.0 -> 2.67 mm, vias 2 -> 1
- net /SPI1_MISO: track 38.6 -> 4.49 mm, vias 1 -> 0
- net /SPI1_MOSI: track 38.5 -> 4.35 mm, vias 1 -> 0
- net /NSS2: track 38.2 -> 4.21 mm, vias 1 -> 0
- net /SPI1_SCK: track 37.7 -> 4.71 mm, vias 1 -> 0
- net /MPU_INT: track 24.3 -> 0.00 mm, vias 2 -> 0
- net Net-(U4-VDD): track 23.2 -> 0.00 mm, vias 3 -> 0
- net /USART2_RX: track 26.8 -> 11.0 mm, vias 1 -> 0
- net /USART2_TX: track 27.8 -> 14.3 mm
- net /I2C1_SCL: track 24.7 -> 17.7 mm, vias 2 -> 1
- net unconnected-(U5-PA4-Pad12): track 0.00 -> 6.78 mm, vias 0 -> 1
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Other:
- board text removed: "V1.2"

Commit message: update pcb
Parts:
- removed TP9: TestPoint, TestPoint:TestPoint_Pad_D1.0mm
- TP10, TP12: moved to F.Cu
- U9: footprint balancerDriver:QFN-24_L3.0-W3.0-P0.40-BL-EP -> balancerDriver:QFN24_3X3X0P9_IVS-L
- moved C23 110.1 mm to (96.8, 34.6), turned to 90 degrees
- moved C24 108.8 mm to (95.3, 34.6), turned to 90 degrees
- moved C22 106.7 mm to (93.4, 32.8), turned to 90 degrees
- moved FB1 105.8 mm to (98.3, 34.6), turned to 90 degrees
- moved C13 105.0 mm to (91.8, 32.8), turned to 90 degrees
- moved U9 98.3 mm to (92.5, 36.6), turned to 0 degrees
- moved C52 84.0 mm to (70.2, 34.7)
- moved SW2 68.1 mm to (69.5, 32.4), turned to 180 degrees
- moved C21 6.05 mm to (75.9, 31.7), turned to 180 degrees
- moved J4 5.19 mm to (108.5, 35.9)
- moved TP22 5.19 mm to (102.5, 37.7)
- moved SW1 2.84 mm to (80.5, 32.3)
- moved J1 1.45 mm to (60.7, 47.8)
- moved TP10 0.54 mm to (81.7, 37.8), turned to 0 degrees
- turned D12 to 180 degrees
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Connections:
- U5 pad 12: unconnected-(U5-PA4-Pad12) -> /SPI1_CS
- U5 pad 3: Net-(U5-PC14) -> /KEY
- U5 pad 45: /I2C1_SDA -> unconnected-(U5-PB7-Pad45)
Routing:
- net /SPI3_MISO: track 2.67 -> 91.4 mm, vias 1 -> 3
- net /SPI3_SCK: track 1.54 -> 86.8 mm, vias 1 -> 3
- net /SPI3_MOSI: track 0.93 -> 81.6 mm
- net +3V3: track 124.4 -> 177.1 mm, vias 7 -> 9
- net /NSS1: track 1.71 -> 36.9 mm
- net /NSS2: track 4.21 -> 36.9 mm, vias 0 -> 1
- net /I2C1_SDA: track 19.6 -> 0.00 mm, vias 1 -> 0
- net /USART2_RX: track 11.0 -> 30.3 mm, vias 0 -> 1
- net GNDD: track 64.9 -> 46.3 mm, vias 46 -> 43
- net /USART2_TX: track 14.3 -> 32.8 mm
- net /I2C1_SCL: track 17.7 -> 2.27 mm
- net /SPI1_CS: track 0.00 -> 14.5 mm, vias 0 -> 2
- net /SPI1_MOSI: track 4.35 -> 15.8 mm
- net /KEY: track 0.00 -> 10.7 mm, vias 0 -> 3
- net /SPI1_MISO: track 4.49 -> 15.2 mm
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Other:
- board text removed: "PA1"
- board text removed: "PC14"

Commit message: update motor pcb
Parts:
- removed C38, C43, C44: 4.7u, Capacitor_SMD:C_0603_1608Metric_Pad1.08x0.95mm_HandSolder
- removed C39, C40, C47, C48: 100n, Capacitor_SMD:C_0603_1608Metric_Pad1.08x0.95mm_HandSolder
- removed R40, R41: 1k, Resistor_SMD:R_0603_1608Metric_Pad0.98x0.95mm_HandSolder
- removed U8: TLV9062xD, Package_SO:SOIC-8_3.9x4.9mm_P1.27mm
- added R49: 3k, Resistor_SMD:R_0603_1608Metric_Pad0.98x0.95mm_HandSolder, B.Cu at (63.7, 54.5)
- added R54: 3k, Resistor_SMD:R_0603_1608Metric_Pad0.98x0.95mm_HandSolder, B.Cu at (62.8, 56.1)
- added R55: 3k, Resistor_SMD:R_0603_1608Metric_Pad0.98x0.95mm_HandSolder, B.Cu at (65.5, 52.9)
- added R56: 3k, Resistor_SMD:R_0603_1608Metric_Pad0.98x0.95mm_HandSolder, B.Cu at (80.5, 51.9)
- added R57: 3k, Resistor_SMD:R_0603_1608Metric_Pad0.98x0.95mm_HandSolder, B.Cu at (90.7, 51.6)
- added R58: 3k, Resistor_SMD:R_0603_1608Metric_Pad0.98x0.95mm_HandSolder, B.Cu at (88.6, 53.3)
- TP21: moved to F.Cu
- moved TP24 85.7 mm to (88.8, 37.2)
- moved TP23 85.2 mm to (88.2, 40.5)
- moved TP25 83.4 mm to (86.5, 41.8)
- moved TP8 7.29 mm to (69.9, 56.0)
- moved J2 5.50 mm to (82.7, 69.2), turned to 0 degrees
- moved TP11 3.89 mm to (82.8, 52.1)
- moved TP18 3.65 mm to (82.7, 56.4)
- moved TP19 3.36 mm to (76.3, 56.8)
- moved R38 3.24 mm to (76.2, 53.8), turned to 0 degrees
- moved TP21 3.19 mm to (44.6, 42.1), turned to 0 degrees
- moved TP10 3.04 mm to (84.7, 37.3)
- moved C11 2.91 mm to (83.6, 58.3)
- moved C27 2.91 mm to (69.5, 58.3)
- moved C45 2.91 mm to (80.2, 58.3)
- moved C46 2.91 mm to (66.1, 58.3)
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Connections:
- J2 pad 1: +3V3 -> /SWCLK
- J2 pad 2: GNDD -> /SWDIO
- J2 pad 3: /USART3_TX -> /USART3_RX
- J2 pad 4: /USART3_RX -> /USART3_TX
- J2 pad 5: /SWDIO -> GNDD
- J2 pad 6: /SWCLK -> +3V3
- R31 pad 2: /VREF_OP2 -> /VREF_OP
- R33 pad 2: /VREF_OP1 -> /VREF_OP
- R38 pad 1: /INA1+ -> /VREF_OP
- R39 pad 2: /INA1+ -> /VREF_OP
- R45 pad 2: /VREF_OP2 -> /VREF_OP
- R47 pad 2: /VREF_OP1 -> /VREF_OP
Routing:
- net /VREF_OP2: track 35.6 -> 0.00 mm, vias 2 -> 0
- net /VREF_OP: track 0.00 -> 34.9 mm, vias 0 -> 3
- net /VREF_OP1: track 31.6 -> 0.00 mm, vias 2 -> 0
- net GNDD: track 46.3 -> 63.5 mm, vias 43 -> 46
- net Net-(U9-VDD): track 0.00 -> 13.4 mm, vias 0 -> 2
- net /INA1+: track 12.0 -> 0.00 mm
- net /OP_VCC: track 39.7 -> 30.0 mm, vias 2 -> 0
- net /TIM1_CH2: track 36.6 -> 45.1 mm, vias 3 -> 4
- net /SWCLK: track 29.7 -> 23.6 mm
- net +3V3: track 177.1 -> 171.4 mm, vias 9 -> 7
- net Net-(U5-PA1): track 2.73 -> 8.27 mm, vias 1 -> 2
- net /SPI3_MISO: track 91.4 -> 86.8 mm
- net /ADC2_IN12: track 24.1 -> 19.7 mm
- net /TIM8_CH3: track 28.7 -> 33.1 mm, vias 1 -> 2
- net /ADC1_IN5: track 20.4 -> 16.2 mm
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
Commit message: update motor pcb
Parts:
- removed J4: Conn_01x03, balancerDriver:CONN-SMD_3P-P1.00_WAFER-SH1.0-3PWB
- removed R49, R54, R55, R56, R57, R58: 3k, Resistor_SMD:R_0603_1608Metric_Pad0.98x0.95mm_HandSolder
- added C38: 100n, Capacitor_SMD:C_0603_1608Metric_Pad1.08x0.95mm_HandSolder, B.Cu at (96.4, 36.0)
- added P1: FPC_0.5MM_4P_Vertical_mounting_type_H2.0mm, balancerDriver:FPC-SMD_4P-L7.5-W2.0-P0.50, F.Cu at (88.8, 41.0)
- added R40: 3k, Resistor_SMD:R_0603_1608Metric_Pad0.98x0.95mm_HandSolder, B.Cu at (63.6, 57.5)
- added RV1: R_Potentiometer, balancerDriver:RES-ADJ-TH_3362P, F.Cu at (101.0, 35.7)
- added TP26: TestPoint, TestPoint:TestPoint_Pad_D1.0mm, F.Cu at (144.5, 54.0)
- added TP27: TestPoint, TestPoint:TestPoint_Pad_D1.0mm, F.Cu at (144.5, 57.0)
- added TP28: TestPoint, TestPoint:TestPoint_Pad_D1.0mm, F.Cu at (144.5, 60.1)
- added TP9: TestPoint, TestPoint:TestPoint_Pad_D1.0mm, F.Cu at (144.5, 51.0)
- TP20, TP7: moved to F.Cu
- moved TP11 72.0 mm to (154.0, 41.1)
- moved TP8 59.9 mm to (129.8, 54.5)
- moved TP17 57.5 mm to (129.8, 57.5)
- moved TP10 55.9 mm to (140.5, 41.1)
- moved TP25 54.6 mm to (140.5, 50.2)
- moved TP24 52.6 mm to (140.5, 47.2)
- moved TP23 52.4 mm to (140.5, 44.1)
- moved TP12 37.6 mm to (67.0, 82.5)
- moved TP13 37.3 mm to (67.0, 85.6)
- moved TP16 36.1 mm to (67.0, 88.7)
- moved TP19 29.1 mm to (72.1, 85.6)
- moved TP18 28.2 mm to (72.1, 82.5)
- moved FB1 23.2 mm to (75.3, 31.5), turned to 180 degrees
- moved C24 20.1 mm to (75.3, 33.0), turned to 180 degrees
- moved C22 20.0 mm to (73.5, 34.9), turned to 180 degrees
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Connections:
- U5 pad 38: /I2C1_SCL -> unconnected-(U5-PA15-Pad38)
Routing:
- net +3V3: track 171.4 -> 211.4 mm
- net GNDD: track 63.5 -> 24.3 mm, vias 46 -> 29
- net /NSS2: track 36.9 -> 0.38 mm, vias 1 -> 0
- net /USART2_TX: track 30.6 -> 1.10 mm
- net /USART2_RX: track 30.3 -> 1.16 mm
- net /TIM1_CH2: track 45.1 -> 33.8 mm, vias 4 -> 3
- net /LED: track 14.0 -> 3.23 mm, vias 2 -> 1
- net /1CS1-: track 35.9 -> 25.4 mm
- net /RESET: track 10.5 -> 0.89 mm, vias 2 -> 1
- net /TIM8_CH3: track 33.1 -> 25.3 mm, vias 2 -> 1
- net Net-(U5-PA1): track 8.27 -> 1.07 mm
- net /SPI3_MOSI: track 81.6 -> 87.9 mm
- net /TIM8_CH2: track 31.2 -> 25.0 mm, vias 4 -> 3
- net Net-(U5-PA11): track 6.47 -> 0.84 mm, vias 2 -> 1
- net /OP_VCC: track 30.0 -> 24.5 mm
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Other:
- board text removed: "PA11"

Commit message: update motor pcb
Parts:
- removed TP10: TestPoint, TestPoint:TestPoint_Pad_D1.0mm
- moved TP27 96.8 mm to (47.9, 50.7)
- moved TP28 96.5 mm to (48.3, 67.1)
- moved TP11 72.6 mm to (83.2, 57.3)
- moved TP8 64.3 mm to (65.8, 61.0)
- moved TP24 64.2 mm to (76.7, 39.4)
- moved TP25 62.6 mm to (78.8, 39.6)
- moved TP23 60.2 mm to (80.6, 37.6)
- moved TP17 58.6 mm to (71.4, 62.4)
- moved TP9 42.1 mm to (106.9, 69.9)
- moved TP26 37.2 mm to (107.3, 55.6)
- moved TP13 36.1 mm to (93.2, 60.7)
- moved TP12 34.2 mm to (94.9, 62.7)
- moved TP16 32.5 mm to (63.7, 56.3)
- moved TP19 30.7 mm to (81.4, 56.3)
- moved TP18 26.7 mm to (84.6, 59.0)
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Connections:
- C38 pad 1: Net-(C38-Pad1) -> /ADC1_IN2
- RV1 pad 2: Net-(C38-Pad1) -> /ADC1_IN2
- U5 pad 9: Net-(U5-PA1) -> /ADC1_IN2
Routing:
- net /ADC1_IN2: track 0.00 -> 27.5 mm, vias 0 -> 2
- net /RESET: track 0.89 -> 18.9 mm, vias 1 -> 2
- net /LED: track 3.23 -> 17.4 mm, vias 1 -> 2
- net +3V3: track 211.4 -> 222.3 mm
- net /1CS1-: track 25.4 -> 33.4 mm
- net /TIM1_CH2: track 33.8 -> 26.6 mm
- net /2CS2-: track 32.2 -> 35.5 mm
- net /1CS2+: track 25.1 -> 22.1 mm
- net Net-(U5-PA11): track 0.84 -> 3.80 mm, vias 1 -> 2
- net /TIM8_CH2: track 25.0 -> 27.9 mm, vias 3 -> 4
- net /ADC1_IN5: track 14.3 -> 17.0 mm, vias 2 -> 3
- net Net-(D12-K): track 0.00 -> 2.29 mm, vias 0 -> 1
- net /TIM1_CH1: track 27.4 -> 29.1 mm, vias 0 -> 1
- net /2CS1-: track 21.8 -> 23.4 mm
- net Net-(Q16-S-Pad1): track 2.02 -> 3.13 mm, vias 0 -> 1
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Other:
- board text added: "A1_IN11"
- board text added: "A1_IN5"
- board text added: "A2_IN12"
- board text added: "A2_IN15"
- board text added: "PA11"
- board text added: "T1_CH1"
- board text added: "T1_CH2"
- board text added: "T1_CH3"
- board text added: "T8_CH1"
- board text added: "T8_CH2"
- board text added: "T8_CH3"

Commit message: update driver pcb
Parts:
- moved P1 4.45 mm to (93.2, 41.1)
Connections:
- P1 pad 3: /USART2_TX -> +3V3
- P1 pad 4: +3V3 -> /USART2_TX
Changed lines of the file:
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@@
 	(footprint "balancerDriver:FPC-SMD_4P-L7.5-W2.0-P0.50"
 		(layer "F.Cu")
-		(at 88.786 41.05 90)
+		(at 93.237 41.099 90)
 		(property "Reference" "P1"
 			(at 1.514 -3.45 270)
@@
 			(size 0.4 1.5)
 			(layers "F.Cu" "F.Paste" "F.Mask")
-			(net 71 "/USART2_TX")
+			(net 3 "+3V3")
 			(pinfunction "3")
 			(pintype "input")
@@
 			(size 0.4 1.5)
 			(layers "F.Cu" "F.Paste" "F.Mask")
-			(net 3 "+3V3")
+			(net 71 "/USART2_TX")
 			(pinfunction "4")
 			(pintype "input")
@@
 		(tags "LED handsolder")
 		(property "Reference" "D12"
-			(at 0 -1.65 360)
+			(at 0 -1.65 0)
 			(layer "F.SilkS")
 			(hide yes)
@@
 		)
 		(property "Value" "LED"
-			(at 0 1.65 360)
+			(at 0 1.65 0)
 			(layer "F.Fab")
 			(effects
@@
 		)
 		(fp_text user "${REFERENCE}"
-			(at 0 0 360)
+			(at 0 0 0)
 			(layer "F.Fab")
 			(effects
@@
 		(tags "resistor handsolder")
 		(property "Reference" "R53"
-			(at 0 1.43 360)
+			(at 0 1.43 0)
 			(layer "B.SilkS")
 			(hide yes)
@@
 		)
 		(property "Value" "4.7k"
-			(at 0 -1.43 360)
+			(at 0 -1.43 0)
 			(layer "B.Fab")
 			(effects
@@
 		)
 		(fp_text user "${REFERENCE}"
-			(at 0 0 360)
+			(at 0 0 0)
 			(layer "B.Fab")
 			(effects
@@
 		(tags "capacitor handsolder")
 		(property "Reference" "C21"
-			(at 0 1.43 270)
+			(at 0 1.43 -90)
 			(layer "B.SilkS")
 			(hide yes)
@@
 		)
 		(property "Value" "100n"
-			(at 0 -1.43 270)
+			(at 0 -1.43 -90)
 			(layer "B.Fab")
 			(effects
@@
 		)
 		(fp_text user "${REFERENCE}"
-			(at 0 0 270)
+			(at 0 0 -90)
 			(layer "B.Fab")
 			(effects
@@
 	)
 	(gr_text "TX"
-		(at 94.1365 39.1 0)
+		(at 93.3 38.9 90)
 		(layer "F.SilkS")
 		(effects
@@
 		)
 	)
+	(gr_text "3V3"
+		(at 92.9 44.4 90)
+		(layer "F.SilkS")
+		(effects
+			(font
+				(size 0.5 0.5)
+				(thickness 0.1)
+				(bold yes)
+			)
+			(justify left bottom)
+		)
+	)
 	(gr_text "T8_CH3"
 		(at 54.8 54.5 0)
@@
 	)
 	(gr_text "MOSI\n"
-		(at 116.05 42.15 180)
+		(at 114 42.9 0)
 		(layer "F.SilkS")
 		(effects
@@
 	)
 	(gr_text "NSS"
-		(at 116.05 41.45 180)
+		(at 114.6 42 0)
 		(layer "F.SilkS")
 		(effects
@@
 	)
 	(gr_text "RX"
-		(at 94.1365 40 0)
+		(at 94.3 39 90)
 		(layer "F.SilkS")
 		(effects
@@
 	)
 	(gr_text "GND"
-		(at 93.8365 41 0)
+		(at 93.7 44.6 90)
 		(layer "F.SilkS")
 		(effects
