File: hardware/motor/bldcDriver.kicad_pcb (KiCad board)
At the start: 4 copper layers, 89.8 x 41.5 mm, 198 parts, among them CN1 MR30PW-F, CN2 MR30PW-F, J1 Conn_01x02, J2 Conn_01x06, P1 FPC_0.5MM_4P_Vertical_mountin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, Q1 EMB09N03V, Q10 EMB09N03V, Q11 EMB09N03V, Q12 EMB09N03V, Q13 EMB09N03V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

Commit message: update motor pcb
Parts:
- removed R53: 4.7k, Resistor_SMD:R_0603_1608Metric_Pad0.98x0.95mm_HandSolder
- added C54: 100n, Capacitor_SMD:C_0603_1608Metric_Pad1.08x0.95mm_HandSolder, B.Cu at (108.4, 43.7)
- added TP10: TestPoint, TestPoint:TestPoint_Pad_D1.0mm, F.Cu at (140.5, 45.8)
- added TP14: TestPoint, TestPoint:TestPoint_Pad_D1.0mm, F.Cu at (155.3, 42.7)
- added TP15: TestPoint, TestPoint:TestPoint_Pad_D1.0mm, F.Cu at (155.3, 45.8)
- added TP16: TestPoint, TestPoint:TestPoint_Pad_D1.0mm, F.Cu at (155.3, 48.8)
- added TP17: TestPoint, TestPoint:TestPoint_Pad_D1.0mm, F.Cu at (140.5, 48.8)
- added TP23: TestPoint, TestPoint:TestPoint_Pad_D1.0mm, F.Cu at (143.6, 42.7)
- added TP24: TestPoint, TestPoint:TestPoint_Pad_D1.0mm, F.Cu at (143.6, 45.8)
- added TP25: TestPoint, TestPoint:TestPoint_Pad_D1.0mm, F.Cu at (143.6, 48.8)
- added TP29: TestPoint, TestPoint:TestPoint_Pad_D1.0mm, F.Cu at (146.6, 42.7)
- added TP30: TestPoint, TestPoint:TestPoint_Pad_D1.0mm, F.Cu at (146.6, 45.8)
- added TP31: TestPoint, TestPoint:TestPoint_Pad_D1.0mm, F.Cu at (146.6, 48.8)
- added TP32: TestPoint, TestPoint:TestPoint_Pad_D1.0mm, F.Cu at (149.7, 42.7)
- added TP34: TestPoint, TestPoint:TestPoint_Pad_D1.0mm, F.Cu at (94.4, 43.1)
- added TP37: TestPoint, TestPoint:TestPoint_Pad_D1.0mm, F.Cu at (149.7, 48.8)
- added TP8: TestPoint, TestPoint:TestPoint_Pad_D1.0mm, F.Cu at (140.5, 42.7)
- D12: value LED -> WS2812B; footprint LED_SMD:LED_0805_2012Metric_Pad1.15x1.40mm_HandSolder -> LED_SMD:LED_WS2812B_PLCC4_5.0x5.0mm_P3.2mm
- FB3: footprint Capacitor_SMD:C_0603_1608Metric_Pad1.08x0.95mm_HandSolder -> Capacitor_SMD:C_0805_2012Metric_Pad1.18x1.45mm_HandSolder
- moved C53 15.0 mm to (77.6, 56.8), turned to 180 degrees
- moved C44 14.6 mm to (77.6, 58.3), turned to 180 degrees
- moved C47 11.0 mm to (73.9, 55.6), turned to 180 degrees
- moved C43 8.63 mm to (66.5, 56.9), turned to 0 degrees
- moved C48 8.63 mm to (66.5, 58.4), turned to 0 degrees
- moved R38 8.63 mm to (66.5, 61.4), turned to 180 degrees
- moved R39 8.63 mm to (66.5, 59.9), turned to 0 degrees
- moved D12 3.11 mm to (103.9, 42.8), turned to 180 degrees
- moved U8 2.94 mm to (72.1, 59.3)
- moved R41 1.74 mm to (77.6, 61.4), turned to 0 degrees
- moved TP35 1.20 mm to (88.6, 38.9)
- moved C68 0.64 mm to (85.4, 42.5)
- moved R49 0.41 mm to (77.6, 59.9), turned to 180 degrees
- moved C67 0.35 mm to (79.6, 42.8)
- moved Y1 0.35 mm to (82.5, 42.7)
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Connections:
- D12 pad 1: Net-(D12-K) -> VCC
- D12 pad 2: +3V3 -> unconnected-(D12-DOUT-Pad2)
- U5 pad 25: /ADC1_IN11 -> unconnected-(U5-PB12-Pad25)
- U5 pad 27: /ADC1_IN5 -> unconnected-(U5-PB14-Pad27)
- U5 pad 8: unconnected-(U5-PA0-Pad8) -> /RGB
- U8 pad 1: /VREF_OP1 -> /VREF_OP2
- U8 pad 2: /VREF_OP1 -> /VREF_OP2
- U8 pad 3: /INA1+ -> /INA2+
- U8 pad 5: /INA2+ -> /INA1+
- U8 pad 6: /VREF_OP2 -> /VREF_OP1
- U8 pad 7: /VREF_OP2 -> /VREF_OP1
Routing:
- net /SPI3_MOSI: track 19.5 -> 86.2 mm, vias 0 -> 1
- net +3V3: track 74.9 -> 139.4 mm, vias 5 -> 6
- net /SPI3_SCK: track 30.2 -> 89.6 mm, vias 2 -> 3
- net /SPI3_MISO: track 32.3 -> 89.7 mm, vias 2 -> 3
- net /NSS1: track 1.48 -> 44.8 mm, vias 0 -> 1
- net /VREF_OP2: track 0.00 -> 34.7 mm, vias 0 -> 2
- net /OP_VCC: track 3.92 -> 36.2 mm, vias 0 -> 3
- net (no net): track 30.5 -> 0.00 mm, vias 2 -> 0
- net /VREF_OP1: track 0.00 -> 27.3 mm, vias 0 -> 2
- net /ADC2_IN15: track 1.41 -> 28.1 mm, vias 1 -> 2
- net /NSS2: track 9.46 -> 33.1 mm, vias 0 -> 1
- net /ADC1_IN12_COMP1_INP: track 4.08 -> 25.8 mm
- net /ADC1_IN2: track 0.00 -> 21.5 mm, vias 0 -> 2
- net /2CS2+: track 16.0 -> 36.3 mm, vias 1 -> 2
- net /SWCLK: track 0.70 -> 19.5 mm, vias 0 -> 1
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
Commit message: update motor pcb
Parts:
- removed TP37, TP39, TP7: TestPoint, TestPoint:TestPoint_Pad_D1.0mm
- moved TP15 92.8 mm to (62.9, 54.4)
- moved TP14 92.6 mm to (63.2, 52.2)
- moved TP16 81.6 mm to (73.8, 53.2)
- moved TP8 80.6 mm to (62.2, 61.6)
- moved TP32 78.4 mm to (71.3, 45.2)
- moved TP30 75.2 mm to (71.5, 49.7)
- moved TP17 68.9 mm to (73.1, 63.1)
- moved TP24 67.4 mm to (76.6, 38.2)
- moved TP10 62.2 mm to (78.6, 51.9)
- moved TP23 61.4 mm to (82.5, 36.3)
- moved TP25 60.3 mm to (84.3, 37.5)
- moved TP40 56.1 mm to (75.0, 59.9)
- moved TP31 51.9 mm to (94.8, 51.0)
- moved TP11 41.5 mm to (85.4, 56.4)
- moved TP19 41.1 mm to (76.1, 62.7)
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Connections:
- C54 pad 2: VCC -> +3V3
- D12 pad 1: VCC -> +3V3
- U5 pad 33: Net-(U5-PA11) -> unconnected-(U5-PA11-Pad33)
Routing:
- net +3V3: track 139.4 -> 181.5 mm, vias 6 -> 10
- net GNDD: track 52.0 -> 89.6 mm, vias 18 -> 37
- net /KEY: track 3.85 -> 19.9 mm, vias 1 -> 2
- net /ADC1_IN11: track 16.2 -> 1.51 mm, vias 2 -> 1
- net GND: track 0.00 -> 7.65 mm, vias 0 -> 1
- net /ADC1_IN2: track 21.5 -> 26.2 mm
- net /YI: track 8.60 -> 5.85 mm
- net /1CS2+: track 20.4 -> 18.0 mm
- net VDDA: track 5.61 -> 7.31 mm
- net /RESET: track 15.8 -> 17.5 mm
- net Net-(U5-PA15): track 0.00 -> 1.15 mm, vias 0 -> 1
- net /SPI1_SCK: track 16.5 -> 17.2 mm, vias 0 -> 1
- net /SWCLK: track 19.5 -> 18.8 mm
- net /TIM1_CH2: track 23.0 -> 22.3 mm
- net +BATT: track 57.8 -> 57.2 mm, vias 54 -> 55
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