File: hardware/motor/bldcDriver.kicad_pcb (KiCad board)
At the start: 4 copper layers, 89.8 x 41.5 mm, 210 parts, among them CN1 MR30PW-F, CN2 MR30PW-F, J1 Conn_01x02, J2 Conn_01x06, P1 FPC_0.5MM_4P_Vertical_mountin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, Q1 EMB09N03V, Q10 EMB09N03V, Q11 EMB09N03V, Q12 EMB09N03V, Q13 EMB09N03V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

Commit message: update motor pcb
Parts:
- added TP7: TestPoint, TestPoint:TestPoint_Pad_D1.0mm, F.Cu at (86.6, 53.6)
Connections:
- U5 pad 25: unconnected-(U5-PB12-Pad25) -> Net-(U5-PB12)
Routing:
- net +3V3: track 181.5 -> 184.9 mm
- net Net-(U5-PB12): track 0.00 -> 1.37 mm, vias 0 -> 1
Other:
- board text added: "CH1"
- board text added: "CH2"
- board text added: "CH3"
- board text added: "INA2+"
- board text added: "PB12"
- board text removed: "T1_CH1"
- board text removed: "T1_CH2"

Commit message: udpate motor firmware
Connections:
- C54 pad 1: GND -> GNDD
- D12 pad 3: GND -> GNDD
Routing:
- net GND: track 7.65 -> 0.00 mm, vias 1 -> 0
- net GNDD: track 89.6 -> 97.3 mm, vias 37 -> 38
Changed lines of the file:
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@@
 	(net 142 "/ADC1_IN12_COMP1_INP")
 	(net 143 "unconnected-(U5-PB2-Pad19)")
-	(net 144 "GND")
-	(net 145 "/RGB")
-	(net 146 "unconnected-(D12-DOUT-Pad2)")
-	(net 147 "Net-(U5-PB12)")
-	(net 148 "unconnected-(U5-PB14-Pad27)")
-	(net 149 "unconnected-(U5-PA11-Pad33)")
+	(net 144 "/RGB")
+	(net 145 "unconnected-(D12-DOUT-Pad2)")
+	(net 146 "Net-(U5-PB12)")
+	(net 147 "unconnected-(U5-PB14-Pad27)")
+	(net 148 "unconnected-(U5-PA11-Pad33)")
 	(footprint "TestPoint:TestPoint_Pad_D1.0mm"
 		(layer "F.Cu")
@@
 			(size 1 1)
 			(layers "F.Cu" "F.Mask")
-			(net 147 "Net-(U5-PB12)")
+			(net 146 "Net-(U5-PB12)")
 			(pinfunction "1")
 			(pintype "passive")
@@
 			(size 1.5 0.9)
 			(layers "F.Cu" "F.Paste" "F.Mask")
-			(net 146 "unconnected-(D12-DOUT-Pad2)")
+			(net 145 "unconnected-(D12-DOUT-Pad2)")
 			(pinfunction "DOUT")
 			(pintype "output+no_connect")
@@
 			(size 1.5 0.9)
 			(layers "F.Cu" "F.Paste" "F.Mask")
-			(net 144 "GND")
+			(net 2 "GNDD")
 			(pinfunction "VSS")
 			(pintype "power_in")
@@
 			(size 1.5 0.9)
 			(layers "F.Cu" "F.Paste" "F.Mask")
-			(net 145 "/RGB")
+			(net 144 "/RGB")
 			(pinfunction "DIN")
 			(pintype "input")
@@
 			(layers "B.Cu" "B.Paste" "B.Mask")
 			(roundrect_rratio 0.25)
-			(net 145 "/RGB")
+			(net 144 "/RGB")
 			(pinfunction "PA0")
 			(pintype "bidirectional")
@@
 			(layers "B.Cu" "B.Paste" "B.Mask")
 			(roundrect_rratio 0.25)
-			(net 147 "Net-(U5-PB12)")
+			(net 146 "Net-(U5-PB12)")
 			(pinfunction "PB12")
 			(pintype "bidirectional")
@@
 			(layers "B.Cu" "B.Paste" "B.Mask")
 			(roundrect_rratio 0.25)
-			(net 148 "unconnected-(U5-PB14-Pad27)")
+			(net 147 "unconnected-(U5-PB14-Pad27)")
 			(pinfunction "PB14")
 			(pintype "bidirectional+no_connect")
@@
 			(layers "B.Cu" "B.Paste" "B.Mask")
 			(roundrect_rratio 0.25)
-			(net 149 "unconnected-(U5-PA11-Pad33)")
+			(net 148 "unconnected-(U5-PA11-Pad33)")
 			(pinfunction "PA11")
 			(pintype "bidirectional+no_connect")
@@
 			(layers "B.Cu" "B.Paste" "B.Mask")
 			(roundrect_rratio 0.25)
-			(net 144 "GND")
+			(net 2 "GNDD")
 			(pintype "passive")
 		)
@@
 	)
 	(segment
+		(start 103.1375 42.8375)
+		(end 108.4 42.8375)
+		(width 0.3)
+		(layer "F.Cu")
+		(net 2)
+	)
+	(segment
 		(start 117.15 44.65)
 		(end 116.8 45)
@@
 		(net 2)
 	)
+	(segment
+		(start 101.45 41.15)
+		(end 103.1375 42.8375)
+		(width 0.3)
+		(layer "F.Cu")
+		(net 2)
+	)
 	(via
 		(at 69.1 68.1)
@@
 	)
 	(via
+		(at 108.4 42.8375)
+		(size 0.6)
+		(drill 0.3)
+		(layers "F.Cu" "B.Cu")
+		(net 2)
+	)
+	(via
 		(at 76.3 45.65)
 		(size 0.9)
@@
 		(net 142)
 	)
-	(segment
-		(start 103.1375 42.8375)
-		(end 108.4 42.8375)
-		(width 0.3)
-		(layer "F.Cu")
-		(net 144)
-	)
-	(segment
-		(start 101.45 41.15)
-		(end 103.1375 42.8375)
-		(width 0.3)
-		(layer "F.Cu")
-		(net 144)
-	)
-	(via
-		(at 108.4 42.8375)
-		(size 0.6)
-		(drill 0.3)
-		(layers "F.Cu" "B.Cu")
-		(net 144)
-	)
 	(via
 		(at 101.45 44.45)
@@
 		(drill 0.25)
 		(layers "F.Cu" "B.Cu")
-		(net 145)
+		(net 144)
 	)
 	(via
@@
 		(drill 0.25)
 		(layers "F.Cu" "B.Cu")
-		(net 145)
+		(net 144)
 	)
 	(segment
@@
 		(width 0.15)
 		(layer "In1.Cu")
-		(net 145)
+		(net 144)
 	)
 	(segment
@@
 		(width 0.15)
 		(layer "In1.Cu")
-		(net 145)
+		(net 144)
 	)
 	(segment
@@
 		(width 0.15)
 		(layer "In1.Cu")
-		(net 145)
+		(net 144)
 	)
 	(segment
@@
 		(width 0.15)
 		(layer "B.Cu")
-		(net 145)
+		(net 144)
 	)
 	(segment
@@
 		(width 0.15)
 		(layer "B.Cu")
-		(net 145)
+		(net 144)
 	)
 	(via
@@
 		(drill 0.25)
 		(layers "F.Cu" "B.Cu")
-		(net 147)
+		(net 146)
 	)
 	(segment
@@
 		(width 0.25)
 		(layer "B.Cu")
-		(net 147)
+		(net 146)
 	)
 	(segment
@@
 		(width 0.25)
 		(layer "B.Cu")
-		(net 147)
+		(net 146)
 	)
 	(zone
