File: hardware/motor/_autosave-bldcDriver.kicad_pcb (KiCad board)
At the start: 4 copper layers, 89.8 x 41.5 mm, 198 parts, among them CN1 MR30PW-F, CN2 MR30PW-F, J1 Conn_01x02, J2 Conn_01x06, P1 FPC_0.5MM_4P_Vertical_mountin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, Q1 EMB09N03V, Q10 EMB09N03V, Q11 EMB09N03V, Q12 EMB09N03V, Q13 EMB09N03V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

Commit message: update motor pcb
Routing:
- net /ADC1_IN12_COMP1_INP: track 4.08 -> 25.5 mm, vias 2 -> 3
- net /2CS2-: track 19.8 -> 9.02 mm
- net (no net): track 30.5 -> 25.4 mm
- net /2CS2+: track 16.0 -> 13.2 mm
Changed lines of the file:
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@@
 	)
 	(segment
-		(start 74.7 66.9)
-		(end 75.925 65.675)
-		(width 0.25)
-		(layer "In2.Cu")
-		(net 0)
-	)
-	(segment
 		(start 76.1 67.9)
 		(end 76.9 68.7)
@@
 	)
 	(segment
-		(start 77.274327 64.3)
-		(end 77.6925 64.3)
-		(width 0.25)
-		(layer "In2.Cu")
-		(net 0)
-	)
-	(segment
-		(start 74.7 67.9)
-		(end 74.7 66.9)
-		(width 0.25)
-		(layer "In2.Cu")
-		(net 0)
-	)
-	(segment
-		(start 75.925 65.649327)
-		(end 77.274327 64.3)
-		(width 0.25)
-		(layer "In2.Cu")
-		(net 0)
-	)
-	(segment
 		(start 74.7 67.9)
 		(end 76.1 67.9)
@@
 	)
 	(segment
-		(start 75.925 65.675)
-		(end 75.925 65.649327)
-		(width 0.25)
-		(layer "In2.Cu")
-		(net 0)
-	)
-	(segment
 		(start 67.6125 70.2)
 		(end 67.3125 69.9)
@@
 	)
 	(segment
-		(start 89 61.703984)
-		(end 81.4125 69.291484)
-		(width 0.25)
-		(layer "In2.Cu")
-		(net 91)
-	)
-	(segment
 		(start 81.4125 69.291484)
 		(end 81.4125 69.9)
@@
 	)
 	(segment
-		(start 79.3125 65.8875)
-		(end 76.5 65.8875)
-		(width 0.25)
-		(layer "In2.Cu")
-		(net 92)
-	)
-	(segment
 		(start 104.85 53.851476)
 		(end 104.85 52.446476)
@@
 	)
 	(via
+		(at 87.17958 48.849681)
+		(size 0.5)
+		(drill 0.25)
+		(layers "F.Cu" "B.Cu")
+		(net 147)
+	)
+	(via
 		(at 72.225 62.9)
 		(size 0.5)
@@
 	)
 	(segment
+		(start 73.129261 62.9)
+		(end 87.17958 48.849681)
+		(width 0.25)
+		(layer "In2.Cu")
+		(net 147)
+	)
+	(segment
+		(start 72.225 62.9)
+		(end 73.129261 62.9)
+		(width 0.25)
+		(layer "In2.Cu")
+		(net 147)
+	)
+	(segment
 		(start 72.145 62.82)
 		(end 71.7575 62.82)
@@
 	)
 	(segment
+		(start 86.5375 48.85)
+		(end 87.179261 48.85)
+		(width 0.25)
+		(layer "B.Cu")
+		(net 147)
+	)
+	(segment
 		(start 72.225 62.9)
 		(end 71.9 62.9)
@@
 		(width 0.25)
 		(layer "B.Cu")
+		(net 147)
+	)
+	(segment
+		(start 87.179261 48.85)
+		(end 87.17958 48.849681)
+		(width 0.25)
+		(layer "B.Cu")
