File: hardware/encoder/encoder.kicad_pcb (KiCad board)
At the start: 2 copper layers, 44.4 x 46.3 mm, 15 parts, among them J1 Conn_01x03, J2 Conn_01x03, J3 Conn_01x06, J5 Conn_01x03, J6 Conn_01x03, U1 AS5047D

Commit message: update controller pcb
Parts:
- removed C1: 100n, Capacitor_SMD:C_0603_1608Metric_Pad1.08x0.95mm_HandSolder
- removed J3: Conn_01x06, Connector_PinHeader_2.54mm:PinHeader_1x06_P2.54mm_Vertical
- added C2: 1u, Capacitor_SMD:C_0603_1608Metric_Pad1.08x0.95mm_HandSolder, F.Cu at (136.3, 74.1)
- added C3: 100n, Capacitor_SMD:C_0603_1608Metric_Pad1.08x0.95mm_HandSolder, F.Cu at (134.8, 74.1)
- added J4: Conn_01x05, Connector_PinSocket_2.54mm:PinSocket_1x05_P2.54mm_Vertical, F.Cu at (146.0, 53.6)
- added U2: SMF5.0CA, encoder:SMF5.0CA, F.Cu at (135.4, 69.9)
- U1: value AS5047D -> MT6701CT; footprint Package_SO:TSSOP-14_4.4x5mm_P0.65mm -> Package_SO:SO-8_3.9x4.9mm_P1.27mm
- moved U1 0.30 mm to (140.8, 73.6)
Connections:
- U1 pad 1: /CS -> +3V3
- U1 pad 2: /CLK -> +3V3
- U1 pad 3: /MISO -> unconnected-(U1-OUT-Pad3)
- U1 pad 4: /MOSI -> GND
- U1 pad 5: GND -> unconnected-(U1-PUSH-Pad5)
- U1 pad 6: unconnected-(U1-B-Pad6) -> /DO
- U1 pad 7: unconnected-(U1-A-Pad7) -> /CLK
- U1 pad 8: unconnected-(U1-W/PWM-Pad8) -> /CSN
Routing:
- net /CSN: track 0.00 -> 23.6 mm
- net /DO: track 0.00 -> 22.2 mm
- net /MOSI: track 22.2 -> 0.00 mm
- net /MISO: track 21.0 -> 0.00 mm
- net /CS: track 19.6 -> 0.00 mm
- net +3V3: track 25.5 -> 20.0 mm
- net GND: track 5.30 -> 7.24 mm, vias 2 -> 3
- added copper zone on F.Cu, net +3V3
Other:
- board text added: "MT6701"
- board text removed: "V2.0"

Commit message: update body
Parts:
- removed H7: MountingHole, MountingHole:MountingHole_3mm_Pad_TopBottom
- H3, H4: footprint dp:MountingHole_2.5mm_Pad_TopBottom -> MountingHole:MountingHole_2.2mm_M2_Pad_Via
- moved H4 50.6 mm to (210.3, 74.7)
- moved H3 50.4 mm to (190.3, 74.7)
Other:
- board size 44.4 x 46.3 mm -> 98.2 x 46.3 mm

Commit message: update rfBat firmware
Parts:
- removed H1, H2: MountingHole, dp:MountingHole_2.5mm_Pad_TopBottom
- removed H5, H6, H8: MountingHole, MountingHole:MountingHole_3mm_Pad_TopBottom
- removed J2: Conn_01x03, Connector_PinSocket_2.54mm:PinSocket_1x03_P2.54mm_Vertical
- removed J4: Conn_01x05, Connector_PinSocket_2.54mm:PinSocket_1x05_P2.54mm_Vertical
- removed J5, J6: Conn_01x03, dp:CONN-SMD_AFC10-S03QCA-00
- J1: value Conn_01x03 -> Conn_01x06; footprint Connector_PinSocket_2.54mm:PinSocket_1x03_P2.54mm_Vertical -> encoder:CONN-SMD_6P-P1.00_BX-SH1.0-6PLT; moved to B.Cu
- moved U2 60.7 mm to (196.1, 71.1), turned to 45 degrees
- moved U1 59.6 mm to (200.4, 74.7)
- moved C2 59.3 mm to (195.6, 75.1)
- moved C3 59.3 mm to (194.1, 75.1)
- moved J1 40.9 mm to (200.3, 75.0)
Connections:
- J1 pad 1: /W -> /CSN
- J1 pad 2: /V -> /MOSI
- J1 pad 3: /U -> /MISO
- U1 pad 6: /DO -> /MISO
Routing:
- net /W: track 96.0 -> 0.00 mm
- net /V: track 81.7 -> 0.00 mm, vias 2 -> 0
- net /U: track 67.5 -> 0.00 mm, vias 4 -> 0
- net /DO: track 22.2 -> 0.00 mm
- net /CSN: track 23.6 -> 3.42 mm, vias 0 -> 1
- net /CLK: track 20.9 -> 3.60 mm, vias 0 -> 1
- net GND: track 7.24 -> 13.3 mm, vias 3 -> 1
- net +3V3: track 20.0 -> 15.0 mm, vias 0 -> 1
- net /MISO: track 0.00 -> 3.08 mm, vias 0 -> 1
- removed copper zone on F.Cu, net +3V3
- removed copper zone on B.Cu, net GND
Other:
- board size 98.2 x 46.3 mm -> 32 x 14 mm
- copper layers 2 -> 4
- board text added: "C"
- board text added: "G"
- board text added: "I"
- board text added: "O"
- board text added: "S"
- board text added: "V"

Commit message: update rfBat firmware
Other:
- copper layers 4 -> 2
Changed lines of the file:
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@@
 	(layers
 		(0 "F.Cu" signal)
-		(1 "In1.Cu" signal)
-		(2 "In2.Cu" signal)
 		(31 "B.Cu" signal)
 		(32 "B.Adhes" user "B.Adhesive")
@@
 			)
 			(layer "dielectric 1"
-				(type "prepreg")
-				(thickness 0.1)
+				(type "core")
+				(thickness 1.51)
 				(material "FR4")
 				(epsilon_r 4.5)
-				(loss_tangent 0.02)
-			)
-			(layer "In1.Cu"
-				(type "copper")
-				(thickness 0.035)
-			)
-			(layer "dielectric 2"
-				(type "core")
-				(thickness 1.24)
-				(material "FR4")
-				(epsilon_r 4.5)
-				(loss_tangent 0.02)
-			)
-			(layer "In2.Cu"
-				(type "copper")
-				(thickness 0.035)
-			)
-			(layer "dielectric 3"
-				(type "prepreg")
-				(thickness 0.1)
-				(material "FR4")
-				(epsilon_r 4.5)

Commit message: update rfBat pcb
Parts:
- J1: footprint encoder:CONN-SMD_6P-P1.00_BX-SH1.0-6PLT -> encoder:FPC-SMD_6P-P0.50_HDGC_0.5K-A-6PB
- moved C3 12.5 mm to (206.6, 74.3), turned to 90 degrees
- moved U2 11.1 mm to (204.6, 78.3), turned to -135 degrees
- moved C2 9.53 mm to (205.1, 74.3), turned to 90 degrees
- moved J1 0.27 mm to (200.3, 74.7), turned to 0 degrees
- moved U1 0.10 mm to (200.3, 74.7), turned to 180 degrees
Connections:
- J1 pad 1: /CSN -> GND
- J1 pad 2: /MOSI -> +3V3
- J1 pad 3: /MISO -> /CLK
- J1 pad 4: /CLK -> /MISO
- J1 pad 5: +3V3 -> /MOSI
- J1 pad 6: GND -> /CSN
Routing:
- net GND: track 13.3 -> 17.0 mm
- net +3V3: track 15.0 -> 12.9 mm
- net /CSN: track 3.42 -> 4.15 mm
Other:
- board text removed: "C"
- board text removed: "I"
- board text removed: "O"
- board text removed: "S"
- board text removed: "V"
