File: hardware/encoder/encoder.kicad_sch (KiCad schematic)
At the start: 15 parts, among them J1 Conn_01x03, J2 Conn_01x03, J3 Conn_01x06, J5 Conn_01x03, J6 Conn_01x03, U1 MT6701CT

Commit message: update controller pcb
Parts:
- removed C1: 100n, Capacitor_SMD:C_0603_1608Metric_Pad1.08x0.95mm_HandSolder, symbol Device:C
- removed J3: Conn_01x06, Connector_PinHeader_2.54mm:PinHeader_1x06_P2.54mm_Vertical, symbol Connector_Generic:Conn_01x06
- added C2: 1u, Capacitor_SMD:C_0603_1608Metric_Pad1.08x0.95mm_HandSolder, symbol Device:C
- added C3: 100n, Capacitor_SMD:C_0603_1608Metric_Pad1.08x0.95mm_HandSolder, symbol Device:C
- added J4: Conn_01x05, Connector_PinSocket_2.54mm:PinSocket_1x05_P2.54mm_Vertical, symbol Connector_Generic:Conn_01x05
- added U2: SMF5.0CA, encoder:SMF5.0CA, symbol encoder:SMF5.0CA
Connections:
- net +3V3: now also U1.1 (VDD), U1.2 (MODE), C2.1, C3.1, J4.4 (Pin_4), U2.1
- net CLK: now also U1.7 (B), J4.2 (Pin_2)
- net GND: now also U1.4 (GND), C2.2, C3.2, J4.5 (Pin_5), U2.2
- net DO: now reaches U1.6 (A)
- net DO: now also J4.1 (Pin_1)
- net CSN: now reaches U1.8 (Z)
- net CSN: now also J4.3 (Pin_3)
- no-connect marks 0 -> 2
Other:
- moved on the sheet: U1

Commit message: update body
Parts:
- removed H1, H2: MountingHole, dp:MountingHole_2.5mm_Pad_TopBottom, symbol Mechanical:MountingHole
- removed H5, H6, H7, H8: MountingHole, MountingHole:MountingHole_3mm_Pad_TopBottom, symbol Mechanical:MountingHole
- removed J1, J2: Conn_01x03, Connector_PinSocket_2.54mm:PinSocket_1x03_P2.54mm_Vertical, symbol Connector_Generic:Conn_01x03
- removed J5, J6: Conn_01x03, dp:CONN-SMD_AFC10-S03QCA-00, symbol Connector_Generic:Conn_01x03
- H3, H4: footprint dp:MountingHole_2.5mm_Pad_TopBottom -> MountingHole:MountingHole_2.2mm_M2_Pad_Via
Other:
- moved on the sheet: H3, H4, J4

Commit message: update rfBat firmware
Parts:
- removed J4: Conn_01x05, Connector_PinSocket_2.54mm:PinSocket_1x05_P2.54mm_Vertical, symbol Connector_Generic:Conn_01x05
- added J1: Conn_01x06, encoder:CONN-SMD_6P-P1.00_BX-SH1.0-6PLT, symbol Connector_Generic:Conn_01x06
Connections:
- net +3V3: now also J1.5 (Pin_5)
- net CLK: now also J1.4 (Pin_4)
- net CSN: now also J1.1 (Pin_1)
- net GND: now also J1.6 (Pin_6)
- net DO renamed MISO
- net MISO: now also J1.3 (Pin_3)
- new net MOSI: J1.2 (Pin_2)
Changed lines of the file:
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@@
 		)
 	)
-	(label "CLK"
-		(at 127 49.53 180)
+	(label "MISO"
+		(at 165.1 76.2 0)
 		(fields_autoplaced yes)
 		(effects
@@
 				(size 1.27 1.27)
 			)
-			(justify right bottom)
-		)
-	)
-	(label "CSN"
-		(at 165.1 81.28 0)
+			(justify left bottom)
+		)
+	)
+	(label "MISO"
+		(at 127 49.53 180)
 		(fields_autoplaced yes)
 		(effects
@@
 				(size 1.27 1.27)
 			)
-			(justify left bottom)
-		)
-	)
-	(label "DO"
-		(at 165.1 76.2 0)
+			(justify right bottom)
+		)
+	)
+	(label "MOSI"
+		(at 127 46.99 180)
 		(fields_autoplaced yes)
 		(effects
@@
 				(size 1.27 1.27)
 			)
-			(justify left bottom)
-		)
-	)
-	(label "CLK"
-		(at 165.1 78.74 0)
+			(justify right bottom)
+		)
+	)
+	(label "CSN"
+		(at 127 44.45 180)
 		(fields_autoplaced yes)
 		(effects
@@
 				(size 1.27 1.27)
 			)
-			(justify left bottom)
+			(justify right bottom)
 		)
 	)
 	(label "CSN"
-		(at 127 52.07 180)
+		(at 165.1 81.28 0)
 		(fields_autoplaced yes)
 		(effects
@@
 				(size 1.27 1.27)
 			)
-			(justify right bottom)
-		)
-	)
-	(label "DO"
-		(at 127 46.99 180)
+			(justify left bottom)
+		)
+	)
+	(label "CLK"
+		(at 165.1 78.74 0)
 		(fields_autoplaced yes)
 		(effects
@@
 				(size 1.27 1.27)
 			)
+			(justify left bottom)
+		)
+	)
+	(label "CLK"
+		(at 127 52.07 180)
+		(fields_autoplaced yes)
+		(effects
+			(font
+				(size 1.27 1.27)
+			)
 			(justify right bottom)
-		)
-	)
-	(symbol
-		(lib_id "Connector_Generic:Conn_01x05")
-		(at 132.08 52.07 0)
-		(unit 1)
-		(exclude_from_sim no)
-		(in_bom yes)
-		(on_board yes)
-		(dnp no)
-		(fields_autoplaced yes)
-		(property "Reference" "J4"
-			(at 134.62 50.7999 0)
-			(effects
-				(font
-					(size 1.27 1.27)
-				)
-				(justify left)
-			)
-		)
-		(property "Value" "Conn_01x05"
-			(at 134.62 53.3399 0)
-			(effects
-				(font
-					(size 1.27 1.27)
-				)
-				(justify left)
-			)
-		)
-		(property "Footprint" "Connector_PinSocket_2.54mm:PinSocket_1x05_P2.54mm_Vertical"
-			(at 132.08 52.07 0)
-			(effects
-				(font
-					(size 1.27 1.27)
-				)
-				(hide yes)
-			)
-		)
-		(property "Datasheet" "~"
-			(at 132.08 52.07 0)
-			(effects
-				(font
-					(size 1.27 1.27)
-				)
-				(hide yes)
-			)
-		)
-		(property "Description" "Generic connector, single row, 01x05, script generated (kicad-library-utils/schlib/autogen/connector/)"
-			(at 132.08 52.07 0)
-			(effects
-				(font
-					(size 1.27 1.27)
-				)
-				(hide yes)
-			)
-		)
-		(pin "4"
-		)
-		(pin "2"
-		)
-		(pin "5"
-		)
-		(pin "1"
-		)
-		(pin "3"
-		)
-		(instances
-			(project "encoder"
-				(path "/cbf7aacc-9925-4e73-a094-13fc31cc8a91"
-					(reference "J4")
-					(unit 1)
-				)
-			)
 		)
 	)
@@
 					(unit 1)
 				)
+			)
+		)
+	)
+	(symbol
+		(lib_id "Connector_Generic:Conn_01x06")
+		(at 132.08 49.53 0)
+		(unit 1)
+		(exclude_from_sim no)
+		(in_bom yes)
+		(on_board yes)
+		(dnp no)
+		(fields_autoplaced yes)
+		(property "Reference" "J1"
+			(at 134.62 49.5299 0)
+			(effects
+				(font
+					(size 1.27 1.27)
+				)
+				(justify left)
+			)
+		)
+		(property "Value" "Conn_01x06"
+			(at 134.62 52.0699 0)
+			(effects
+				(font
+					(size 1.27 1.27)
+				)
+				(justify left)
+			)
+		)
+		(property "Footprint" "encoder:CONN-SMD_6P-P1.00_BX-SH1.0-6PLT"
+			(at 132.08 49.53 0)
+			(effects
+				(font
+					(size 1.27 1.27)
+				)
+				(hide yes)
+			)
+		)
+		(property "Datasheet" "~"
+			(at 132.08 49.53 0)
+			(effects
+				(font
+					(size 1.27 1.27)
+				)
+				(hide yes)
+			)
+		)
+		(property "Description" "Generic connector, single row, 01x06, script generated (kicad-library-utils/schlib/autogen/connector/)"
+			(at 132.08 49.53 0)
+			(effects
+				(font
+					(size 1.27 1.27)
+				)
+				(hide yes)
+			)
+		)
+		(pin "4"
+		)
+		(pin "1"
+		)
+		(pin "3"
+		)
+		(pin "5"
+		)
+		(pin "6"
+		)
+		(pin "2"
+		)
+		(instances
+			(project "encoder"
+				(path "/cbf7aacc-9925-4e73-a094-13fc31cc8a91"
+					(reference "J1")
+					(unit 1)
+				)

Commit message: update rfBat pcb
Parts:
- J1: footprint encoder:CONN-SMD_6P-P1.00_BX-SH1.0-6PLT -> encoder:FPC-SMD_6P-P0.50_HDGC_0.5K-A-6PB
Connections:
- net +3V3: now also J1.2 (Pin_2); no longer J1.5 (Pin_5)
- net CLK: now also J1.3 (Pin_3); no longer J1.4 (Pin_4)
- net CSN: now also J1.6 (Pin_6); no longer J1.1 (Pin_1)
- net GND: now also J1.1 (Pin_1); no longer J1.6 (Pin_6)
- net MISO: now also J1.4 (Pin_4); no longer J1.3 (Pin_3)
- net MOSI: now also J1.5 (Pin_5); no longer J1.2 (Pin_2)
Other:
- moved on the sheet: J1
Changed lines of the file:
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@@
+	(wire
+		(pts
+			(xy 124.46 54.61) (xy 124.46 55.88)
+		)
+		(stroke
+			(width 0)
+			(type default)
+		)
+	)
+	(wire
+		(pts
+			(xy 152.4 106.68) (xy 152.4 107.95)
+		)
+		(stroke
+			(width 0)
+			(type default)
+		)
+	)
+	(wire
+		(pts
+			(xy 124.46 52.07) (xy 127 52.07)
+		)
+		(stroke
+			(width 0)
+			(type default)
+		)
+	)
 	(wire
 		(pts
@@
 	(wire
 		(pts
-			(xy 124.46 57.15) (xy 124.46 58.42)
+			(xy 138.43 88.9) (xy 139.7 88.9)
 		)
 		(stroke
@@
 	(wire
 		(pts
-			(xy 152.4 106.68) (xy 152.4 107.95)
+			(xy 152.4 66.04) (xy 152.4 67.31)
 		)
 		(stroke
@@
 	(wire
 		(pts
-			(xy 138.43 88.9) (xy 139.7 88.9)
-		)
-		(stroke
-			(width 0)
-			(type default)
-		)
-	)
-	(wire
-		(pts
-			(xy 152.4 66.04) (xy 152.4 67.31)
-		)
-		(stroke
-			(width 0)
-			(type default)
-		)
-	)
-	(wire
-		(pts
 			(xy 134.62 81.28) (xy 128.27 81.28)
-		)
-		(stroke
-			(width 0)
-			(type default)
-		)
-	)
-	(wire
-		(pts
-			(xy 124.46 57.15) (xy 127 57.15)
 		)
 		(stroke
@@
 		)
 	)
-	(label "MISO"
-		(at 127 49.53 180)
+	(label "CSN"
+		(at 127 41.91 180)
 		(fields_autoplaced yes)
 		(effects
@@
 		)
 	)
-	(label "MOSI"
-		(at 127 46.99 180)
-		(fields_autoplaced yes)
-		(effects
-			(font
-				(size 1.27 1.27)
-			)
-			(justify right bottom)
-		)
-	)
-	(label "CSN"
-		(at 127 44.45 180)
+	(label "CLK"
+		(at 127 49.53 180)
 		(fields_autoplaced yes)
 		(effects
@@
 		)
 	)
-	(label "CLK"
-		(at 127 52.07 180)
+	(label "MOSI"
+		(at 127 44.45 180)
 		(fields_autoplaced yes)
 		(effects
@@
 		)
 	)
+	(label "MISO"
+		(at 127 46.99 180)
+		(fields_autoplaced yes)
+		(effects
+			(font
+				(size 1.27 1.27)
+			)
+			(justify right bottom)
+		)
+	)
+	(symbol
+		(lib_id "power:+3V3")
+		(at 124.46 52.07 90)
+		(unit 1)
+		(exclude_from_sim no)
+		(in_bom yes)
+		(on_board yes)
+		(dnp no)
+		(property "Reference" "#PWR02"
+			(at 128.27 52.07 0)
+			(effects
+				(font
+					(size 1.27 1.27)
+				)
+				(hide yes)
+			)
+		)
+		(property "Value" "+3V3"
+			(at 119.126 52.324 90)
+			(effects
+				(font
+					(size 1.27 1.27)
+				)
+			)
+		)
+		(property "Footprint" ""
+			(at 124.46 52.07 0)
+			(effects
+				(font
+					(size 1.27 1.27)
+				)
+				(hide yes)
+			)
+		)
+		(property "Datasheet" ""
+			(at 124.46 52.07 0)
+			(effects
+				(font
+					(size 1.27 1.27)
+				)
+				(hide yes)
+			)
+		)
+		(property "Description" "Power symbol creates a global label with name \"+3V3\""
+			(at 124.46 52.07 0)
+			(effects
+				(font
+					(size 1.27 1.27)
+				)
+				(hide yes)
+			)
+		)
+		(pin "1"
+		)
+		(instances
+			(project "encoder"
+				(path "/cbf7aacc-9925-4e73-a094-13fc31cc8a91"
+					(reference "#PWR02")
+					(unit 1)
+				)
+			)
+		)
+	)
 	(symbol
 		(lib_id "encoder:SMF5.0CA")
@@
 	)
 	(symbol
+		(lib_id "power:GND")
+		(at 124.46 55.88 0)
+		(unit 1)
+		(exclude_from_sim no)
+		(in_bom yes)
+		(on_board yes)
+		(dnp no)
+		(property "Reference" "#PWR03"
+			(at 124.46 62.23 0)
+			(effects
+				(font
+					(size 1.27 1.27)
+				)
+				(hide yes)
+			)
+		)
+		(property "Value" "GND"
+			(at 128.27 57.15 0)
+			(effects
+				(font
+					(size 1.27 1.27)
+				)
+				(hide yes)
+			)
+		)
+		(property "Footprint" ""
+			(at 124.46 55.88 0)
+			(effects
+				(font
+					(size 1.27 1.27)
+				)
+				(hide yes)
+			)
+		)
+		(property "Datasheet" ""
+			(at 124.46 55.88 0)
+			(effects
+				(font
+					(size 1.27 1.27)
+				)
+				(hide yes)
+			)
+		)
+		(property "Description" ""
+			(at 124.46 55.88 0)
+			(effects
+				(font
+					(size 1.27 1.27)
+				)
+				(hide yes)
+			)
+		)
+		(pin "1"
+		)
+		(instances
+			(project "encoder"
+				(path "/cbf7aacc-9925-4e73-a094-13fc31cc8a91"
+					(reference "#PWR03")
+					(unit 1)
+				)
+			)
+		)
+	)
+	(symbol
 		(lib_id "Device:C")
 		(at 128.27 72.39 0)
@@
 	)
 	(symbol
-		(lib_id "power:+3V3")
-		(at 124.46 54.61 90)
-		(unit 1)
-		(exclude_from_sim no)
-		(in_bom yes)
-		(on_board yes)
-		(dnp no)
-		(property "Reference" "#PWR05"
-			(at 128.27 54.61 0)
-			(effects
-				(font
-					(size 1.27 1.27)
-				)
-				(hide yes)
-			)
-		)
-		(property "Value" "+3V3"
-			(at 119.126 54.864 90)
-			(effects
-				(font
-					(size 1.27 1.27)
-				)
-			)
-		)
-		(property "Footprint" ""
-			(at 124.46 54.61 0)
-			(effects
-				(font
-					(size 1.27 1.27)
-				)
-				(hide yes)
-			)
-		)
-		(property "Datasheet" ""
-			(at 124.46 54.61 0)
-			(effects
-				(font
-					(size 1.27 1.27)
-				)
-				(hide yes)
-			)
-		)
-		(property "Description" "Power symbol creates a global label with name \"+3V3\""
-			(at 124.46 54.61 0)
-			(effects
-				(font
-					(size 1.27 1.27)
-				)
-				(hide yes)
-			)
-		)
-		(pin "1"
-		)
-		(instances
-			(project "encoder"
-				(path "/cbf7aacc-9925-4e73-a094-13fc31cc8a91"
-					(reference "#PWR05")
-					(unit 1)
-				)
-			)
-		)
-	)
-	(symbol
 		(lib_id "power:GND")
 		(at 152.4 107.95 0)
@@
 		(lib_id "Connector_Generic:Conn_01x06")
 		(at 132.08 49.53 0)
-		(unit 1)
-		(exclude_from_sim no)
-		(in_bom yes)
-		(on_board yes)
-		(dnp no)
-		(fields_autoplaced yes)
+		(mirror x)
+		(unit 1)
+		(exclude_from_sim no)
+		(in_bom yes)
+		(on_board yes)
+		(dnp no)
 		(property "Reference" "J1"
-			(at 134.62 49.5299 0)
+			(at 134.62 49.5301 0)
 			(effects
 				(font
@@
 		)
 		(property "Value" "Conn_01x06"
-			(at 134.62 52.0699 0)
-			(effects
-				(font
-					(size 1.27 1.27)
-				)
-				(justify left)
-			)
-		)
-		(property "Footprint" "encoder:CONN-SMD_6P-P1.00_BX-SH1.0-6PLT"
+			(at 134.62 46.9901 0)
+			(effects
+				(font
+					(size 1.27 1.27)
+				)
+				(justify left)
+			)
+		)
+		(property "Footprint" "encoder:FPC-SMD_6P-P0.50_HDGC_0.5K-A-6PB"
 			(at 132.08 49.53 0)
 			(effects
@@
 					(unit 1)
 				)
-			)
-		)
-	)
-	(symbol
-		(lib_id "power:GND")
-		(at 124.46 58.42 0)
-		(unit 1)
-		(exclude_from_sim no)
-		(in_bom yes)
-		(on_board yes)
-		(dnp no)
-		(property "Reference" "#PWR06"
-			(at 124.46 64.77 0)
-			(effects
-				(font
-					(size 1.27 1.27)
-				)
-				(hide yes)
-			)
-		)
-		(property "Value" "GND"
-			(at 128.27 59.69 0)
-			(effects
-				(font
-					(size 1.27 1.27)
-				)
-				(hide yes)
-			)
-		)
-		(property "Footprint" ""
-			(at 124.46 58.42 0)
-			(effects
-				(font
-					(size 1.27 1.27)
-				)
-				(hide yes)
-			)
-		)
-		(property "Datasheet" ""
-			(at 124.46 58.42 0)
-			(effects
-				(font
-					(size 1.27 1.27)
-				)
-				(hide yes)
-			)
-		)
-		(property "Description" ""
-			(at 124.46 58.42 0)
-			(effects
-				(font
-					(size 1.27 1.27)
-				)
-				(hide yes)
-			)
-		)
-		(pin "1"
-		)
-		(instances
-			(project "encoder"
-				(path "/cbf7aacc-9925-4e73-a094-13fc31cc8a91"
-					(reference "#PWR06")
-					(unit 1)
-				)
